File: switch.sch (KiCad schematic (older format))
At the start: 188 parts

Commit message: maybe use a premade powerbrick
Parts:
- removed C? (x4): 0.1uF, Capacitor_SMD:C_0402_1005Metric, symbol Device:C_Small
- removed FB?: BLM18EG221SN1D, kicad-lib:ferrite-blm18, symbol Device:Ferrite_Bead_Small
- removed J?: JK0654219, Connector_RJ:RJ45_Pulse_JK0654219NL_Horizontal, symbol Connector:JK0654219
- removed R?: 10K, Resistor_SMD:R_0402_1005Metric, symbol Device:R_Small_US
- removed TP? (x2): TestPoint, TestPoint:TestPoint_Pad_D1.0mm, symbol Connector:TestPoint
- removed U?: MDT420M02001, dg_connectors:m.2_pcie_nvme, symbol dg_connectors:m.2_pcie_nvme
- added T3, T4, T5, T6, T7: QT24A01, dg_transformers:SOP100P1000X450-24N, symbol dg_transformers:QT24A01
- gave numbers to parts that had none: 176
Connections:
- net labels removed: 3V3_PCIE, GNDREF, RPI_PCIe_CLK_N, RPI_PCIe_CLK_P, RPI_PCIe_CLK_nREQ, RPI_PCIe_RX_N, RPI_PCIe_RX_P, RPI_PCIe_TX_N, RPI_PCIe_TX_P, RPI_PCIe_nRST
- wire segments 693 -> 609
- no-connect marks 45 -> 13
Other:
- note removed: "M.2 SSD Connector"
