File: dcdc.sch (KiCad schematic (older format))
At the start: 0 parts

Commit message: Added Schematic Design for 12V->5V DC-DC.
Parts:
- added C? (x6): 10uF 25V, Capacitor_SMD:C_1206_3216Metric, symbol Device:C_Small
- added C?: 4.7uF 25V, Capacitor_SMD:C_0805_2012Metric, symbol Device:C_Small
- added C?: 15nF, Capacitor_SMD:C_0402_1005Metric, symbol Device:C_Small
- added C?: 33nF, Capacitor_SMD:C_0402_1005Metric, symbol Device:C_Small
- added C?: 68pF, Capacitor_SMD:C_0402_1005Metric, symbol Device:C_Small
- added C?: 100nF, Capacitor_SMD:C_0805_2012Metric, symbol Device:C_Small
- added L?: 4.7uH, dg_transformers:IND_1350, symbol Device:L
- added R? (x2): 53.6K, Resistor_SMD:R_0402_1005Metric, symbol Device:R
- added R?: 2.55K, Resistor_SMD:R_0402_1005Metric, symbol Device:R
- added R? (x2): 102K, Resistor_SMD:R_0402_1005Metric, symbol Device:R
- added R?: 36.5K, Resistor_SMD:R_0402_1005Metric, symbol Device:R
- added U?: TPS54620, dg_ic:Texas_S-PVQFN-N14_ThermalVias, symbol dg_ic:TPS54620
- added U?: RT8065, dg_ic:DFN-8-1EP_3x3mm_P0.65mm_EP1.55x2.4mm, symbol dg_ic:RT8065
Connections:
- net labels added: +12V, +5V, GND, TPS_EN, TPS_FB, TPS_PWRGD
- wire segments 0 -> 66
Other:
- note added: "DNP Enable Resistors \nto disable UVLO."

Commit message: dcdc: dont use global labels for rails
Connections:
- net labels removed: +12V, +5V, TPS_FB
- wire segments 66 -> 78
Other:
- moved on the sheet: R?
Changed lines of the file:
@@
 Comment4 ""
 $EndDescr
-Text HLabel 1550 1400 0    50   Input ~ 0
+Text HLabel 7250 1250 1    50   Input ~ 0
 5V
 Text HLabel 1550 1700 0    50   Input ~ 0
 3.3V
-Text HLabel 1550 1100 0    50   Input ~ 0
+Text HLabel 2850 1250 0    50   Input ~ 0
 VIN
 Text HLabel 1550 1950 0    50   Input ~ 0
@@
 $EndComp
 $Comp
-L power:+12V #PWR?
-U 1 1 61114473
-P 3150 1400
-F 0 "#PWR?" H 3150 1250 50  0001 C CNN
-F 1 "+12V" H 3165 1573 50  0000 C CNN
-F 2 "" H 3150 1400 50  0001 C CNN
-F 3 "" H 3150 1400 50  0001 C CNN
-	1    3150 1400
-	1    0    0    -1
-$EndComp
-Connection ~ 3150 1400
-$Comp
-L power:+12V #PWR?
-U 1 1 61114CBD
-P 3150 2150
-F 0 "#PWR?" H 3150 2000 50  0001 C CNN
-F 1 "+12V" H 3165 2323 50  0000 C CNN
-F 2 "" H 3150 2150 50  0001 C CNN
-F 3 "" H 3150 2150 50  0001 C CNN
-	1    3150 2150
-	1    0    0    -1
-$EndComp
-$Comp
 L Device:R R?
 U 1 1 61113B66
@@
 L Device:R R?
 U 1 1 6111DEF4
-P 5950 2500
-F 0 "R?" V 5950 2450 50  0000 L CNN
-F 1 "102K" V 5850 2400 50  0000 L CNN
-F 2 "Resistor_SMD:R_0402_1005Metric" V 5880 2500 50  0001 C CNN
-F 3 "~" H 5950 2500 50  0001 C CNN
-	1    5950 2500
+P 8300 1850
+F 0 "R?" V 8300 1800 50  0000 L CNN
+F 1 "102K" V 8200 1750 50  0000 L CNN
+F 2 "Resistor_SMD:R_0402_1005Metric" V 8230 1850 50  0001 C CNN
+F 3 "~" H 8300 1850 50  0001 C CNN
+	1    8300 1850
 	1    0    0    -1
 $EndComp
@@
 L Device:R R?
 U 1 1 6111E4B3
-P 6450 2350
-F 0 "R?" V 6450 2300 50  0000 L CNN
-F 1 "53.6K" V 6350 2250 50  0000 L CNN
-F 2 "Resistor_SMD:R_0402_1005Metric" V 6380 2350 50  0001 C CNN
-F 3 "~" H 6450 2350 50  0001 C CNN
-	1    6450 2350
-	0    1    1    0
+P 7800 1700
+F 0 "R?" V 7800 1650 50  0000 L CNN
+F 1 "53.6K" V 7700 1600 50  0000 L CNN
+F 2 "Resistor_SMD:R_0402_1005Metric" V 7730 1700 50  0001 C CNN
+F 3 "~" H 7800 1700 50  0001 C CNN
+	1    7800 1700
+	0    -1   -1   0
 $EndComp
 $Comp
 L power:GND #PWR?
 U 1 1 611237EC
-P 5950 2650
-F 0 "#PWR?" H 5950 2400 50  0001 C CNN
-F 1 "GND" H 5955 2477 50  0000 C CNN
-F 2 "" H 5950 2650 50  0001 C CNN
-F 3 "" H 5950 2650 50  0001 C CNN
-	1    5950 2650
+P 8300 2000
+F 0 "#PWR?" H 8300 1750 50  0001 C CNN
+F 1 "GND" H 8305 1827 50  0000 C CNN
+F 2 "" H 8300 2000 50  0001 C CNN
+F 3 "" H 8300 2000 50  0001 C CNN
+	1    8300 2000
 	1    0    0    -1
 $EndComp
@@
 Wire Wire Line
 	6950 1800 6950 1700
-Connection ~ 7250 1700
 Wire Wire Line
 	6350 1700 6650 1700
@@
 	1    0    0    -1
 $EndComp
-$Comp
-L power:+5V #PWR?
-U 1 1 61124A2B
-P 7250 1700
-F 0 "#PWR?" H 7250 1550 50  0001 C CNN
-F 1 "+5V" H 7265 1873 50  0000 C CNN
-F 2 "" H 7250 1700 50  0001 C CNN
-F 3 "" H 7250 1700 50  0001 C CNN
-	1    7250 1700
-	1    0    0    -1
-$EndComp
 Wire Wire Line
 	6250 1700 6350 1700
@@
 	5600 1700 5850 1700
 Connection ~ 5850 1700
-Text Label 5600 1900 0    50   ~ 0
-TPS_FB
 Wire Wire Line
 	5500 1900 5900 1900
-Text Label 5950 2350 0    50   ~ 0
-TPS_FB
-Wire Wire Line
-	5950 2350 6300 2350
-$Comp
-L power:+5V #PWR?
-U 1 1 611559B1
-P 6600 2350
-F 0 "#PWR?" H 6600 2200 50  0001 C CNN
-F 1 "+5V" V 6615 2478 50  0000 L CNN
-F 2 "" H 6600 2350 50  0001 C CNN
-F 3 "" H 6600 2350 50  0001 C CNN
-	1    6600 2350
-	0    1    1    0
-$EndComp
+Wire Wire Line
+	8300 1700 8050 1700
 Text Notes 2850 3300 0    50   ~ 0
 DNP Enable Resistors \nto disable UVLO.
+Connection ~ 7250 1700
+Wire Wire Line
+	7650 1700 7250 1700
+Wire Wire Line
+	7250 1250 7250 1700
+Wire Wire Line
+	8050 1700 8050 2650
+Wire Wire Line
+	8050 2650 5900 2650
+Wire Wire Line
+	5900 2650 5900 1900
+Connection ~ 8050 1700
+Wire Wire Line
+	8050 1700 7950 1700
+Wire Wire Line
+	2850 1250 2950 1250
+Wire Wire Line
+	3150 1250 3150 1400
+Connection ~ 3150 1400
+Wire Wire Line
+	3150 2150 3150 2050
+Wire Wire Line
+	3150 2050 2950 2050
+Wire Wire Line
+	2950 2050 2950 1250
+Connection ~ 2950 1250
+Wire Wire Line
+	2950 1250 3150 1250
 $EndSCHEMATC

Commit message: add the ksz switch
Parts:
- gave numbers to parts that had none: 20
Changed lines of the file:
@@
 $Descr A4 11693 8268
 encoding utf-8
-Sheet 4 4
+Sheet 4 5
 Title ""
 Date ""
@@
 DISABLE
 $Comp
-L dg_ic:TPS54620 U?
+L dg_ic:TPS54620 U4
 U 1 1 610FC53B
 P 5050 1300
-F 0 "U?" H 5025 1555 50  0000 C CNN
+F 0 "U4" H 5025 1555 50  0000 C CNN
 F 1 "TPS54620" H 5025 1464 50  0000 C CNN
 F 2 "dg_ic:Texas_S-PVQFN-N14_ThermalVias" H 5050 -50 50  0001 C CNN
@@
 $EndComp
 $Comp
-L dg_ic:RT8065 U?
+L dg_ic:RT8065 U5
 U 1 1 610FCD44
 P 5200 4650
-F 0 "U?" H 5225 4905 50  0000 C CNN
+F 0 "U5" H 5225 4905 50  0000 C CNN
 F 1 "RT8065" H 5225 4814 50  0000 C CNN
 F 2 "dg_ic:DFN-8-1EP_3x3mm_P0.65mm_EP1.55x2.4mm" H 5200 3650 50  0001 C CNN
@@
 $EndComp
 $Comp
-L Device:C_Small C?
+L Device:C_Small C2
 U 1 1 610FE465
 P 3500 1600
-F 0 "C?" H 3550 1700 50  0000 L CNN
+F 0 "C2" H 3550 1700 50  0000 L CNN
 F 1 "10uF 25V" V 3400 1400 50  0000 L CNN
 F 2 "Capacitor_SMD:C_1206_3216Metric" H 3500 1600 50  0001 C CNN
@@
 $EndComp
 $Comp
-L Device:C_Small C?
+L Device:C_Small C4
 U 1 1 610FF2E2
 P 3850 1600
-F 0 "C?" H 3900 1700 50  0000 L CNN
+F 0 "C4" H 3900 1700 50  0000 L CNN
 F 1 "4.7uF 25V" V 3750 1400 50  0000 L CNN
 F 2 "Capacitor_SMD:C_0805_2012Metric" H 3850 1600 50  0001 C CNN
@@
 $EndComp
 $Comp
-L Device:R R?
+L Device:R R3
 U 1 1 6110002E
 P 4000 2650
-F 0 "R?" V 4000 2600 50  0000 L CNN
+F 0 "R3" V 4000 2600 50  0000 L CNN
 F 1 "53.6K" V 3900 2550 50  0000 L CNN
 F 2 "Resistor_SMD:R_0402_1005Metric" V 3930 2650 50  0001 C CNN
@@
 $EndComp
 $Comp
-L Device:C_Small C?
+L Device:C_Small C3
 U 1 1 61100BC3
 P 3750 2600
-F 0 "C?" H 3650 2750 50  0000 L CNN
+F 0 "C3" H 3650 2750 50  0000 L CNN
 F 1 "15nF" V 3650 2500 50  0000 L CNN
 F 2 "Capacitor_SMD:C_0402_1005Metric" H 3750 2600 50  0001 C CNN
@@
 $EndComp
 $Comp
-L Device:R R?
+L Device:R R4
 U 1 1 61102728
 P 4250 2650
-F 0 "R?" V 4250 2600 50  0000 L CNN
+F 0 "R4" V 4250 2600 50  0000 L CNN
 F 1 "2.55K" V 4150 2550 50  0000 L CNN
 F 2 "Resistor_SMD:R_0402_1005Metric" V 4180 2650 50  0001 C CNN
@@
 $EndComp
 $Comp
-L Device:C_Small C?
+L Device:C_Small C7
 U 1 1 61102A9D
 P 4250 3000
-F 0 "C?" H 4342 3046 50  0000 L CNN
+F 0 "C7" H 4342 3046 50  0000 L CNN
 F 1 "33nF" V 4150 2900 50  0000 L CNN
 F 2 "Capacitor_SMD:C_0402_1005Metric" H 4250 3000 50  0001 C CNN
@@
 $EndComp
 $Comp
-L Device:C_Small C?
+L Device:C_Small C8
 U 1 1 61102F15
 P 4450 2750
-F 0 "C?" H 4500 2850 50  0000 L CNN
+F 0 "C8" H 4500 2850 50  0000 L CNN
 F 1 "68pF" H 4500 2650 50  0000 L CNN
 F 2 "Capacitor_SMD:C_0402_1005Metric" H 4450 2750 50  0001 C CNN
@@
 	4450 2850 4450 3200
 $Comp
-L power:GND #PWR?
+L power:GND #PWR0103
 U 1 1 611056D6
 P 4250 3200
-F 0 "#PWR?" H 4250 2950 50  0001 C CNN
+F 0 "#PWR0103" H 4250 2950 50  0001 C CNN
 F 1 "GND" H 4255 3027 50  0000 C CNN
 F 2 "" H 4250 3200 50  0001 C CNN
@@
 Connection ~ 4250 3200
 $Comp
-L power:GND #PWR?
+L power:GND #PWR0104
 U 1 1 61105D35
 P 4000 2900
-F 0 "#PWR?" H 4000 2650 50  0001 C CNN
+F 0 "#PWR0104" H 4000 2650 50  0001 C CNN
 F 1 "GND" H 4005 2727 50  0000 C CNN
 F 2 "" H 4000 2900 50  0001 C CNN
@@
 $EndComp
 $Comp
-L power:GND #PWR?
+L power:GND #PWR0106
 U 1 1 61105FF4
 P 3750 2800
-F 0 "#PWR?" H 3750 2550 50  0001 C CNN
+F 0 "#PWR0106" H 3750 2550 50  0001 C CNN
 F 1 "GND" H 3755 2627 50  0000 C CNN
 F 2 "" H 3750 2800 50  0001 C CNN
@@
 	4550 1900 4000 1900
 $Comp
-L Device:C_Small C?
+L Device:C_Small C1
 U 1 1 61109F56
 P 3150 1600
-F 0 "C?" H 3200 1700 50  0000 L CNN
+F 0 "C1" H 3200 1700 50  0000 L CNN
 F 1 "10uF 25V" V 3050 1400 50  0000 L CNN
 F 2 "Capacitor_SMD:C_1206_3216Metric" H 3150 1600 50  0001 C CNN
@@
 	3500 1850 3850 1850
 $Comp
-L power:GND #PWR?
+L power:GND #PWR0107
 U 1 1 6110CCCF
 P 3500 1850
-F 0 "#PWR?" H 3500 1600 50  0001 C CNN
+F 0 "#PWR0107" H 3500 1600 50  0001 C CNN
 F 1 "GND" H 3505 1677 50  0000 C CNN
 F 2 "" H 3500 1850 50  0001 C CNN
@@
 	3750 2500 3750 2200
 $Comp
-L power:GND #PWR?
+L power:GND #PWR0108
 U 1 1 611119B4
 P 5600 2450
-F 0 "#PWR?" H 5600 2200 50  0001 C CNN
+F 0 "#PWR0108" H 5600 2200 50  0001 C CNN
 F 1 "GND" H 5605 2277 50  0000 C CNN
 F 2 "" H 5600 2450 50  0001 C CNN
@@
 	5600 2300 5600 2400
 $Comp
-L Device:R R?
+L Device:R R2
 U 1 1 6111402F
 P 3150 2750
-F 0 "R?" V 3150 2700 50  0000 L CNN
+F 0 "R2" V 3150 2700 50  0000 L CNN
 F 1 "36.5K" V 3050 2650 50  0000 L CNN
 F 2 "Resistor_SMD:R_0402_1005Metric" V 3080 2750 50  0001 C CNN
@@
 $EndComp
 $Comp
-L Device:R R?
+L Device:R R1
 U 1 1 61113B66
 P 3150 2300
-F 0 "R?" V 3150 2250 50  0000 L CNN
+F 0 "R1" V 3150 2250 50  0000 L CNN
 F 1 "102K" V 3050 2200 50  0000 L CNN
 F 2 "Resistor_SMD:R_0402_1005Metric" V 3080 2300 50  0001 C CNN
@@
 $EndComp
 $Comp
-L power:GND #PWR?
+L power:GND #PWR0109
 U 1 1 61116DFC
 P 3150 2900
-F 0 "#PWR?" H 3150 2650 50  0001 C CNN
+F 0 "#PWR0109" H 3150 2650 50  0001 C CNN
 F 1 "GND" H 3155 2727 50  0000 C CNN
 F 2 "" H 3150 2900 50  0001 C CNN
@@
 	3150 2550 3450 2550
 $Comp
-L Device:R R?
+L Device:R R6
 U 1 1 6111DEF4
 P 8300 1850
-F 0 "R?" V 8300 1800 50  0000 L CNN
+F 0 "R6" V 8300 1800 50  0000 L CNN
 F 1 "102K" V 8200 1750 50  0000 L CNN
 F 2 "Resistor_SMD:R_0402_1005Metric" V 8230 1850 50  0001 C CNN
@@
 $EndComp
 $Comp
-L Device:R R?
+L Device:R R5
 U 1 1 6111E4B3
 P 7800 1700
-F 0 "R?" V 7800 1650 50  0000 L CNN
+F 0 "R5" V 7800 1650 50  0000 L CNN
 F 1 "53.6K" V 7700 1600 50  0000 L CNN
 F 2 "Resistor_SMD:R_0402_1005Metric" V 7730 1700 50  0001 C CNN
@@
 $EndComp
 $Comp
-L power:GND #PWR?
+L power:GND #PWR0110
 U 1 1 611237EC
 P 8300 2000
-F 0 "#PWR?" H 8300 1750 50  0001 C CNN
+F 0 "#PWR0110" H 8300 1750 50  0001 C CNN
 F 1 "GND" H 8305 1827 50  0000 C CNN
 F 2 "" H 8300 2000 50  0001 C CNN
@@
 $EndComp
 $Comp
-L Device:L L?
+L Device:L L1
 U 1 1 6113C80A
 P 6100 1700
-F 0 "L?" V 6200 1800 50  0000 C CNN
+F 0 "L1" V 6200 1800 50  0000 C CNN
 F 1 "4.7uH" V 6200 1600 50  0000 C CNN
 F 2 "dg_transformers:IND_1350" H 6100 1700 50  0001 C CNN
@@
 $EndComp
 $Comp
-L Device:C_Small C?
+L Device:C_Small C9
 U 1 1 6113D3E0
 P 5700 1400
-F 0 "C?" V 5650 1250 50  0000 L CNN
+F 0 "C9" V 5650 1250 50  0000 L CNN
 F 1 "100nF" V 5800 1300 50  0000 L CNN
 F 2 "Capacitor_SMD:C_0805_2012Metric" H 5700 1400 50  0001 C CNN
@@
 	6350 2000 6350 2150
 $Comp
-L power:GND #PWR?
+L power:GND #PWR0111
 U 1 1 6112B198
 P 7250 2150
-F 0 "#PWR?" H 7250 1900 50  0001 C CNN
+F 0 "#PWR0111" H 7250 1900 50  0001 C CNN
 F 1 "GND" H 7255 1977 50  0000 C CNN
 F 2 "" H 7250 2150 50  0001 C CNN
@@
 $EndComp
 $Comp
-L Device:C_Small C?
+L Device:C_Small C17
 U 1 1 61126AF1
 P 7250 1900
-F 0 "C?" H 7300 2000 50  0000 L CNN
+F 0 "C17" H 7300 2000 50  0000 L CNN
 F 1 "10uF 25V" V 7150 1700 50  0000 L CNN
 F 2 "Capacitor_SMD:C_1206_3216Metric" H 7250 1900 50  0001 C CNN
@@
 $EndComp
 $Comp
-L Device:C_Small C?
+L Device:C_Small C16
 U 1 1 611267EB
 P 6950 1900
-F 0 "C?" H 7000 2000 50  0000 L CNN
+F 0 "C16" H 7000 2000 50  0000 L CNN
 F 1 "10uF 25V" V 6850 1700 50  0000 L CNN
 F 2 "Capacitor_SMD:C_1206_3216Metric" H 6950 1900 50  0001 C CNN
@@
 $EndComp
 $Comp
-L Device:C_Small C?
+L Device:C_Small C15
 U 1 1 611264DE
 P 6650 1900
-F 0 "C?" H 6700 2000 50  0000 L CNN
+F 0 "C15" H 6700 2000 50  0000 L CNN
 F 1 "10uF 25V" V 6550 1700 50  0000 L CNN
 F 2 "Capacitor_SMD:C_1206_3216Metric" H 6650 1900 50  0001 C CNN
@@
 $EndComp
 $Comp
-L Device:C_Small C?
+L Device:C_Small C10
 U 1 1 61125B5C
 P 6350 1900
-F 0 "C?" H 6400 2000 50  0000 L CNN
+F 0 "C10" H 6400 2000 50  0000 L CNN
 F 1 "10uF 25V" V 6250 1700 50  0000 L CNN
 F 2 "Capacitor_SMD:C_1206_3216Metric" H 6350 1900 50  0001 C CNN

Commit message: maybe use a premade powerbrick
Parts:
- removed C1, C10, C15, C16, C17, C2: 10uF 25V, Capacitor_SMD:C_1206_3216Metric, symbol Device:C_Small
- removed C3: 15nF, Capacitor_SMD:C_0402_1005Metric, symbol Device:C_Small
- removed C4: 4.7uF 25V, Capacitor_SMD:C_0805_2012Metric, symbol Device:C_Small
- removed C7: 33nF, Capacitor_SMD:C_0402_1005Metric, symbol Device:C_Small
- removed C8: 68pF, Capacitor_SMD:C_0402_1005Metric, symbol Device:C_Small
- removed C9: 100nF, Capacitor_SMD:C_0805_2012Metric, symbol Device:C_Small
- removed L1: 4.7uH, dg_transformers:IND_1350, symbol Device:L
- removed R1, R6: 102K, Resistor_SMD:R_0402_1005Metric, symbol Device:R
- removed R2: 36.5K, Resistor_SMD:R_0402_1005Metric, symbol Device:R
- removed R4: 2.55K, Resistor_SMD:R_0402_1005Metric, symbol Device:R
- removed R5: 53.6K, Resistor_SMD:R_0402_1005Metric, symbol Device:R
- removed U4: TPS54620, dg_ic:Texas_S-PVQFN-N14_ThermalVias, symbol dg_ic:TPS54620
- removed U5: RT8065, dg_ic:DFN-8-1EP_3x3mm_P0.65mm_EP1.55x2.4mm, symbol dg_ic:RT8065
- added F?: Polyfuse, symbol Device:Polyfuse
- added IC2 (x2): OKR-T_6-W12-C, dg_power:MURATACASEC90, symbol dg_power:OKR-T_6-W12-C
- added J2: Conn_02x03_Counter_Clockwise, Connector_PinHeader_2.54mm:PinHeader_2x03_P2.54mm_Vertical, symbol Connector_Generic:Conn_02x03_Odd_Even
- added R2: 268, symbol Device:R
- added R2: 436, symbol Device:R
- R3: value 53.6K -> 100K; footprint Resistor_SMD:R_0402_1005Metric -> (none)
Connections:
- net labels added: VIN1, VIN2
- net labels removed: TPS_EN, TPS_PWRGD
- wire segments 78 -> 26
Other:
- note added: "best efficiency isnt entirely clear yet,\nwe can switch input for 3.3 between 5V and 12V here"
- note removed: "DNP Enable Resistors \nto disable UVLO."

Commit message: just use two usb hubs
Parts:
- gave numbers to parts that had none: 1
Changed lines of the file:
@@
 $Descr A4 11693 8268
 encoding utf-8
-Sheet 3 3
+Sheet 3 5
 Title ""
 Date ""
@@
 VIN1
 $Comp
-L Device:Polyfuse F?
+L Device:Polyfuse F1
 U 1 1 624CFE29
 P 800 800
-F 0 "F?" H 888 846 50  0000 L CNN
+F 0 "F1" H 888 846 50  0000 L CNN
 F 1 "Polyfuse" H 888 755 50  0000 L CNN
 F 2 "" H 850 600 50  0001 L CNN

Commit message: use native rpi uarts instead of extra chip
Parts:
- added R4: 1K, Resistor_SMD:R_0402_1005Metric_Pad0.72x0.64mm_HandSolder, symbol Device:R
- added RLA1: G3VM-61VY2-TR, dg_relay:G3VM-SOP, symbol dg_relay:G3VM-61VY2-TR
- R2: footprint (none) -> Resistor_SMD:R_0402_1005Metric_Pad0.72x0.64mm_HandSolder
- R3: value 100K -> DNC; footprint (none) -> Resistor_SMD:R_0402_1005Metric_Pad0.72x0.64mm_HandSolder
Connections:
- wire segments 26 -> 34
Other:
- moved on the sheet: R28
Changed lines of the file:
@@
 $Descr A4 11693 8268
 encoding utf-8
-Sheet 3 5
+Sheet 3 6
 Title ""
 Date ""
@@
 AR Path="/62171C70/61F5E18B" Ref="#PWR027"  Part="1"
 AR Path="/6218DDBF/61F5E18B" Ref="#PWR041"  Part="1"
-F 0 "#PWR0103" H 3050 1300 50  0001 C CNN
+AR Path="/61DCBD06/61F5E18B" Ref="#PWR0124"  Part="1"
+F 0 "#PWR0124" H 3050 1300 50  0001 C CNN
 F 1 "GND" H 3055 1377 50  0000 C CNN
 F 2 "" H 3050 1550 50  0001 C CNN
@@
 AR Path="/62171C70/6205DE31" Ref="IC7"  Part="1"
 AR Path="/6218DDBF/6205DE31" Ref="IC9"  Part="1"
-F 0 "IC1" H 5678 946 50  0000 L CNN
+AR Path="/61DCBD06/6205DE31" Ref="IC3"  Part="1"
+F 0 "IC3" H 5678 946 50  0000 L CNN
 F 1 "OKR-T_6-W12-C" H 5678 855 50  0000 L CNN
 F 2 "dg_power:MURATACASEC90" H 5700 1200 50  0001 L CNN
@@
 AR Path="/62171C70/6205EE37" Ref="R95"  Part="1"
 AR Path="/6218DDBF/6205EE37" Ref="R110"  Part="1"
-F 0 "R1" H 3520 1146 50  0000 L CNN
+AR Path="/61DCBD06/6205EE37" Ref="R14"  Part="1"
+F 0 "R14" H 3520 1146 50  0000 L CNN
 F 1 "268" H 3520 1055 50  0000 L CNN
-F 2 "" V 3380 1100 50  0001 C CNN
+F 2 "Resistor_SMD:R_0402_1005Metric_Pad0.72x0.64mm_HandSolder" V 3380 1100 50  0001 C CNN
 F 3 "~" H 3450 1100 50  0001 C CNN
 	1    3450 1100
@@
 AR Path="/62171C70/620C55C1" Ref="IC8"  Part="1"
 AR Path="/6218DDBF/620C55C1" Ref="IC10"  Part="1"
-F 0 "IC2" H 5678 2496 50  0000 L CNN
+AR Path="/61DCBD06/620C55C1" Ref="IC4"  Part="1"
+F 0 "IC4" H 5678 2496 50  0000 L CNN
 F 1 "OKR-T_6-W12-C" H 5678 2405 50  0000 L CNN
 F 2 "dg_power:MURATACASEC90" H 5700 2750 50  0001 L CNN
@@
 AR Path="/62171C70/620C890B" Ref="#PWR028"  Part="1"
 AR Path="/6218DDBF/620C890B" Ref="#PWR042"  Part="1"
-F 0 "#PWR0104" H 3050 2850 50  0001 C CNN
+AR Path="/61DCBD06/620C890B" Ref="#PWR0125"  Part="1"
+F 0 "#PWR0125" H 3050 2850 50  0001 C CNN
 F 1 "GND" H 3055 2927 50  0000 C CNN
 F 2 "" H 3050 3100 50  0001 C CNN
@@
 AR Path="/62171C70/620C8913" Ref="R96"  Part="1"
 AR Path="/6218DDBF/620C8913" Ref="R111"  Part="1"
-F 0 "R2" V 3657 2650 50  0000 C CNN
+AR Path="/61DCBD06/620C8913" Ref="R15"  Part="1"
+F 0 "R15" V 3657 2650 50  0000 C CNN
 F 1 "436" V 3566 2650 50  0000 C CNN
-F 2 "" V 3380 2650 50  0001 C CNN
+F 2 "Resistor_SMD:R_0402_1005Metric_Pad0.72x0.64mm_HandSolder" V 3380 2650 50  0001 C CNN
 F 3 "~" H 3450 2650 50  0001 C CNN
 	1    3450 2650
@@
 AR Path="/62171C70/620CBF19" Ref="J12"  Part="1"
 AR Path="/6218DDBF/620CBF19" Ref="J13"  Part="1"
-F 0 "J2" V 2004 2380 50  0000 L CNN
+AR Path="/61DCBD06/620CBF19" Ref="J4"  Part="1"
+F 0 "J4" V 2004 2380 50  0000 L CNN
 F 1 "Conn_02x03_Counter_Clockwise" V 2095 2380 50  0000 L CNN
 F 2 "Connector_PinHeader_2.54mm:PinHeader_2x03_P2.54mm_Vertical" H 2000 2200 50  0001 C CNN
@@
 L Device:R R?
 U 1 1 620D7FAF
-P 1950 1000
+P 3900 3900
 AR Path="/611D29B0/620D7FAF" Ref="R?"  Part="1"
 AR Path="/613B6F05/620D7FAF" Ref="R3"  Part="1"
@@
 AR Path="/62171C70/620D7FAF" Ref="R93"  Part="1"
 AR Path="/6218DDBF/620D7FAF" Ref="R109"  Part="1"
-F 0 "R3" V 2157 1000 50  0000 C CNN
-F 1 "100K" V 2066 1000 50  0000 C CNN
-F 2 "" V 1880 1000 50  0001 C CNN
-F 3 "~" H 1950 1000 50  0001 C CNN
-	1    1950 1000
-	0    -1   -1   0
-$EndComp
-Text HLabel 1750 1000 0    50   Input ~ 0
+AR Path="/61DCBD06/620D7FAF" Ref="R28"  Part="1"
+F 0 "R28" V 4107 3900 50  0000 C CNN
+F 1 "DNC" V 4016 3900 50  0000 C CNN
+F 2 "Resistor_SMD:R_0402_1005Metric_Pad0.72x0.64mm_HandSolder" V 3830 3900 50  0001 C CNN
+F 3 "~" H 3900 3900 50  0001 C CNN
+	1    3900 3900
+	-1   0    0    1
+$EndComp
+Text HLabel 1950 4200 0    50   Input ~ 0
 DISABLE
 Wire Wire Line
-	1800 1000 1750 1000
-Wire Wire Line
-	2200 1000 2100 1000
+	3900 3650 3900 3750
 Text Notes 1000 3400 1    50   ~ 0
 best efficiency isnt entirely clear yet,\nwe can switch input for 3.3 between 5V and 12V here
@@
 Text Label 3900 1400 2    50   ~ 0
 VIN1
-Text Label 2200 1000 0    50   ~ 0
+Text Label 3900 3650 1    50   ~ 0
 VIN1
 $Comp
@@
 U 1 1 624CFE29
 P 800 800
-F 0 "F1" H 888 846 50  0000 L CNN
+AR Path="/613B6F05/624CFE29" Ref="F1"  Part="1"
+AR Path="/61DCBD06/624CFE29" Ref="F2"  Part="1"
+F 0 "F2" H 888 846 50  0000 L CNN
 F 1 "Polyfuse" H 888 755 50  0000 L CNN
 F 2 "" H 850 600 50  0001 L CNN
@@
 	1    0    0    -1
 $EndComp
+$Comp
+L dg_relay:G3VM-61VY2-TR RLA1
+U 1 1 61CDA64C
+P 2450 4100
+AR Path="/613B6F05/61CDA64C" Ref="RLA1"  Part="1"
+AR Path="/61DCBD06/61CDA64C" Ref="RLA2"  Part="1"
+F 0 "RLA2" H 3150 4327 60  0000 C CNN
+F 1 "G3VM-61VY2-TR" H 3150 4221 60  0000 C CNN
+F 2 "dg_relay:G3VM-SOP" H 3350 4240 60  0001 C CNN
+F 3 "https://www.mouser.de/datasheet/2/307/omron_04102018_G3VM-6_G__61VY1_DS_E-1317117.pdf" H 2450 4100 60  0001 C CNN
+F 4 "C306896" H 3150 4123 50  0000 C CNN "LCSC#"
+	1    2450 4100
+	1    0    0    -1
+$EndComp
+Text HLabel 4100 4200 2    50   Input ~ 0
+DISABLE
+Wire Wire Line
+	3700 4200 3900 4200
+Wire Wire Line
+	3900 4050 3900 4200
+Connection ~ 3900 4200
+Wire Wire Line
+	3900 4200 4100 4200
+$Comp
+L power:GND #PWR0116
+U 1 1 61CE1EC9
+P 2300 4700
+AR Path="/613B6F05/61CE1EC9" Ref="#PWR0116"  Part="1"
+AR Path="/611D29B0/61CE1EC9" Ref="#PWR?"  Part="1"
+AR Path="/620E19B9/61CE1EC9" Ref="#PWR?"  Part="1"
+AR Path="/620FBA52/61CE1EC9" Ref="#PWR?"  Part="1"
+AR Path="/62117961/61CE1EC9" Ref="#PWR?"  Part="1"
+AR Path="/62132900/61CE1EC9" Ref="#PWR?"  Part="1"
+AR Path="/62156477/61CE1EC9" Ref="#PWR?"  Part="1"
+AR Path="/62171C70/61CE1EC9" Ref="#PWR?"  Part="1"
+AR Path="/6218DDBF/61CE1EC9" Ref="#PWR?"  Part="1"
+AR Path="/61DCBD06/61CE1EC9" Ref="#PWR0126"  Part="1"
+F 0 "#PWR0126" H 2300 4450 50  0001 C CNN
+F 1 "GND" H 2305 4527 50  0000 C CNN
+F 2 "" H 2300 4700 50  0001 C CNN
+F 3 "" H 2300 4700 50  0001 C CNN
+	1    2300 4700
+	1    0    0    -1
+$EndComp
+Wire Wire Line
+	2300 4700 2300 4600
+Wire Wire Line
+	2300 4600 2600 4600
+$Comp
+L power:GND #PWR0117
+U 1 1 61CE3867
+P 4000 4700
+AR Path="/613B6F05/61CE3867" Ref="#PWR0117"  Part="1"
+AR Path="/611D29B0/61CE3867" Ref="#PWR?"  Part="1"
+AR Path="/620E19B9/61CE3867" Ref="#PWR?"  Part="1"
+AR Path="/620FBA52/61CE3867" Ref="#PWR?"  Part="1"
+AR Path="/62117961/61CE3867" Ref="#PWR?"  Part="1"
+AR Path="/62132900/61CE3867" Ref="#PWR?"  Part="1"
+AR Path="/62156477/61CE3867" Ref="#PWR?"  Part="1"
+AR Path="/62171C70/61CE3867" Ref="#PWR?"  Part="1"
+AR Path="/6218DDBF/61CE3867" Ref="#PWR?"  Part="1"
+AR Path="/61DCBD06/61CE3867" Ref="#PWR0127"  Part="1"
+F 0 "#PWR0127" H 4000 4450 50  0001 C CNN
+F 1 "GND" H 4005 4527 50  0000 C CNN
+F 2 "" H 4000 4700 50  0001 C CNN
+F 3 "" H 4000 4700 50  0001 C CNN
+	1    4000 4700
+	-1   0    0    -1
+$EndComp
+Wire Wire Line
+	4000 4700 4000 4600
+Wire Wire Line
+	4000 4600 3700 4600
+$Comp
+L Device:R R?
+U 1 1 61CE43D9
+P 2350 4200
+AR Path="/611D29B0/61CE43D9" Ref="R?"  Part="1"
+AR Path="/613B6F05/61CE43D9" Ref="R4"  Part="1"
+AR Path="/620E19B9/61CE43D9" Ref="R?"  Part="1"
+AR Path="/620FBA52/61CE43D9" Ref="R?"  Part="1"
+AR Path="/62117961/61CE43D9" Ref="R?"  Part="1"
+AR Path="/62132900/61CE43D9" Ref="R?"  Part="1"
+AR Path="/62156477/61CE43D9" Ref="R?"  Part="1"
+AR Path="/62171C70/61CE43D9" Ref="R?"  Part="1"
+AR Path="/6218DDBF/61CE43D9" Ref="R?"  Part="1"
+AR Path="/61DCBD06/61CE43D9" Ref="R13"  Part="1"
+F 0 "R13" V 2557 4200 50  0000 C CNN
+F 1 "1K" V 2466 4200 50  0000 C CNN
+F 2 "Resistor_SMD:R_0402_1005Metric_Pad0.72x0.64mm_HandSolder" V 2280 4200 50  0001 C CNN
+F 3 "~" H 2350 4200 50  0001 C CNN
+	1    2350 4200
+	0    -1   -1   0
+$EndComp
+Wire Wire Line
+	1950 4200 2200 4200
+Wire Wire Line
+	2500 4200 2600 4200
 $EndSCHEMATC
