File: dcdc.sch (KiCad schematic (older format))
At the start: 9 parts, among them IC2 OKR-T_6-W12-C, J2 Conn_02x03_Counter_Clockwise

Commit message: Organized DC-DC Schematic.
Parts:
- removed IC2: OKR-T_6-W12-C, dg_power:MURATACASEC90, symbol dg_power:OKR-T_6-W12-C
- removed R2: 436, Resistor_SMD:R_0402_1005Metric_Pad0.72x0.64mm_HandSolder, symbol Device:R
- added D? (x2): LED, LED_SMD:LED_0603_1608Metric, symbol Device:LED
- added IC?: OKR-T_6-W12-C, dg_power:MURATACASEC90, symbol dg_power:OKR-T_6-W12-C
- added R? (x2): 1k, Resistor_SMD:R_0402_1005Metric, symbol Device:R
- added R?: 436, Resistor_SMD:R_0402_1005Metric_Pad0.72x0.64mm_HandSolder, symbol Device:R
- J2: value Conn_02x03_Counter_Clockwise -> Header_2x6_2.54mm
Connections:
- net labels added: VIN_3V3_DCDC, VIN_5V_DCDC
- net labels removed: VIN2
Other:
- note added: "Best efficiency isnt entirely clear yet,\nWe can switch input for 3.3 between 5V and 12V here"
- note added: "RTRIM (kOhm) = 1.182 / (Vout-0.591)"
- note added: "RTRIM_3V3 = 436 = 1.182 / (3.3-0.591)"
- note added: "RTRIM_5V = 268 = 1.182 / (5-0.591)"
- note removed: "best efficiency isnt entirely clear yet,\nwe can switch input for 3.3 between 5V and 12V here"
- moved on the sheet: F1, IC1, J2, R1, R3, R4, RLA1

Commit message: Organized sch.
Parts:
- removed R3: DNC, Resistor_SMD:R_0402_1005Metric_Pad0.72x0.64mm_HandSolder, symbol Device:R
- added R?: 1k, Resistor_SMD:R_0402_1005Metric, symbol Device:R
- added R?: DNC, Resistor_SMD:R_0402_1005Metric, symbol Device:R
Connections:
- net labels added: DISABLE_DCDC, VIN_DCDC_3V3, VIN_DCDC_5V
- net labels removed: VIN1, VIN_3V3_DCDC, VIN_5V_DCDC
Other:
- note added: "Jumper to Bypass Mosfet Disable Control."
- moved on the sheet: R4, RLA1

Commit message: Organized pi.sch document.
Other:
- moved on the sheet: D?, F1, IC1, IC?, J2, R1, R4, R?, RLA1

Commit message: Revised main schematic.
Connections:
- net labels added: 3V3
- net labels removed: 3.3V
Changed lines of the file:
@@
 	7800 2650 7900 2650
 Text HLabel 7250 1900 0    50   Input ~ 0
-3.3V
+3V3
 $Comp
 L Device:LED D?
@@
 VIN_DCDC_3V3
 Text HLabel 4450 2500 0    50   Input ~ 0
-3.3V
+3V3
 $Comp
 L Device:R R?

Commit message: move BEL rj45 to dg library
Changed lines of the file:
@@
 $Descr A4 11693 8268
 encoding utf-8
-Sheet 3 6
+Sheet 5 6
 Title ""
 Date ""
@@
 AR Path="/6218DDBF/61F5E18B" Ref="#PWR041"  Part="1"
 AR Path="/61DCBD06/61F5E18B" Ref="#PWR0124"  Part="1"
-F 0 "#PWR0103" H 4000 1550 50  0001 C CNN
+F 0 "#PWR0124" H 4000 1550 50  0001 C CNN
 F 1 "GND" H 4005 1627 50  0000 C CNN
 F 2 "" H 4000 1800 50  0001 C CNN
@@
 AR Path="/6218DDBF/6205DE31" Ref="IC9"  Part="1"
 AR Path="/61DCBD06/6205DE31" Ref="IC3"  Part="1"
-F 0 "IC1" H 6000 1750 50  0000 L CNN
+F 0 "IC3" H 6000 1750 50  0000 L CNN
 F 1 "OKR-T_6-W12-C" H 5450 1650 50  0000 L CNN
 F 2 "dg_power:MURATACASEC90" H 6200 1700 50  0001 L CNN
@@
 AR Path="/6218DDBF/6205EE37" Ref="R110"  Part="1"
 AR Path="/61DCBD06/6205EE37" Ref="R14"  Part="1"
-F 0 "R1" V 4250 1550 50  0000 L CNN
+F 0 "R14" V 4250 1550 50  0000 L CNN
 F 1 "268" V 4150 1500 50  0000 L CNN
 F 2 "Resistor_SMD:R_0402_1005Metric_Pad0.72x0.64mm_HandSolder" V 4080 1600 50  0001 C CNN
@@
 AR Path="/6218DDBF/620CBF19" Ref="J13"  Part="1"
 AR Path="/61DCBD06/620CBF19" Ref="J4"  Part="1"
-F 0 "J2" H 2400 2700 50  0000 L CNN
+F 0 "J4" H 2400 2700 50  0000 L CNN
 F 1 "Header_2x6_2.54mm" H 2050 2250 50  0000 L CNN
 F 2 "Connector_PinHeader_2.54mm:PinHeader_2x03_P2.54mm_Vertical" H 2400 2500 50  0001 C CNN
@@
 AR Path="/613B6F05/624CFE29" Ref="F1"  Part="1"
 AR Path="/61DCBD06/624CFE29" Ref="F2"  Part="1"
-F 0 "F1" V 2400 1550 50  0000 L CNN
+F 0 "F2" V 2400 1550 50  0000 L CNN
 F 1 "Polyfuse" V 2200 1400 50  0000 L CNN
 F 2 "" H 2350 1400 50  0001 L CNN
@@
 AR Path="/613B6F05/61CDA64C" Ref="RLA1"  Part="1"
 AR Path="/61DCBD06/61CDA64C" Ref="RLA2"  Part="1"
-F 0 "RLA1" H 8450 2777 60  0000 C CNN
+F 0 "RLA2" H 8450 2777 60  0000 C CNN
 F 1 "G3VM-61VY2-TR" H 8450 2671 60  0000 C CNN
 F 2 "dg_relay:G3VM-SOP" H 8650 2690 60  0001 C CNN
@@
 AR Path="/6218DDBF/61CE3867" Ref="#PWR?"  Part="1"
 AR Path="/61DCBD06/61CE3867" Ref="#PWR0127"  Part="1"
-F 0 "#PWR0117" H 9000 2900 50  0001 C CNN
+F 0 "#PWR0127" H 9000 2900 50  0001 C CNN
 F 1 "GND" H 9005 2977 50  0000 C CNN
 F 2 "" H 9000 3150 50  0001 C CNN
@@
 AR Path="/6218DDBF/61CE43D9" Ref="R?"  Part="1"
 AR Path="/61DCBD06/61CE43D9" Ref="R13"  Part="1"
-F 0 "R4" V 7857 2650 50  0000 C CNN
+F 0 "R13" V 7857 2650 50  0000 C CNN
 F 1 "1K" V 7766 2650 50  0000 C CNN
 F 2 "Resistor_SMD:R_0402_1005Metric_Pad0.72x0.64mm_HandSolder" V 7580 2650 50  0001 C CNN
@@
 AR Path="/6218DDB9/611489B3" Ref="D?"  Part="1"
 AR Path="/613B6F05/611489B3" Ref="D?"  Part="1"
+AR Path="/61DCBD06/611489B3" Ref="D?"  Part="1"
 F 0 "D?" H 7600 1550 50  0000 C CNN
 F 1 "LED" H 7350 1700 50  0000 C CNN
@@
 AR Path="/6218DDB9/611489C2" Ref="D?"  Part="1"
 AR Path="/613B6F05/611489C2" Ref="D?"  Part="1"
+AR Path="/61DCBD06/611489C2" Ref="D?"  Part="1"
 F 0 "D?" H 7600 1800 50  0000 C CNN
 F 1 "LED" H 7350 1950 50  0000 C CNN
@@
 AR Path="/6218DDB9/611489D8" Ref="#PWR?"  Part="1"
 AR Path="/613B6F05/611489D8" Ref="#PWR?"  Part="1"
+AR Path="/61DCBD06/611489D8" Ref="#PWR?"  Part="1"
 F 0 "#PWR?" H 8250 1400 50  0001 C CNN
 F 1 "GND" H 8255 1477 50  0000 C CNN
@@
 AR Path="/6218DDB9/6114B6A4" Ref="#PWR?"  Part="1"
 AR Path="/613B6F05/6114B6A4" Ref="#PWR?"  Part="1"
+AR Path="/61DCBD06/6114B6A4" Ref="#PWR?"  Part="1"
 F 0 "#PWR?" H 8250 1650 50  0001 C CNN
 F 1 "GND" H 8255 1727 50  0000 C CNN

Commit message: use a 2x2 and a magjack
Parts:
- gave numbers to parts that had none: 8
Changed lines of the file:
@@
 AR Path="/62171C6A/611489B3" Ref="D?"  Part="1"
 AR Path="/6218DDB9/611489B3" Ref="D?"  Part="1"
-AR Path="/613B6F05/611489B3" Ref="D?"  Part="1"
-AR Path="/61DCBD06/611489B3" Ref="D?"  Part="1"
-F 0 "D?" H 7600 1550 50  0000 C CNN
+AR Path="/613B6F05/611489B3" Ref="D8"  Part="1"
+AR Path="/61DCBD06/611489B3" Ref="D10"  Part="1"
+F 0 "D10" H 7600 1550 50  0000 C CNN
 F 1 "LED" H 7350 1700 50  0000 C CNN
 F 2 "LED_SMD:LED_0603_1608Metric" H 7500 1650 50  0001 C CNN
@@
 AR Path="/62171C6A/611489C2" Ref="D?"  Part="1"
 AR Path="/6218DDB9/611489C2" Ref="D?"  Part="1"
-AR Path="/613B6F05/611489C2" Ref="D?"  Part="1"
-AR Path="/61DCBD06/611489C2" Ref="D?"  Part="1"
-F 0 "D?" H 7600 1800 50  0000 C CNN
+AR Path="/613B6F05/611489C2" Ref="D9"  Part="1"
+AR Path="/61DCBD06/611489C2" Ref="D11"  Part="1"
+F 0 "D11" H 7600 1800 50  0000 C CNN
 F 1 "LED" H 7350 1950 50  0000 C CNN
 F 2 "LED_SMD:LED_0603_1608Metric" H 7500 1900 50  0001 C CNN
@@
 AR Path="/62171C6A/611489D8" Ref="#PWR?"  Part="1"
 AR Path="/6218DDB9/611489D8" Ref="#PWR?"  Part="1"
-AR Path="/613B6F05/611489D8" Ref="#PWR?"  Part="1"
-AR Path="/61DCBD06/611489D8" Ref="#PWR?"  Part="1"
-F 0 "#PWR?" H 8250 1400 50  0001 C CNN
+AR Path="/613B6F05/611489D8" Ref="#PWR0126"  Part="1"
+AR Path="/61DCBD06/611489D8" Ref="#PWR0135"  Part="1"
+F 0 "#PWR0135" H 8250 1400 50  0001 C CNN
 F 1 "GND" H 8255 1477 50  0000 C CNN
 F 2 "" H 8250 1650 50  0001 C CNN
@@
 P 7950 1650
 AR Path="/611D29B0/61149574" Ref="R?"  Part="1"
-AR Path="/613B6F05/61149574" Ref="R?"  Part="1"
+AR Path="/613B6F05/61149574" Ref="R3"  Part="1"
 AR Path="/620E19B9/61149574" Ref="R?"  Part="1"
 AR Path="/620FBA52/61149574" Ref="R?"  Part="1"
@@
 AR Path="/62171C70/61149574" Ref="R?"  Part="1"
 AR Path="/6218DDBF/61149574" Ref="R?"  Part="1"
-AR Path="/61DCBD06/61149574" Ref="R?"  Part="1"
-F 0 "R?" V 8050 1650 50  0000 C CNN
+AR Path="/61DCBD06/61149574" Ref="R21"  Part="1"
+F 0 "R21" V 8050 1650 50  0000 C CNN
 F 1 "1k" V 7950 1650 50  0000 C CNN
 F 2 "Resistor_SMD:R_0402_1005Metric" V 7880 1650 50  0001 C CNN
@@
 AR Path="/62171C6A/6114B6A4" Ref="#PWR?"  Part="1"
 AR Path="/6218DDB9/6114B6A4" Ref="#PWR?"  Part="1"
-AR Path="/613B6F05/6114B6A4" Ref="#PWR?"  Part="1"
-AR Path="/61DCBD06/6114B6A4" Ref="#PWR?"  Part="1"
-F 0 "#PWR?" H 8250 1650 50  0001 C CNN
+AR Path="/613B6F05/6114B6A4" Ref="#PWR0128"  Part="1"
+AR Path="/61DCBD06/6114B6A4" Ref="#PWR0137"  Part="1"
+F 0 "#PWR0137" H 8250 1650 50  0001 C CNN
 F 1 "GND" H 8255 1727 50  0000 C CNN
 F 2 "" H 8250 1900 50  0001 C CNN
@@
 P 7950 1900
 AR Path="/611D29B0/6114B6AB" Ref="R?"  Part="1"
-AR Path="/613B6F05/6114B6AB" Ref="R?"  Part="1"
+AR Path="/613B6F05/6114B6AB" Ref="R15"  Part="1"
 AR Path="/620E19B9/6114B6AB" Ref="R?"  Part="1"
 AR Path="/620FBA52/6114B6AB" Ref="R?"  Part="1"
@@
 AR Path="/62171C70/6114B6AB" Ref="R?"  Part="1"
 AR Path="/6218DDBF/6114B6AB" Ref="R?"  Part="1"
-AR Path="/61DCBD06/6114B6AB" Ref="R?"  Part="1"
-F 0 "R?" V 8050 1900 50  0000 C CNN
+AR Path="/61DCBD06/6114B6AB" Ref="R22"  Part="1"
+F 0 "R22" V 8050 1900 50  0000 C CNN
 F 1 "1k" V 7950 1900 50  0000 C CNN
 F 2 "Resistor_SMD:R_0402_1005Metric" V 7880 1900 50  0001 C CNN
@@
 	4300 1600 4550 1600
 $Comp
-L power:GND #PWR?
+L power:GND #PWR0129
 U 1 1 6115EC66
 P 4000 1600
-AR Path="/613B6F05/6115EC66" Ref="#PWR?"  Part="1"
+AR Path="/613B6F05/6115EC66" Ref="#PWR0129"  Part="1"
 AR Path="/611D29B0/6115EC66" Ref="#PWR?"  Part="1"
 AR Path="/620E19B9/6115EC66" Ref="#PWR?"  Part="1"
@@
 AR Path="/62171C70/6115EC66" Ref="#PWR?"  Part="1"
 AR Path="/6218DDBF/6115EC66" Ref="#PWR?"  Part="1"
-AR Path="/61DCBD06/6115EC66" Ref="#PWR?"  Part="1"
-F 0 "#PWR?" H 4000 1350 50  0001 C CNN
+AR Path="/61DCBD06/6115EC66" Ref="#PWR0139"  Part="1"
+F 0 "#PWR0139" H 4000 1350 50  0001 C CNN
 F 1 "GND" H 4005 1427 50  0000 C CNN
 F 2 "" H 4000 1600 50  0001 C CNN
@@
 	4000 1800 4550 1800
 $Comp
-L power:GND #PWR?
+L power:GND #PWR0130
 U 1 1 61162826
 P 4000 2600
-AR Path="/613B6F05/61162826" Ref="#PWR?"  Part="1"
+AR Path="/613B6F05/61162826" Ref="#PWR0130"  Part="1"
 AR Path="/611D29B0/61162826" Ref="#PWR?"  Part="1"
 AR Path="/620E19B9/61162826" Ref="#PWR?"  Part="1"
@@
 AR Path="/62171C70/61162826" Ref="#PWR?"  Part="1"
 AR Path="/6218DDBF/61162826" Ref="#PWR?"  Part="1"
-AR Path="/61DCBD06/61162826" Ref="#PWR?"  Part="1"
-F 0 "#PWR?" H 4000 2350 50  0001 C CNN
+AR Path="/61DCBD06/61162826" Ref="#PWR0140"  Part="1"
+F 0 "#PWR0140" H 4000 2350 50  0001 C CNN
 F 1 "GND" H 4005 2427 50  0000 C CNN
 F 2 "" H 4000 2600 50  0001 C CNN
@@
 P 4550 2400
 AR Path="/611D29B0/61162834" Ref="IC?"  Part="1"
-AR Path="/613B6F05/61162834" Ref="IC?"  Part="1"
+AR Path="/613B6F05/61162834" Ref="IC2"  Part="1"
 AR Path="/620E19B9/61162834" Ref="IC?"  Part="1"
 AR Path="/620FBA52/61162834" Ref="IC?"  Part="1"
@@
 AR Path="/62171C70/61162834" Ref="IC?"  Part="1"
 AR Path="/6218DDBF/61162834" Ref="IC?"  Part="1"
-AR Path="/61DCBD06/61162834" Ref="IC?"  Part="1"
-F 0 "IC?" H 6000 2550 50  0000 L CNN
+AR Path="/61DCBD06/61162834" Ref="IC4"  Part="1"
+F 0 "IC4" H 6000 2550 50  0000 L CNN
 F 1 "OKR-T_6-W12-C" H 5450 2450 50  0000 L CNN
 F 2 "dg_power:MURATACASEC90" H 6200 2500 50  0001 L CNN
@@
 P 4150 2400
 AR Path="/611D29B0/6116283A" Ref="R?"  Part="1"
-AR Path="/613B6F05/6116283A" Ref="R?"  Part="1"
+AR Path="/613B6F05/6116283A" Ref="R2"  Part="1"
 AR Path="/620E19B9/6116283A" Ref="R?"  Part="1"
 AR Path="/620FBA52/6116283A" Ref="R?"  Part="1"
@@
 AR Path="/62171C70/6116283A" Ref="R?"  Part="1"
 AR Path="/6218DDBF/6116283A" Ref="R?"  Part="1"
-AR Path="/61DCBD06/6116283A" Ref="R?"  Part="1"
-F 0 "R?" V 4250 2350 50  0000 L CNN
+AR Path="/61DCBD06/6116283A" Ref="R20"  Part="1"
+F 0 "R20" V 4250 2350 50  0000 L CNN
 F 1 "436" V 4150 2300 50  0000 L CNN
 F 2 "Resistor_SMD:R_0402_1005Metric_Pad0.72x0.64mm_HandSolder" V 4080 2400 50  0001 C CNN
@@
 	4300 2400 4550 2400
 $Comp
-L power:GND #PWR?
+L power:GND #PWR0131
 U 1 1 61162845
 P 4000 2400
-AR Path="/613B6F05/61162845" Ref="#PWR?"  Part="1"
+AR Path="/613B6F05/61162845" Ref="#PWR0131"  Part="1"
 AR Path="/611D29B0/61162845" Ref="#PWR?"  Part="1"
 AR Path="/620E19B9/61162845" Ref="#PWR?"  Part="1"
@@
 AR Path="/62171C70/61162845" Ref="#PWR?"  Part="1"
 AR Path="/6218DDBF/61162845" Ref="#PWR?"  Part="1"
-AR Path="/61DCBD06/61162845" Ref="#PWR?"  Part="1"
-F 0 "#PWR?" H 4000 2150 50  0001 C CNN
+AR Path="/61DCBD06/61162845" Ref="#PWR0141"  Part="1"
+F 0 "#PWR0141" H 4000 2150 50  0001 C CNN
 F 1 "GND" H 4005 2227 50  0000 C CNN
 F 2 "" H 4000 2400 50  0001 C CNN
@@
 P 9200 2450
 AR Path="/611D29B0/6116D895" Ref="R?"  Part="1"
-AR Path="/613B6F05/6116D895" Ref="R?"  Part="1"
+AR Path="/613B6F05/6116D895" Ref="R18"  Part="1"
 AR Path="/620E19B9/6116D895" Ref="R?"  Part="1"
 AR Path="/620FBA52/6116D895" Ref="R?"  Part="1"
@@
 AR Path="/62171C70/6116D895" Ref="R?"  Part="1"
 AR Path="/6218DDBF/6116D895" Ref="R?"  Part="1"
-AR Path="/61DCBD06/6116D895" Ref="R?"  Part="1"
-F 0 "R?" V 9300 2450 50  0000 C CNN
+AR Path="/61DCBD06/6116D895" Ref="R23"  Part="1"
+F 0 "R23" V 9300 2450 50  0000 C CNN
 F 1 "1k" V 9200 2450 50  0000 C CNN
 F 2 "Resistor_SMD:R_0402_1005Metric" V 9130 2450 50  0001 C CNN
@@
 	9350 2450 9850 2450
 $Comp
-L power:GND #PWR?
+L power:GND #PWR0134
 U 1 1 61173063
 P 7900 3150
-AR Path="/613B6F05/61173063" Ref="#PWR?"  Part="1"
+AR Path="/613B6F05/61173063" Ref="#PWR0134"  Part="1"
 AR Path="/611D29B0/61173063" Ref="#PWR?"  Part="1"
 AR Path="/620E19B9/61173063" Ref="#PWR?"  Part="1"
@@
 AR Path="/62171C70/61173063" Ref="#PWR?"  Part="1"
 AR Path="/6218DDBF/61173063" Ref="#PWR?"  Part="1"
-AR Path="/61DCBD06/61173063" Ref="#PWR?"  Part="1"
-F 0 "#PWR?" H 7900 2900 50  0001 C CNN
+AR Path="/61DCBD06/61173063" Ref="#PWR0142"  Part="1"
+F 0 "#PWR0142" H 7900 2900 50  0001 C CNN
 F 1 "GND" H 7905 2977 50  0000 C CNN
 F 2 "" H 7900 3150 50  0001 C CNN
@@
 P 9250 1650
 AR Path="/611D29B0/61184138" Ref="R?"  Part="1"
-AR Path="/613B6F05/61184138" Ref="R?"  Part="1"
+AR Path="/613B6F05/61184138" Ref="R19"  Part="1"
 AR Path="/620E19B9/61184138" Ref="R?"  Part="1"
 AR Path="/620FBA52/61184138" Ref="R?"  Part="1"
@@
 AR Path="/62171C70/61184138" Ref="R?"  Part="1"
 AR Path="/6218DDBF/61184138" Ref="R?"  Part="1"
-AR Path="/61DCBD06/61184138" Ref="R?"  Part="1"
-F 0 "R?" V 9350 1650 50  0000 C CNN
+AR Path="/61DCBD06/61184138" Ref="R28"  Part="1"
+F 0 "R28" V 9350 1650 50  0000 C CNN
 F 1 "DNC" V 9250 1650 50  0000 C CNN
 F 2 "Resistor_SMD:R_0402_1005Metric" V 9180 1650 50  0001 C CNN
