File: dcdc.sch (KiCad schematic (older format))
At the start: 14 parts, among them IC1 OKR-T_6-W12-C, IC2 OKR-T_6-W12-C, J7 Header_2x6_2.54mm

Commit message: Changed fuse footprint and updated Part num.
Parts:
- F1: footprint Fuse:Fuse_1210_3225Metric_Castellated -> Fuse:Fuse_2920_7451Metric_Castellated; #LCSC (none) -> C315905
Changed lines of the file:
@@
 $Descr A4 11693 8268
 encoding utf-8
-Sheet 11 12
+Sheet 7 12
 Title ""
 Date ""
@@
 AR Path="/6144BA6D/61F5E18B" Ref="#PWR079"  Part="1"
 AR Path="/614B514C/61F5E18B" Ref="#PWR097"  Part="1"
-F 0 "#PWR016" H 4000 1550 50  0001 C CNN
+F 0 "#PWR079" H 4000 1550 50  0001 C CNN
 F 1 "GND" H 4005 1627 50  0000 C CNN
 F 2 "" H 4000 1800 50  0001 C CNN
@@
 AR Path="/6144BA6D/6205DE31" Ref="IC7"  Part="1"
 AR Path="/614B514C/6205DE31" Ref="IC9"  Part="1"
-F 0 "IC1" H 6000 1750 50  0000 L CNN
+F 0 "IC7" H 6000 1750 50  0000 L CNN
 F 1 "OKR-T_6-W12-C" H 5450 1650 50  0000 L CNN
 F 2 "dg_power:MURATACASEC90" H 6200 1700 50  0001 L CNN
@@
 AR Path="/6144BA6D/6205EE37" Ref="R50"  Part="1"
 AR Path="/614B514C/6205EE37" Ref="R64"  Part="1"
-F 0 "R1" V 4250 1550 50  0000 L CNN
+F 0 "R50" V 4250 1550 50  0000 L CNN
 F 1 "268" V 4150 1500 50  0000 L CNN
 F 2 "Resistor_SMD:R_0402_1005Metric_Pad0.72x0.64mm_HandSolder" V 4080 1600 50  0001 C CNN
@@
 AR Path="/6144BA6D/620CBF19" Ref="J11"  Part="1"
 AR Path="/614B514C/620CBF19" Ref="J12"  Part="1"
-F 0 "J7" H 2400 2700 50  0000 L CNN
+F 0 "J11" H 2400 2700 50  0000 L CNN
 F 1 "Header_2x6_2.54mm" H 2050 2250 50  0000 L CNN
 F 2 "Connector_PinHeader_2.54mm:PinHeader_2x03_P2.54mm_Vertical" H 2400 2500 50  0001 C CNN
@@
 AR Path="/6144BA6D/624CFE29" Ref="F4"  Part="1"
 AR Path="/614B514C/624CFE29" Ref="F5"  Part="1"
-F 0 "F1" V 2400 1550 50  0000 L CNN
+F 0 "F4" V 2400 1550 50  0000 L CNN
 F 1 "Polyfuse" V 2200 1400 50  0000 L CNN
-F 2 "Fuse:Fuse_1210_3225Metric_Castellated" H 2350 1400 50  0001 L CNN
+F 2 "Fuse:Fuse_2920_7451Metric_Castellated" H 2350 1400 50  0001 L CNN
 F 3 "~" H 2300 1600 50  0001 C CNN
+F 4 "C315905" V 2300 1600 50  0001 C CNN "#LCSC"
 	1    2300 1600
 	0    -1   -1   0
@@
 AR Path="/6144BA6D/61CDA64C" Ref="RLA4"  Part="1"
 AR Path="/614B514C/61CDA64C" Ref="RLA5"  Part="1"
-F 0 "RLA1" H 8450 2777 60  0000 C CNN
+F 0 "RLA4" H 8450 2777 60  0000 C CNN
 F 1 "G3VM-61VY2-TR" H 8450 2671 60  0000 C CNN
 F 2 "dg_relay:G3VM-SOP" H 8650 2690 60  0001 C CNN
@@
 AR Path="/6144BA6D/61CE3867" Ref="#PWR085"  Part="1"
 AR Path="/614B514C/61CE3867" Ref="#PWR0103"  Part="1"
-F 0 "#PWR022" H 9000 2900 50  0001 C CNN
+F 0 "#PWR085" H 9000 2900 50  0001 C CNN
 F 1 "GND" H 9005 2977 50  0000 C CNN
 F 2 "" H 9000 3150 50  0001 C CNN
@@
 AR Path="/6144BA6D/61CE43D9" Ref="R52"  Part="1"
 AR Path="/614B514C/61CE43D9" Ref="R66"  Part="1"
-F 0 "R3" V 7857 2650 50  0000 C CNN
+F 0 "R52" V 7857 2650 50  0000 C CNN
 F 1 "1K" V 7766 2650 50  0000 C CNN
 F 2 "Resistor_SMD:R_0402_1005Metric_Pad0.72x0.64mm_HandSolder" V 7580 2650 50  0001 C CNN
@@
 AR Path="/6144BA6D/611489B3" Ref="D15"  Part="1"
 AR Path="/614B514C/611489B3" Ref="D19"  Part="1"
-F 0 "D3" H 7600 1550 50  0000 C CNN
+F 0 "D15" H 7600 1550 50  0000 C CNN
 F 1 "LED" H 7350 1700 50  0000 C CNN
 F 2 "LED_SMD:LED_0603_1608Metric" H 7500 1650 50  0001 C CNN
@@
 AR Path="/6144BA6D/611489C2" Ref="D16"  Part="1"
 AR Path="/614B514C/611489C2" Ref="D20"  Part="1"
-F 0 "D4" H 7600 1800 50  0000 C CNN
+F 0 "D16" H 7600 1800 50  0000 C CNN
 F 1 "LED" H 7350 1950 50  0000 C CNN
 F 2 "LED_SMD:LED_0603_1608Metric" H 7500 1900 50  0001 C CNN
@@
 AR Path="/6144BA6D/611489D8" Ref="#PWR083"  Part="1"
 AR Path="/614B514C/611489D8" Ref="#PWR0101"  Part="1"
-F 0 "#PWR020" H 8250 1400 50  0001 C CNN
+F 0 "#PWR083" H 8250 1400 50  0001 C CNN
 F 1 "GND" H 8255 1477 50  0000 C CNN
 F 2 "" H 8250 1650 50  0001 C CNN
@@
 AR Path="/6144BA6D/61149574" Ref="R53"  Part="1"
 AR Path="/614B514C/61149574" Ref="R67"  Part="1"
-F 0 "R4" V 8050 1650 50  0000 C CNN
+F 0 "R53" V 8050 1650 50  0000 C CNN
 F 1 "1k" V 7950 1650 50  0000 C CNN
 F 2 "Resistor_SMD:R_0402_1005Metric" V 7880 1650 50  0001 C CNN
@@
 AR Path="/6144BA6D/6114B6A4" Ref="#PWR084"  Part="1"
 AR Path="/614B514C/6114B6A4" Ref="#PWR0102"  Part="1"
-F 0 "#PWR021" H 8250 1650 50  0001 C CNN
+F 0 "#PWR084" H 8250 1650 50  0001 C CNN
 F 1 "GND" H 8255 1727 50  0000 C CNN
 F 2 "" H 8250 1900 50  0001 C CNN
@@
 AR Path="/6144BA6D/6114B6AB" Ref="R54"  Part="1"
 AR Path="/614B514C/6114B6AB" Ref="R68"  Part="1"
-F 0 "R5" V 8050 1900 50  0000 C CNN
+F 0 "R54" V 8050 1900 50  0000 C CNN
 F 1 "1k" V 7950 1900 50  0000 C CNN
 F 2 "Resistor_SMD:R_0402_1005Metric" V 7880 1900 50  0001 C CNN
@@
 AR Path="/6144BA6D/6115EC66" Ref="#PWR078"  Part="1"
 AR Path="/614B514C/6115EC66" Ref="#PWR096"  Part="1"
-F 0 "#PWR015" H 4000 1350 50  0001 C CNN
+F 0 "#PWR078" H 4000 1350 50  0001 C CNN
 F 1 "GND" H 4005 1427 50  0000 C CNN
 F 2 "" H 4000 1600 50  0001 C CNN
@@
 AR Path="/6144BA6D/61162826" Ref="#PWR081"  Part="1"
 AR Path="/614B514C/61162826" Ref="#PWR099"  Part="1"
-F 0 "#PWR018" H 4000 2350 50  0001 C CNN
+F 0 "#PWR081" H 4000 2350 50  0001 C CNN
 F 1 "GND" H 4005 2427 50  0000 C CNN
 F 2 "" H 4000 2600 50  0001 C CNN
@@
 AR Path="/6144BA6D/61162834" Ref="IC8"  Part="1"
 AR Path="/614B514C/61162834" Ref="IC10"  Part="1"
-F 0 "IC2" H 6000 2550 50  0000 L CNN
+F 0 "IC8" H 6000 2550 50  0000 L CNN
 F 1 "OKR-T_6-W12-C" H 5450 2450 50  0000 L CNN
 F 2 "dg_power:MURATACASEC90" H 6200 2500 50  0001 L CNN
@@
 AR Path="/6144BA6D/6116283A" Ref="R51"  Part="1"
 AR Path="/614B514C/6116283A" Ref="R65"  Part="1"
-F 0 "R2" V 4250 2350 50  0000 L CNN
+F 0 "R51" V 4250 2350 50  0000 L CNN
 F 1 "436" V 4150 2300 50  0000 L CNN
 F 2 "Resistor_SMD:R_0402_1005Metric_Pad0.72x0.64mm_HandSolder" V 4080 2400 50  0001 C CNN
@@
 AR Path="/6144BA6D/61162845" Ref="#PWR080"  Part="1"
 AR Path="/614B514C/61162845" Ref="#PWR098"  Part="1"
-F 0 "#PWR017" H 4000 2150 50  0001 C CNN
+F 0 "#PWR080" H 4000 2150 50  0001 C CNN
 F 1 "GND" H 4005 2227 50  0000 C CNN
 F 2 "" H 4000 2400 50  0001 C CNN
@@
 AR Path="/6144BA6D/6116D895" Ref="R55"  Part="1"
 AR Path="/614B514C/6116D895" Ref="R69"  Part="1"
-F 0 "R6" V 8000 2850 50  0000 C CNN
+F 0 "R55" V 8000 2850 50  0000 C CNN
 F 1 "100k" H 7750 2850 50  0000 C CNN
 F 2 "Resistor_SMD:R_0402_1005Metric" V 7830 2850 50  0001 C CNN
@@
 AR Path="/6144BA6D/61173063" Ref="#PWR082"  Part="1"
 AR Path="/614B514C/61173063" Ref="#PWR0100"  Part="1"
-F 0 "#PWR019" H 7900 2900 50  0001 C CNN
+F 0 "#PWR082" H 7900 2900 50  0001 C CNN
 F 1 "GND" H 7905 2977 50  0000 C CNN
 F 2 "" H 7900 3150 50  0001 C CNN
@@
 AR Path="/613B6F05/61DF2ADC" Ref="JP1"  Part="1"
 AR Path="/6144BA6D/61DF2ADC" Ref="JP16"  Part="1"
-F 0 "JP1" H 9400 1700 50  0000 C CNN
+F 0 "JP16" H 9400 1700 50  0000 C CNN
 F 1 "SolderJumper_2_Open" H 9250 1764 50  0001 C CNN
 F 2 "Jumper:SolderJumper-2_P1.3mm_Open_RoundedPad1.0x1.5mm" H 9250 1650 50  0001 C CNN

Commit message: DFM
Parts:
- F1: #LCSC C315905 -> (none); JLC# (none) -> C315905
- R1: JLC# (none) -> C204354
- R2: JLC# (none) -> C100430

Commit message: Added Part numbers.
Parts:
- R1: value 268 -> 261; JLC# C204354 -> C25097
- R2: value 436 -> 432
Other:
- note added: "RTRIM_3V3 = 432 = 1.182 / (3.32-0.591)"
- note added: "RTRIM_5V = 261 = 1.182 / (5.11-0.591)"
- note removed: "RTRIM_3V3 = 436 = 1.182 / (3.3-0.591)"
- note removed: "RTRIM_5V = 268 = 1.182 / (5-0.591)"
Changed lines of the file:
@@
 $Descr A4 11693 8268
 encoding utf-8
-Sheet 11 12
+Sheet 9 12
 Title ""
 Date ""
@@
 AR Path="/6144BA6D/61F5E18B" Ref="#PWR079"  Part="1"
 AR Path="/614B514C/61F5E18B" Ref="#PWR097"  Part="1"
-F 0 "#PWR016" H 4000 1550 50  0001 C CNN
+F 0 "#PWR097" H 4000 1550 50  0001 C CNN
 F 1 "GND" H 4005 1627 50  0000 C CNN
 F 2 "" H 4000 1800 50  0001 C CNN
@@
 AR Path="/6144BA6D/6205DE31" Ref="IC7"  Part="1"
 AR Path="/614B514C/6205DE31" Ref="IC9"  Part="1"
-F 0 "IC1" H 6000 1750 50  0000 L CNN
+F 0 "IC9" H 6000 1750 50  0000 L CNN
 F 1 "OKR-T_6-W12-C" H 5450 1650 50  0000 L CNN
 F 2 "dg_power:MURATACASEC90" H 6200 1700 50  0001 L CNN
@@
 AR Path="/6144BA6D/6205EE37" Ref="R50"  Part="1"
 AR Path="/614B514C/6205EE37" Ref="R64"  Part="1"
-F 0 "R1" V 4250 1550 50  0000 L CNN
-F 1 "268" V 4150 1500 50  0000 L CNN
+F 0 "R64" V 4250 1550 50  0000 L CNN
+F 1 "261" V 4150 1500 50  0000 L CNN
 F 2 "Resistor_SMD:R_0402_1005Metric_Pad0.72x0.64mm_HandSolder" V 4080 1600 50  0001 C CNN
 F 3 "~" H 4150 1600 50  0001 C CNN
-F 4 "C204354" V 4150 1600 50  0001 C CNN "JLC#"
+F 4 "C25097" V 4150 1600 50  0001 C CNN "JLC#"
 	1    4150 1600
 	0    -1   -1   0
@@
 AR Path="/6144BA6D/620CBF19" Ref="J11"  Part="1"
 AR Path="/614B514C/620CBF19" Ref="J12"  Part="1"
-F 0 "J7" H 2400 2700 50  0000 L CNN
+F 0 "J12" H 2400 2700 50  0000 L CNN
 F 1 "Header_2x6_2.54mm" H 2050 2250 50  0000 L CNN
 F 2 "Connector_PinHeader_2.54mm:PinHeader_2x03_P2.54mm_Vertical" H 2400 2500 50  0001 C CNN
@@
 AR Path="/6144BA6D/624CFE29" Ref="F4"  Part="1"
 AR Path="/614B514C/624CFE29" Ref="F5"  Part="1"
-F 0 "F1" V 2400 1550 50  0000 L CNN
+F 0 "F5" V 2400 1550 50  0000 L CNN
 F 1 "Polyfuse" V 2200 1400 50  0000 L CNN
 F 2 "Fuse:Fuse_2920_7451Metric_Castellated" H 2350 1400 50  0001 L CNN
@@
 AR Path="/6144BA6D/61CDA64C" Ref="RLA4"  Part="1"
 AR Path="/614B514C/61CDA64C" Ref="RLA5"  Part="1"
-F 0 "RLA1" H 8450 2777 60  0000 C CNN
+F 0 "RLA5" H 8450 2777 60  0000 C CNN
 F 1 "G3VM-61VY2-TR" H 8450 2671 60  0000 C CNN
 F 2 "dg_relay:G3VM-SOP" H 8650 2690 60  0001 C CNN
@@
 AR Path="/6144BA6D/61CE3867" Ref="#PWR085"  Part="1"
 AR Path="/614B514C/61CE3867" Ref="#PWR0103"  Part="1"
-F 0 "#PWR022" H 9000 2900 50  0001 C CNN
+F 0 "#PWR0103" H 9000 2900 50  0001 C CNN
 F 1 "GND" H 9005 2977 50  0000 C CNN
 F 2 "" H 9000 3150 50  0001 C CNN
@@
 AR Path="/6144BA6D/61CE43D9" Ref="R52"  Part="1"
 AR Path="/614B514C/61CE43D9" Ref="R66"  Part="1"
-F 0 "R3" V 7857 2650 50  0000 C CNN
+F 0 "R66" V 7857 2650 50  0000 C CNN
 F 1 "1K" V 7766 2650 50  0000 C CNN
 F 2 "Resistor_SMD:R_0402_1005Metric_Pad0.72x0.64mm_HandSolder" V 7580 2650 50  0001 C CNN
@@
 AR Path="/6144BA6D/611489B3" Ref="D15"  Part="1"
 AR Path="/614B514C/611489B3" Ref="D19"  Part="1"
-F 0 "D3" H 7600 1550 50  0000 C CNN
+F 0 "D19" H 7600 1550 50  0000 C CNN
 F 1 "LED" H 7350 1700 50  0000 C CNN
 F 2 "LED_SMD:LED_0603_1608Metric" H 7500 1650 50  0001 C CNN
@@
 AR Path="/6144BA6D/611489C2" Ref="D16"  Part="1"
 AR Path="/614B514C/611489C2" Ref="D20"  Part="1"
-F 0 "D4" H 7600 1800 50  0000 C CNN
+F 0 "D20" H 7600 1800 50  0000 C CNN
 F 1 "LED" H 7350 1950 50  0000 C CNN
 F 2 "LED_SMD:LED_0603_1608Metric" H 7500 1900 50  0001 C CNN
@@
 AR Path="/6144BA6D/611489D8" Ref="#PWR083"  Part="1"
 AR Path="/614B514C/611489D8" Ref="#PWR0101"  Part="1"
-F 0 "#PWR020" H 8250 1400 50  0001 C CNN
+F 0 "#PWR0101" H 8250 1400 50  0001 C CNN
 F 1 "GND" H 8255 1477 50  0000 C CNN
 F 2 "" H 8250 1650 50  0001 C CNN
@@
 AR Path="/6144BA6D/61149574" Ref="R53"  Part="1"
 AR Path="/614B514C/61149574" Ref="R67"  Part="1"
-F 0 "R4" V 8050 1650 50  0000 C CNN
+F 0 "R67" V 8050 1650 50  0000 C CNN
 F 1 "1k" V 7950 1650 50  0000 C CNN
 F 2 "Resistor_SMD:R_0402_1005Metric" V 7880 1650 50  0001 C CNN
@@
 AR Path="/6144BA6D/6114B6A4" Ref="#PWR084"  Part="1"
 AR Path="/614B514C/6114B6A4" Ref="#PWR0102"  Part="1"
-F 0 "#PWR021" H 8250 1650 50  0001 C CNN
+F 0 "#PWR0102" H 8250 1650 50  0001 C CNN
 F 1 "GND" H 8255 1727 50  0000 C CNN
 F 2 "" H 8250 1900 50  0001 C CNN
@@
 AR Path="/6144BA6D/6114B6AB" Ref="R54"  Part="1"
 AR Path="/614B514C/6114B6AB" Ref="R68"  Part="1"
-F 0 "R5" V 8050 1900 50  0000 C CNN
+F 0 "R68" V 8050 1900 50  0000 C CNN
 F 1 "1k" V 7950 1900 50  0000 C CNN
 F 2 "Resistor_SMD:R_0402_1005Metric" V 7880 1900 50  0001 C CNN
@@
 RTRIM (kOhm) = 1.182 / (Vout-0.591)
 Text Notes 4500 3300 0    50   ~ 0
-RTRIM_3V3 = 436 = 1.182 / (3.3-0.591)
+RTRIM_3V3 = 432 = 1.182 / (3.32-0.591)
 Text Notes 4550 3200 0    50   ~ 0
-RTRIM_5V = 268 = 1.182 / (5-0.591)
+RTRIM_5V = 261 = 1.182 / (5.11-0.591)
 Wire Wire Line
 	4050 1900 4550 1900
@@
 AR Path="/6144BA6D/6115EC66" Ref="#PWR078"  Part="1"
 AR Path="/614B514C/6115EC66" Ref="#PWR096"  Part="1"
-F 0 "#PWR015" H 4000 1350 50  0001 C CNN
+F 0 "#PWR096" H 4000 1350 50  0001 C CNN
 F 1 "GND" H 4005 1427 50  0000 C CNN
 F 2 "" H 4000 1600 50  0001 C CNN
@@
 AR Path="/6144BA6D/61162826" Ref="#PWR081"  Part="1"
 AR Path="/614B514C/61162826" Ref="#PWR099"  Part="1"
-F 0 "#PWR018" H 4000 2350 50  0001 C CNN
+F 0 "#PWR099" H 4000 2350 50  0001 C CNN
 F 1 "GND" H 4005 2427 50  0000 C CNN
 F 2 "" H 4000 2600 50  0001 C CNN
@@
 AR Path="/6144BA6D/6116283A" Ref="R51"  Part="1"
 AR Path="/614B514C/6116283A" Ref="R65"  Part="1"
-F 0 "R2" V 4250 2350 50  0000 L CNN
-F 1 "436" V 4150 2300 50  0000 L CNN
+F 0 "R65" V 4250 2350 50  0000 L CNN
+F 1 "432" V 4150 2300 50  0000 L CNN
 F 2 "Resistor_SMD:R_0402_1005Metric_Pad0.72x0.64mm_HandSolder" V 4080 2400 50  0001 C CNN
 F 3 "~" H 4150 2400 50  0001 C CNN
@@
 AR Path="/6144BA6D/61162845" Ref="#PWR080"  Part="1"
 AR Path="/614B514C/61162845" Ref="#PWR098"  Part="1"
-F 0 "#PWR017" H 4000 2150 50  0001 C CNN
+F 0 "#PWR098" H 4000 2150 50  0001 C CNN
 F 1 "GND" H 4005 2227 50  0000 C CNN
 F 2 "" H 4000 2400 50  0001 C CNN
@@
 AR Path="/6144BA6D/6116D895" Ref="R55"  Part="1"
 AR Path="/614B514C/6116D895" Ref="R69"  Part="1"
-F 0 "R6" V 8000 2850 50  0000 C CNN
+F 0 "R69" V 8000 2850 50  0000 C CNN
 F 1 "100k" H 7750 2850 50  0000 C CNN
 F 2 "Resistor_SMD:R_0402_1005Metric" V 7830 2850 50  0001 C CNN
@@
 AR Path="/6144BA6D/61173063" Ref="#PWR082"  Part="1"
 AR Path="/614B514C/61173063" Ref="#PWR0100"  Part="1"
-F 0 "#PWR019" H 7900 2900 50  0001 C CNN
+F 0 "#PWR0100" H 7900 2900 50  0001 C CNN
 F 1 "GND" H 7905 2977 50  0000 C CNN
 F 2 "" H 7900 3150 50  0001 C CNN
@@
 AR Path="/613B6F05/61DF2ADC" Ref="JP1"  Part="1"
 AR Path="/6144BA6D/61DF2ADC" Ref="JP16"  Part="1"
-F 0 "JP1" H 9400 1700 50  0000 C CNN
+F 0 "JP21" H 9400 1700 50  0000 C CNN
 F 1 "SolderJumper_2_Open" H 9250 1764 50  0001 C CNN
 F 2 "Jumper:SolderJumper-2_P1.3mm_Open_RoundedPad1.0x1.5mm" H 9250 1650 50  0001 C CNN
@@
 AR Path="/6144BA6D/61162834" Ref="IC8"  Part="1"
 AR Path="/614B514C/61162834" Ref="IC10"  Part="1"
-F 0 "IC2" H 6000 2550 50  0000 L CNN
+F 0 "IC10" H 6000 2550 50  0000 L CNN
 F 1 "OKR-T_6-W12-C" H 5450 2450 50  0000 L CNN
 F 2 "dg_power:MURATACASEC90" H 6200 2500 50  0001 L CNN

Commit message: DFM
Changed lines of the file:
@@
 $Descr A4 11693 8268
 encoding utf-8
-Sheet 9 12
+Sheet 3 12
 Title ""
 Date ""
@@
 AR Path="/6144BA6D/61F5E18B" Ref="#PWR079"  Part="1"
 AR Path="/614B514C/61F5E18B" Ref="#PWR097"  Part="1"
-F 0 "#PWR097" H 4000 1550 50  0001 C CNN
+F 0 "#PWR043" H 4000 1550 50  0001 C CNN
 F 1 "GND" H 4005 1627 50  0000 C CNN
 F 2 "" H 4000 1800 50  0001 C CNN
@@
 AR Path="/6144BA6D/6205DE31" Ref="IC7"  Part="1"
 AR Path="/614B514C/6205DE31" Ref="IC9"  Part="1"
-F 0 "IC9" H 6000 1750 50  0000 L CNN
+F 0 "IC3" H 6000 1750 50  0000 L CNN
 F 1 "OKR-T_6-W12-C" H 5450 1650 50  0000 L CNN
 F 2 "dg_power:MURATACASEC90" H 6200 1700 50  0001 L CNN
@@
 AR Path="/6144BA6D/6205EE37" Ref="R50"  Part="1"
 AR Path="/614B514C/6205EE37" Ref="R64"  Part="1"
-F 0 "R64" V 4250 1550 50  0000 L CNN
+F 0 "R22" V 4250 1550 50  0000 L CNN
 F 1 "261" V 4150 1500 50  0000 L CNN
 F 2 "Resistor_SMD:R_0402_1005Metric_Pad0.72x0.64mm_HandSolder" V 4080 1600 50  0001 C CNN
@@
 AR Path="/6144BA6D/620CBF19" Ref="J11"  Part="1"
 AR Path="/614B514C/620CBF19" Ref="J12"  Part="1"
-F 0 "J12" H 2400 2700 50  0000 L CNN
+F 0 "J9" H 2400 2700 50  0000 L CNN
 F 1 "Header_2x6_2.54mm" H 2050 2250 50  0000 L CNN
 F 2 "Connector_PinHeader_2.54mm:PinHeader_2x03_P2.54mm_Vertical" H 2400 2500 50  0001 C CNN
@@
 AR Path="/6144BA6D/624CFE29" Ref="F4"  Part="1"
 AR Path="/614B514C/624CFE29" Ref="F5"  Part="1"
-F 0 "F5" V 2400 1550 50  0000 L CNN
+F 0 "F2" V 2400 1550 50  0000 L CNN
 F 1 "Polyfuse" V 2200 1400 50  0000 L CNN
 F 2 "Fuse:Fuse_2920_7451Metric_Castellated" H 2350 1400 50  0001 L CNN
@@
 AR Path="/6144BA6D/61CDA64C" Ref="RLA4"  Part="1"
 AR Path="/614B514C/61CDA64C" Ref="RLA5"  Part="1"
-F 0 "RLA5" H 8450 2777 60  0000 C CNN
+F 0 "RLA2" H 8450 2777 60  0000 C CNN
 F 1 "G3VM-61VY2-TR" H 8450 2671 60  0000 C CNN
 F 2 "dg_relay:G3VM-SOP" H 8650 2690 60  0001 C CNN
@@
 AR Path="/6144BA6D/61CE3867" Ref="#PWR085"  Part="1"
 AR Path="/614B514C/61CE3867" Ref="#PWR0103"  Part="1"
-F 0 "#PWR0103" H 9000 2900 50  0001 C CNN
+F 0 "#PWR049" H 9000 2900 50  0001 C CNN
 F 1 "GND" H 9005 2977 50  0000 C CNN
 F 2 "" H 9000 3150 50  0001 C CNN
@@
 AR Path="/6144BA6D/61CE43D9" Ref="R52"  Part="1"
 AR Path="/614B514C/61CE43D9" Ref="R66"  Part="1"
-F 0 "R66" V 7857 2650 50  0000 C CNN
+F 0 "R24" V 7857 2650 50  0000 C CNN
 F 1 "1K" V 7766 2650 50  0000 C CNN
 F 2 "Resistor_SMD:R_0402_1005Metric_Pad0.72x0.64mm_HandSolder" V 7580 2650 50  0001 C CNN
@@
 AR Path="/6144BA6D/611489B3" Ref="D15"  Part="1"
 AR Path="/614B514C/611489B3" Ref="D19"  Part="1"
-F 0 "D19" H 7600 1550 50  0000 C CNN
+F 0 "D7" H 7600 1550 50  0000 C CNN
 F 1 "LED" H 7350 1700 50  0000 C CNN
 F 2 "LED_SMD:LED_0603_1608Metric" H 7500 1650 50  0001 C CNN
@@
 AR Path="/6144BA6D/611489C2" Ref="D16"  Part="1"
 AR Path="/614B514C/611489C2" Ref="D20"  Part="1"
-F 0 "D20" H 7600 1800 50  0000 C CNN
+F 0 "D8" H 7600 1800 50  0000 C CNN
 F 1 "LED" H 7350 1950 50  0000 C CNN
 F 2 "LED_SMD:LED_0603_1608Metric" H 7500 1900 50  0001 C CNN
@@
 AR Path="/6144BA6D/611489D8" Ref="#PWR083"  Part="1"
 AR Path="/614B514C/611489D8" Ref="#PWR0101"  Part="1"
-F 0 "#PWR0101" H 8250 1400 50  0001 C CNN
+F 0 "#PWR047" H 8250 1400 50  0001 C CNN
 F 1 "GND" H 8255 1477 50  0000 C CNN
 F 2 "" H 8250 1650 50  0001 C CNN
@@
 AR Path="/6144BA6D/61149574" Ref="R53"  Part="1"
 AR Path="/614B514C/61149574" Ref="R67"  Part="1"
-F 0 "R67" V 8050 1650 50  0000 C CNN
+F 0 "R25" V 8050 1650 50  0000 C CNN
 F 1 "1k" V 7950 1650 50  0000 C CNN
 F 2 "Resistor_SMD:R_0402_1005Metric" V 7880 1650 50  0001 C CNN
@@
 AR Path="/6144BA6D/6114B6A4" Ref="#PWR084"  Part="1"
 AR Path="/614B514C/6114B6A4" Ref="#PWR0102"  Part="1"
-F 0 "#PWR0102" H 8250 1650 50  0001 C CNN
+F 0 "#PWR048" H 8250 1650 50  0001 C CNN
 F 1 "GND" H 8255 1727 50  0000 C CNN
 F 2 "" H 8250 1900 50  0001 C CNN
@@
 AR Path="/6144BA6D/6114B6AB" Ref="R54"  Part="1"
 AR Path="/614B514C/6114B6AB" Ref="R68"  Part="1"
-F 0 "R68" V 8050 1900 50  0000 C CNN
+F 0 "R26" V 8050 1900 50  0000 C CNN
 F 1 "1k" V 7950 1900 50  0000 C CNN
 F 2 "Resistor_SMD:R_0402_1005Metric" V 7880 1900 50  0001 C CNN
@@
 AR Path="/6144BA6D/6115EC66" Ref="#PWR078"  Part="1"
 AR Path="/614B514C/6115EC66" Ref="#PWR096"  Part="1"
-F 0 "#PWR096" H 4000 1350 50  0001 C CNN
+F 0 "#PWR042" H 4000 1350 50  0001 C CNN
 F 1 "GND" H 4005 1427 50  0000 C CNN
 F 2 "" H 4000 1600 50  0001 C CNN
@@
 AR Path="/6144BA6D/61162826" Ref="#PWR081"  Part="1"
 AR Path="/614B514C/61162826" Ref="#PWR099"  Part="1"
-F 0 "#PWR099" H 4000 2350 50  0001 C CNN
+F 0 "#PWR045" H 4000 2350 50  0001 C CNN
 F 1 "GND" H 4005 2427 50  0000 C CNN
 F 2 "" H 4000 2600 50  0001 C CNN
@@
 AR Path="/6144BA6D/6116283A" Ref="R51"  Part="1"
 AR Path="/614B514C/6116283A" Ref="R65"  Part="1"
-F 0 "R65" V 4250 2350 50  0000 L CNN
+F 0 "R23" V 4250 2350 50  0000 L CNN
 F 1 "432" V 4150 2300 50  0000 L CNN
 F 2 "Resistor_SMD:R_0402_1005Metric_Pad0.72x0.64mm_HandSolder" V 4080 2400 50  0001 C CNN
@@
 AR Path="/6144BA6D/61162845" Ref="#PWR080"  Part="1"
 AR Path="/614B514C/61162845" Ref="#PWR098"  Part="1"
-F 0 "#PWR098" H 4000 2150 50  0001 C CNN
+F 0 "#PWR044" H 4000 2150 50  0001 C CNN
 F 1 "GND" H 4005 2227 50  0000 C CNN
 F 2 "" H 4000 2400 50  0001 C CNN
@@
 AR Path="/6144BA6D/6116D895" Ref="R55"  Part="1"
 AR Path="/614B514C/6116D895" Ref="R69"  Part="1"
-F 0 "R69" V 8000 2850 50  0000 C CNN
+F 0 "R27" V 8000 2850 50  0000 C CNN
 F 1 "100k" H 7750 2850 50  0000 C CNN
 F 2 "Resistor_SMD:R_0402_1005Metric" V 7830 2850 50  0001 C CNN
@@
 AR Path="/6144BA6D/61173063" Ref="#PWR082"  Part="1"
 AR Path="/614B514C/61173063" Ref="#PWR0100"  Part="1"
-F 0 "#PWR0100" H 7900 2900 50  0001 C CNN
+F 0 "#PWR046" H 7900 2900 50  0001 C CNN
 F 1 "GND" H 7905 2977 50  0000 C CNN
 F 2 "" H 7900 3150 50  0001 C CNN
@@
 AR Path="/613B6F05/61DF2ADC" Ref="JP1"  Part="1"
 AR Path="/6144BA6D/61DF2ADC" Ref="JP16"  Part="1"
-F 0 "JP21" H 9400 1700 50  0000 C CNN
+F 0 "JP6" H 9400 1700 50  0000 C CNN
 F 1 "SolderJumper_2_Open" H 9250 1764 50  0001 C CNN
 F 2 "Jumper:SolderJumper-2_P1.3mm_Open_RoundedPad1.0x1.5mm" H 9250 1650 50  0001 C CNN
@@
 AR Path="/6144BA6D/61162834" Ref="IC8"  Part="1"
 AR Path="/614B514C/61162834" Ref="IC10"  Part="1"
-F 0 "IC10" H 6000 2550 50  0000 L CNN
+F 0 "IC4" H 6000 2550 50  0000 L CNN
 F 1 "OKR-T_6-W12-C" H 5450 2450 50  0000 L CNN
 F 2 "dg_power:MURATACASEC90" H 6200 2500 50  0001 L CNN
