File: currypi.sch (KiCad schematic (older format))
At the start: 0 parts

Commit message: nvme
Parts:
- added D1: D_TVS, Diode_SMD:D_SMA, symbol Device:D_TVS
- added J1: Conn_02x04_Odd_Even, symbol Connector_Generic:Conn_02x04_Odd_Even
Connections:
- net labels added: +24V, GND
- wire segments 0 -> 20
Changed lines of the file:
@@
 $Descr A4 11693 8268
 encoding utf-8
-Sheet 1 3
+Sheet 1 4
 Title ""
 Date ""
@@
 Comment4 ""
 $EndDescr
+$Comp
+L Connector_Generic:Conn_02x04_Odd_Even J1
+U 1 1 611A366D
+P 1050 1350
+F 0 "J1" H 1100 1667 50  0000 C CNN
+F 1 "Conn_02x04_Odd_Even" H 1100 1576 50  0000 C CNN
+F 2 "" H 1050 1350 50  0001 C CNN
+F 3 "~" H 1050 1350 50  0001 C CNN
+	1    1050 1350
+	0    -1   -1   0
+$EndComp
+Wire Wire Line
+	1250 1000 1250 1050
+Wire Wire Line
+	1150 1050 1150 1000
+Connection ~ 1150 1000
+Wire Wire Line
+	1150 1000 1250 1000
+Wire Wire Line
+	1050 1050 1050 1000
+Connection ~ 1050 1000
+Wire Wire Line
+	1050 1000 1150 1000
+Wire Wire Line
+	950  1050 950  1000
+Wire Wire Line
+	950  1000 1050 1000
+Wire Wire Line
+	950  1550 1050 1550
+Connection ~ 1050 1550
+Wire Wire Line
+	1050 1550 1150 1550
+Connection ~ 1150 1550
+Wire Wire Line
+	1150 1550 1250 1550
+$Comp
+L Device:D_TVS D1
+U 1 1 61298C46
+P 1550 1300
+F 0 "D1" V 1504 1380 50  0000 L CNN
+F 1 "D_TVS" V 1595 1380 50  0000 L CNN
+F 2 "Diode_SMD:D_SMA" H 1550 1300 50  0001 C CNN
+F 3 "~" H 1550 1300 50  0001 C CNN
+	1    1550 1300
+	0    1    1    0
+$EndComp
+Wire Wire Line
+	1250 1000 1550 1000
+Wire Wire Line
+	1550 1000 1550 1150
+Connection ~ 1250 1000
+Wire Wire Line
+	1250 1550 1550 1550
+Wire Wire Line
+	1550 1550 1550 1450
+Connection ~ 1250 1550
+$Comp
+L power:+24V #PWR0101
+U 1 1 612995AA
+P 1250 800
+F 0 "#PWR0101" H 1250 650 50  0001 C CNN
+F 1 "+24V" H 1265 973 50  0000 C CNN
+F 2 "" H 1250 800 50  0001 C CNN
+F 3 "" H 1250 800 50  0001 C CNN
+	1    1250 800
+	1    0    0    -1
+$EndComp
+Wire Wire Line
+	1250 800  1250 1000
+$Comp
+L power:GND #PWR0102
+U 1 1 61299E64
+P 1250 1900
+F 0 "#PWR0102" H 1250 1650 50  0001 C CNN
+F 1 "GND" H 1255 1727 50  0000 C CNN
+F 2 "" H 1250 1900 50  0001 C CNN
+F 3 "" H 1250 1900 50  0001 C CNN
+	1    1250 1900
+	1    0    0    -1
+$EndComp
+Wire Wire Line
+	1250 1550 1250 1900
 $Sheet
-S 4350 2300 1000 2300
-U 610DBB8D
-F0 "pi" 50
-F1 "pi.sch" 50
-F2 "5V" I R 5350 2650 50
-F3 "BOOT" I L 4350 2700 50
-F4 "RX" I L 4350 2800 50
-F5 "TX" I L 4350 2900 50
-F6 "USB+" I L 4350 3050 50
-F7 "USB-" I L 4350 3150 50
-F8 "ETH0+" I L 4350 3450 50
-F9 "ETH0-" I L 4350 3550 50
-F10 "ETH1+" I L 4350 3700 50
-F11 "ETH1-" I L 4350 3800 50
-F12 "ETH2+" I L 4350 3950 50
-F13 "ETH2-" I L 4350 4050 50
-F14 "ETH3+" I L 4350 4200 50
-F15 "ETH3-" I L 4350 4300 50
-F16 "3.3V" I R 5350 2750 50
+S 650  6150 2150 1450
+U 61328729
+F0 "mgm" 50
+F1 "mgm.sch" 50
+F2 "5V" I L 650 6400 50
+F3 "BOOT" I L 650 6600 50
+F4 "RX" I L 650 6800 50
+F5 "TX" I L 650 6950 50
+F6 "USB+" I L 650 7100 50
+F7 "USB-" I L 650 7250 50
+F8 "ETH0+" I R 2800 6500 50
+F9 "ETH0-" I R 2800 6600 50
+F10 "ETH1+" I R 2800 6700 50
+F11 "ETH1-" I R 2800 6800 50
+F12 "ETH2+" I R 2800 6900 50
+F13 "ETH2-" I R 2800 7000 50
+F14 "ETH3+" I R 2800 7100 50
+F15 "ETH3-" I R 2800 7200 50
 $EndSheet
 $Sheet
-S 5550 2300 700  1050
-U 610F006D
-F0 "dcdc" 50
+S 4400 1050 1000 2300
+U 613B6EFF
+F0 "sheet613B6EED" 50
+F1 "pi.sch" 50
+F2 "5V" I R 5400 1400 50
+F3 "BOOT" I L 4400 1450 50
+F4 "RX" I L 4400 1550 50
+F5 "TX" I L 4400 1650 50
+F6 "USB+" I L 4400 1800 50
+F7 "USB-" I L 4400 1900 50
+F8 "ETH0+" I L 4400 2200 50
+F9 "ETH0-" I L 4400 2300 50
+F10 "ETH1+" I L 4400 2450 50
+F11 "ETH1-" I L 4400 2550 50
+F12 "ETH2+" I L 4400 2700 50
+F13 "ETH2-" I L 4400 2800 50
+F14 "ETH3+" I L 4400 2950 50
+F15 "ETH3-" I L 4400 3050 50
+F16 "3.3V" I R 5400 1500 50
+$EndSheet
+$Sheet
+S 5600 1050 700  1050
+U 613B6F05
+F0 "sheet613B6EEE" 50
 F1 "dcdc.sch" 50
+F2 "5V" I L 5600 1400 50
+F3 "3.3V" I L 5600 1500 50
+F4 "VIN" I R 6300 1250 50
+F5 "DISABLE" I R 6300 1500 50
 $EndSheet
+$Comp
+L power:+24V #PWR0105
+U 1 1 613B6F0B
+P 6350 950
+F 0 "#PWR0105" H 6350 800 50  0001 C CNN
+F 1 "+24V" H 6365 1123 50  0000 C CNN
+F 2 "" H 6350 950 50  0001 C CNN
+F 3 "" H 6350 950 50  0001 C CNN
+	1    6350 950
+	1    0    0    -1
+$EndComp
+Wire Wire Line
+	6350 950  6350 1250
+Wire Wire Line
+	5600 1400 5400 1400
+Wire Wire Line
+	5400 1500 5600 1500
+Wire Wire Line
+	6350 1250 6300 1250
 $EndSCHEMATC

Commit message: add the ksz switch
Changed lines of the file:
@@
 $Descr A4 11693 8268
 encoding utf-8
-Sheet 1 4
+Sheet 1 5
 Title ""
 Date ""
@@
 Wire Wire Line
 	6350 1250 6300 1250
+$Sheet
+S 5500 3800 2650 1900
+U 611254CF
+F0 "switch" 50
+F1 "switch.sch" 50
+$EndSheet
 $EndSCHEMATC

Commit message: possible layout example
Connections:
- wire segments 20 -> 24
Changed lines of the file:
@@
 F1 "switch.sch" 50
 $EndSheet
+$Sheet
+S 7050 1100 1000 2300
+U 611D29AA
+F0 "sheet611D2998" 50
+F1 "pi.sch" 50
+F2 "5V" I R 8050 1450 50
+F3 "BOOT" I L 7050 1500 50
+F4 "RX" I L 7050 1600 50
+F5 "TX" I L 7050 1700 50
+F6 "USB+" I L 7050 1850 50
+F7 "USB-" I L 7050 1950 50
+F8 "ETH0+" I L 7050 2250 50
+F9 "ETH0-" I L 7050 2350 50
+F10 "ETH1+" I L 7050 2500 50
+F11 "ETH1-" I L 7050 2600 50
+F12 "ETH2+" I L 7050 2750 50
+F13 "ETH2-" I L 7050 2850 50
+F14 "ETH3+" I L 7050 3000 50
+F15 "ETH3-" I L 7050 3100 50
+F16 "3.3V" I R 8050 1550 50
+$EndSheet
+$Sheet
+S 8250 1100 700  1050
+U 611D29B0
+F0 "sheet611D2999" 50
+F1 "dcdc.sch" 50
+F2 "5V" I L 8250 1450 50
+F3 "3.3V" I L 8250 1550 50
+F4 "VIN" I R 8950 1300 50
+F5 "DISABLE" I R 8950 1550 50
+$EndSheet
+$Comp
+L power:+24V #PWR?
+U 1 1 611D29B6
+P 9000 1000
+F 0 "#PWR?" H 9000 850 50  0001 C CNN
+F 1 "+24V" H 9015 1173 50  0000 C CNN
+F 2 "" H 9000 1000 50  0001 C CNN
+F 3 "" H 9000 1000 50  0001 C CNN
+	1    9000 1000
+	1    0    0    -1
+$EndComp
+Wire Wire Line
+	9000 1000 9000 1300
+Wire Wire Line
+	8250 1450 8050 1450
+Wire Wire Line
+	8050 1550 8250 1550
+Wire Wire Line
+	9000 1300 8950 1300
 $EndSCHEMATC

Commit message: maybe use a premade powerbrick
Parts:
- added C126, C127, C132, C133: 14pF, Capacitor_SMD:C_0603_1608Metric, symbol Device:C
- added C128: 100nF, Capacitor_SMD:C_0603_1608Metric, symbol Device:C
- added C129, C134: 10uF, Capacitor_SMD:C_0603_1608Metric, symbol Device:C
- added C130, C131: 0.1uF, Capacitor_SMD:C_0603_1608Metric, symbol Device:C
- added J4: Conn_02x03_Odd_Even, Connector_PinHeader_2.54mm:PinHeader_2x03_P2.54mm_Vertical, symbol Connector_Generic:Conn_02x03_Odd_Even
- added J5: 2x20, Connector_PinHeader_2.54mm:PinHeader_2x20_P2.54mm_Vertical, symbol Connector_Generic:Conn_02x20_Odd_Even
- added J6: Conn_02x03_Odd_Even, Connector:Tag-Connect_TC2030-IDC-FP_2x03_P1.27mm_Vertical, symbol Connector_Generic:Conn_02x03_Odd_Even
- added J7, J9: USB_B, aep:CUI_UJ2-BH-1-TH, symbol Connector:USB_B
- added J8: SS-74500-024, aep:BEL_SS-74500-024, symbol aep:SS-74500-024
- added M1, M2: Fan_4pin, Connector:FanPinHeader_1x04_P2.54mm_Vertical, symbol Motor:Fan_4pin
- added R100, R101, R102, R97, R98, R99: 10K, Resistor_SMD:R_0603_1608Metric, symbol Device:R
- added R86, R87: NC, Resistor_SMD:R_0603_1608Metric, symbol Device:R
- added R88, R89: 36K 1%, Resistor_SMD:R_0603_1608Metric, symbol Device:R
- added R94: 12K 1%, Resistor_SMD:R_0603_1608Metric, symbol Device:R
- added U13: EMC2301, Package_SO:MSOP-8_3x3mm_P0.65mm, symbol aep:EMC2301
- added U14: STM32L151C8T6, Package_QFP:LQFP-48_7x7mm_P0.5mm, symbol MCU_ST_STM32L1:STM32L151C8Tx
- added U15: USB2514B_Bi, Package_DFN_QFN:QFN-36-1EP_6x6mm_P0.5mm_EP3.7x3.7mm, symbol Interface_USB:USB2514B_Bi
- added Y2, Y3: 24Mhz X1E0000210264, Crystal:Crystal_SMD_SeikoEpson_TSX3225-4Pin_3.2x2.5mm, symbol Device:Crystal_GND24_Small
Connections:
- net labels added: +12V, +3V3, c1_act, c1_boot, c1_eth_act, c1_eth_link, c1_reset, c1_rx, c1_tx, c1_usb+, c1_usb-, c1_vref, c1_wp, c2_act, c2_boot, c2_eth_act, c2_eth_link, c2_eth_p1+, c2_eth_p1-, c2_eth_p2+, c2_eth_p2-, c2_eth_p3+, c2_eth_p3-, c2_eth_p4+, c2_eth_p4-, c2_reset, c2_rx, c2_tx, c2_usb+, c2_usb-, c2_vref, c2_wp, c3_act, c3_boot, c3_eth_act, c3_eth_link, c3_eth_p1+, c3_eth_p1-, c3_eth_p2+, c3_eth_p2-, c3_eth_p3+, c3_eth_p3-, c3_eth_p4+, c3_eth_p4-, c3_reset, c3_rx, c3_tx, c3_usb+, c3_usb-, c3_vref, c3_wp, c4_act, c4_boot, c4_eth_act, c4_eth_link, c4_eth_p1+, c4_eth_p1-, c4_eth_p2+, c4_eth_p2-, c4_eth_p3+, c4_eth_p3-, c4_eth_p4+, c4_eth_p4-, c4_gpio1, c4_reset, c4_rx, c4_tx, c4_usb+, c4_usb-, c4_vref, c4_wp, mcu_reset, mcu_scl, mcu_sda, mcu_swclk, mcu_swdio, mcu_tdo, mcu_usb+, mcu_usb-, root_usb+, root_usb-
- net labels removed: +24V
- wire segments 24 -> 298
- no-connect marks 0 -> 18
Other:
- note added: "TODO: this is wrong?"
- note added: "c4 is soft uart, because thats just mgm to mcu\ncustomers get hard uart"

Commit message: just use two usb hubs
Parts:
- removed C126, C127, C132, C133: 14pF, Capacitor_SMD:C_0603_1608Metric, symbol Device:C
- removed C128: 100nF, Capacitor_SMD:C_0603_1608Metric, symbol Device:C
- removed C129, C134: 10uF, Capacitor_SMD:C_0603_1608Metric, symbol Device:C
- removed C130, C131: 0.1uF, Capacitor_SMD:C_0603_1608Metric, symbol Device:C
- removed J4: Conn_02x03_Odd_Even, Connector_PinHeader_2.54mm:PinHeader_2x03_P2.54mm_Vertical, symbol Connector_Generic:Conn_02x03_Odd_Even
- removed J5: 2x20, Connector_PinHeader_2.54mm:PinHeader_2x20_P2.54mm_Vertical, symbol Connector_Generic:Conn_02x20_Odd_Even
- removed J6: Conn_02x03_Odd_Even, Connector:Tag-Connect_TC2030-IDC-FP_2x03_P1.27mm_Vertical, symbol Connector_Generic:Conn_02x03_Odd_Even
- removed J7, J9: USB_B, aep:CUI_UJ2-BH-1-TH, symbol Connector:USB_B
- removed unit 2 of J8
- removed unit 3 of J8
- removed unit 4 of J8
- removed M1, M2: Fan_4pin, Connector:FanPinHeader_1x04_P2.54mm_Vertical, symbol Motor:Fan_4pin
- removed R100, R101, R102, R97, R98, R99: 10K, Resistor_SMD:R_0603_1608Metric, symbol Device:R
- removed R86, R87: NC, Resistor_SMD:R_0603_1608Metric, symbol Device:R
- removed R88, R89: 36K 1%, Resistor_SMD:R_0603_1608Metric, symbol Device:R
- removed R94: 12K 1%, Resistor_SMD:R_0603_1608Metric, symbol Device:R
- removed U13: EMC2301, Package_SO:MSOP-8_3x3mm_P0.65mm, symbol aep:EMC2301
- removed U14: STM32L151C8T6, Package_QFP:LQFP-48_7x7mm_P0.5mm, symbol MCU_ST_STM32L1:STM32L151C8Tx
- removed U15: USB2514B_Bi, Package_DFN_QFN:QFN-36-1EP_6x6mm_P0.5mm_EP3.7x3.7mm, symbol Interface_USB:USB2514B_Bi
- removed Y2, Y3: 24Mhz X1E0000210264, Crystal:Crystal_SMD_SeikoEpson_TSX3225-4Pin_3.2x2.5mm, symbol Device:Crystal_GND24_Small
- added J3: SS-74500-024, aep:BEL_SS-74500-024, symbol aep:SS-74500-024
- J1: footprint (none) -> Connector_Molex:Molex_Mini-Fit_Jr_5569-08A1_2x04_P4.20mm_Horizontal; symbol Connector_Generic:Conn_02x04_Odd_Even -> Connector_Generic:Conn_02x04_Counter_Clockwise
Connections:
- net +12V: now also J1.5 (Pin_5), J1.7 (Pin_7); no longer J1.2 (Pin_2), J1.4 (Pin_4)
- net GND: now also J1.2 (Pin_2), J1.4 (Pin_4); no longer J1.5 (Pin_5), J1.7 (Pin_7)
- net c2_eth_act: now also J3.12_2
- net c2_eth_link: now also J3.10_2
- net c2_eth_p1+: now also J3.8_2
- net c2_eth_p1-: now also J3.7_2
- net c2_eth_p2+: now also J3.6_2
- net c2_eth_p2-: now also J3.5_2
- net c2_eth_p3+: now also J3.4_2
- net c2_eth_p3-: now also J3.3_2
- net c2_eth_p4+: now also J3.2_2
- net c2_eth_p4-: now also J3.1_2
- net c2_vref: now also J3.11_2, J3.9_2
- net c3_eth_act: now also J3.12_3
- net c3_eth_link: now also J3.10_3
- net c3_eth_p1+: now also J3.8_3
- net c3_eth_p1-: now also J3.7_3
- net c3_eth_p2+: now also J3.6_3
- net c3_eth_p2-: now also J3.5_3
- net c3_eth_p3+: now also J3.4_3
- net c3_eth_p3-: now also J3.3_3
- net c3_eth_p4+: now also J3.2_3
- net c3_eth_p4-: now also J3.1_3
- net c3_vref: now also J3.11_3, J3.9_3
- net c4_eth_act: now also J3.12_4
- net c4_eth_link: now also J3.10_4
- net c4_eth_p1+: now also J3.8_4
- net c4_eth_p1-: now also J3.7_4
- net c4_eth_p2+: now also J3.6_4
- net c4_eth_p2-: now also J3.5_4
- net c4_eth_p3+: now also J3.4_4
- net c4_eth_p3-: now also J3.3_4
- net c4_eth_p4+: now also J3.2_4
- net c4_eth_p4-: now also J3.1_4
- net c4_vref: now also J3.11_4, J3.9_4
- net sheet613B6EED/ETH0+ renamed pi/ETH0+
- net sheet613B6EED/ETH0- renamed pi/ETH0-
- net sheet613B6EED/ETH1+ renamed pi/ETH1+
- net sheet613B6EED/ETH1- renamed pi/ETH1-
- net sheet613B6EED/ETH2+ renamed pi/ETH2+
- net sheet613B6EED/ETH2- renamed pi/ETH2-
- net sheet613B6EED/ETH3+ renamed pi/ETH3+
- net sheet613B6EED/ETH3- renamed pi/ETH3-
- no-connect marks 18 -> 0
Other:
- note added: "TODO: switch usb detect is wrong\nTODO: usb connectors have D+/- reversed\nTODO: RJ45 is cursed. https://i.pinimg.com/originals/46/e6/6c/46e66c1fcbe21f8910b95691846599ba.jpg\n\n\nTODO: slice smith termination is shorted instead of with cap"
- note removed: "c4 is soft uart, because thats just mgm to mcu\ncustomers get hard uart"

Commit message: use native rpi uarts instead of extra chip
Parts:
- added D7: D_TVS, Diode_SMD:D_SMA, symbol Device:D_TVS
- added H1, H? (x5): MountingHole, MountingHole:MountingHole_3.2mm_M3_Pad, symbol Mechanical:MountingHole_Pad
- added J5: Conn_02x04_Odd_Even, Connector_Molex:Molex_Mini-Fit_Jr_5569-08A2_2x04_P4.20mm_Horizontal, symbol Connector_Generic:Conn_02x04_Counter_Clockwise
- J1: footprint Connector_Molex:Molex_Mini-Fit_Jr_5569-08A1_2x04_P4.20mm_Horizontal -> Connector_Molex:Molex_Mini-Fit_Jr_5569-08A2_2x04_P4.20mm_Horizontal
- renumbered J8 to J3
Connections:
- net +12V: now also D7.1 (A1), J5.5 (Pin_5), J5.6 (Pin_6), J5.7 (Pin_7), J5.8 (Pin_8)
- net GND: now also D7.2 (A2), H1.1, H?.1, H?.1, H?.1, H?.1, H?.1, J5.1 (Pin_1), J5.2 (Pin_2), J5.3 (Pin_3), J5.4 (Pin_4)
