File: currypi.sch (KiCad schematic (older format))
At the start: 14 parts, among them J1 Conn_02x04_Odd_Even, J3 SS-74500-020, J5 Conn_02x04_Odd_Even

Commit message: Created .gitignore file. Completed schematic organization. Added Fan Driver alternative.
Parts:
- removed H1, H2, H3, H4, H5, H6: MountingHole, MountingHole:MountingHole_3.2mm_M3_Pad, symbol Mechanical:MountingHole_Pad
- added FID? (x3): Fiducial, Fiducial:Fiducial_1mm_Mask2mm, symbol Mechanical:Fiducial
- added H? (x6): MountingHole, MountingHole:MountingHole_3.2mm_M3_Pad, symbol Mechanical:MountingHole_Pad
Connections:
- wire segments 206 -> 204
Other:
- moved on the sheet: D1, D7, J1, J3B, J3C, J3D, J5

Commit message: Schematics annotated.
Parts:
- gave numbers to parts that had none: 12
- renumbered D7 to D2, J3 to J1, J1 to J5, J5 to J6

Commit message: Updated PCB Design.
Parts:
- removed J2, J3, J4: SS-74500-020, dg_connectors:BEL_SS-74500-020, symbol dg_connectors:SS-74500-020
Connections:
- wire segments 204 -> 198
Changed lines of the file:
@@
 $EndSheet
-$Comp
-L dg_connectors:SS-74500-020 J1
-U 2 1 611D8906
-P 3850 -1750
-F 0 "J1" H 3500 -1000 50  0000 L CNN
-F 1 "SS-74500-020" H 3600 -2500 50  0000 L CNN
-F 2 "dg_connectors:BEL_SS-74500-020" H 3850 -1750 50  0001 L BNN
-F 3 "" H 3850 -1750 50  0001 L BNN
-F 4 "A4" H 3850 -1750 50  0001 L BNN "PARTREV"
-F 5 "Bel Magnetic Solutions" H 3850 -1750 50  0001 L BNN "MANUFACTURER"
-F 6 "Manufacturer Recommendations" H 3850 -1750 50  0001 L BNN "STANDARD"
-F 7 "27.41mm" H 3850 -1750 50  0001 L BNN "MAXIMUM_PACKAGE_HEIGHT"
-	2    3850 -1750
-	-1   0    0    -1
-$EndComp
-$Comp
-L dg_connectors:SS-74500-020 J1
-U 3 1 611DAAD0
-P 4900 -1750
-F 0 "J1" H 4500 -1000 50  0000 L CNN
-F 1 "SS-74500-020" H 4700 -2500 50  0000 L CNN
-F 2 "dg_connectors:BEL_SS-74500-020" H 4900 -1750 50  0001 L BNN
-F 3 "" H 4900 -1750 50  0001 L BNN
-F 4 "A4" H 4900 -1750 50  0001 L BNN "PARTREV"
-F 5 "Bel Magnetic Solutions" H 4900 -1750 50  0001 L BNN "MANUFACTURER"
-F 6 "Manufacturer Recommendations" H 4900 -1750 50  0001 L BNN "STANDARD"
-F 7 "27.41mm" H 4900 -1750 50  0001 L BNN "MAXIMUM_PACKAGE_HEIGHT"
-	3    4900 -1750
-	-1   0    0    -1
-$EndComp
-$Comp
-L dg_connectors:SS-74500-020 J1
-U 4 1 611DD33A
-P 5950 -1750
-F 0 "J1" H 5600 -1000 50  0000 L CNN
-F 1 "SS-74500-020" H 5750 -2500 50  0000 L CNN
-F 2 "dg_connectors:BEL_SS-74500-020" H 5950 -1750 50  0001 L BNN
-F 3 "" H 5950 -1750 50  0001 L BNN
-F 4 "A4" H 5950 -1750 50  0001 L BNN "PARTREV"
-F 5 "Bel Magnetic Solutions" H 5950 -1750 50  0001 L BNN "MANUFACTURER"
-F 6 "Manufacturer Recommendations" H 5950 -1750 50  0001 L BNN "STANDARD"
-F 7 "27.41mm" H 5950 -1750 50  0001 L BNN "MAXIMUM_PACKAGE_HEIGHT"
-	4    5950 -1750
-	-1   0    0    -1
-$EndComp
 $Comp
 L power:GND #PWR01
@@
 	1    1750 2150
 	1    0    0    -1
-$EndComp
-$Comp
-L dg_connectors:SS-74500-020 J1
-U 1 1 611D6319
-P 1100 1500
-F 0 "J1" H 993 633 50  0000 C CNN
-F 1 "SS-74500-020" H 993 724 50  0000 C CNN
-F 2 "dg_connectors:BEL_SS-74500-020" H 1100 1500 50  0001 L BNN
-F 3 "" H 1100 1500 50  0001 L BNN
-F 4 "A4" H 1100 1500 50  0001 L BNN "PARTREV"
-F 5 "Bel Magnetic Solutions" H 1100 1500 50  0001 L BNN "MANUFACTURER"
-F 6 "Manufacturer Recommendations" H 1100 1500 50  0001 L BNN "STANDARD"
-F 7 "27.41mm" H 1100 1500 50  0001 L BNN "MAXIMUM_PACKAGE_HEIGHT"
-	1    1100 1500
-	-1   0    0    -1
 $EndComp
 Wire Wire Line
@@
 F18 "eth_speed_ledy" I L 2850 3550 50
 $EndSheet
-$Comp
-L power:GND #PWR02
-U 1 1 6142DCA5
-P 1750 3800
-AR Path="/6142DCA5" Ref="#PWR02"  Part="1"
-AR Path="/5FEB1CB4/6142DCA5" Ref="#PWR?"  Part="1"
-AR Path="/5FECBD46/6142DCA5" Ref="#PWR?"  Part="1"
-AR Path="/5FECD465/6142DCA5" Ref="#PWR?"  Part="1"
-AR Path="/5FECEB82/6142DCA5" Ref="#PWR?"  Part="1"
-AR Path="/5FDF5C30/6142DCA5" Ref="#PWR?"  Part="1"
-AR Path="/5FDF9B9D/6142DCA5" Ref="#PWR?"  Part="1"
-AR Path="/5FDFE7F4/6142DCA5" Ref="#PWR?"  Part="1"
-AR Path="/6133068E/6142DCA5" Ref="#PWR?"  Part="1"
-F 0 "#PWR02" H 1750 3550 50  0001 C CNN
-F 1 "GND" H 1755 3627 50  0000 C CNN
-F 2 "" H 1750 3800 50  0001 C CNN
-F 3 "" H 1750 3800 50  0001 C CNN
-	1    1750 3800
-	1    0    0    -1
-$EndComp
-$Comp
-L dg_connectors:SS-74500-020 J2
-U 1 1 6142DCAF
-P 1100 3150
-F 0 "J2" H 993 2283 50  0000 C CNN
-F 1 "SS-74500-020" H 993 2374 50  0000 C CNN
-F 2 "dg_connectors:BEL_SS-74500-020" H 1100 3150 50  0001 L BNN
-F 3 "" H 1100 3150 50  0001 L BNN
-F 4 "A4" H 1100 3150 50  0001 L BNN "PARTREV"
-F 5 "Bel Magnetic Solutions" H 1100 3150 50  0001 L BNN "MANUFACTURER"
-F 6 "Manufacturer Recommendations" H 1100 3150 50  0001 L BNN "STANDARD"
-F 7 "27.41mm" H 1100 3150 50  0001 L BNN "MAXIMUM_PACKAGE_HEIGHT"
-	1    1100 3150
-	-1   0    0    -1
-$EndComp
 Wire Wire Line
 	1700 3550 1800 3550
@@
 Wire Wire Line
 	1800 3350 1700 3350
-Wire Wire Line
-	1700 3750 1750 3750
-Wire Wire Line
-	1750 3750 1750 3800
 Wire Wire Line
 	2850 2550 1700 2550
@@
 F18 "eth_speed_ledy" I L 2850 5200 50
 $EndSheet
-$Comp
-L power:GND #PWR03
-U 1 1 6143BBDA
-P 1750 5450
-AR Path="/6143BBDA" Ref="#PWR03"  Part="1"
-AR Path="/5FEB1CB4/6143BBDA" Ref="#PWR?"  Part="1"
-AR Path="/5FECBD46/6143BBDA" Ref="#PWR?"  Part="1"
-AR Path="/5FECD465/6143BBDA" Ref="#PWR?"  Part="1"
-AR Path="/5FECEB82/6143BBDA" Ref="#PWR?"  Part="1"
-AR Path="/5FDF5C30/6143BBDA" Ref="#PWR?"  Part="1"
-AR Path="/5FDF9B9D/6143BBDA" Ref="#PWR?"  Part="1"
-AR Path="/5FDFE7F4/6143BBDA" Ref="#PWR?"  Part="1"
-AR Path="/6133068E/6143BBDA" Ref="#PWR?"  Part="1"
-F 0 "#PWR03" H 1750 5200 50  0001 C CNN
-F 1 "GND" H 1755 5277 50  0000 C CNN
-F 2 "" H 1750 5450 50  0001 C CNN
-F 3 "" H 1750 5450 50  0001 C CNN
-	1    1750 5450
-	1    0    0    -1
-$EndComp
-$Comp
-L dg_connectors:SS-74500-020 J3
-U 1 1 6143BBE4
-P 1100 4800
-F 0 "J3" H 993 3933 50  0000 C CNN
-F 1 "SS-74500-020" H 993 4024 50  0000 C CNN
-F 2 "dg_connectors:BEL_SS-74500-020" H 1100 4800 50  0001 L BNN
-F 3 "" H 1100 4800 50  0001 L BNN
-F 4 "A4" H 1100 4800 50  0001 L BNN "PARTREV"
-F 5 "Bel Magnetic Solutions" H 1100 4800 50  0001 L BNN "MANUFACTURER"
-F 6 "Manufacturer Recommendations" H 1100 4800 50  0001 L BNN "STANDARD"
-F 7 "27.41mm" H 1100 4800 50  0001 L BNN "MAXIMUM_PACKAGE_HEIGHT"
-	1    1100 4800
-	-1   0    0    -1
-$EndComp
 Wire Wire Line
 	1700 5200 1800 5200
@@
 Wire Wire Line
 	1800 5000 1700 5000
-Wire Wire Line
-	1700 5400 1750 5400
-Wire Wire Line
-	1750 5400 1750 5450
 Wire Wire Line
 	2850 4200 1700 4200
@@
 F18 "eth_speed_ledy" I L 2850 6850 50
 $EndSheet
-$Comp
-L power:GND #PWR04
-U 1 1 6144BA95
-P 1750 7100
-AR Path="/6144BA95" Ref="#PWR04"  Part="1"
-AR Path="/5FEB1CB4/6144BA95" Ref="#PWR?"  Part="1"
-AR Path="/5FECBD46/6144BA95" Ref="#PWR?"  Part="1"
-AR Path="/5FECD465/6144BA95" Ref="#PWR?"  Part="1"
-AR Path="/5FECEB82/6144BA95" Ref="#PWR?"  Part="1"
-AR Path="/5FDF5C30/6144BA95" Ref="#PWR?"  Part="1"
-AR Path="/5FDF9B9D/6144BA95" Ref="#PWR?"  Part="1"
-AR Path="/5FDFE7F4/6144BA95" Ref="#PWR?"  Part="1"
-AR Path="/6133068E/6144BA95" Ref="#PWR?"  Part="1"
-F 0 "#PWR04" H 1750 6850 50  0001 C CNN
-F 1 "GND" H 1755 6927 50  0000 C CNN
-F 2 "" H 1750 7100 50  0001 C CNN
-F 3 "" H 1750 7100 50  0001 C CNN
-	1    1750 7100
-	1    0    0    -1
-$EndComp
-$Comp
-L dg_connectors:SS-74500-020 J4
-U 1 1 6144BA9F
-P 1100 6450
-F 0 "J4" H 993 5583 50  0000 C CNN
-F 1 "SS-74500-020" H 993 5674 50  0000 C CNN
-F 2 "dg_connectors:BEL_SS-74500-020" H 1100 6450 50  0001 L BNN
-F 3 "" H 1100 6450 50  0001 L BNN
-F 4 "A4" H 1100 6450 50  0001 L BNN "PARTREV"
-F 5 "Bel Magnetic Solutions" H 1100 6450 50  0001 L BNN "MANUFACTURER"
-F 6 "Manufacturer Recommendations" H 1100 6450 50  0001 L BNN "STANDARD"
-F 7 "27.41mm" H 1100 6450 50  0001 L BNN "MAXIMUM_PACKAGE_HEIGHT"
-	1    1100 6450
-	-1   0    0    -1
-$EndComp
 Wire Wire Line
 	1700 6850 1800 6850
@@
 Wire Wire Line
 	1800 6650 1700 6650
-Wire Wire Line
-	1700 7050 1750 7050
-Wire Wire Line
-	1750 7050 1750 7100
 Wire Wire Line
 	2850 5850 1700 5850
@@
 	1    0    0    -1
 $EndComp
+$Comp
+L dg_connectors:SS-74500-020 J1
+U 1 1 6133EDC5
+P 1100 1500
+F 0 "J1" H 993 2367 50  0000 C CNN
+F 1 "SS-74500-020" H 993 2276 50  0000 C CNN
+F 2 "dg_connectors:BEL_SS-74500-020" H 1100 1500 50  0001 L BNN
+F 3 "" H 1100 1500 50  0001 L BNN
+F 4 "A4" H 1100 1500 50  0001 L BNN "PARTREV"
+F 5 "Bel Magnetic Solutions" H 1100 1500 50  0001 L BNN "MANUFACTURER"
+F 6 "Manufacturer Recommendations" H 1100 1500 50  0001 L BNN "STANDARD"
+F 7 "27.41mm" H 1100 1500 50  0001 L BNN "MAXIMUM_PACKAGE_HEIGHT"
+	1    1100 1500
+	-1   0    0    -1
+$EndComp
+$Comp
+L dg_connectors:SS-74500-020 J1
+U 2 1 61344D1A
+P 1100 3150
+F 0 "J1" H 993 4017 50  0000 C CNN
+F 1 "SS-74500-020" H 993 3926 50  0000 C CNN
+F 2 "dg_connectors:BEL_SS-74500-020" H 1100 3150 50  0001 L BNN
+F 3 "" H 1100 3150 50  0001 L BNN
+F 4 "A4" H 1100 3150 50  0001 L BNN "PARTREV"
+F 5 "Bel Magnetic Solutions" H 1100 3150 50  0001 L BNN "MANUFACTURER"
+F 6 "Manufacturer Recommendations" H 1100 3150 50  0001 L BNN "STANDARD"
+F 7 "27.41mm" H 1100 3150 50  0001 L BNN "MAXIMUM_PACKAGE_HEIGHT"
+	2    1100 3150
+	-1   0    0    -1
+$EndComp
+$Comp
+L dg_connectors:SS-74500-020 J1
+U 3 1 6134B0E3
+P 1100 4800
+F 0 "J1" H 993 5667 50  0000 C CNN
+F 1 "SS-74500-020" H 993 5576 50  0000 C CNN
+F 2 "dg_connectors:BEL_SS-74500-020" H 1100 4800 50  0001 L BNN
+F 3 "" H 1100 4800 50  0001 L BNN
+F 4 "A4" H 1100 4800 50  0001 L BNN "PARTREV"
+F 5 "Bel Magnetic Solutions" H 1100 4800 50  0001 L BNN "MANUFACTURER"
+F 6 "Manufacturer Recommendations" H 1100 4800 50  0001 L BNN "STANDARD"
+F 7 "27.41mm" H 1100 4800 50  0001 L BNN "MAXIMUM_PACKAGE_HEIGHT"
+	3    1100 4800
+	-1   0    0    -1
+$EndComp
+$Comp
+L dg_connectors:SS-74500-020 J1
+U 4 1 613511D5
+P 1100 6450
+F 0 "J1" H 993 7317 50  0000 C CNN
+F 1 "SS-74500-020" H 993 7226 50  0000 C CNN
+F 2 "dg_connectors:BEL_SS-74500-020" H 1100 6450 50  0001 L BNN
+F 3 "" H 1100 6450 50  0001 L BNN
+F 4 "A4" H 1100 6450 50  0001 L BNN "PARTREV"
+F 5 "Bel Magnetic Solutions" H 1100 6450 50  0001 L BNN "MANUFACTURER"
+F 6 "Manufacturer Recommendations" H 1100 6450 50  0001 L BNN "STANDARD"
+F 7 "27.41mm" H 1100 6450 50  0001 L BNN "MAXIMUM_PACKAGE_HEIGHT"
+	4    1100 6450
+	-1   0    0    -1
+$EndComp
 $EndSCHEMATC

Commit message: Completed PCIE and Eth. Routing.
Changed lines of the file:
@@
 S 4050 750  700  400
 U 613B6F05
-F0 "dcdc" 50
+F0 "C1_PWR" 50
 F1 "dcdc.sch" 50
 F2 "5V" I L 4050 900 50
@@
 S 2850 750  1000 1350
 U 613B6EFF
-F0 "pi" 50
+F0 "C1" 50
 F1 "pi.sch" 50
 F2 "5V" I R 3850 900 50
@@
 S 4050 2400 700  400
 U 6142DC7D
-F0 "sheet6142DC76" 50
+F0 "C2_PWR" 50
 F1 "dcdc.sch" 50
 F2 "5V" I L 4050 2550 50
@@
 S 2850 2400 1000 1350
 U 6142DC9F
-F0 "sheet6142DC77" 50
+F0 "C2" 50
 F1 "pi.sch" 50
 F2 "5V" I R 3850 2550 50
@@
 S 4050 4050 700  400
 U 6143BBB2
-F0 "sheet6143BBAB" 50
+F0 "C3_PWR" 50
 F1 "dcdc.sch" 50
 F2 "5V" I L 4050 4200 50
@@
 S 2850 4050 1000 1350
 U 6143BBD4
-F0 "sheet6143BBAC" 50
+F0 "C3" 50
 F1 "pi.sch" 50
 F2 "5V" I R 3850 4200 50
@@
 S 4050 5700 700  400
 U 6144BA6D
-F0 "sheet6144BA66" 50
+F0 "C4_PWR" 50
 F1 "dcdc.sch" 50
 F2 "5V" I L 4050 5850 50
@@
 S 2850 5700 1000 1350
 U 6144BA8F
-F0 "sheet6144BA67" 50
+F0 "C4" 50
 F1 "pi.sch" 50
 F2 "5V" I R 3850 5850 50

Commit message: Fixed Eth. Schematic issue and Completed Eth. Routing.
Connections:
- wire segments 198 -> 206
Changed lines of the file:
@@
 Wire Wire Line
 	1700 1600 2850 1600
-Wire Wire Line
-	2850 1300 1700 1300
-Wire Wire Line
-	2850 1400 2650 1400
-Wire Wire Line
-	2450 1200 1700 1200
 Text Notes 1900 1200 0    50   ~ 0
 Blue
@@
 Text Notes 1900 3050 0    50   ~ 0
 Green
-Wire Wire Line
-	2550 3050 2550 2850
-Wire Wire Line
-	2550 2850 2850 2850
-Wire Wire Line
-	1700 3050 2550 3050
 Text Notes 1900 3150 0    50   ~ 0
 Brown White
@@
 Wire Wire Line
 	1700 3250 2850 3250
-Wire Wire Line
-	2850 2950 1700 2950
-Wire Wire Line
-	2850 3050 2650 3050
-Wire Wire Line
-	2650 3050 2650 2900
-Wire Wire Line
-	2650 2900 2450 2900
-Wire Wire Line
-	2450 2900 2450 2850
-Wire Wire Line
-	2450 2850 1700 2850
 Text Notes 1900 2850 0    50   ~ 0
 Blue
@@
 Text Notes 1900 4700 0    50   ~ 0
 Green
-Wire Wire Line
-	2550 4700 2550 4500
-Wire Wire Line
-	2550 4500 2850 4500
-Wire Wire Line
-	1700 4700 2550 4700
 Text Notes 1900 4800 0    50   ~ 0
 Brown White
@@
 Wire Wire Line
 	1700 4900 2850 4900
-Wire Wire Line
-	2850 4600 1700 4600
-Wire Wire Line
-	2850 4700 2650 4700
-Wire Wire Line
-	2650 4700 2650 4550
-Wire Wire Line
-	2650 4550 2450 4550
-Wire Wire Line
-	2450 4550 2450 4500
-Wire Wire Line
-	2450 4500 1700 4500
 Text Notes 1900 4500 0    50   ~ 0
 Blue
@@
 Text Notes 1900 6350 0    50   ~ 0
 Green
-Wire Wire Line
-	2550 6350 2550 6150
-Wire Wire Line
-	2550 6150 2850 6150
-Wire Wire Line
-	1700 6350 2550 6350
 Text Notes 1900 6450 0    50   ~ 0
 Brown White
@@
 Wire Wire Line
 	1700 6550 2850 6550
-Wire Wire Line
-	2850 6250 1700 6250
-Wire Wire Line
-	2850 6350 2650 6350
-Wire Wire Line
-	2650 6350 2650 6200
-Wire Wire Line
-	2650 6200 2450 6200
-Wire Wire Line
-	2450 6200 2450 6150
-Wire Wire Line
-	2450 6150 1700 6150
 Text Notes 1900 6150 0    50   ~ 0
 Blue
@@
 Wire Wire Line
 	4750 5850 5150 5850
-Wire Wire Line
-	2450 1250 2450 1200
-Wire Wire Line
-	2650 1250 2450 1250
-Wire Wire Line
-	2650 1400 2650 1250
 $Sheet
 S 7950 2400 700  400
@@
 	-1   0    0    -1
 $EndComp
+Wire Wire Line
+	2850 1300 2450 1300
+Wire Wire Line
+	2450 1300 2450 1200
+Wire Wire Line
+	2450 1200 1700 1200
+Wire Wire Line
+	1700 1300 2400 1300
+Wire Wire Line
+	2400 1300 2400 1350
+Wire Wire Line
+	2400 1350 2600 1350
+Wire Wire Line
+	2600 1350 2600 1400
+Wire Wire Line
+	2600 1400 2850 1400
+Wire Wire Line
+	2550 3050 2550 2850
+Wire Wire Line
+	2550 2850 2850 2850
+Wire Wire Line
+	1700 3050 2550 3050
+Text Notes 1900 3150 0    50   ~ 0
+Brown White
+Wire Wire Line
+	2850 2950 2450 2950
+Wire Wire Line
+	2450 2950 2450 2850
+Wire Wire Line
+	2450 2850 1700 2850
+Wire Wire Line
+	1700 2950 2400 2950
+Wire Wire Line
+	2400 2950 2400 3000
+Wire Wire Line
+	2400 3000 2600 3000
+Wire Wire Line
+	2600 3000 2600 3050
+Wire Wire Line
+	2600 3050 2850 3050
+Wire Wire Line
+	2550 4700 2550 4500
+Wire Wire Line
+	2550 4500 2850 4500
+Wire Wire Line
+	1700 4700 2550 4700
+Text Notes 1900 4800 0    50   ~ 0
+Brown White
+Wire Wire Line
+	2850 4600 2450 4600
+Wire Wire Line
+	2450 4600 2450 4500
+Wire Wire Line
+	2450 4500 1700 4500
+Wire Wire Line
+	1700 4600 2400 4600
+Wire Wire Line
+	2400 4600 2400 4650
+Wire Wire Line
+	2400 4650 2600 4650
+Wire Wire Line
+	2600 4650 2600 4700
+Wire Wire Line
+	2600 4700 2850 4700
+Wire Wire Line
+	2550 6350 2550 6150
+Wire Wire Line
+	2550 6150 2850 6150
+Wire Wire Line
+	1700 6350 2550 6350
+Text Notes 1900 6450 0    50   ~ 0
+Brown White
+Wire Wire Line
+	2850 6250 2450 6250
+Wire Wire Line
+	2450 6250 2450 6150
+Wire Wire Line
+	2450 6150 1700 6150
+Wire Wire Line
+	1700 6250 2400 6250
+Wire Wire Line
+	2400 6250 2400 6300
+Wire Wire Line
+	2400 6300 2600 6300
+Wire Wire Line
+	2600 6300 2600 6350
+Wire Wire Line
+	2600 6350 2850 6350
 $EndSCHEMATC

Commit message: Added jumper for RJ45 Ind. leds.
Parts:
- added JP?: SolderJumper_2_Open, Jumper:SolderJumper-2_P1.3mm_Open_RoundedPad1.0x1.5mm, symbol Jumper:SolderJumper_2_Open
Connections:
- wire segments 206 -> 208
Changed lines of the file:
@@
 Wire Wire Line
 	2600 6350 2850 6350
+$Comp
+L Jumper:SolderJumper_2_Open JP?
+U 1 1 615BF249
+P 7900 3150
+AR Path="/610DBB8D/615BF249" Ref="JP?"  Part="1"
+AR Path="/613B6218/615BF249" Ref="JP?"  Part="1"
+AR Path="/613B6EFF/615BF249" Ref="JP?"  Part="1"
+AR Path="/613B79B7/615BF249" Ref="JP?"  Part="1"
+AR Path="/613B8664/615BF249" Ref="JP?"  Part="1"
+AR Path="/613B8F90/615BF249" Ref="JP?"  Part="1"
+AR Path="/611D29AA/615BF249" Ref="JP?"  Part="1"
+AR Path="/620E19B3/615BF249" Ref="JP?"  Part="1"
+AR Path="/620FBA4C/615BF249" Ref="JP?"  Part="1"
+AR Path="/6211795B/615BF249" Ref="JP?"  Part="1"
+AR Path="/621328FA/615BF249" Ref="JP?"  Part="1"
+AR Path="/62156471/615BF249" Ref="JP?"  Part="1"
+AR Path="/62171C6A/615BF249" Ref="JP?"  Part="1"
+AR Path="/6218DDB9/615BF249" Ref="JP?"  Part="1"
+AR Path="/61E646BE/615BF249" Ref="JP?"  Part="1"
+AR Path="/612EF6EF/615BF249" Ref="JP?"  Part="1"
+AR Path="/612FBF86/615BF249" Ref="JP?"  Part="1"
+AR Path="/61339A05/615BF249" Ref="JP?"  Part="1"
+AR Path="/61347D57/615BF249" Ref="JP?"  Part="1"
+AR Path="/6135BFD5/615BF249" Ref="JP?"  Part="1"
+AR Path="/61397EC7/615BF249" Ref="JP?"  Part="1"
+AR Path="/613FE9A0/615BF249" Ref="JP?"  Part="1"
+AR Path="/61409D83/615BF249" Ref="JP?"  Part="1"
+AR Path="/61416F70/615BF249" Ref="JP?"  Part="1"
+AR Path="/6142DC9F/615BF249" Ref="JP?"  Part="1"
+AR Path="/6143BBD4/615BF249" Ref="JP?"  Part="1"
+AR Path="/6144BA8F/615BF249" Ref="JP?"  Part="1"
+AR Path="/613B5606/615BF249" Ref="JP?"  Part="1"
+AR Path="/6142DC7D/615BF249" Ref="JP?"  Part="1"
+AR Path="/6143BBB2/615BF249" Ref="JP?"  Part="1"
+AR Path="/614B514C/615BF249" Ref="JP?"  Part="1"
+AR Path="/613B6F05/615BF249" Ref="JP?"  Part="1"
+AR Path="/6144BA6D/615BF249" Ref="JP?"  Part="1"
+F 0 "JP?" H 8050 3200 50  0000 C CNN
+F 1 "SolderJumper_2_Open" H 7900 3264 50  0001 C CNN
+F 2 "Jumper:SolderJumper-2_P1.3mm_Open_RoundedPad1.0x1.5mm" H 7900 3150 50  0001 C CNN
+F 3 "~" H 7900 3150 50  0001 C CNN
+	1    7900 3150
+	1    0    0    -1
+$EndComp
+Text Label 8600 3150 2    50   ~ 0
+3V3_MGMT
+Text Label 7450 3150 0    50   ~ 0
+LED_3V3
+Wire Wire Line
+	8050 3150 8600 3150
+Wire Wire Line
+	7750 3150 7450 3150
 $EndSCHEMATC

Commit message: Added PN for PCIE Connector.
Parts:
- gave numbers to parts that had none: 1
Changed lines of the file:
@@
 AR Path="/613B6F05/615BF249" Ref="JP?"  Part="1"
 AR Path="/6144BA6D/615BF249" Ref="JP?"  Part="1"
-F 0 "JP?" H 8050 3200 50  0000 C CNN
+AR Path="/615BF249" Ref="JP27"  Part="1"
+F 0 "JP27" H 8050 3200 50  0000 C CNN
 F 1 "SolderJumper_2_Open" H 7900 3264 50  0001 C CNN
 F 2 "Jumper:SolderJumper-2_P1.3mm_Open_RoundedPad1.0x1.5mm" H 7900 3150 50  0001 C CNN
