File: currypi.sch (KiCad schematic (older format))
At the start: 15 parts, among them J1 SS-74500-020, J5 Conn_02x04_Odd_Even, J6 Conn_02x04_Odd_Even

Commit message: Changed Eth. Led supply to rpi internal 3v3.
Changed lines of the file:
@@
 Wire Wire Line
 	4050 900  3850 900
-Wire Wire Line
-	3850 1000 4050 1000
 $Comp
 L power:+12V #PWR05
@@
 F17 "eth_act_ledg" I L 2850 1800 50
 F18 "eth_speed_ledy" I L 2850 1900 50
+F19 "3V3_INT" I L 2850 1700 50
 $EndSheet
 $Comp
@@
 Wire Wire Line
 	1900 2000 1700 2000
-Text Label 1900 1700 0    50   ~ 0
-LED_3V3
-Wire Wire Line
-	1800 1700 2250 1700
 Wire Wire Line
 	7300 3750 7450 3750
@@
 Wire Wire Line
 	4050 2550 3850 2550
-Wire Wire Line
-	3850 2650 4050 2650
 $Comp
 L power:+12V #PWR06
@@
 F17 "eth_act_ledg" I L 2850 3450 50
 F18 "eth_speed_ledy" I L 2850 3550 50
+F19 "3V3_INT" I L 2850 3350 50
 $EndSheet
 Wire Wire Line
@@
 Wire Wire Line
 	1900 3650 1700 3650
-Text Label 1900 3350 0    50   ~ 0
-LED_3V3
-Wire Wire Line
-	1800 3350 2250 3350
 Wire Wire Line
 	5150 2550 5150 2500
@@
 Wire Wire Line
 	4050 4200 3850 4200
-Wire Wire Line
-	3850 4300 4050 4300
 $Comp
 L power:+12V #PWR07
@@
 F17 "eth_act_ledg" I L 2850 5100 50
 F18 "eth_speed_ledy" I L 2850 5200 50
+F19 "3V3_INT" I L 2850 5000 50
 $EndSheet
 Wire Wire Line
@@
 Wire Wire Line
 	1900 5300 1700 5300
-Text Label 1900 5000 0    50   ~ 0
-LED_3V3
-Wire Wire Line
-	1800 5000 2250 5000
 Wire Wire Line
 	5150 4200 5150 4150
@@
 Wire Wire Line
 	4050 5850 3850 5850
-Wire Wire Line
-	3850 5950 4050 5950
 $Comp
 L power:+12V #PWR08
@@
 F17 "eth_act_ledg" I L 2850 6750 50
 F18 "eth_speed_ledy" I L 2850 6850 50
+F19 "3V3_INT" I L 2850 6650 50
 $EndSheet
 Wire Wire Line
@@
 Wire Wire Line
 	1900 6950 1700 6950
-Text Label 1900 6650 0    50   ~ 0
-LED_3V3
-Wire Wire Line
-	1800 6650 2250 6650
 Wire Wire Line
 	5150 5850 5150 5800
@@
 Wire Wire Line
 	7750 3150 7450 3150
+Wire Wire Line
+	3850 1000 4050 1000
+Wire Wire Line
+	3850 2650 4050 2650
+Wire Wire Line
+	3850 4300 4050 4300
+Wire Wire Line
+	3850 5950 4050 5950
+Wire Wire Line
+	1800 3350 2850 3350
+Wire Wire Line
+	1800 1700 2850 1700
+Wire Wire Line
+	1800 5000 2850 5000
+Wire Wire Line
+	1800 6650 2850 6650
 $EndSCHEMATC

Commit message: Changed DCDC Disable Signal. Added Labels.
Parts:
- added LOGO1: Logo_Open_Hardware_Small, Symbol:OSHW-Logo2_9.8x8mm_SilkScreen, symbol Graphic:Logo_Open_Hardware_Small
Changed lines of the file:
@@
 $EndComp
 $Comp
-L Graphic:Logo_Open_Hardware_Small #LOGO1
+L Graphic:Logo_Open_Hardware_Small LOGO1
 U 1 1 61DA8664
 P 6500 7450
-F 0 "#LOGO1" H 6500 7725 50  0001 C CNN
+F 0 "LOGO1" H 6500 7725 50  0001 C CNN
 F 1 "Logo_Open_Hardware_Small" H 6500 7225 50  0001 C CNN
-F 2 "Symbol:OSHW-Logo2_7.3x6mm_SilkScreen" H 6500 7450 50  0001 C CNN
+F 2 "Symbol:OSHW-Logo2_9.8x8mm_SilkScreen" H 6500 7450 50  0001 C CNN
 F 3 "~" H 6500 7450 50  0001 C CNN
 	1    6500 7450

Commit message: replace transformers, since out of stock
Parts:
- removed JP27: SolderJumper_2_Open, Jumper:SolderJumper-2_P1.3mm_Open_RoundedPad1.0x1.5mm, symbol Jumper:SolderJumper_2_Open
Connections:
- net labels removed: LED_3V3
- wire segments 208 -> 206
Changed lines of the file:
@@
 	1    0    0    -1
 $EndComp
-Text Notes -150 22200 0    394  ~ 0
+Text Notes -4750 13700 0    394  ~ 0
 TODO: switch usb detect is wrong\nTODO: usb connectors have D+/- reversed\nTODO: RJ45 is cursed. https://i.pinimg.com/originals/46/e6/6c/46e66c1fcbe21f8910b95691846599ba.jpg\n\n\nTODO: slice smith termination is shorted instead of with cap
 Text Label 3950 1400 0    50   ~ 0
@@
 Wire Wire Line
 	2600 6350 2850 6350
-$Comp
-L Jumper:SolderJumper_2_Open JP?
-U 1 1 615BF249
-P 7900 3150
-AR Path="/610DBB8D/615BF249" Ref="JP?"  Part="1"
-AR Path="/613B6218/615BF249" Ref="JP?"  Part="1"
-AR Path="/613B6EFF/615BF249" Ref="JP?"  Part="1"
-AR Path="/613B79B7/615BF249" Ref="JP?"  Part="1"
-AR Path="/613B8664/615BF249" Ref="JP?"  Part="1"
-AR Path="/613B8F90/615BF249" Ref="JP?"  Part="1"
-AR Path="/611D29AA/615BF249" Ref="JP?"  Part="1"
-AR Path="/620E19B3/615BF249" Ref="JP?"  Part="1"
-AR Path="/620FBA4C/615BF249" Ref="JP?"  Part="1"
-AR Path="/6211795B/615BF249" Ref="JP?"  Part="1"
-AR Path="/621328FA/615BF249" Ref="JP?"  Part="1"
-AR Path="/62156471/615BF249" Ref="JP?"  Part="1"
-AR Path="/62171C6A/615BF249" Ref="JP?"  Part="1"
-AR Path="/6218DDB9/615BF249" Ref="JP?"  Part="1"
-AR Path="/61E646BE/615BF249" Ref="JP?"  Part="1"
-AR Path="/612EF6EF/615BF249" Ref="JP?"  Part="1"
-AR Path="/612FBF86/615BF249" Ref="JP?"  Part="1"
-AR Path="/61339A05/615BF249" Ref="JP?"  Part="1"
-AR Path="/61347D57/615BF249" Ref="JP?"  Part="1"
-AR Path="/6135BFD5/615BF249" Ref="JP?"  Part="1"
-AR Path="/61397EC7/615BF249" Ref="JP?"  Part="1"
-AR Path="/613FE9A0/615BF249" Ref="JP?"  Part="1"
-AR Path="/61409D83/615BF249" Ref="JP?"  Part="1"
-AR Path="/61416F70/615BF249" Ref="JP?"  Part="1"
-AR Path="/6142DC9F/615BF249" Ref="JP?"  Part="1"
-AR Path="/6143BBD4/615BF249" Ref="JP?"  Part="1"
-AR Path="/6144BA8F/615BF249" Ref="JP?"  Part="1"
-AR Path="/613B5606/615BF249" Ref="JP?"  Part="1"
-AR Path="/6142DC7D/615BF249" Ref="JP?"  Part="1"
-AR Path="/6143BBB2/615BF249" Ref="JP?"  Part="1"
-AR Path="/614B514C/615BF249" Ref="JP?"  Part="1"
-AR Path="/613B6F05/615BF249" Ref="JP?"  Part="1"
-AR Path="/6144BA6D/615BF249" Ref="JP?"  Part="1"
-AR Path="/615BF249" Ref="JP27"  Part="1"
-F 0 "JP27" H 8050 3200 50  0000 C CNN
-F 1 "SolderJumper_2_Open" H 7900 3264 50  0001 C CNN
-F 2 "Jumper:SolderJumper-2_P1.3mm_Open_RoundedPad1.0x1.5mm" H 7900 3150 50  0001 C CNN
-F 3 "~" H 7900 3150 50  0001 C CNN
-	1    7900 3150
-	1    0    0    -1
-$EndComp
-Text Label 8600 3150 2    50   ~ 0
-3V3_MGMT
-Text Label 7450 3150 0    50   ~ 0
-LED_3V3
-Wire Wire Line
-	8050 3150 8600 3150
-Wire Wire Line
-	7750 3150 7450 3150
 Wire Wire Line
 	3850 1000 4050 1000

Commit message: floating all post-transformer ethernet
as per azonenbergs suggestion,
external ethernet traces shouldnt use the local ground as reference.

I have no idea how to calculate the impedance for free floating
differential pairs.  i THINK they need to be treated as single ended?
but targeting which impedance? 100? 50?
Connections:
- wire segments 206 -> 205
Other:
- moved on the sheet: H1, H2
Changed lines of the file:
@@
 L power:GND #PWR09
 U 1 1 61D74BD2
-P 5650 6950
-F 0 "#PWR09" H 5650 6700 50  0001 C CNN
-F 1 "GND" H 5655 6777 50  0000 C CNN
-F 2 "" H 5650 6950 50  0001 C CNN
-F 3 "" H 5650 6950 50  0001 C CNN
-	1    5650 6950
+P 5850 6950
+F 0 "#PWR09" H 5850 6700 50  0001 C CNN
+F 1 "GND" H 5855 6777 50  0000 C CNN
+F 2 "" H 5850 6950 50  0001 C CNN
+F 3 "" H 5850 6950 50  0001 C CNN
+	1    5850 6950
 	1    0    0    -1
 $EndComp
@@
 	1    0    0    -1
 $EndComp
-Wire Wire Line
-	5650 6950 5850 6950
 $Comp
 L Mechanical:MountingHole_Pad H1
 U 1 1 61DAAD7C
-P 5650 6850
-F 0 "H1" H 5600 7050 50  0000 L CNN
-F 1 "MountingHole" H 5750 6808 50  0001 L CNN
-F 2 "MountingHole:MountingHole_3.2mm_M3_Pad" H 5650 6850 50  0001 C CNN
-F 3 "~" H 5650 6850 50  0001 C CNN
-	1    5650 6850
-	1    0    0    -1
-$EndComp
-Connection ~ 5650 6950
-$Comp
-L Mechanical:MountingHole_Pad H2
-U 1 1 61DAAF7A
 P 5850 6850
-F 0 "H2" H 5800 7050 50  0000 L CNN
+F 0 "H1" H 5800 7050 50  0000 L CNN
 F 1 "MountingHole" H 5950 6808 50  0001 L CNN
 F 2 "MountingHole:MountingHole_3.2mm_M3_Pad" H 5850 6850 50  0001 C CNN
@@
 	1    0    0    -1
 $EndComp
+$Comp
+L Mechanical:MountingHole_Pad H2
+U 1 1 61DAAF7A
+P 5450 6850
+F 0 "H2" H 5400 7050 50  0000 L CNN
+F 1 "MountingHole" H 5550 6808 50  0001 L CNN
+F 2 "MountingHole:MountingHole_3.2mm_M3_Pad" H 5450 6850 50  0001 C CNN
+F 3 "~" H 5450 6850 50  0001 C CNN
+	1    5450 6850
+	1    0    0    -1
+$EndComp

Commit message: replace transformer/jack combo with magjack
we learned from andrew that the pre-transformer length loss isn't actually that bad.

On the other hand the pre-transformer signals carry alot of EMI.

I find the EMI more scary because it depends on outside factors,
while the pre-transformer loss is a work or no-work situation.
Parts:
- removed J1: SS-74500-020, dg_connectors:BEL_SS-74500-020, symbol dg_connectors:SS-74500-020
- added C17, C18, C31, C33: 100nF, Capacitor_SMD:C_0402_1005Metric, symbol Device:C
- added J20: 0879-2C2R-54, dg_connectors:BEL_0879-2C2R-54, symbol dg_connectors:0879-2C2R-54
Connections:
- wire segments 205 -> 261
Other:
- note added: "TODO: replace usb hub"
- note removed: "Blue"
- note removed: "Blue White"
- note removed: "Brown"
- note removed: "Brown White"
- note removed: "Green"
- note removed: "Green White"
- note removed: "Orange"
- note removed: "Orange White"
- note removed: "TODO: switch usb detect is wrong\nTODO: usb connectors have D+/- reversed\nTODO: RJ45 is cursed. https://i.pinimg.com/originals/46/e6/6c/46e66c1fcbe21f8910b95691846599ba.jpg\n\n\nTODO: slice smith termination is shorted instead of with cap"
- moved on the sheet: D1, D2, FID1, FID2, FID3, H1, H2, H3, H4, H5, H6, J5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

Commit message: Changed fuse footprint and updated Part num.
Other:
- moved on the sheet: H2
Changed lines of the file:
@@
 L Mechanical:MountingHole_Pad H2
 U 1 1 61DAAF7A
-P 10400 7750
-F 0 "H2" H 10350 7950 50  0000 L CNN
-F 1 "MountingHole" H 10500 7708 50  0001 L CNN
-F 2 "MountingHole:MountingHole_3.2mm_M3_Pad" H 10400 7750 50  0001 C CNN
-F 3 "~" H 10400 7750 50  0001 C CNN
-	1    10400 7750
+P 10600 7750
+F 0 "H2" H 10550 7950 50  0000 L CNN
+F 1 "MountingHole" H 10700 7708 50  0001 L CNN
+F 2 "MountingHole:MountingHole_3.2mm_M3_Pad" H 10600 7750 50  0001 C CNN
+F 3 "~" H 10600 7750 50  0001 C CNN
+	1    10600 7750
 	1    0    0    -1
 $EndComp
@@
 	2950 10200 2000 10200
 Wire Wire Line
-	10800 7850 10400 7850
+	10800 7850 10600 7850
 $EndSCHEMATC

Commit message: Added Part numbers.
Parts:
- D1, D2: #LCSC (none) -> C110519
Changed lines of the file:
@@
 F 2 "Diode_SMD:D_SMA" H 12650 2100 50  0001 C CNN
 F 3 "~" H 12650 2100 50  0001 C CNN
+F 4 "C110519" V 12650 2100 50  0001 C CNN "#LCSC"
 	1    12650 2100
 	0    1    1    0
@@
 F 2 "Diode_SMD:D_SMA" H 11650 2100 50  0001 C CNN
 F 3 "~" H 11650 2100 50  0001 C CNN
+F 4 "C110519" V 11650 2100 50  0001 C CNN "#LCSC"
 	1    11650 2100
 	0    1    1    0
