File: pi.sch (KiCad schematic (older format))
At the start: 16 parts

Commit message: nvme
Parts:
- added C1, C3: C, Capacitor_SMD:C_0805_2012Metric, symbol Device:C
- added C2, C4: C, Capacitor_SMD:C_0603_1608Metric, symbol Device:C
- added D3, D4: LED, LED_SMD:LED_0603_1608Metric, symbol Device:LED
- added R2, R3: R, Resistor_SMD:R_0603_1608Metric, symbol Device:R
- added U2: m.2_pcie_nvme, dg_connectors:m.2_pcie_nvme, symbol dg_connectors:m.2_pcie_nvme
- gave numbers to parts that had none: 13
Connections:
- net 3.3V: now also C3.1, C4.1, D4.2 (A), U2.12 (3V3), U2.14 (3V3), U2.16 (3V3), U2.18 (3V3), U2.2 (3V3), U2.4 (3V3)
- net 5V: now also C1.1, C2.1, D3.2 (A)
- net GND: now also C1.2, C2.2, C3.2, C4.2, R2.1, R3.1
- net pcie_clkreq: now reaches U1.102 (PCIe_CLK_nREQ)
- net pcie_clkreq: now also U2.52 (CLKREQ#/NC)
- net pcie_nrst: now reaches U1.109 (PCIe_nRST)
- net pcie_nrst: now also U2.50 (PERST#/NC)
- net pcie_clk+: now reaches U1.110 (PCIe_CLK_P)
- net pcie_clk+: now also U2.55 (REFCLKP)
- net pcie_clk-: now reaches U1.112 (PCIe_CLK_N)
- net pcie_clk-: now also U2.53 (REFCLKN)
- new net: D3.1 (K), R2.2
- new net: D4.1 (K), R3.2
Other:
- moved on the sheet: D22, D23, D24, R21, R22, R23, U1B, U1C, U1D

Commit message: maybe use a premade powerbrick
Parts:
- added T2: QT24A01, dg_transformers:SOP100P1000X450-24N, symbol dg_transformers:QT24A01
- added TP13, TP14, TP15: TestPoint, TestPoint:TestPoint_Pad_D1.0mm, symbol Connector:TestPoint
Connections:
- net pcie_clk+ is gone; now on net GND: U1.110 (PCIe_CLK_P), U2.55 (REFCLKP)
- net pcie_clk- is gone; now on net GND: U1.112 (PCIe_CLK_N), U2.53 (REFCLKN)
- net 3.3V: now also U2.70 (3V3), U2.72 (3V3), U2.74 (3V3)
- net GND: now also U2.1 (GND), U2.15 (GND), U2.21 (GND), U2.27 (GND), U2.3 (GND), U2.33 (GND), U2.39 (GND), U2.45 (GND), U2.51 (GND), U2.57 (GND), U2.71 (GND), U2.73 (GND), U2.75 (GND), U2.9 (GND), U2.MP
- net RPI_PCIe_RX_P: now reaches U1.116 (PCIe_RX_P)
- net RPI_PCIe_RX_P: now also U2.43 (PERP0/SATA_B-)
- net RPI_PCIe_RX_N: now reaches U1.118 (PCIe_RX_N)
- net RPI_PCIe_RX_N: now also U2.41 (PERN0/SATA_B+)
- net RPI_PCIe_TX_P: now reaches U1.122 (PCIe_TX_P)
- net RPI_PCIe_TX_P: now also U2.49 (PETP0/SATA_A+)
- net RPI_PCIe_TX_N: now reaches U1.124 (PCIe_TX_N)
- net RPI_PCIe_TX_N: now also U2.47 (PETN0/SATA_A-)
- net at U2.10 (DAS/DSS#): now also TP14.1
- net at U2.54 (PEWAKE#/NC): now also TP15.1
- net at U2.69 (PEDET): now also TP13.1
- net pcie_clkreq renamed RPI_PCIe_CLK_nREQ
- net pcie_nrst renamed RPI_PCIe_nRST
Other:
- moved on the sheet: C13, C14, U1B, U1D

Commit message: just use two usb hubs
Other:
- moved on the sheet: T1
Changed lines of the file:
@@
 $Descr A4 11693 8268
 encoding utf-8
-Sheet 2 3
+Sheet 2 5
 Title ""
 Date ""
@@
 L dg_transformers:QT24A01 T2
 U 1 1 62435BC4
-P 6900 850
+P 6450 900
 AR Path="/620E19B3/62435BC4" Ref="T2"  Part="1"
 AR Path="/613B6EFF/62435BC4" Ref="T1"  Part="1"
@@
 AR Path="/62171C6A/62435BC4" Ref="T4"  Part="1"
 AR Path="/6218DDB9/62435BC4" Ref="T5"  Part="1"
-F 0 "T1" H 7450 1205 50  0000 C CNN
-F 1 "QT24A01" H 7450 1114 50  0000 C CNN
-F 2 "dg_transformers:SOP100P1000X450-24N" H 7050 -500 50  0001 L CNN
-F 3 "https://datasheet.lcsc.com/szlcsc/TNK-QT24A01_C216359.pdf" H 7850 850 50  0001 L CNN
-F 4 "10/100/1000Base-T Single Port Transformer Module" H 7050 -600 50  0001 L CNN "Description"
-F 5 "4.5" H 7850 -700 50  0001 L CNN "Height"
-F 6 "TNK" H 7050 -700 50  0001 L CNN "Manufacturer_Name"
-F 7 "QT24A01" H 7300 -700 50  0001 L CNN "Manufacturer_Part_Number"
-F 8 "C216359" H 7450 1023 50  0000 C CNN "LCSC#"
-	1    6900 850
-	1    0    0    -1
-$EndComp
+F 0 "T1" H 7000 1255 50  0000 C CNN
+F 1 "QT24A01" H 7000 1164 50  0000 C CNN
+F 2 "dg_transformers:SOP100P1000X450-24N" H 6600 -450 50  0001 L CNN
+F 3 "https://datasheet.lcsc.com/szlcsc/TNK-QT24A01_C216359.pdf" H 7400 900 50  0001 L CNN
+F 4 "10/100/1000Base-T Single Port Transformer Module" H 6600 -550 50  0001 L CNN "Description"
+F 5 "4.5" H 7400 -650 50  0001 L CNN "Height"
+F 6 "TNK" H 6600 -650 50  0001 L CNN "Manufacturer_Name"
+F 7 "QT24A01" H 6850 -650 50  0001 L CNN "Manufacturer_Part_Number"
+F 8 "C216359" H 7000 1073 50  0000 C CNN "LCSC#"
+	1    6450 900
+	1    0    0    -1
+$EndComp

Commit message: Organized DC-DC Schematic.
Changed lines of the file:
@@
 	2100 850  2200 850
-$Comp
-L power:GND #PWR0112
-U 1 1 612B9481
-P 3200 1050
-AR Path="/610DBB8D/612B9481" Ref="#PWR0112"  Part="1"
-AR Path="/613B6218/612B9481" Ref="#PWR0126"  Part="1"
-AR Path="/613B6EFF/612B9481" Ref="#PWR0134"  Part="1"
-AR Path="/613B79B7/612B9481" Ref="#PWR0142"  Part="1"
-AR Path="/613B8664/612B9481" Ref="#PWR0150"  Part="1"
-AR Path="/613B8F90/612B9481" Ref="#PWR0158"  Part="1"
-AR Path="/611D29AA/612B9481" Ref="#PWR0231"  Part="1"
-AR Path="/620E19B3/612B9481" Ref="#PWR0117"  Part="1"
-AR Path="/620FBA4C/612B9481" Ref="#PWR0226"  Part="1"
-AR Path="/6211795B/612B9481" Ref="#PWR0239"  Part="1"
-AR Path="/621328FA/612B9481" Ref="#PWR0252"  Part="1"
-AR Path="/62156471/612B9481" Ref="#PWR05"  Part="1"
-AR Path="/62171C6A/612B9481" Ref="#PWR019"  Part="1"
-AR Path="/6218DDB9/612B9481" Ref="#PWR033"  Part="1"
-F 0 "#PWR0134" H 3200 800 50  0001 C CNN
-F 1 "GND" H 3205 877 50  0000 C CNN
-F 2 "" H 3200 1050 50  0001 C CNN
-F 3 "" H 3200 1050 50  0001 C CNN
-	1    3200 1050
-	1    0    0    -1
-$EndComp
-Wire Wire Line
-	3200 1050 3200 850
-Wire Wire Line
-	3200 850  2950 850
 $Comp
 L Device:LED D4
@@
 L power:GND #PWR0113
 U 1 1 612CB2FE
-P 4900 1050
+P 4800 950
 AR Path="/610DBB8D/612CB2FE" Ref="#PWR0113"  Part="1"
 AR Path="/613B6218/612CB2FE" Ref="#PWR0127"  Part="1"
@@
 AR Path="/62171C6A/612CB2FE" Ref="#PWR021"  Part="1"
 AR Path="/6218DDB9/612CB2FE" Ref="#PWR035"  Part="1"
-F 0 "#PWR0135" H 4900 800 50  0001 C CNN
-F 1 "GND" H 4905 877 50  0000 C CNN
-F 2 "" H 4900 1050 50  0001 C CNN
-F 3 "" H 4900 1050 50  0001 C CNN
-	1    4900 1050
-	1    0    0    -1
-$EndComp
-Wire Wire Line
-	4900 1050 4900 850
-Wire Wire Line
-	4900 850  4650 850
+F 0 "#PWR0135" H 4800 700 50  0001 C CNN
+F 1 "GND" H 4805 777 50  0000 C CNN
+F 2 "" H 4800 950 50  0001 C CNN
+F 3 "" H 4800 950 50  0001 C CNN
+	1    4800 950
+	1    0    0    -1
+$EndComp
 $Comp
 L Device:C C1
@@
 	1    0    0    -1
 $EndComp
+Wire Wire Line
+	4650 850  4800 850
+Wire Wire Line
+	4800 850  4800 950
+$Comp
+L power:GND #PWR?
+U 1 1 6113A7DA
+P 3100 950
+AR Path="/610DBB8D/6113A7DA" Ref="#PWR?"  Part="1"
+AR Path="/613B6218/6113A7DA" Ref="#PWR?"  Part="1"
+AR Path="/613B6EFF/6113A7DA" Ref="#PWR?"  Part="1"
+AR Path="/613B79B7/6113A7DA" Ref="#PWR?"  Part="1"
+AR Path="/613B8664/6113A7DA" Ref="#PWR?"  Part="1"
+AR Path="/613B8F90/6113A7DA" Ref="#PWR?"  Part="1"
+AR Path="/611D29AA/6113A7DA" Ref="#PWR?"  Part="1"
+AR Path="/620E19B3/6113A7DA" Ref="#PWR?"  Part="1"
+AR Path="/620FBA4C/6113A7DA" Ref="#PWR?"  Part="1"
+AR Path="/6211795B/6113A7DA" Ref="#PWR?"  Part="1"
+AR Path="/621328FA/6113A7DA" Ref="#PWR?"  Part="1"
+AR Path="/62156471/6113A7DA" Ref="#PWR?"  Part="1"
+AR Path="/62171C6A/6113A7DA" Ref="#PWR?"  Part="1"
+AR Path="/6218DDB9/6113A7DA" Ref="#PWR?"  Part="1"
+F 0 "#PWR?" H 3100 700 50  0001 C CNN
+F 1 "GND" H 3105 777 50  0000 C CNN
+F 2 "" H 3100 950 50  0001 C CNN
+F 3 "" H 3100 950 50  0001 C CNN
+	1    3100 950
+	1    0    0    -1
+$EndComp
+Wire Wire Line
+	2950 850  3100 850
+Wire Wire Line
+	3100 850  3100 950
 $EndSCHEMATC

Commit message: Organized pi.sch document.
Parts:
- removed C2, C4: C, Capacitor_SMD:C_0603_1608Metric, symbol Device:C
- removed C3: C, Capacitor_SMD:C_0805_2012Metric, symbol Device:C
- removed D3, D4: LED, LED_SMD:LED_0603_1608Metric, symbol Device:LED
- removed R1, R2, R3, R4, R5, R6: R, Resistor_SMD:R_0603_1608Metric, symbol Device:R
- added C? (x8): 10uF, Capacitor_SMD:C_0805_2012Metric, symbol Device:C
- added C? (x2): 100uF, Capacitor_SMD:C_1206_3216Metric, symbol Device:C
- added C? (x6): 100nF, Capacitor_SMD:C_0402_1005Metric, symbol Device:C
- added C?: 1000pF 2kV, Capacitor_SMD:C_1206_3216Metric, symbol Device:C
- added R? (x4): 1k, Resistor_SMD:R_0402_1005Metric, symbol Device:R
- added R? (x4): 75, Resistor_SMD:R_0402_1005Metric, symbol Device:R
- C1: value C -> 10uF
Connections:
- net 5V: now also C?.1, C?.1, C?.1, C?.1, C?.1, C?.1
- net ETH0+: now also T2.23 (MX1+); no longer U1.12 (Ethernet_Pair0_P)
- net ETH0-: now also T2.22 (MX1-); no longer U1.10 (Ethernet_Pair0_N)
- net ETH1+: now also T2.20 (MX2+); no longer U1.4 (Ethernet_Pair1_P)
- net ETH1-: now also T2.19 (MX2-); no longer U1.6 (Ethernet_Pair1_N)
- net ETH2+: now also T2.17 (MX3+); no longer U1.11 (Ethernet_Pair2_P)
- net ETH2-: now also T2.16 (MX3-); no longer U1.9 (Ethernet_Pair2_N)
- net ETH3+: now also T2.14 (MX4+); no longer U1.3 (Ethernet_Pair3_P)
- net ETH3-: now also T2.13 (MX4-); no longer U1.5 (Ethernet_Pair3_N)
- net GND: now also C?.1, C?.2, C?.2, C?.2, C?.2, C?.2, C?.2, C?.2, C?.2, C?.2, C?.2, C?.2, C?.2, C?.2, C?.2, C?.2, C?.2; no longer U1.110 (PCIe_CLK_P), U1.112 (PCIe_CLK_N), U2.53 (REFCLKN), U2.55 (REFCLKP)
- net at U1.21 (Pi_nLED_Activity): now also R?.2
- net at U1.15 (Ethernet_nLED3_(act,green,_3.3V)): now also R?.2
- net at U1.17 (Ethernet_nLED2_(speed,yellow,_3.3V)): now also R?.2
- net at U1.19 (Ethernet_nLED1_(speed,yellow,_3.3V)): now also R?.2
- net at D2.1 (K): now also R?.1
- net at D5.2 (A): now also R?.1
- net at D6.2 (A): now also R?.1
- net at D7.2 (A): now also R?.1
- net at T2.1 (TCT1): now also T2.10 (TCT4), T2.4 (TCT2), T2.7 (TCT3), C?.1
- net TD4_P: now reaches T2.11 (TD4+)
- net TD4_P: now also U1.3 (Ethernet_Pair3_P)
- net TD4_N: now reaches T2.12 (TD4-)
- net TD4_N: now also U1.5 (Ethernet_Pair3_N)
- net at T2.15 (MCT4): now also R?.1
- net at T2.18 (MCT3): now also R?.1
- net TD1_P: now reaches T2.2 (TD1+)
- net TD1_P: now also U1.12 (Ethernet_Pair0_P)
- net at T2.21 (MCT2): now also R?.1
- net at T2.24 (MCT1): now also R?.1
- net TD1_N: now reaches T2.3 (TD1-)
- net TD1_N: now also U1.10 (Ethernet_Pair0_N)
- net TD2_P: now reaches T2.5 (TD2+)
- net TD2_P: now also U1.4 (Ethernet_Pair1_P)
- net TD2_N: now reaches T2.6 (TD2-)
- net TD2_N: now also U1.6 (Ethernet_Pair1_N)
- net TD3_P: now reaches T2.8 (TD3+)
- net TD3_P: now also U1.11 (Ethernet_Pair2_P)
- net TD3_N: now reaches T2.9 (TD3-)
- net TD3_N: now also U1.9 (Ethernet_Pair2_N)
- net pi3.3 renamed pi3V3
- new net: C?.2, R?.2, R?.2, R?.2, R?.2
- new net 3V3: C?.1, C?.1, C?.1, C?.1, C?.1, C?.1, C?.1, C?.1, C?.1
- new net RPI_PCIe_CLK_N: U1.112 (PCIe_CLK_N), U2.53 (REFCLKN)
- new net RPI_PCIe_CLK_P: U1.110 (PCIe_CLK_P), U2.55 (REFCLKP)
Other:
- note added: "CM4 Decoupling"
- note added: "NVMe Decoupling"
- moved on the sheet: C11, D19, D22, D23, D24, JP13, JP14, JP15, JP16, T1, TP12, TP6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
