File: pi.sch (KiCad schematic (older format))
At the start: 36 parts, among them T1 QT24A01, U1 rpi_cm4, U2 m.2_pcie_nvme

Commit message: Added PN for PCIE Connector.
Parts:
- U2: LCSC# (none) -> C364435

Commit message: Completed Signal & Power Routing.
Parts:
- removed TP1, TP2, TP3: TestPoint, TestPoint:TestPoint_Pad_D1.0mm, symbol Connector:TestPoint
Connections:
- wire segments 245 -> 242

Commit message: Changed Eth. Led supply to rpi internal 3v3.
Connections:
- net pi3V3 renamed 3V3_INT
Changed lines of the file:
@@
 Wire Wire Line
 	2050 7500 2600 7500
+Text HLabel 1400 2450 0    50   Input ~ 0
+3V3_INT
+Wire Wire Line
+	1600 2450 1400 2450
+Connection ~ 1600 2450
 $EndSCHEMATC
