File: pi.sch (KiCad schematic (older format))
At the start: 28 parts, among them J2 DF40HC_3.0_-100DS-0.4V_51_PNP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, J3 DF40HC_3.0_-100DS-0.4V_51_PNP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, U1 rpi_cm4, U2 m.2_pcie_nvme

Commit message: Changed fuse footprint and updated Part num.
Other:
- moved on the sheet: J16, J17

Commit message: DFM
Parts:
- C1, C8: JLC# (none) -> C312983
- C10, C11, C12, C13, C2, C3, C4, C9: JLC# (none) -> C15850
- C14, C15, C16, C6: JLC# (none) -> C1525

Commit message: Added Part numbers.
Parts:
- R7: #LCSC (none) -> C11702
Changed lines of the file:
@@
 F 2 "Resistor_SMD:R_0402_1005Metric" V 1380 5450 50  0001 C CNN
 F 3 "~" H 1450 5450 50  0001 C CNN
+F 4 "C11702" V 1450 5450 50  0001 C CNN "#LCSC"
 	1    1450 5450
 	0    -1   -1   0
