File: mgm.sch (KiCad schematic (older format))
At the start: 17 parts, among them U3 rpi_cm4

Commit message: just use two usb hubs
Parts:
- removed C5: C, Capacitor_SMD:C_0805_2012Metric, symbol Device:C
- removed C6: C, Capacitor_SMD:C_0603_1608Metric, symbol Device:C
- removed D10, D11, D12, D8, D9: LED, LED_SMD:LED_0603_1608Metric, symbol Device:LED
- removed JP5, JP6, JP7, JP8: SolderJumper_2_Open, Jumper:SolderJumper-2_P1.3mm_Open_RoundedPad1.0x1.5mm, symbol Jumper:SolderJumper_2_Open
- removed R10, R11, R8, R9: R, Resistor_SMD:R_0603_1608Metric, symbol Device:R
- removed U3: rpi_cm4, dg_rpi:rpi_cm4, symbol dg_rpi:rpi_cm4
- added C1, C2: 14pF, Capacitor_SMD:C_0603_1608Metric, symbol Device:C
- added C3: 100nF, Capacitor_SMD:C_0603_1608Metric, symbol Device:C
- added C4: 10uF, Capacitor_SMD:C_0603_1608Metric, symbol Device:C
- added J4: Conn_02x03_Odd_Even, Connector_PinHeader_2.54mm:PinHeader_2x03_P2.54mm_Vertical, symbol Connector_Generic:Conn_02x03_Odd_Even
- added J5: Conn_02x03_Odd_Even, Connector:Tag-Connect_TC2030-IDC-FP_2x03_P1.27mm_Vertical, symbol Connector_Generic:Conn_02x03_Odd_Even
- added J6: 2x20, Connector_PinHeader_2.54mm:PinHeader_2x20_P2.54mm_Vertical, symbol Connector_Generic:Conn_02x20_Odd_Even
- added M1, M2: Fan_4pin, Connector:FanPinHeader_1x04_P2.54mm_Vertical, symbol Motor:Fan_4pin
- added R4, R5: NC, Resistor_SMD:R_0603_1608Metric, symbol Device:R
- added R6: 36K 1%, Resistor_SMD:R_0603_1608Metric, symbol Device:R
- added U3: EMC2301, Package_SO:MSOP-8_3x3mm_P0.65mm, symbol aep:EMC2301
- added U4: STM32L151C8T6, Package_QFP:LQFP-48_7x7mm_P0.5mm, symbol MCU_ST_STM32L1:STM32L151C8Tx
- added Y1: 24Mhz X1E0000210264, Crystal:Crystal_SMD_SeikoEpson_TSX3225-4Pin_3.2x2.5mm, symbol Device:Crystal_GND24_Small
- R7: value R -> 36K 1%
Connections:
- net labels added: +12V, +3V3, c1_act, c1_boot, c1_reset, c1_rx, c1_tx, c1_vref, c1_wp, c2_act, c2_boot, c2_reset, c2_rx, c2_tx, c2_vref, c2_wp, c3_act, c3_boot, c3_reset, c3_rx, c3_tx, c3_vref, c3_wp, c4_act, c4_boot, c4_gpio1, c4_reset, c4_rx, c4_tx, c4_vref, c4_wp, mcu_reset, mcu_scl, mcu_sda, mcu_swclk, mcu_swdio, mcu_tdo, mcu_usb+, mcu_usb-
- net labels removed: 5V, BOOT, ETH0+, ETH0-, ETH1+, ETH1-, ETH2+, ETH2-, ETH3+, ETH3-, RX, TX, USB+, USB-, pi3.3
- wire segments 111 -> 138
- no-connect marks 4 -> 9
Other:
- note added: "c4 is soft uart, because thats just mgm to mcu\ncustomers get hard uart"

Commit message: use native rpi uarts instead of extra chip
Parts:
- removed C4: 10uF, Capacitor_SMD:C_0603_1608Metric, symbol Device:C
- removed J4: Conn_02x03_Odd_Even, Connector_PinHeader_2.54mm:PinHeader_2x03_P2.54mm_Vertical, symbol Connector_Generic:Conn_02x03_Odd_Even
- removed J5: Conn_02x03_Odd_Even, Connector:Tag-Connect_TC2030-IDC-FP_2x03_P1.27mm_Vertical, symbol Connector_Generic:Conn_02x03_Odd_Even
- removed J6: 2x20, Connector_PinHeader_2.54mm:PinHeader_2x20_P2.54mm_Vertical, symbol Connector_Generic:Conn_02x20_Odd_Even
- removed R4: NC, Resistor_SMD:R_0603_1608Metric, symbol Device:R
- removed U4: STM32L151C8T6, Package_QFP:LQFP-48_7x7mm_P0.5mm, symbol MCU_ST_STM32L1:STM32L151C8Tx
- removed Y1: 24Mhz X1E0000210264, Crystal:Crystal_SMD_SeikoEpson_TSX3225-4Pin_3.2x2.5mm, symbol Device:Crystal_GND24_Small
- added D2, D3, D4, D5, D6: LED, LED_SMD:LED_0603_1608Metric, symbol Device:LED
- added JP1, JP2, JP3, JP4: SolderJumper_2_Open, Jumper:SolderJumper-2_P1.3mm_Open_RoundedPad1.0x1.5mm, symbol Jumper:SolderJumper_2_Open
- added R10, R11, R12, R8: R, Resistor_SMD:R_0603_1608Metric, symbol Device:R
- added T2: QT24A01, dg_transformers:SOP100P1000X450-24N, symbol dg_transformers:QT24A01
- added U1, U4: rpi_cm4, dg_rpi:rpi_cm4, symbol dg_rpi:rpi_cm4
- C1: value 14pF -> C; footprint Capacitor_SMD:C_0603_1608Metric -> Capacitor_SMD:C_0805_2012Metric
- C2: value 14pF -> C
- R5: value NC -> R
Connections:
- net labels added: 5V, ETH0+, ETH0-, ETH1+, ETH1-, ETH2+, ETH2-, ETH3+, ETH3-, RXD3, RXD4, RXD5, SCL, SDA, TXD3, TXD4, TXD5, USB+, USB-, c1_disable, c2_disable, c3_disable, c4_disable, pi3.3
- net labels removed: c1_act, c1_reset, c1_vref, c1_wp, c2_act, c2_reset, c2_vref, c2_wp, c3_act, c3_reset, c3_vref, c3_wp, c4_act, c4_gpio1, c4_reset, c4_vref, c4_wp, mcu_reset, mcu_scl, mcu_sda, mcu_swclk, mcu_swdio, mcu_tdo, mcu_usb+, mcu_usb-
- wire segments 138 -> 151
- no-connect marks 9 -> 7
Other:
- note removed: "c4 is soft uart, because thats just mgm to mcu\ncustomers get hard uart"
- moved on the sheet: C3, M1, M2, R6, R7, U3

Commit message: use a 2x2 and a magjack
Parts:
- removed T2: QT24A01, dg_transformers:SOP100P1000X450-24N, symbol dg_transformers:QT24A01
- added J6: 0826-1X1T-GH-F, dg_connectors:BEL_0826-1X1T-GH-F, symbol dg_connectors:0826-1X1T-GH-F
Connections:
- wire segments 151 -> 159
Changed lines of the file:
@@
-$EndComp
-$Comp
-L dg_transformers:QT24A01 T?
-U 1 1 618693F9
-P 6550 3900
-AR Path="/620E19B3/618693F9" Ref="T?"  Part="1"
-AR Path="/613B6EFF/618693F9" Ref="T?"  Part="1"
-AR Path="/62156471/618693F9" Ref="T?"  Part="1"
-AR Path="/62171C6A/618693F9" Ref="T?"  Part="1"
-AR Path="/6218DDB9/618693F9" Ref="T?"  Part="1"
-AR Path="/613B5606/618693F9" Ref="T2"  Part="1"
-F 0 "T2" H 7100 4255 50  0000 C CNN
-F 1 "QT24A01" H 7100 4164 50  0000 C CNN
-F 2 "dg_transformers:SOP100P1000X450-24N" H 6700 2550 50  0001 L CNN
-F 3 "https://datasheet.lcsc.com/szlcsc/TNK-QT24A01_C216359.pdf" H 7500 3900 50  0001 L CNN
-F 4 "10/100/1000Base-T Single Port Transformer Module" H 6700 2450 50  0001 L CNN "Description"
-F 5 "4.5" H 7500 2350 50  0001 L CNN "Height"
-F 6 "TNK" H 6700 2350 50  0001 L CNN "Manufacturer_Name"
-F 7 "QT24A01" H 6950 2350 50  0001 L CNN "Manufacturer_Part_Number"
-F 8 "C216359" H 7100 4073 50  0000 C CNN "LCSC#"
-	1    6550 3900
-	1    0    0    -1
 $EndComp
 $Comp
@@
 Text HLabel 4600 2650 0    50   Input ~ 0
 c1_boot
+$Comp
+L dg_connectors:0826-1X1T-GH-F J6
+U 1 1 612127DD
+P 6200 5200
+F 0 "J6" H 6100 6767 50  0000 C CNN
+F 1 "0826-1X1T-GH-F" H 6100 6676 50  0000 C CNN
+F 2 "dg_connectors:BEL_0826-1X1T-GH-F" H 5750 6950 50  0001 L BNN
+F 3 "" H 6250 7100 50  0001 L BNN
+	1    6200 5200
+	-1   0    0    -1
+$EndComp
+Wire Wire Line
+	7400 4300 7150 4300
+Wire Wire Line
+	7150 4100 7400 4100
+Wire Wire Line
+	7400 3900 7150 3900
+Text HLabel 7400 4300 2    50   Input ~ 0
+ETH1+
+Text HLabel 7400 4100 2    50   Input ~ 0
+ETH0-
+Text HLabel 7400 3900 2    50   Input ~ 0
+ETH0+
+Text HLabel 7400 4500 2    50   Input ~ 0
+ETH1-
+Text HLabel 7400 4700 2    50   Input ~ 0
+ETH2+
+Wire Wire Line
+	7150 4500 7400 4500
+Wire Wire Line
+	7400 4700 7150 4700
+Text HLabel 7400 4900 2    50   Input ~ 0
+ETH2-
+Text HLabel 7400 5100 2    50   Input ~ 0
+ETH3+
+Wire Wire Line
+	7150 4900 7400 4900
+Wire Wire Line
+	7400 5100 7150 5100
+Text HLabel 7400 5300 2    50   Input ~ 0
+ETH3-
+Wire Wire Line
+	7150 5300 7400 5300
 $EndSCHEMATC

Commit message: Organized schematics.
Parts:
- removed U3: EMC2301, Package_SO:MSOP-8_3x3mm_P0.65mm, symbol aep:EMC2301
- added U?: EMC2301, Package_SO:MSOP-8_3x3mm_P0.65mm, symbol dg_ic:EMC2301

Commit message: replace fan controller with rpi gpio
the chip is out of stock until 2022
Parts:
- removed C3: 100nF, Capacitor_SMD:C_0603_1608Metric, symbol Device:C
- removed R6, R7: 36K 1%, Resistor_SMD:R_0603_1608Metric, symbol Device:R
- removed U?: EMC2301, Package_SO:MSOP-8_3x3mm_P0.65mm, symbol dg_ic:EMC2301
- added C?: 100nF, Capacitor_SMD:C_0402_1005Metric, symbol Device:C
- added R? (x4): 0Ohm, Resistor_SMD:R_0402_1005Metric, symbol Device:R
- R8: footprint Resistor_SMD:R_0603_1608Metric -> Resistor_SMD:R_0402_1005Metric
Connections:
- net labels added: fanpwm, tach1, tach2
- net labels removed: +3V3
- wire segments 159 -> 162
- no-connect marks 7 -> 4
Other:
- moved on the sheet: J6, M1, M2
