File: mgm.sch (KiCad schematic (older format))
At the start: 26 parts, among them J6 0826-1X1T-GH-F, M1 Fan_4pin, M2 Fan_4pin, U1 rpi_cm4, U4 rpi_cm4

Commit message: Created .gitignore file. Completed schematic organization. Added Fan Driver alternative.
Parts:
- removed C1: C, Capacitor_SMD:C_0805_2012Metric, symbol Device:C
- removed C2: C, Capacitor_SMD:C_0603_1608Metric, symbol Device:C
- removed C?: 100nF, Capacitor_SMD:C_0402_1005Metric, symbol Device:C
- removed D2, D3, D4, D5, D6: LED, LED_SMD:LED_0603_1608Metric, symbol Device:LED
- removed JP1, JP2, JP3, JP4: SolderJumper_2_Open, Jumper:SolderJumper-2_P1.3mm_Open_RoundedPad1.0x1.5mm, symbol Jumper:SolderJumper_2_Open
- removed M2: Fan_4pin, Connector:FanPinHeader_1x04_P2.54mm_Vertical, symbol Motor:Fan_4pin
- removed R10, R11, R12, R5: R, Resistor_SMD:R_0603_1608Metric, symbol Device:R
- removed R8: R, Resistor_SMD:R_0402_1005Metric, symbol Device:R
- removed R? (x4): 0Ohm, Resistor_SMD:R_0402_1005Metric, symbol Device:R
- added C? (x4): 10uF, Capacitor_SMD:C_0805_2012Metric, symbol Device:C
- added C?: 100uF, Capacitor_SMD:C_1206_3216Metric, symbol Device:C
- added C? (x3): 100nF, Capacitor_SMD:C_0402_1005Metric, symbol Device:C
- added D? (x2): LED, LED_SMD:LED_0603_1608Metric, symbol Device:LED
- added JP? (x5): SolderJumper_2_Open, Jumper:SolderJumper-2_P1.3mm_Open_RoundedPad1.0x1.5mm, symbol Jumper:SolderJumper_2_Open
- added M?: Fan_4pin, Connector:FanPinHeader_1x04_P2.54mm_Vertical, symbol Motor:Fan_4pin
- added Q?: 2N7002K, Package_TO_SOT_SMD:SOT-23, symbol Transistor_FET:2N7002K
- added R? (x4): 1k, Resistor_SMD:R_0402_1005Metric, symbol Device:R
- added R? (x3): 470, Resistor_SMD:R_0402_1005Metric, symbol Device:R
- added R? (x2): 0, Resistor_SMD:R_0402_1005Metric, symbol Device:R
- added R?: 7.2K, Resistor_SMD:R_0402_1005Metric, symbol Device:R
- added R?: 5K, Resistor_SMD:R_0402_1005Metric, symbol Device:R
- added R?: DNP, Resistor_SMD:R_0402_1005Metric, symbol Device:R
Connections:
- net labels added: eth_act_ledg, eth_speed_ledy, fan_pwm_in, pi3V3
- net labels removed: SCL, SDA, pi3.3
- wire segments 162 -> 190
Other:
- note added: "CM4 Decoupling"
- note added: "Two Options to drive Fans.\nResistor between fanpwm-fan_pwm_in is to \nbypass mosfet drive. \n12V must be disabled before bypassing."
- note added: "UART RX/TX Pairs \nSwapped in this section."
- moved on the sheet: J6, M1, U1F, U4A, U4C

Commit message: Schematics annotated.
Parts:
- gave numbers to parts that had none: 29
- renumbered J6 to J13, U4 to U10

Commit message: Completed PCB Placement.
Parts:
- removed C85: 10uF, Capacitor_SMD:C_0805_2012Metric, symbol Device:C
- removed C87: 100nF, Capacitor_SMD:C_0402_1005Metric, symbol Device:C
- renumbered U1 to U10
Connections:
- wire segments 190 -> 182
Changed lines of the file:
@@
 AR Path="/62171C6A/618D9DD5" Ref="U?"  Part="1"
 AR Path="/6218DDB9/618D9DD5" Ref="U?"  Part="1"
-AR Path="/613B5606/618D9DD5" Ref="U1"  Part="6"
-F 0 "U1" H 4600 1165 50  0000 C CNN
+AR Path="/613B5606/618D9DD5" Ref="U10"  Part="6"
+F 0 "U10" H 4600 1165 50  0000 C CNN
 F 1 "rpi_cm4" H 4600 1074 50  0000 C CNN
 F 2 "dg_rpi:rpi_cm4" H 4750 -4550 50  0001 C CNN
@@
 Text HLabel 1450 7000 0    50   Input ~ 0
 5V
-$Comp
-L Device:C C?
-U 1 1 612AF71F
-P 2550 7200
-AR Path="/610DBB8D/612AF71F" Ref="C?"  Part="1"
-AR Path="/613B6218/612AF71F" Ref="C?"  Part="1"
-AR Path="/613B6EFF/612AF71F" Ref="C?"  Part="1"
-AR Path="/613B79B7/612AF71F" Ref="C?"  Part="1"
-AR Path="/613B8664/612AF71F" Ref="C?"  Part="1"
-AR Path="/613B8F90/612AF71F" Ref="C?"  Part="1"
-AR Path="/611D29AA/612AF71F" Ref="C?"  Part="1"
-AR Path="/620E19B3/612AF71F" Ref="C?"  Part="1"
-AR Path="/620FBA4C/612AF71F" Ref="C?"  Part="1"
-AR Path="/6211795B/612AF71F" Ref="C?"  Part="1"
-AR Path="/621328FA/612AF71F" Ref="C?"  Part="1"
-AR Path="/62156471/612AF71F" Ref="C?"  Part="1"
-AR Path="/62171C6A/612AF71F" Ref="C?"  Part="1"
-AR Path="/6218DDB9/612AF71F" Ref="C?"  Part="1"
-AR Path="/61E646BE/612AF71F" Ref="C?"  Part="1"
-AR Path="/612EF6EF/612AF71F" Ref="C?"  Part="1"
-AR Path="/612FBF86/612AF71F" Ref="C?"  Part="1"
-AR Path="/61339A05/612AF71F" Ref="C?"  Part="1"
-AR Path="/61347D57/612AF71F" Ref="C?"  Part="1"
-AR Path="/6135BFD5/612AF71F" Ref="C?"  Part="1"
-AR Path="/61397EC7/612AF71F" Ref="C?"  Part="1"
-AR Path="/613FE9A0/612AF71F" Ref="C?"  Part="1"
-AR Path="/61409D83/612AF71F" Ref="C?"  Part="1"
-AR Path="/61416F70/612AF71F" Ref="C?"  Part="1"
-AR Path="/6142DC9F/612AF71F" Ref="C?"  Part="1"
-AR Path="/6143BBD4/612AF71F" Ref="C?"  Part="1"
-AR Path="/6144BA8F/612AF71F" Ref="C?"  Part="1"
-AR Path="/613B5606/612AF71F" Ref="C85"  Part="1"
-F 0 "C85" H 2600 7300 50  0000 L CNN
-F 1 "10uF" H 2600 7100 50  0000 L CNN
-F 2 "Capacitor_SMD:C_0805_2012Metric" H 2588 7050 50  0001 C CNN
-F 3 "~" H 2550 7200 50  0001 C CNN
-	1    2550 7200
-	1    0    0    -1
-$EndComp
 $Comp
 L power:GND #PWR?
@@
 	1    0    0    -1
 $EndComp
-Wire Wire Line
-	2850 7000 2550 7000
-Wire Wire Line
-	2550 7050 2550 7000
-Connection ~ 2550 7000
 $Comp
 L Device:C C?
@@
 	1500 7400 1800 7400
 Wire Wire Line
-	2550 7400 2550 7350
-Wire Wire Line
 	1450 7000 1500 7000
 Wire Wire Line
@@
 Connection ~ 2300 7400
 Wire Wire Line
-	2300 7400 2550 7400
-Wire Wire Line
 	2300 7050 2300 7000
 Connection ~ 2300 7000
 Wire Wire Line
-	2300 7000 2550 7000
-Wire Wire Line
 	2050 7050 2050 7000
 Connection ~ 2050 7000
@@
 Wire Wire Line
 	1800 7000 2050 7000
-$Comp
-L Device:C C?
-U 1 1 612AF760
-P 3150 7200
-AR Path="/610DBB8D/612AF760" Ref="C?"  Part="1"
-AR Path="/613B6218/612AF760" Ref="C?"  Part="1"
-AR Path="/613B6EFF/612AF760" Ref="C?"  Part="1"
-AR Path="/613B79B7/612AF760" Ref="C?"  Part="1"
-AR Path="/613B8664/612AF760" Ref="C?"  Part="1"
-AR Path="/613B8F90/612AF760" Ref="C?"  Part="1"
-AR Path="/611D29AA/612AF760" Ref="C?"  Part="1"
-AR Path="/620E19B3/612AF760" Ref="C?"  Part="1"
-AR Path="/620FBA4C/612AF760" Ref="C?"  Part="1"
-AR Path="/6211795B/612AF760" Ref="C?"  Part="1"
-AR Path="/621328FA/612AF760" Ref="C?"  Part="1"
-AR Path="/62156471/612AF760" Ref="C?"  Part="1"
-AR Path="/62171C6A/612AF760" Ref="C?"  Part="1"
-AR Path="/6218DDB9/612AF760" Ref="C?"  Part="1"
-AR Path="/61E646BE/612AF760" Ref="C?"  Part="1"
-AR Path="/612EF6EF/612AF760" Ref="C?"  Part="1"
-AR Path="/612FBF86/612AF760" Ref="C?"  Part="1"
-AR Path="/61339A05/612AF760" Ref="C?"  Part="1"
-AR Path="/61347D57/612AF760" Ref="C?"  Part="1"
-AR Path="/6135BFD5/612AF760" Ref="C?"  Part="1"
-AR Path="/61397EC7/612AF760" Ref="C?"  Part="1"
-AR Path="/613FE9A0/612AF760" Ref="C?"  Part="1"
-AR Path="/61409D83/612AF760" Ref="C?"  Part="1"
-AR Path="/61416F70/612AF760" Ref="C?"  Part="1"
-AR Path="/6142DC9F/612AF760" Ref="C?"  Part="1"
-AR Path="/6143BBD4/612AF760" Ref="C?"  Part="1"
-AR Path="/6144BA8F/612AF760" Ref="C?"  Part="1"
-AR Path="/613B5606/612AF760" Ref="C87"  Part="1"
-F 0 "C87" H 3200 7300 50  0000 L CNN
-F 1 "100nF" H 3200 7100 50  0000 L CNN
-F 2 "Capacitor_SMD:C_0402_1005Metric" H 3188 7050 50  0001 C CNN
-F 3 "~" H 3150 7200 50  0001 C CNN
-	1    3150 7200
-	1    0    0    -1
-$EndComp
 $Comp
 L Device:C C?
@@
 $EndComp
 Wire Wire Line
-	3150 7400 3150 7350
-Wire Wire Line
-	3150 7400 2850 7400
-Wire Wire Line
 	2850 7400 2850 7350
 Wire Wire Line
-	2850 7400 2550 7400
-Connection ~ 2850 7400
-Connection ~ 2550 7400
-Wire Wire Line
 	2850 7050 2850 7000
-Wire Wire Line
-	2850 7000 3150 7000
-Wire Wire Line
-	3150 7000 3150 7050
-Connection ~ 2850 7000
 Text Notes 2050 6950 0    50   ~ 0
 CM4 Decoupling
@@
 Wire Wire Line
 	5550 1350 5150 1350
-Wire Wire Line
-	5550 2750 5150 2750
-Wire Wire Line
-	5550 2850 5150 2850
-Wire Wire Line
-	5550 2950 5150 2950
-Wire Wire Line
-	5550 3050 5150 3050
-Wire Wire Line
-	5550 3150 5150 3150
-Wire Wire Line
-	5550 3250 5150 3250
-Wire Wire Line
-	5550 3350 5150 3350
-Wire Wire Line
-	5550 3450 5150 3450
 Text Notes 5100 1000 0    50   ~ 0
 UART RX/TX Pairs \nSwapped in this section.
@@
 Wire Wire Line
 	7250 1150 7400 1150
+Wire Wire Line
+	2300 7000 2850 7000
+Wire Wire Line
+	2300 7400 2850 7400
+Wire Wire Line
+	5550 2750 5150 2750
+Wire Wire Line
+	5150 2850 5550 2850
+Wire Wire Line
+	5550 2950 5150 2950
+Wire Wire Line
+	5150 3050 5550 3050
+Wire Wire Line
+	5550 3150 5150 3150
+Wire Wire Line
+	5150 3250 5550 3250
+Wire Wire Line
+	5550 3350 5150 3350
+Wire Wire Line
+	5150 3450 5550 3450
 $EndSCHEMATC

Commit message: Fixed fan pwm connection.
Connections:
- wire segments 182 -> 184
Changed lines of the file:
@@
 	6500 1750 6150 1750
 Wire Wire Line
-	7400 1450 7400 1600
+	7400 1450 7400 1500
 Wire Wire Line
 	7100 1500 7100 1550
@@
 Text Label 7900 1500 2    50   ~ 0
 fan_pwm_in
-Wire Wire Line
-	7100 1500 7900 1500
-Connection ~ 7100 1500
 Text Notes 6400 2550 0    50   ~ 0
 Two Options to drive Fans.\nResistor between fanpwm-fan_pwm_in is to \nbypass mosfet drive. \n12V must be disabled before bypassing.
@@
 Wire Wire Line
 	5150 3450 5550 3450
+Connection ~ 7100 1500
+Wire Wire Line
+	7100 1500 7400 1500
+Connection ~ 7400 1500
+Wire Wire Line
+	7400 1500 7400 1600
+Wire Wire Line
+	7400 1500 7900 1500
 $EndSCHEMATC

Commit message: Added 3th Fan Connector.
Parts:
- added M3: Fan_4pin, Connector:FanPinHeader_1x04_P2.54mm_Vertical, symbol Motor:Fan_4pin
- added R82: 1k, Resistor_SMD:R_0402_1005Metric, symbol Device:R
- added R83: 0, Resistor_SMD:R_0402_1005Metric, symbol Device:R
Connections:
- net labels added: tach3
- wire segments 184 -> 192
Changed lines of the file:
@@
 Wire Wire Line
 	7400 1500 7900 1500
+$Comp
+L Motor:Fan_4pin M?
+U 1 1 61425EE3
+P 7550 3250
+AR Path="/6133068E/61425EE3" Ref="M?"  Part="1"
+AR Path="/61425EE3" Ref="M?"  Part="1"
+AR Path="/613B5606/61425EE3" Ref="M3"  Part="1"
+F 0 "M3" H 7708 3346 50  0000 L CNN
+F 1 "Fan_4pin" H 7708 3255 50  0000 L CNN
+F 2 "Connector:FanPinHeader_1x04_P2.54mm_Vertical" H 7550 3260 50  0001 C CNN
+F 3 "http://www.formfactors.org/developer%5Cspecs%5Crev1_2_public.pdf" H 7550 3260 50  0001 C CNN
+	1    7550 3250
+	1    0    0    -1
+$EndComp
+$Comp
+L power:GND #PWR?
+U 1 1 61425EE9
+P 7550 3450
+AR Path="/61425EE9" Ref="#PWR?"  Part="1"
+AR Path="/5FEB1CB4/61425EE9" Ref="#PWR?"  Part="1"
+AR Path="/5FECBD46/61425EE9" Ref="#PWR?"  Part="1"
+AR Path="/5FECD465/61425EE9" Ref="#PWR?"  Part="1"
+AR Path="/5FECEB82/61425EE9" Ref="#PWR?"  Part="1"
+AR Path="/5FDF5C30/61425EE9" Ref="#PWR?"  Part="1"
+AR Path="/5FDF9B9D/61425EE9" Ref="#PWR?"  Part="1"
+AR Path="/5FDFE7F4/61425EE9" Ref="#PWR?"  Part="1"
+AR Path="/6133068E/61425EE9" Ref="#PWR?"  Part="1"
+AR Path="/613B5606/61425EE9" Ref="#PWR03"  Part="1"
+F 0 "#PWR03" H 7550 3200 50  0001 C CNN
+F 1 "GND" H 7555 3277 50  0000 C CNN
+F 2 "" H 7550 3450 50  0001 C CNN
+F 3 "" H 7550 3450 50  0001 C CNN
+	1    7550 3450
+	1    0    0    -1
+$EndComp
+$Comp
+L power:+12V #PWR?
+U 1 1 61425EEF
+P 7550 2950
+AR Path="/6133068E/61425EEF" Ref="#PWR?"  Part="1"
+AR Path="/61425EEF" Ref="#PWR?"  Part="1"
+AR Path="/613B5606/61425EEF" Ref="#PWR02"  Part="1"
+F 0 "#PWR02" H 7550 2800 50  0001 C CNN
+F 1 "+12V" H 7565 3123 50  0000 C CNN
+F 2 "" H 7550 2950 50  0001 C CNN
+F 3 "" H 7550 2950 50  0001 C CNN
+	1    7550 2950
+	1    0    0    -1
+$EndComp
+Text Label 6600 3150 2    50   ~ 0
+tach3
+Wire Wire Line
+	7000 3150 7100 3150
+Text Label 6600 2950 2    50   ~ 0
+pi3V3
+Wire Wire Line
+	6700 2950 6400 2950
+$Comp
+L Device:R R?
+U 1 1 61425EF9
+P 6850 3150
+AR Path="/611D29B0/61425EF9" Ref="R?"  Part="1"
+AR Path="/613B6F05/61425EF9" Ref="R?"  Part="1"
+AR Path="/620E19B9/61425EF9" Ref="R?"  Part="1"
+AR Path="/620FBA52/61425EF9" Ref="R?"  Part="1"
+AR Path="/62117961/61425EF9" Ref="R?"  Part="1"
+AR Path="/62132900/61425EF9" Ref="R?"  Part="1"
+AR Path="/62156477/61425EF9" Ref="R?"  Part="1"
+AR Path="/62171C70/61425EF9" Ref="R?"  Part="1"
+AR Path="/6218DDBF/61425EF9" Ref="R?"  Part="1"
+AR Path="/61DCBD06/61425EF9" Ref="R?"  Part="1"
+AR Path="/613B6EFF/61425EF9" Ref="R?"  Part="1"
+AR Path="/61E646BE/61425EF9" Ref="R?"  Part="1"
+AR Path="/612EF6EF/61425EF9" Ref="R?"  Part="1"
+AR Path="/612FBF86/61425EF9" Ref="R?"  Part="1"
+AR Path="/61339A05/61425EF9" Ref="R?"  Part="1"
+AR Path="/61347D57/61425EF9" Ref="R?"  Part="1"
+AR Path="/6135BFD5/61425EF9" Ref="R?"  Part="1"
+AR Path="/61397EC7/61425EF9" Ref="R?"  Part="1"
+AR Path="/613FE9A0/61425EF9" Ref="R?"  Part="1"
+AR Path="/61409D83/61425EF9" Ref="R?"  Part="1"
+AR Path="/61416F70/61425EF9" Ref="R?"  Part="1"
+AR Path="/6142DC9F/61425EF9" Ref="R?"  Part="1"
+AR Path="/6143BBD4/61425EF9" Ref="R?"  Part="1"
+AR Path="/6144BA8F/61425EF9" Ref="R?"  Part="1"
+AR Path="/613B5606/61425EF9" Ref="R83"  Part="1"
+F 0 "R83" V 6950 3150 50  0000 C CNN
+F 1 "0" V 6850 3150 50  0000 C CNN
+F 2 "Resistor_SMD:R_0402_1005Metric" V 6780 3150 50  0001 C CNN
+F 3 "~" H 6850 3150 50  0001 C CNN
+	1    6850 3150
+	0    -1   -1   0
+$EndComp
+Wire Wire Line
+	7100 3150 7100 2950
+Wire Wire Line
+	7100 2950 7000 2950
+Connection ~ 7100 3150
+Wire Wire Line
+	7100 3150 7250 3150
+Wire Wire Line
+	6700 3150 6400 3150
+$Comp
+L Device:R R?
+U 1 1 61425F04
+P 6850 2950
+AR Path="/611D29B0/61425F04" Ref="R?"  Part="1"
+AR Path="/613B6F05/61425F04" Ref="R?"  Part="1"
+AR Path="/620E19B9/61425F04" Ref="R?"  Part="1"
+AR Path="/620FBA52/61425F04" Ref="R?"  Part="1"
+AR Path="/62117961/61425F04" Ref="R?"  Part="1"
+AR Path="/62132900/61425F04" Ref="R?"  Part="1"
+AR Path="/62156477/61425F04" Ref="R?"  Part="1"
+AR Path="/62171C70/61425F04" Ref="R?"  Part="1"
+AR Path="/6218DDBF/61425F04" Ref="R?"  Part="1"
+AR Path="/61DCBD06/61425F04" Ref="R?"  Part="1"
+AR Path="/613B6EFF/61425F04" Ref="R?"  Part="1"
+AR Path="/61E646BE/61425F04" Ref="R?"  Part="1"
+AR Path="/612EF6EF/61425F04" Ref="R?"  Part="1"
+AR Path="/612FBF86/61425F04" Ref="R?"  Part="1"
+AR Path="/61339A05/61425F04" Ref="R?"  Part="1"
+AR Path="/61347D57/61425F04" Ref="R?"  Part="1"
+AR Path="/6135BFD5/61425F04" Ref="R?"  Part="1"
+AR Path="/61397EC7/61425F04" Ref="R?"  Part="1"
+AR Path="/613FE9A0/61425F04" Ref="R?"  Part="1"
+AR Path="/61409D83/61425F04" Ref="R?"  Part="1"
+AR Path="/61416F70/61425F04" Ref="R?"  Part="1"
+AR Path="/6142DC9F/61425F04" Ref="R?"  Part="1"
+AR Path="/6143BBD4/61425F04" Ref="R?"  Part="1"
+AR Path="/6144BA8F/61425F04" Ref="R?"  Part="1"
+AR Path="/613B5606/61425F04" Ref="R82"  Part="1"
+F 0 "R82" V 6950 2950 50  0000 C CNN
+F 1 "1k" V 6850 2950 50  0000 C CNN
+F 2 "Resistor_SMD:R_0402_1005Metric" V 6780 2950 50  0001 C CNN
+F 3 "~" H 6850 2950 50  0001 C CNN
+	1    6850 2950
+	0    -1   -1   0
+$EndComp
+Text Label 7200 3350 2    50   ~ 0
+fan_pwm_in
+Wire Wire Line
+	6750 3350 7250 3350
+Text Label 5250 2650 0    50   ~ 0
+tach3
+Wire Wire Line
+	5450 2650 5150 2650
 $EndSCHEMATC

Commit message: replace transformers, since out of stock
Parts:
- added J18, J19: DF40HC_3.0_-100DS-0.4V_51_PNP_OVERLAY, dg_rpi:HRS_DF40HC(3.0)-100DS-0.4V(58)_PNP_OVERLAY, symbol dg_rpi:DF40HC_3.0_-100DS-0.4V_51_PNP_OVERLAY
Changed lines of the file:
@@
 Wire Wire Line
 	5450 2650 5150 2650
+$Comp
+L dg_rpi:DF40HC_3.0_-100DS-0.4V_51_PNP_OVERLAY J?
+U 1 1 61404CBC
+P 11550 6800
+AR Path="/613B6EFF/61404CBC" Ref="J?"  Part="1"
+AR Path="/6142DC9F/61404CBC" Ref="J?"  Part="1"
+AR Path="/6143BBD4/61404CBC" Ref="J?"  Part="1"
+AR Path="/6144BA8F/61404CBC" Ref="J?"  Part="1"
+AR Path="/613B5606/61404CBC" Ref="J19"  Part="1"
+F 0 "J19" H 11828 6891 50  0000 L CNN
+F 1 "DF40HC_3.0_-100DS-0.4V_51_PNP_OVERLAY" H 11828 6800 50  0000 L CNN
+F 2 "dg_rpi:HRS_DF40HC(3.0)-100DS-0.4V(58)_PNP_OVERLAY" H 12400 6900 50  0001 L CNN
+F 3 "https://componentsearchengine.com/Datasheets/1/DF40HC(3.0)-100DS-0.4V(51.pdf" H 12400 6800 50  0001 L CNN
+F 4 "Board to Board & Mezzanine Connectors 100P 2R 3MM RECPT SMT VERT 0.4MM PITCH" H 12400 6700 50  0001 L CNN "Description"
+F 5 "3.05" H 12400 6600 50  0001 L CNN "Height"
+F 6 "Hirose" H 12400 6500 50  0001 L CNN "Manufacturer_Name"
+F 7 "DF40HC(3.0)-100DS-0.4V(51" H 12400 6400 50  0001 L CNN "Manufacturer_Part_Number"
+F 8 "798-DF40HC30100DS451" H 12400 6300 50  0001 L CNN "Mouser Part Number"
+F 9 "https://www.mouser.co.uk/ProductDetail/Hirose-Connector/DF40HC30-100DS-04V51?qs=%252BAZVS4b%2FkgIV%252B3vHYy2dCA%3D%3D" H 12400 6200 50  0001 L CNN "Mouser Price/Stock"
+F 10 "DF40HC(3.0)-100DS-0.4V(51" H 12400 6100 50  0001 L CNN "Arrow Part Number"
+F 11 "https://www.arrow.com/en/products/df40hc-3.0-100ds-0.4v-51/hirose-electric" H 12400 6000 50  0001 L CNN "Arrow Price/Stock"
+F 12 "C424649" H 11828 6709 50  0000 L CNN "LCSC#"
+	1    11550 6800
+	1    0    0    -1
+$EndComp
+$Comp
+L dg_rpi:DF40HC_3.0_-100DS-0.4V_51_PNP_OVERLAY J?
+U 1 1 61404CCB
+P 11550 6350
+AR Path="/613B6EFF/61404CCB" Ref="J?"  Part="1"
+AR Path="/6142DC9F/61404CCB" Ref="J?"  Part="1"
+AR Path="/6143BBD4/61404CCB" Ref="J?"  Part="1"
+AR Path="/6144BA8F/61404CCB" Ref="J?"  Part="1"
+AR Path="/613B5606/61404CCB" Ref="J18"  Part="1"
+F 0 "J18" H 11828 6441 50  0000 L CNN
+F 1 "DF40HC_3.0_-100DS-0.4V_51_PNP_OVERLAY" H 11828 6350 50  0000 L CNN
+F 2 "dg_rpi:HRS_DF40HC(3.0)-100DS-0.4V(58)_PNP_OVERLAY" H 12400 6450 50  0001 L CNN
+F 3 "https://componentsearchengine.com/Datasheets/1/DF40HC(3.0)-100DS-0.4V(51.pdf" H 12400 6350 50  0001 L CNN
+F 4 "Board to Board & Mezzanine Connectors 100P 2R 3MM RECPT SMT VERT 0.4MM PITCH" H 12400 6250 50  0001 L CNN "Description"
+F 5 "3.05" H 12400 6150 50  0001 L CNN "Height"
+F 6 "Hirose" H 12400 6050 50  0001 L CNN "Manufacturer_Name"
+F 7 "DF40HC(3.0)-100DS-0.4V(51" H 12400 5950 50  0001 L CNN "Manufacturer_Part_Number"
+F 8 "798-DF40HC30100DS451" H 12400 5850 50  0001 L CNN "Mouser Part Number"
+F 9 "https://www.mouser.co.uk/ProductDetail/Hirose-Connector/DF40HC30-100DS-04V51?qs=%252BAZVS4b%2FkgIV%252B3vHYy2dCA%3D%3D" H 12400 5750 50  0001 L CNN "Mouser Price/Stock"
+F 10 "DF40HC(3.0)-100DS-0.4V(51" H 12400 5650 50  0001 L CNN "Arrow Part Number"
+F 11 "https://www.arrow.com/en/products/df40hc-3.0-100ds-0.4v-51/hirose-electric" H 12400 5550 50  0001 L CNN "Arrow Price/Stock"
+F 12 "C424649" H 11828 6259 50  0000 L CNN "LCSC#"
+	1    11550 6350
+	1    0    0    -1
+$EndComp
 $EndSCHEMATC
