File: usbhub.sch (KiCad schematic (older format))
At the start: 34 parts, among them J7 USB_C_Receptacle, U5 USB2514B_Bi, U6 USB2514B_Bi, Y2 24Mhz X1E0000210264, Y3 24Mhz X1E0000210264

Commit message: use native rpi uarts instead of extra chip
Parts:
- removed C10, C9: 14pF, Capacitor_SMD:C_0603_1608Metric, symbol Device:C
- removed C17: 10uF, Capacitor_SMD:C_0603_1608Metric, symbol Device:C
- removed C5, C6: 0.1uF, Capacitor_SMD:C_0603_1608Metric, symbol Device:C
- removed H1, H2, H3, H4: MountingHole, MountingHole:MountingHole_3.2mm_M3_Pad_Via, symbol Mechanical:MountingHole
- removed J?: USB_C_Receptacle, symbol Connector:USB_C_Receptacle
- removed R10, R11, R12, R13, R14, R15: 10K, Resistor_SMD:R_0603_1608Metric, symbol Device:R
- removed R8: 12K 1%, Resistor_SMD:R_0603_1608Metric, symbol Device:R
- removed U5: USB2514B_Bi, Package_DFN_QFN:QFN-36-1EP_6x6mm_P0.5mm_EP3.7x3.7mm, symbol Interface_USB:USB2514B_Bi
- removed Y2: 24Mhz X1E0000210264, Crystal:Crystal_SMD_SeikoEpson_TSX3225-4Pin_3.2x2.5mm, symbol Device:Crystal_GND24_Small
Connections:
- net labels added: 3.3V
- net labels removed: +3V3, ext_usb+, ext_usb-, mcu_usb+, mcu_usb-, r2_usb+, r2_usb-
- wire segments 146 -> 76
- no-connect marks 18 -> 9
Other:
- moved on the sheet: C15, C16, C18, C7, C8, J7, R16, R17, R24, R25, R26, R27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
