File: usbhub.sch (KiCad schematic (older format))
At the start: 19 parts, among them U3 USB2514B_Bi, Y1 24Mhz Q24FA20H00339

Commit message: Added Part numbers.
Parts:
- C22, C23: value 14pF -> 18pF; JLC# C458857 -> C1549
- R15, R18, R19, R20, R21: #LCSC (none) -> C25744
- Y1: value 24Mhz Q24FA20H00339 -> X1E0000210129 24Mhz 12pF; JLC# C255952 -> C255917
Other:
- note added: "6pF Input Capacitance"
Changed lines of the file:
@@
 AR Path="/6130ED51/617667F3" Ref="Y1"  Part="1"
 F 0 "Y1" H 5700 5650 50  0000 L CNN
-F 1 "24Mhz Q24FA20H00339" H 5450 5350 50  0000 L CNN
+F 1 "X1E0000210129 24Mhz 12pF" H 5300 5350 50  0000 L CNN
 F 2 "Crystal:Crystal_SMD_SeikoEpson_TSX3225-4Pin_3.2x2.5mm" H 5900 5500 50  0001 C CNN
 F 3 "~" H 5900 5500 50  0001 C CNN
-F 4 "C255952" H 5900 5500 50  0001 C CNN "JLC#"
+F 4 "C255917" H 5900 5500 50  0001 C CNN "JLC#"
 	1    5900 5500
 	-1   0    0    1
@@
 F 2 "Resistor_SMD:R_0402_1005Metric" V 5280 4750 50  0001 C CNN
 F 3 "~" H 5350 4750 50  0001 C CNN
+F 4 "C25744" V 5350 4750 50  0001 C CNN "#LCSC"
 	1    5350 4750
 	-1   0    0    1
@@
 F 2 "Resistor_SMD:R_0402_1005Metric" V 5080 4750 50  0001 C CNN
 F 3 "~" H 5150 4750 50  0001 C CNN
+F 4 "C25744" V 5150 4750 50  0001 C CNN "#LCSC"
 	1    5150 4750
 	-1   0    0    1
@@
 F 2 "Resistor_SMD:R_0402_1005Metric" V 4880 4300 50  0001 C CNN
 F 3 "~" H 4950 4300 50  0001 C CNN
+F 4 "C25744" V 4950 4300 50  0001 C CNN "#LCSC"
 	1    4950 4300
 	0    -1   -1   0
@@
 F 2 "Resistor_SMD:R_0402_1005Metric" V 4880 4400 50  0001 C CNN
 F 3 "~" H 4950 4400 50  0001 C CNN
+F 4 "C25744" V 4950 4400 50  0001 C CNN "#LCSC"
 	1    4950 4400
 	0    -1   -1   0
@@
 AR Path="/6130ED51/617B578E" Ref="C22"  Part="1"
 F 0 "C22" H 5550 5750 50  0000 L CNN
-F 1 "14pF" H 5550 5550 50  0000 L CNN
+F 1 "18pF" H 5550 5550 50  0000 L CNN
 F 2 "Capacitor_SMD:C_0402_1005Metric" H 5538 5500 50  0001 C CNN
 F 3 "~" H 5500 5650 50  0001 C CNN
-F 4 "C458857" H 5500 5650 50  0001 C CNN "JLC#"
+F 4 "C1549" H 5500 5650 50  0001 C CNN "JLC#"
 	1    5500 5650
 	1    0    0    -1
@@
 AR Path="/6130ED51/617B5AAC" Ref="C23"  Part="1"
 F 0 "C23" H 6300 5750 50  0000 L CNN
-F 1 "14pF" H 6300 5550 50  0000 L CNN
+F 1 "18pF" H 6300 5550 50  0000 L CNN
 F 2 "Capacitor_SMD:C_0402_1005Metric" H 6288 5500 50  0001 C CNN
 F 3 "~" H 6250 5650 50  0001 C CNN
-F 4 "C458857" H 6250 5650 50  0001 C CNN "JLC#"
+F 4 "C1549" H 6250 5650 50  0001 C CNN "JLC#"
 	1    6250 5650
 	1    0    0    -1
@@
 F 2 "Resistor_SMD:R_0402_1005Metric" V 6980 5500 50  0001 C CNN
 F 3 "~" H 7050 5500 50  0001 C CNN
+F 4 "C25744" V 7050 5500 50  0001 C CNN "#LCSC"
 	1    7050 5500
 	0    -1   -1   0
@@
 	4000 5350 3700 5350
 Connection ~ 4000 5350
+Text Notes 5450 5300 0    50   ~ 0
+6pF Input Capacitance
 $EndSCHEMATC

Commit message: Changed USB Hub with Mux.
Parts:
- removed C19: 10uF, Capacitor_SMD:C_0805_2012Metric, symbol Device:C
- removed C20, C21, C24, C25, C26, C5, C7: 100nF, Capacitor_SMD:C_0402_1005Metric, symbol Device:C
- removed C22, C23: 18pF, Capacitor_SMD:C_0402_1005Metric, symbol Device:C
- removed R15, R16, R18, R19, R20, R21: 10k, Resistor_SMD:R_0402_1005Metric, symbol Device:R
- removed R17: 12k 1%, Resistor_SMD:R_0402_1005Metric, symbol Device:R
- removed U3: USB2514B_Bi, Package_DFN_QFN:QFN-36-1EP_6x6mm_P0.5mm_EP3.7x3.7mm, symbol Interface_USB:USB2514B_Bi
- removed Y1: X1E0000210129 24Mhz 12pF, Crystal:Crystal_SMD_SeikoEpson_TSX3225-4Pin_3.2x2.5mm, symbol Device:Crystal_GND24_Small
- added C? (x3): 100nF, Capacitor_SMD:C_0402_1005Metric, symbol Device:C
- added R? (x6): 10k, Resistor_SMD:R_0402_1005Metric, symbol Device:R
- added U? (x3): FSUSB30MUX, Package_SO:MSOP-10_3x3mm_P0.5mm, symbol dg_ic:FSUSB30MUX
Connections:
- net 3.3V: now also C?.1, C?.1, C?.1, R?.2, R?.2, U?.10 (VCC), U?.10 (VCC), U?.10 (VCC)
- net GND: now also C?.2, C?.2, C?.2, R?.2, R?.2, R?.2, R?.2, U?.5 (GND), U?.5 (GND), U?.5 (GND)
- net c1_usb+: now also U?.2 (HSD1+)
- net c1_usb-: now also U?.8 (HSD1-)
- net c2_usb+: now also U?.3 (HSD2+)
- net c2_usb-: now also U?.7 (HSD2-)
- net c3_usb+: now also U?.2 (HSD1+)
- net c3_usb-: now also U?.8 (HSD1-)
- net c4_usb+: now also U?.3 (HSD2+)
- net c4_usb-: now also U?.7 (HSD2-)
- net root_usb+: now also U?.4 (D+)
- net root_usb-: now also U?.6 (D-)
- new net: U?.2 (HSD1+), U?.4 (D+)
- new net: U?.6 (D-), U?.8 (HSD1-)
- new net: U?.3 (HSD2+), U?.4 (D+)
- new net: U?.6 (D-), U?.7 (HSD2-)
- new net USB_SW_OE1: R?.1, U?.9 (OE)
- new net USB_SW_OE2: R?.1, U?.9 (OE)
- new net root_usb_enable: R?.1, U?.9 (OE)
- new net root_usb_sel0: R?.1, U?.1 (Select)
- new net root_usb_sel1: R?.1, U?.1 (Select)
- new net root_usb_sel2: R?.1, U?.1 (Select)
- no-connect marks 9 -> 0
Other:
- note added: "In default output is disabled (OE0)."
- note added: "OE1 & OE2 is not used."
- note removed: "6pF Input Capacitance"

Commit message: Routing Damned USB Mux.
Parts:
- gave numbers to parts that had none: 12
Connections:
- net usb_sw0_sw1+: now reaches U11.4 (D+), U3.2 (HSD1+)
- net usb_sw0_sw1-: now reaches U11.6 (D-), U3.8 (HSD1-)
- net usb_sw0_sw2+: now reaches U12.4 (D+), U3.3 (HSD2+)
- net usb_sw0_sw2-: now reaches U12.6 (D-), U3.7 (HSD2-)
Changed lines of the file:
@@
 $EndDescr
 $Comp
-L dg_ic:FSUSB30MUX U?
+L dg_ic:FSUSB30MUX U11
 U 1 1 6162937C
 P 6250 2650
-F 0 "U?" H 6250 3165 50  0000 C CNN
+F 0 "U11" H 6250 3165 50  0000 C CNN
 F 1 "FSUSB30MUX" H 6250 3074 50  0000 C CNN
 F 2 "Package_SO:MSOP-10_3x3mm_P0.5mm" H 6200 3150 50  0001 C CNN
@@
 $EndComp
 $Comp
-L dg_ic:FSUSB30MUX U?
+L dg_ic:FSUSB30MUX U3
 U 1 1 616299D6
 P 4250 2650
-F 0 "U?" H 4250 3165 50  0000 C CNN
+F 0 "U3" H 4250 3165 50  0000 C CNN
 F 1 "FSUSB30MUX" H 4250 3074 50  0000 C CNN
 F 2 "Package_SO:MSOP-10_3x3mm_P0.5mm" H 4200 3150 50  0001 C CNN
@@
 $EndComp
 $Comp
-L dg_ic:FSUSB30MUX U?
+L dg_ic:FSUSB30MUX U12
 U 1 1 61629C2B
 P 6250 4150
-F 0 "U?" H 6250 4665 50  0000 C CNN
+F 0 "U12" H 6250 4665 50  0000 C CNN
 F 1 "FSUSB30MUX" H 6250 4574 50  0000 C CNN
 F 2 "Package_SO:MSOP-10_3x3mm_P0.5mm" H 6200 4650 50  0001 C CNN
@@
 AR Path="/5FDFE7F4/61638038" Ref="#PWR?"  Part="1"
 AR Path="/6133068E/61638038" Ref="#PWR?"  Part="1"
-AR Path="/6130ED51/61638038" Ref="#PWR?"  Part="1"
-F 0 "#PWR?" H 6750 2800 50  0001 C CNN
+AR Path="/6130ED51/61638038" Ref="#PWR037"  Part="1"
+F 0 "#PWR037" H 6750 2800 50  0001 C CNN
 F 1 "GND" H 6755 2877 50  0000 C CNN
 F 2 "" H 6750 3050 50  0001 C CNN
@@
 AR Path="/5FDFE7F4/61638758" Ref="#PWR?"  Part="1"
 AR Path="/6133068E/61638758" Ref="#PWR?"  Part="1"
-AR Path="/6130ED51/61638758" Ref="#PWR?"  Part="1"
-F 0 "#PWR?" H 6750 4300 50  0001 C CNN
+AR Path="/6130ED51/61638758" Ref="#PWR038"  Part="1"
+F 0 "#PWR038" H 6750 4300 50  0001 C CNN
 F 1 "GND" H 6755 4377 50  0000 C CNN
 F 2 "" H 6750 4550 50  0001 C CNN
@@
 AR Path="/5FDFE7F4/61638AD0" Ref="#PWR?"  Part="1"
 AR Path="/6133068E/61638AD0" Ref="#PWR?"  Part="1"
-AR Path="/6130ED51/61638AD0" Ref="#PWR?"  Part="1"
-F 0 "#PWR?" H 4750 2800 50  0001 C CNN
+AR Path="/6130ED51/61638AD0" Ref="#PWR034"  Part="1"
+F 0 "#PWR034" H 4750 2800 50  0001 C CNN
 F 1 "GND" H 4755 2877 50  0000 C CNN
 F 2 "" H 4750 3050 50  0001 C CNN
@@
 AR Path="/6143BBD4/6163BB77" Ref="C?"  Part="1"
 AR Path="/6144BA8F/6163BB77" Ref="C?"  Part="1"
-AR Path="/6130ED51/6163BB77" Ref="C?"  Part="1"
-F 0 "C?" H 5700 3350 50  0000 L CNN
+AR Path="/6130ED51/6163BB77" Ref="C7"  Part="1"
+F 0 "C7" H 5700 3350 50  0000 L CNN
 F 1 "100nF" H 5700 3150 50  0000 L CNN
 F 2 "Capacitor_SMD:C_0402_1005Metric" H 5688 3100 50  0001 C CNN
@@
 AR Path="/5FDFE7F4/6164128D" Ref="#PWR?"  Part="1"
 AR Path="/6133068E/6164128D" Ref="#PWR?"  Part="1"
-AR Path="/6130ED51/6164128D" Ref="#PWR?"  Part="1"
-F 0 "#PWR?" H 5650 3150 50  0001 C CNN
+AR Path="/6130ED51/6164128D" Ref="#PWR035"  Part="1"
+F 0 "#PWR035" H 5650 3150 50  0001 C CNN
 F 1 "GND" H 5655 3227 50  0000 C CNN
 F 2 "" H 5650 3400 50  0001 C CNN
@@
 AR Path="/6143BBD4/6164261A" Ref="C?"  Part="1"
 AR Path="/6144BA8F/6164261A" Ref="C?"  Part="1"
-AR Path="/6130ED51/6164261A" Ref="C?"  Part="1"
-F 0 "C?" H 3700 3350 50  0000 L CNN
+AR Path="/6130ED51/6164261A" Ref="C5"  Part="1"
+F 0 "C5" H 3700 3350 50  0000 L CNN
 F 1 "100nF" H 3700 3150 50  0000 L CNN
 F 2 "Capacitor_SMD:C_0402_1005Metric" H 3688 3100 50  0001 C CNN
@@
 AR Path="/5FDFE7F4/61642625" Ref="#PWR?"  Part="1"
 AR Path="/6133068E/61642625" Ref="#PWR?"  Part="1"
-AR Path="/6130ED51/61642625" Ref="#PWR?"  Part="1"
-F 0 "#PWR?" H 3650 3150 50  0001 C CNN
+AR Path="/6130ED51/61642625" Ref="#PWR01"  Part="1"
+F 0 "#PWR01" H 3650 3150 50  0001 C CNN
 F 1 "GND" H 3655 3227 50  0000 C CNN
 F 2 "" H 3650 3400 50  0001 C CNN
@@
 AR Path="/6143BBD4/616458EF" Ref="C?"  Part="1"
 AR Path="/6144BA8F/616458EF" Ref="C?"  Part="1"
-AR Path="/6130ED51/616458EF" Ref="C?"  Part="1"
-F 0 "C?" H 5700 4850 50  0000 L CNN
+AR Path="/6130ED51/616458EF" Ref="C19"  Part="1"
+F 0 "C19" H 5700 4850 50  0000 L CNN
 F 1 "100nF" H 5700 4650 50  0000 L CNN
 F 2 "Capacitor_SMD:C_0402_1005Metric" H 5688 4600 50  0001 C CNN
@@
 AR Path="/5FDFE7F4/616458FA" Ref="#PWR?"  Part="1"
 AR Path="/6133068E/616458FA" Ref="#PWR?"  Part="1"
-AR Path="/6130ED51/616458FA" Ref="#PWR?"  Part="1"
-F 0 "#PWR?" H 5650 4650 50  0001 C CNN
+AR Path="/6130ED51/616458FA" Ref="#PWR036"  Part="1"
+F 0 "#PWR036" H 5650 4650 50  0001 C CNN
 F 1 "GND" H 5655 4727 50  0000 C CNN
 F 2 "" H 5650 4900 50  0001 C CNN
@@
 AR Path="/6143BBD4/616779A8" Ref="R?"  Part="1"
 AR Path="/6144BA8F/616779A8" Ref="R?"  Part="1"
-AR Path="/6130ED51/616779A8" Ref="R?"  Part="1"
-F 0 "R?" V 4450 4650 50  0000 C CNN
+AR Path="/6130ED51/616779A8" Ref="R15"  Part="1"
+F 0 "R15" V 4450 4650 50  0000 C CNN
 F 1 "10k" V 4400 4450 50  0000 C CNN
 F 2 "Resistor_SMD:R_0402_1005Metric" V 4330 4450 50  0001 C CNN
@@
 AR Path="/6143BBD4/616779AF" Ref="R?"  Part="1"
 AR Path="/6144BA8F/616779AF" Ref="R?"  Part="1"
-AR Path="/6130ED51/616779AF" Ref="R?"  Part="1"
-F 0 "R?" V 4450 4750 50  0000 C CNN
+AR Path="/6130ED51/616779AF" Ref="R16"  Part="1"
+F 0 "R16" V 4450 4750 50  0000 C CNN
 F 1 "10k" V 4400 4550 50  0000 C CNN
 F 2 "Resistor_SMD:R_0402_1005Metric" V 4330 4550 50  0001 C CNN
@@
 AR Path="/6143BBD4/616EF1BF" Ref="R?"  Part="1"
 AR Path="/6144BA8F/616EF1BF" Ref="R?"  Part="1"
-AR Path="/6130ED51/616EF1BF" Ref="R?"  Part="1"
-F 0 "R?" V 4450 4100 50  0000 C CNN
+AR Path="/6130ED51/616EF1BF" Ref="R8"  Part="1"
+F 0 "R8" V 4450 4100 50  0000 C CNN
 F 1 "10k" V 4400 3900 50  0000 C CNN
 F 2 "Resistor_SMD:R_0402_1005Metric" V 4330 3900 50  0001 C CNN
@@
 AR Path="/5FDFE7F4/616EF3E5" Ref="#PWR?"  Part="1"
 AR Path="/6133068E/616EF3E5" Ref="#PWR?"  Part="1"
-AR Path="/6130ED51/616EF3E5" Ref="#PWR?"  Part="1"
-F 0 "#PWR?" H 4650 3650 50  0001 C CNN
+AR Path="/6130ED51/616EF3E5" Ref="#PWR04"  Part="1"
+F 0 "#PWR04" H 4650 3650 50  0001 C CNN
 F 1 "GND" V 4650 3700 50  0000 C CNN
 F 2 "" H 4650 3900 50  0001 C CNN
@@
 AR Path="/6143BBD4/6170A575" Ref="R?"  Part="1"
 AR Path="/6144BA8F/6170A575" Ref="R?"  Part="1"
-AR Path="/6130ED51/6170A575" Ref="R?"  Part="1"
-F 0 "R?" V 4450 4200 50  0000 C CNN
+AR Path="/6130ED51/6170A575" Ref="R9"  Part="1"
+F 0 "R9" V 4450 4200 50  0000 C CNN
 F 1 "10k" V 4400 4000 50  0000 C CNN
 F 2 "Resistor_SMD:R_0402_1005Metric" V 4330 4000 50  0001 C CNN
@@
 AR Path="/5FDFE7F4/6170A57B" Ref="#PWR?"  Part="1"
 AR Path="/6133068E/6170A57B" Ref="#PWR?"  Part="1"
-AR Path="/6130ED51/6170A57B" Ref="#PWR?"  Part="1"
-F 0 "#PWR?" H 4650 3750 50  0001 C CNN
+AR Path="/6130ED51/6170A57B" Ref="#PWR031"  Part="1"
+F 0 "#PWR031" H 4650 3750 50  0001 C CNN
 F 1 "GND" V 4650 3800 50  0000 C CNN
 F 2 "" H 4650 4000 50  0001 C CNN
@@
 AR Path="/6143BBD4/617107C6" Ref="R?"  Part="1"
 AR Path="/6144BA8F/617107C6" Ref="R?"  Part="1"
-AR Path="/6130ED51/617107C6" Ref="R?"  Part="1"
-F 0 "R?" V 4450 4300 50  0000 C CNN
+AR Path="/6130ED51/617107C6" Ref="R10"  Part="1"
+F 0 "R10" V 4450 4300 50  0000 C CNN
 F 1 "10k" V 4400 4100 50  0000 C CNN
 F 2 "Resistor_SMD:R_0402_1005Metric" V 4330 4100 50  0001 C CNN
@@
 AR Path="/5FDFE7F4/617107CC" Ref="#PWR?"  Part="1"
 AR Path="/6133068E/617107CC" Ref="#PWR?"  Part="1"
-AR Path="/6130ED51/617107CC" Ref="#PWR?"  Part="1"
-F 0 "#PWR?" H 4650 3850 50  0001 C CNN
+AR Path="/6130ED51/617107CC" Ref="#PWR032"  Part="1"
+F 0 "#PWR032" H 4650 3850 50  0001 C CNN
 F 1 "GND" V 4650 3900 50  0000 C CNN
 F 2 "" H 4650 4100 50  0001 C CNN
@@
 AR Path="/6143BBD4/61716888" Ref="R?"  Part="1"
 AR Path="/6144BA8F/61716888" Ref="R?"  Part="1"
-AR Path="/6130ED51/61716888" Ref="R?"  Part="1"
-F 0 "R?" V 4450 4400 50  0000 C CNN
+AR Path="/6130ED51/61716888" Ref="R11"  Part="1"
+F 0 "R11" V 4450 4400 50  0000 C CNN
 F 1 "10k" V 4400 4200 50  0000 C CNN
 F 2 "Resistor_SMD:R_0402_1005Metric" V 4330 4200 50  0001 C CNN
@@
 AR Path="/5FDFE7F4/6171688E" Ref="#PWR?"  Part="1"
 AR Path="/6133068E/6171688E" Ref="#PWR?"  Part="1"
-AR Path="/6130ED51/6171688E" Ref="#PWR?"  Part="1"
-F 0 "#PWR?" H 4650 3950 50  0001 C CNN
+AR Path="/6130ED51/6171688E" Ref="#PWR033"  Part="1"
+F 0 "#PWR033" H 4650 3950 50  0001 C CNN
 F 1 "GND" V 4650 4000 50  0000 C CNN
 F 2 "" H 4650 4200 50  0001 C CNN
@@
 Wire Wire Line
 	3400 4200 4250 4200
+Text Label 5050 2400 0    50   ~ 0
+usb_sw0_sw1+
+Text Label 5050 2500 0    50   ~ 0
+usb_sw0_sw1-
+Text Label 5200 3900 0    50   ~ 0
+usb_sw0_sw2+
+Text Label 5200 4000 0    50   ~ 0
+usb_sw0_sw2-
 $EndSCHEMATC
