File: currypi.kicad_pcb (KiCad board)
At the start: 2 copper layers, 80 x 500 mm, 40 parts, among them U1 rpi_cm4, U2 m.2_pcie_nvme, U3 rpi_cm4

Commit message: add the ksz switch
Parts:
- added C1: 10uF 25V, Capacitor_SMD:C_1206_3216Metric, F.Cu at (66.8, 105.4)
- added C10: 10uF 25V, Capacitor_SMD:C_1206_3216Metric, F.Cu at (61.2, 105.4)
- added C15: 10uF 25V, Capacitor_SMD:C_1206_3216Metric, F.Cu at (43.5, 119.9)
- added C16: 10uF 25V, Capacitor_SMD:C_1206_3216Metric, F.Cu at (49.4, 110.7)
- added C17: 10uF 25V, Capacitor_SMD:C_1206_3216Metric, F.Cu at (55.5, 105.4)
- added C2: 10uF 25V, Capacitor_SMD:C_1206_3216Metric, F.Cu at (49.4, 114.0)
- added C3: 15nF, Capacitor_SMD:C_0402_1005Metric, F.Cu at (48.3, 105.0)
- added C4: 4.7uF 25V, Capacitor_SMD:C_0805_2012Metric, F.Cu at (44.3, 109.5)
- added C7: 33nF, Capacitor_SMD:C_0402_1005Metric, F.Cu at (39.8, 112.6)
- added C8: 68pF, Capacitor_SMD:C_0402_1005Metric, F.Cu at (46.3, 107.0)
- added C9: 100nF, Capacitor_SMD:C_0805_2012Metric, F.Cu at (50.0, 107.5)
- added L1: 4.7uH, dg_transformers:IND_1350, F.Cu at (60.9, 114.3)
- added R1: 102K, Resistor_SMD:R_0402_1005Metric, F.Cu at (44.9, 117.2)
- added R2: 36.5K, Resistor_SMD:R_0402_1005Metric, F.Cu at (39.2, 120.5)
- added R3: 53.6K, Resistor_SMD:R_0402_1005Metric, F.Cu at (39.2, 118.5)
- added R4: 2.55K, Resistor_SMD:R_0402_1005Metric, F.Cu at (51.2, 105.0)
- added R5: 53.6K, Resistor_SMD:R_0402_1005Metric, F.Cu at (39.8, 116.6)
- added R6: 102K, Resistor_SMD:R_0402_1005Metric, F.Cu at (39.8, 114.6)
- added U1: rpi_cm4, dg_rpi:rpi_cm4, F.Cu at (65.8, 176.5)
- added U1: rpi_cm4, dg_rpi:rpi_cm4, F.Cu at (66.9, 133.3)
- added U1: rpi_cm4, dg_rpi:rpi_cm4, F.Cu at (67.8, 48.3)
- added U2: m.2_pcie_nvme, dg_connectors:m.2_pcie_nvme, B.Cu at (31.2, 93.4)
- added U2: m.2_pcie_nvme, dg_connectors:m.2_pcie_nvme, B.Cu at (41.1, 109.1)
- added U2: m.2_pcie_nvme, dg_connectors:m.2_pcie_nvme, B.Cu at (66.8, 109.6)
- added U2: m.2_pcie_nvme, dg_connectors:m.2_pcie_nvme, B.Cu at (57.1, 19.3)
- added U4: TPS54620, dg_ic:Texas_S-PVQFN-N14_ThermalVias, F.Cu at (49.3, 118.6)
- added U5: RT8065, dg_ic:DFN-8-1EP_3x3mm_P0.65mm_EP1.55x2.4mm, F.Cu at (43.9, 113.3)
- U2: moved to B.Cu
- moved C5 481.0 mm to (193.1, -30.1)
- moved C6 481.0 mm to (191.1, -30.1)
- moved D1 481.0 mm to (207.1, 32.9)
- moved D10 481.0 mm to (219.2, -30.0)
- moved D11 481.0 mm to (221.1, -30.1)
- moved D12 481.0 mm to (208.1, -30.1)
- moved D8 481.0 mm to (216.1, -30.1)
- moved D9 481.0 mm to (188.1, -30.1)
- moved JP5 481.0 mm to (196.1, -30.1)
- moved JP6 481.0 mm to (199.1, -30.1)
- moved JP7 481.0 mm to (213.1, -30.1)
- moved JP8 481.0 mm to (224.1, -30.1)
- moved R10 481.0 mm to (204.1, -29.9)
- moved R11 481.0 mm to (210.1, -30.1)
- moved R7 481.0 mm to (202.1, -30.1)
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Connections:
- D1 pad 1: (no net) -> +24V
Other:
- board size 80 x 500 mm -> 80 x 350 mm

Commit message: possible layout example
Parts:
- removed the C1 at (66.8, 105.4)
- removed the C10 at (61.2, 105.4)
- removed C12, C14, C6: C, Capacitor_SMD:C_0603_1608Metric
- removed the C15 at (43.5, 119.9)
- removed the C16 at (49.4, 110.7)
- removed the C17 at (55.5, 105.4)
- removed the C2 at (49.4, 114.0)
- removed the C3 at (48.3, 105.0)
- removed the C4 at (44.3, 109.5)
- removed C5: C, Capacitor_SMD:C_0805_2012Metric
- removed the C7 at (39.8, 112.6)
- removed the C8 at (46.3, 107.0)
- removed the C9 at (50.0, 107.5)
- removed the D1 at (207.1, 32.9)
- removed D10, D11, D12, D19, D20, D21, D22, D23, D24, D8, D9: LED, LED_SMD:LED_0603_1608Metric
- removed JP13, JP5, JP6, JP7, JP8: SolderJumper_2_Open, Jumper:SolderJumper-2_P1.3mm_Open_RoundedPad1.0x1.5mm
- removed the L1 at (60.9, 114.3)
- removed the R1 at (44.9, 117.2)
- removed R10, R11, R18, R19, R20, R21, R22, R23, R7, R8, R9: R, Resistor_SMD:R_0603_1608Metric
- removed the R2 at (39.2, 120.5)
- removed the R3 at (39.2, 118.5)
- removed the R4 at (51.2, 105.0)
- removed the R5 at (39.8, 116.6)
- removed the R6 at (39.8, 114.6)
- removed the U1 at (65.8, 176.5)
- removed the U1 at (66.9, 133.3)
- removed the U1 at (67.8, 48.3)
- removed the U1 at (66.3, 4.06)
- removed the U2 at (31.2, 93.4)
- removed the U2 at (41.1, 109.1)
- removed the U2 at (66.8, 109.6)
- removed the U2 at (57.1, 19.3)
- removed the U2 at (104.1, 206.8)
- removed the U4 at (49.3, 118.6)
- removed the U5 at (43.9, 113.3)
- added C1: 10uF 25V, Capacitor_SMD:C_1206_3216Metric, F.Cu at (70.1, 225.8)
- added C1: 10uF 25V, Capacitor_SMD:C_1206_3216Metric, F.Cu at (71.9, 103.9)
- added C10: 10uF 25V, Capacitor_SMD:C_1206_3216Metric, F.Cu at (55.7, 202.5)
- added C10: 10uF 25V, Capacitor_SMD:C_1206_3216Metric, F.Cu at (57.4, 80.6)
- added C101: 0.1uF, Capacitor_SMD:C_0402_1005Metric, F.Cu at (39.1, 343.8)
- added C102: 0.1uF, Capacitor_SMD:C_0402_1005Metric, F.Cu at (33.2, 348.8)
- added C103: 0.1uF, Capacitor_SMD:C_0402_1005Metric, F.Cu at (30.4, 350.8)
- added C104: 0.1uF, Capacitor_SMD:C_0402_1005Metric, F.Cu at (65.6, 305.5)
- added C105: 0.1uF, Capacitor_SMD:C_0402_1005Metric, F.Cu at (68.4, 301.5)
- added C106: 0.1uF, Capacitor_SMD:C_0402_1005Metric, F.Cu at (68.4, 303.5)
- added C107: 0.1uF, Capacitor_SMD:C_0402_1005Metric, F.Cu at (51.8, 330.9)
- added C108: 0.1uF, Capacitor_SMD:C_0402_1005Metric, F.Cu at (48.9, 334.8)
- added C109: 0.1uF, Capacitor_SMD:C_0402_1005Metric, F.Cu at (44.8, 338.8)
- added C110: 0.1uF, Capacitor_SMD:C_0402_1005Metric, F.Cu at (62.7, 309.1)
- added C111: C, Capacitor_SMD:C_0805_2012Metric, F.Cu at (386.1, 59.7)
- added C114: C, Capacitor_SMD:C_0805_2012Metric, F.Cu at (390.6, 59.7)
- added C115: 10uF 25V, Capacitor_SMD:C_1206_3216Metric, F.Cu at (13.2, 145.0)
- added C115: 10uF 25V, Capacitor_SMD:C_1206_3216Metric, F.Cu at (29.0, 30.5)
- added C116: 10uF 25V, Capacitor_SMD:C_1206_3216Metric, F.Cu at (13.2, 139.3)
- added C116: 10uF 25V, Capacitor_SMD:C_1206_3216Metric, F.Cu at (29.0, 36.2)
- added C117: 15nF, Capacitor_SMD:C_0402_1005Metric, F.Cu at (20.4, 166.4)
- added C117: 15nF, Capacitor_SMD:C_0402_1005Metric, F.Cu at (21.8, 9.14)
- added C118: 4.7uF 25V, Capacitor_SMD:C_0805_2012Metric, F.Cu at (15.3, 156.2)
- added C118: 4.7uF 25V, Capacitor_SMD:C_0805_2012Metric, F.Cu at (26.9, 19.3)
- added C119: 33nF, Capacitor_SMD:C_0402_1005Metric, F.Cu at (14.8, 159.9)
- added C119: 33nF, Capacitor_SMD:C_0402_1005Metric, F.Cu at (27.3, 15.7)
- added C120: 68pF, Capacitor_SMD:C_0402_1005Metric, F.Cu at (12.8, 157.8)
- added C120: 68pF, Capacitor_SMD:C_0402_1005Metric, F.Cu at (29.4, 17.7)
- added C121: 100nF, Capacitor_SMD:C_0805_2012Metric, F.Cu at (17.3, 161.8)
- added C121: 100nF, Capacitor_SMD:C_0805_2012Metric, F.Cu at (24.9, 13.7)
- added C122: 10uF 25V, Capacitor_SMD:C_1206_3216Metric, F.Cu at (13.2, 150.7)
- added C122: 10uF 25V, Capacitor_SMD:C_1206_3216Metric, F.Cu at (29.0, 24.9)
- added C123: 10uF 25V, Capacitor_SMD:C_1206_3216Metric, F.Cu at (18.5, 156.8)
- added C123: 10uF 25V, Capacitor_SMD:C_1206_3216Metric, F.Cu at (23.7, 18.7)
- added C124: 10uF 25V, Capacitor_SMD:C_1206_3216Metric, F.Cu at (21.8, 156.8)
- added C124: 10uF 25V, Capacitor_SMD:C_1206_3216Metric, F.Cu at (20.4, 18.7)
- added C125: 10uF 25V, Capacitor_SMD:C_1206_3216Metric, F.Cu at (27.7, 162.7)
- added C125: 10uF 25V, Capacitor_SMD:C_1206_3216Metric, F.Cu at (14.5, 12.9)
- added C15: 10uF 25V, Capacitor_SMD:C_1206_3216Metric, F.Cu at (70.1, 214.5)
- added C15: 10uF 25V, Capacitor_SMD:C_1206_3216Metric, F.Cu at (71.9, 92.6)
- added C16: 10uF 25V, Capacitor_SMD:C_1206_3216Metric, F.Cu at (70.1, 220.2)
- added C16: 10uF 25V, Capacitor_SMD:C_1206_3216Metric, F.Cu at (71.9, 98.2)
- added C17: 10uF 25V, Capacitor_SMD:C_1206_3216Metric, F.Cu at (61.5, 208.4)
- added C17: 10uF 25V, Capacitor_SMD:C_1206_3216Metric, F.Cu at (63.3, 86.4)
- added C18: 0.1uF, Capacitor_SMD:C_0402_1005Metric, F.Cu at (36.1, 348.8)
- added C19: 0.1uF, Capacitor_SMD:C_0402_1005Metric, F.Cu at (39.0, 345.8)
- added C2: 10uF 25V, Capacitor_SMD:C_1206_3216Metric, F.Cu at (64.9, 208.4)
- added C2: 10uF 25V, Capacitor_SMD:C_1206_3216Metric, F.Cu at (66.6, 86.4)
- added C21: 0.1uF, Capacitor_SMD:C_0402_1005Metric, F.Cu at (71.2, 299.6)
- added C22: 10uF, Capacitor_SMD:C_0603_1608Metric, F.Cu at (34.9, 314.9)
- added C23: 0.1uF, Capacitor_SMD:C_0402_1005Metric, F.Cu at (78.2, 353.1)
- added C24: 10uF, Capacitor_SMD:C_0603_1608Metric, F.Cu at (30.9, 314.9)
- added C29: 0.1uF, Capacitor_SMD:C_0402_1005Metric, F.Cu at (78.2, 292.7)
- added C3: 15nF, Capacitor_SMD:C_0402_1005Metric, F.Cu at (70.5, 207.3)
- added C3: 15nF, Capacitor_SMD:C_0402_1005Metric, F.Cu at (72.3, 85.4)
- added C31: 0.1uF, Capacitor_SMD:C_0402_1005Metric, F.Cu at (74.0, 299.5)
- added C34: 0.1uF, Capacitor_SMD:C_0402_1005Metric, F.Cu at (75.4, 292.7)
- added C35: 0.1uF, Capacitor_SMD:C_0402_1005Metric, F.Cu at (56.6, 311.1)
- added C36: 0.1uF, Capacitor_SMD:C_0402_1005Metric, F.Cu at (62.7, 307.1)
- added C37: 0.1uF, Capacitor_SMD:C_0402_1005Metric, F.Cu at (68.3, 299.6)
- added C38: 10uF, Capacitor_SMD:C_0603_1608Metric, F.Cu at (39.0, 312.4)
- added C39: 0.1uF, Capacitor_SMD:C_0402_1005Metric, F.Cu at (59.6, 309.2)
- added C4: 4.7uF 25V, Capacitor_SMD:C_0805_2012Metric, F.Cu at (68.0, 209.0)
- added C4: 4.7uF 25V, Capacitor_SMD:C_0805_2012Metric, F.Cu at (69.8, 87.0)
- added C40: 0.1uF, Capacitor_SMD:C_0402_1005Metric, F.Cu at (62.7, 305.2)
- added C41: 0.1uF, Capacitor_SMD:C_0402_1005Metric, F.Cu at (33.3, 346.8)
- added C43: 0.1uF, Capacitor_SMD:C_0402_1005Metric, F.Cu at (36.2, 343.8)
- added C45: 0.1uF, Capacitor_SMD:C_0402_1005Metric, F.Cu at (65.6, 309.5)
- added C46: 0.1uF, Capacitor_SMD:C_0402_1005Metric, F.Cu at (65.6, 303.6)
- added C47: 0.1uF, Capacitor_SMD:C_0402_1005Metric, F.Cu at (48.9, 332.8)
- added C49: 0.1uF, Capacitor_SMD:C_0402_1005Metric, F.Cu at (59.5, 311.1)
- added C50: 0.1uF, Capacitor_SMD:C_0402_1005Metric, F.Cu at (30.4, 352.8)
- added C51: 0.1uF, Capacitor_SMD:C_0402_1005Metric, F.Cu at (58.1, 313.1)
- added C52: 15pF, Capacitor_SMD:C_0402_1005Metric, F.Cu at (55.8, 315.8)
- added C53: 15pF, Capacitor_SMD:C_0402_1005Metric, F.Cu at (52.9, 317.8)
- added C54: 10uF, Capacitor_SMD:C_0603_1608Metric, F.Cu at (78.1, 283.7)
- added C55: 10uF, Capacitor_SMD:C_0603_1608Metric, F.Cu at (30.9, 336.1)
- added C56: 10uF, Capacitor_SMD:C_0603_1608Metric, F.Cu at (39.0, 317.4)
- added C57: 10uF, Capacitor_SMD:C_0603_1608Metric, F.Cu at (44.3, 307.3)
- added C58: 10uF, Capacitor_SMD:C_0603_1608Metric, F.Cu at (30.9, 338.6)
- added C59: 10uF, Capacitor_SMD:C_0603_1608Metric, F.Cu at (43.0, 312.4)
- added C60: 10uF, Capacitor_SMD:C_0603_1608Metric, F.Cu at (34.9, 333.6)
- added C61: 10uF, Capacitor_SMD:C_0603_1608Metric, F.Cu at (30.9, 299.5)
- added C62: 10uF, Capacitor_SMD:C_0603_1608Metric, F.Cu at (43.0, 314.9)
- added C63: 10uF, Capacitor_SMD:C_0603_1608Metric, F.Cu at (44.3, 299.5)
- added C64: 10uF, Capacitor_SMD:C_0603_1608Metric, F.Cu at (30.9, 333.6)
- added C65: 10uF, Capacitor_SMD:C_0603_1608Metric, F.Cu at (34.9, 331.1)
- added C66: 100 uF, Capacitor_SMD:CP_Elec_5x5.3, F.Cu at (69.5, 291.2)
- added C67: 10uF, Capacitor_SMD:C_0603_1608Metric, F.Cu at (30.9, 331.1)
- added C68: 10uF, Capacitor_SMD:C_0603_1608Metric, F.Cu at (34.9, 317.4)
- added C69: 10uF, Capacitor_SMD:C_0603_1608Metric, F.Cu at (30.9, 317.4)
- added C7: 33nF, Capacitor_SMD:C_0402_1005Metric, F.Cu at (62.9, 198.8)
- added C7: 33nF, Capacitor_SMD:C_0402_1005Metric, F.Cu at (64.7, 76.9)
- added C70: 10uF, Capacitor_SMD:C_0603_1608Metric, F.Cu at (39.0, 314.9)
- added C71: 1uF, Capacitor_SMD:C_0402_1005Metric, F.Cu at (47.7, 338.8)
- added C72: 1uF, Capacitor_SMD:C_0402_1005Metric, F.Cu at (62.5, 311.1)
- added C73: 0.1uF, Capacitor_SMD:C_0402_1005Metric, F.Cu at (65.6, 307.5)
- added C76: 0.1uF, Capacitor_SMD:C_0402_1005Metric, F.Cu at (78.3, 289.9)
- added C77: 0.1uF, Capacitor_SMD:C_0402_1005Metric, F.Cu at (70.5, 297.6)
- added C78: 0.1uF, Capacitor_SMD:C_0402_1005Metric, F.Cu at (39.1, 339.8)
- added C79: 0.1uF, Capacitor_SMD:C_0402_1005Metric, F.Cu at (43.1, 336.8)
- added C8: 68pF, Capacitor_SMD:C_0402_1005Metric, F.Cu at (68.5, 205.3)
- added C8: 68pF, Capacitor_SMD:C_0402_1005Metric, F.Cu at (70.3, 83.4)
- added C80: 0.1uF, Capacitor_SMD:C_0402_1005Metric, F.Cu at (46.0, 334.3)
- added C81: 0.1uF, Capacitor_SMD:C_0402_1005Metric, F.Cu at (30.4, 348.8)
- added C82: 10uF, Capacitor_SMD:C_0603_1608Metric, F.Cu at (40.2, 309.9)
- added C83: 10uF, Capacitor_SMD:C_0603_1608Metric, F.Cu at (36.2, 309.9)
- added C84: 0.1uF, Capacitor_SMD:C_0402_1005Metric, F.Cu at (50.0, 317.8)
- added C85: 0.1uF, Capacitor_SMD:C_0402_1005Metric, F.Cu at (52.9, 315.8)
- added C86: 0.1uF, Capacitor_SMD:C_0402_1005Metric, F.Cu at (50.0, 315.8)
- added C87: 10uF, Capacitor_SMD:C_0603_1608Metric, F.Cu at (44.3, 309.8)
- added C88: 10uF, Capacitor_SMD:C_0603_1608Metric, F.Cu at (35.0, 312.4)
- added C89: 0.1uF, Capacitor_SMD:C_0402_1005Metric, F.Cu at (42.0, 338.8)
- added C9: 100nF, Capacitor_SMD:C_0805_2012Metric, F.Cu at (66.0, 203.3)
- added C9: 100nF, Capacitor_SMD:C_0805_2012Metric, F.Cu at (67.8, 81.4)
- added C90: 0.1uF, Capacitor_SMD:C_0402_1005Metric, F.Cu at (39.1, 341.8)
- added C91: 0.1uF, Capacitor_SMD:C_0402_1005Metric, F.Cu at (46.0, 336.8)
- added C92: 0.1uF, Capacitor_SMD:C_0402_1005Metric, F.Cu at (42.0, 340.8)
- added C93: 0.1uF, Capacitor_SMD:C_0402_1005Metric, F.Cu at (73.5, 295.6)
- added C95: 0.1uF, Capacitor_SMD:C_0402_1005Metric, F.Cu at (55.3, 313.8)
- added C97: 0.1uF, Capacitor_SMD:C_0402_1005Metric, F.Cu at (76.3, 294.7)
- added C98: 0.1uF, Capacitor_SMD:C_0402_1005Metric, F.Cu at (36.1, 346.8)
- added C99: 0.1uF, Capacitor_SMD:C_0402_1005Metric, F.Cu at (73.5, 297.6)
- added D1: D_TVS, Diode_SMD:D_SMA, F.Cu at (56.3, 188.7)
- added D1: D_TVS, Diode_SMD:D_SMA, F.Cu at (58.0, 66.8)
- added D13: 150060GS75000, LED_SMD:LED_0603_1608Metric, F.Cu at (43.1, 302.2)
- added D14: 150060GS75000, LED_SMD:LED_0603_1608Metric, F.Cu at (36.2, 304.7)
- added D15: 150060GS75000, LED_SMD:LED_0603_1608Metric, F.Cu at (40.3, 304.7)
- added D16: 150060RS75000, LED_SMD:LED_0603_1608Metric, F.Cu at (40.3, 307.3)
- added D17: 150060RS75000, LED_SMD:LED_0603_1608Metric, F.Cu at (44.3, 304.7)
- added D18: 150060RS75000, LED_SMD:LED_0603_1608Metric, F.Cu at (36.2, 307.3)
- added D2: 150060RS75000, LED_SMD:LED_0603_1608Metric, F.Cu at (35.0, 302.2)
- added D25: 150060RS75000, LED_SMD:LED_0603_1608Metric, F.Cu at (40.3, 299.6)
- added D3: 150060GS75000, LED_SMD:LED_0603_1608Metric, F.Cu at (36.2, 299.6)
- added D4: 150060RS75000, LED_SMD:LED_0603_1608Metric, F.Cu at (31.0, 310.5)
- added D5: SMAJ5.0CA-TR, Diode_SMD:D_SMA, F.Cu at (51.3, 294.5)
- added D6: 150060GS75000, LED_SMD:LED_0603_1608Metric, F.Cu at (31.0, 302.2)
- added D7: 150060GS75000, LED_SMD:LED_0603_1608Metric, F.Cu at (39.1, 302.2)
- added H1: VIN+, MountingHole:MountingHole_3.2mm_M3_Pad, F.Cu at (51.3, 300.8)
- added H2: VIN-, MountingHole:MountingHole_3.2mm_M3_Pad, F.Cu at (59.3, 296.2)
- added J3: 1367073-1, dg_connectors:SFP_with_Cage, F.Cu at (10.7, 299.0)
- added JP1: SolderJumper_2_Open, Jumper:SolderJumper-2_P1.3mm_Open_RoundedPad1.0x1.5mm, F.Cu at (390.4, 62.9)
- added JP2: SolderJumper_2_Open, Jumper:SolderJumper-2_P1.3mm_Open_RoundedPad1.0x1.5mm, F.Cu at (386.1, 62.9)
- added JP3: SolderJumper_2_Open, Jumper:SolderJumper-2_P1.3mm_Open_RoundedPad1.0x1.5mm, F.Cu at (386.1, 66.5)
- added L1: 4.7uH, dg_transformers:IND_1350, F.Cu at (61.2, 219.9)
- added L1: 4.7uH, dg_transformers:IND_1350, F.Cu at (63.0, 98.0)
- added L2: 4.7uH, dg_transformers:IND_1350, F.Cu at (22.1, 145.2)
- added L2: 4.7uH, dg_transformers:IND_1350, F.Cu at (20.1, 30.3)
- added R1: 102K, Resistor_SMD:R_0402_1005Metric, F.Cu at (58.3, 203.9)
- added R1: 102K, Resistor_SMD:R_0402_1005Metric, F.Cu at (60.1, 82.0)
- added R13: 10K, Resistor_SMD:R_0402_1005Metric, F.Cu at (30.4, 344.9)
- added R14: 10K, Resistor_SMD:R_0402_1005Metric, F.Cu at (44.2, 319.1)
- added R15: 4.7K, Resistor_SMD:R_0402_1005Metric, F.Cu at (64.7, 297.6)
- added R16: 4.7K, Resistor_SMD:R_0402_1005Metric, F.Cu at (37.3, 337.9)
- added R17: 1K, Resistor_SMD:R_0402_1005Metric, F.Cu at (77.6, 285.9)
- added R2: 36.5K, Resistor_SMD:R_0402_1005Metric, F.Cu at (60.9, 198.8)
- added R2: 36.5K, Resistor_SMD:R_0402_1005Metric, F.Cu at (62.7, 76.8)
- added R24: 1K, Resistor_SMD:R_0402_1005Metric, F.Cu at (64.7, 295.6)
- added R25: 1K, Resistor_SMD:R_0402_1005Metric, F.Cu at (33.3, 342.9)
- added R26: 6.04K %1, Resistor_SMD:R_0402_1005Metric, F.Cu at (44.2, 332.3)
- added R27: 191 %1, Resistor_SMD:R_0402_1005Metric, F.Cu at (47.1, 317.7)
- added R28: 22R, Resistor_SMD:R_0402_1005Metric, F.Cu at (40.2, 336.8)
- added R29: 22R, Resistor_SMD:R_0402_1005Metric, F.Cu at (36.2, 339.8)
- added R3: 53.6K, Resistor_SMD:R_0402_1005Metric, F.Cu at (59.0, 198.8)
- added R3: 53.6K, Resistor_SMD:R_0402_1005Metric, F.Cu at (60.7, 76.8)
- added R30: 22R, Resistor_SMD:R_0402_1005Metric, F.Cu at (40.2, 334.8)
- added R32: 22R, Resistor_SMD:R_0402_1005Metric, F.Cu at (67.7, 297.6)
- added R33: 22R, Resistor_SMD:R_0402_1005Metric, F.Cu at (56.9, 307.2)
- added R35: 4.7K, Resistor_SMD:R_0402_1005Metric, F.Cu at (77.6, 280.9)
- added R36: 10K, Resistor_SMD:R_0402_1005Metric, F.Cu at (67.7, 295.6)
- added R37: 10K, Resistor_SMD:R_0402_1005Metric, F.Cu at (78.3, 287.9)
- added R38: 10K, Resistor_SMD:R_0402_1005Metric, F.Cu at (33.3, 344.9)
- added R39: 10K, Resistor_SMD:R_0402_1005Metric, F.Cu at (38.4, 319.7)
- added R4: 2.55K, Resistor_SMD:R_0402_1005Metric, F.Cu at (70.5, 210.2)
- added R4: 2.55K, Resistor_SMD:R_0402_1005Metric, F.Cu at (72.3, 88.3)
- added R40: 10K, Resistor_SMD:R_0402_1005Metric, F.Cu at (30.4, 340.9)
- added R41: 4.7K, Resistor_SMD:R_0402_1005Metric, F.Cu at (38.4, 332.8)
- added R42: 750R, Resistor_SMD:R_0402_1005Metric, F.Cu at (34.4, 335.9)
- added R43: 750R, Resistor_SMD:R_0402_1005Metric, F.Cu at (56.7, 301.2)
- added R44: 750R, Resistor_SMD:R_0402_1005Metric, F.Cu at (59.6, 301.2)
- added R45: 750R, Resistor_SMD:R_0402_1005Metric, F.Cu at (56.7, 303.2)
- added R46: 750R, Resistor_SMD:R_0402_1005Metric, F.Cu at (75.4, 288.8)
- added R47: 750R, Resistor_SMD:R_0402_1005Metric, F.Cu at (59.6, 303.2)
- added R48: 750R, Resistor_SMD:R_0402_1005Metric, F.Cu at (62.5, 301.2)
- added R49: 1K, Resistor_SMD:R_0402_1005Metric, F.Cu at (70.6, 295.6)
- added R5: 53.6K, Resistor_SMD:R_0402_1005Metric, F.Cu at (57.0, 198.2)
- added R5: 53.6K, Resistor_SMD:R_0402_1005Metric, F.Cu at (58.7, 76.3)
- added R50: 1K, Resistor_SMD:R_0402_1005Metric, F.Cu at (37.3, 335.9)
- added R51: 1K, Resistor_SMD:R_0402_1005Metric, F.Cu at (34.4, 337.9)
- added R52: 1K, Resistor_SMD:R_0402_1005Metric, F.Cu at (41.3, 319.7)
- added R53: 1K, Resistor_SMD:R_0402_1005Metric, F.Cu at (42.4, 317.2)
- added R54: 1K, Resistor_SMD:R_0402_1005Metric, F.Cu at (41.3, 332.8)
- added R55: 1K, Resistor_SMD:R_0402_1005Metric, F.Cu at (49.5, 313.8)
- added R56: 1K, Resistor_SMD:R_0402_1005Metric, F.Cu at (50.8, 311.9)
- added R57: 1K, Resistor_SMD:R_0402_1005Metric, F.Cu at (53.8, 308.8)
- added R58: 1K, Resistor_SMD:R_0402_1005Metric, F.Cu at (56.9, 305.2)
- added R59: 0R_DNP, Resistor_SMD:R_0402_1005Metric, F.Cu at (30.4, 342.9)
- added R6: 102K, Resistor_SMD:R_0402_1005Metric, F.Cu at (55.0, 198.2)
- added R6: 102K, Resistor_SMD:R_0402_1005Metric, F.Cu at (56.8, 76.3)
- added R60: 0R_DNP, Resistor_SMD:R_0402_1005Metric, F.Cu at (33.3, 340.9)
- added R61: 0R_DNP, Resistor_SMD:R_0402_1005Metric, F.Cu at (75.4, 290.7)
- added R62: 0R_DNP, Resistor_SMD:R_0402_1005Metric, F.Cu at (62.5, 303.2)
- added R63: 0R_DNP, Resistor_SMD:R_0402_1005Metric, F.Cu at (53.7, 311.9)
- added R64: 0R_DNP, Resistor_SMD:R_0402_1005Metric, F.Cu at (59.8, 305.2)
- added R65: 0R_DNP, Resistor_SMD:R_0402_1005Metric, F.Cu at (30.4, 346.9)
- added R66: 0R_DNP, Resistor_SMD:R_0402_1005Metric, F.Cu at (36.2, 341.8)
- added R67: 0R_DNP, Resistor_SMD:R_0402_1005Metric, F.Cu at (43.1, 334.8)
- added R68: 24K, Resistor_SMD:R_0402_1005Metric, F.Cu at (56.8, 309.2)
- added R69: 10K, Resistor_SMD:R_0402_1005Metric, F.Cu at (52.4, 313.8)
- added R70: 40.2K, Resistor_SMD:R_0402_1005Metric, F.Cu at (65.4, 299.6)
- added R71: 10K, Resistor_SMD:R_0402_1005Metric, F.Cu at (47.1, 319.7)
- added R72: 10K, Resistor_SMD:R_0402_1005Metric, F.Cu at (65.4, 301.6)
- added R73: 22R, Resistor_SMD:R_0402_1005Metric, F.Cu at (59.8, 307.2)
- added R80: 102K, Resistor_SMD:R_0402_1005Metric, F.Cu at (22.4, 166.4)
- added R80: 102K, Resistor_SMD:R_0402_1005Metric, F.Cu at (19.8, 9.12)
- added R81: 36.5K, Resistor_SMD:R_0402_1005Metric, F.Cu at (24.4, 166.4)
- added R81: 36.5K, Resistor_SMD:R_0402_1005Metric, F.Cu at (17.8, 9.12)
- added R82: 53.6K, Resistor_SMD:R_0402_1005Metric, F.Cu at (12.8, 154.9)
- added R82: 53.6K, Resistor_SMD:R_0402_1005Metric, F.Cu at (29.4, 20.6)
- added R83: 2.55K, Resistor_SMD:R_0402_1005Metric, F.Cu at (26.3, 166.9)
- added R83: 2.55K, Resistor_SMD:R_0402_1005Metric, F.Cu at (15.8, 8.58)
- added R84: 53.6K, Resistor_SMD:R_0402_1005Metric, F.Cu at (28.3, 166.9)
- added R84: 53.6K, Resistor_SMD:R_0402_1005Metric, F.Cu at (13.8, 8.58)
- added R85: 102K, Resistor_SMD:R_0402_1005Metric, F.Cu at (25.0, 161.3)
- added R85: 102K, Resistor_SMD:R_0402_1005Metric, F.Cu at (17.2, 14.2)
- added SW1: PTS645SM43SMTR92 LFS, Button_Switch_SMD:SW_SPST_PTS645, F.Cu at (70.5, 283.8)
- added TP1: TestPoint_Small, TestPoint:TestPoint_Pad_D1.0mm, F.Cu at (53.9, 306.3)
- added TP2: TestPoint, TestPoint:TestPoint_Pad_D1.0mm, F.Cu at (50.9, 309.3)
- added TP3: TestPoint, TestPoint:TestPoint_Pad_D1.0mm, F.Cu at (46.5, 315.2)
- added TP4: TestPoint, TestPoint:TestPoint_Pad_D1.0mm, F.Cu at (47.8, 310.6)
- added TP5: TestPoint, TestPoint:TestPoint_Pad_D1.0mm, F.Cu at (50.9, 306.3)
- added TP7: TestPoint, TestPoint:TestPoint_Pad_D1.0mm, F.Cu at (47.8, 307.6)
- added U1: rpi_cm4, dg_rpi:rpi_cm4, F.Cu at (48.5, 235.7)
- added U1: rpi_cm4, dg_rpi:rpi_cm4, F.Cu at (50.8, 113.0)
- added U10: m.2_pcie_nvme, dg_connectors:m.2_pcie_nvme, B.Cu at (59.7, 145.3)
- added U10: m.2_pcie_nvme, dg_connectors:m.2_pcie_nvme, B.Cu at (57.1, 11.7)
- added U11: TPS54620, dg_ic:Texas_S-PVQFN-N14_ThermalVias, F.Cu at (26.4, 156.9)
- added U11: TPS54620, dg_ic:Texas_S-PVQFN-N14_ThermalVias, F.Cu at (15.8, 18.6)
- added U12: RT8065, dg_ic:DFN-8-1EP_3x3mm_P0.65mm_EP1.55x2.4mm, F.Cu at (21.1, 162.3)
- added U12: RT8065, dg_ic:DFN-8-1EP_3x3mm_P0.65mm_EP1.55x2.4mm, F.Cu at (21.1, 13.2)
- added U2: m.2_pcie_nvme, dg_connectors:m.2_pcie_nvme, B.Cu at (24.6, 241.3)
- added U2: m.2_pcie_nvme, dg_connectors:m.2_pcie_nvme, B.Cu at (22.1, 107.7)
- added U4: TPS54620, dg_ic:Texas_S-PVQFN-N14_ThermalVias, F.Cu at (56.9, 208.3)
- added U4: TPS54620, dg_ic:Texas_S-PVQFN-N14_ThermalVias, F.Cu at (58.7, 86.3)
- added U5: RT8065, dg_ic:DFN-8-1EP_3x3mm_P0.65mm_EP1.55x2.4mm, F.Cu at (62.2, 202.9)
- added U5: RT8065, dg_ic:DFN-8-1EP_3x3mm_P0.65mm_EP1.55x2.4mm, F.Cu at (64.0, 81.0)
- added U6: KSZ9477S, dg_ic:128-TQFP-EP, F.Cu at (14.0, 270.3)
- added U7: LM1085ISX-3.3/NOPB, Package_TO_SOT_SMD:TO-263-3_TabPin2, F.Cu at (56.1, 286.1)
- added U9: rpi_cm4, dg_rpi:rpi_cm4, F.Cu at (35.1, 121.4)
- added U9: rpi_cm4, dg_rpi:rpi_cm4, F.Cu at (79.5, 55.9)
- added Y1: ABM8G-25.000MHZ-B4Y-T, Crystal:Crystal_SMD_Abracon_ABM8G-4Pin_3.2x2.5mm, F.Cu at (31.6, 307.0)
- moved JP15 372.1 mm to (390.4, 156.4), turned to 0 degrees
- moved C13 368.9 mm to (390.6, 153.1), turned to 0 degrees
- moved C11 367.4 mm to (386.1, 153.1), turned to 0 degrees
- moved JP14 364.7 mm to (386.1, 159.9), turned to 0 degrees
- moved JP16 361.4 mm to (386.1, 156.4), turned to 0 degrees
- moved U3 330.2 mm to (37.6, 238.3), turned to 270 degrees
Connections:
- U3 pad 102: (no net) -> /sheet611D2998/pcie_clkreq
- U3 pad 109: (no net) -> /sheet611D2998/pcie_nrst
- U3 pad 110: (no net) -> /sheet611D2998/pcie_clk+
- U3 pad 112: (no net) -> /sheet611D2998/pcie_clk-

Commit message: maybe use a premade powerbrick
Parts:
- removed C1 (x2), C10 (x2), C115 (x2), C116 (x2), C122 (x2), C123 (x2), C124 (x2), C125 (x2), C15 (x2), C16 (x2), C17 (x2), C2 (x2): 10uF 25V, Capacitor_SMD:C_1206_3216Metric
- removed C101, C102, C103, C104, C105, C106, C107, C108, C109, C110, C18, C19, C21, C23, C29, C31, C34, C35, C36, C37, C39, C40, C41, C43, C45, C46, C47, C49, C50, C51, C73, C76, C77, C78, C79, C80, C81, C84, C85, C86, C89, C90, C91, C92, C93, C95, C97, C98, C99: 0.1uF, Capacitor_SMD:C_0402_1005Metric
- removed the C11 at (386.1, 153.1)
- removed C111, C114: C, Capacitor_SMD:C_0805_2012Metric
- removed C117 (x2), C3 (x2): 15nF, Capacitor_SMD:C_0402_1005Metric
- removed C118 (x2), C4 (x2): 4.7uF 25V, Capacitor_SMD:C_0805_2012Metric
- removed C119 (x2), C7 (x2): 33nF, Capacitor_SMD:C_0402_1005Metric
- removed C120 (x2), C8 (x2): 68pF, Capacitor_SMD:C_0402_1005Metric
- removed C121 (x2), C9 (x2): 100nF, Capacitor_SMD:C_0805_2012Metric
- removed C22, C24, C38, C54, C55, C56, C57, C58, C59, C60, C61, C62, C63, C64, C65, C67, C68, C69, C70, C82, C83, C87, C88: 10uF, Capacitor_SMD:C_0603_1608Metric
- removed C52, C53: 15pF, Capacitor_SMD:C_0402_1005Metric
- removed C66: 100 uF, Capacitor_SMD:CP_Elec_5x5.3
- removed C71, C72: 1uF, Capacitor_SMD:C_0402_1005Metric
- removed the D1 at (56.3, 188.7)
- removed the D1 at (58.0, 66.8)
- removed D13, D14, D15, D3, D6, D7: 150060GS75000, LED_SMD:LED_0603_1608Metric
- removed D16, D17, D18, D2, D25, D4: 150060RS75000, LED_SMD:LED_0603_1608Metric
- removed D5: SMAJ5.0CA-TR, Diode_SMD:D_SMA
- removed H1: VIN+, MountingHole:MountingHole_3.2mm_M3_Pad
- removed H2: VIN-, MountingHole:MountingHole_3.2mm_M3_Pad
- removed J3: 1367073-1, dg_connectors:SFP_with_Cage
- removed JP1, JP2, JP3: SolderJumper_2_Open, Jumper:SolderJumper-2_P1.3mm_Open_RoundedPad1.0x1.5mm
- removed the JP14 at (386.1, 159.9)
- removed the JP15 at (390.4, 156.4)
- removed the JP16 at (386.1, 156.4)
- removed L1 (x2), L2 (x2): 4.7uH, dg_transformers:IND_1350
- removed R1 (x2), R6 (x2), R80 (x2), R85 (x2): 102K, Resistor_SMD:R_0402_1005Metric
- removed R13, R14, R36, R37, R38, R39, R40, R69, R71, R72: 10K, Resistor_SMD:R_0402_1005Metric
- removed R15, R16, R35, R41: 4.7K, Resistor_SMD:R_0402_1005Metric
- removed R17, R24, R25, R49, R50, R51, R52, R53, R54, R55, R56, R57, R58: 1K, Resistor_SMD:R_0402_1005Metric
- removed R2 (x2), R81 (x2): 36.5K, Resistor_SMD:R_0402_1005Metric
- removed R26: 6.04K %1, Resistor_SMD:R_0402_1005Metric
- removed R27: 191 %1, Resistor_SMD:R_0402_1005Metric
- removed R28, R29, R30, R32, R33, R73: 22R, Resistor_SMD:R_0402_1005Metric
- removed R3 (x2), R5 (x2), R82 (x2), R84 (x2): 53.6K, Resistor_SMD:R_0402_1005Metric
- removed R4 (x2), R83 (x2): 2.55K, Resistor_SMD:R_0402_1005Metric
- removed R42, R43, R44, R45, R46, R47, R48: 750R, Resistor_SMD:R_0402_1005Metric
- removed R59, R60, R61, R62, R63, R64, R65, R66, R67: 0R_DNP, Resistor_SMD:R_0402_1005Metric
- removed R68: 24K, Resistor_SMD:R_0402_1005Metric
- removed R70: 40.2K, Resistor_SMD:R_0402_1005Metric
- removed SW1: PTS645SM43SMTR92 LFS, Button_Switch_SMD:SW_SPST_PTS645
- removed TP1: TestPoint_Small, TestPoint:TestPoint_Pad_D1.0mm
- removed TP2, TP3, TP4, TP5: TestPoint, TestPoint:TestPoint_Pad_D1.0mm
- removed the U1 at (48.5, 235.7)
- removed the U1 at (50.8, 113.0)
- removed U10 (x2): m.2_pcie_nvme, dg_connectors:m.2_pcie_nvme
- removed U11 (x2), U4 (x2): TPS54620, dg_ic:Texas_S-PVQFN-N14_ThermalVias
- removed U12 (x2), U5 (x2): RT8065, dg_ic:DFN-8-1EP_3x3mm_P0.65mm_EP1.55x2.4mm
- removed the U2 at (24.6, 241.3)
- removed the U2 at (22.1, 107.7)
- removed U3, U9 (x2): rpi_cm4, dg_rpi:rpi_cm4
- removed U6: KSZ9477S, dg_ic:128-TQFP-EP
- removed U7: LM1085ISX-3.3/NOPB, Package_TO_SOT_SMD:TO-263-3_TabPin2
- removed Y1: ABM8G-25.000MHZ-B4Y-T, Crystal:Crystal_SMD_Abracon_ABM8G-4Pin_3.2x2.5mm
- added C11: C, Capacitor_SMD:C_0805_2012Metric, F.Cu at (48.5, 261.1)
- added C11: C, Capacitor_SMD:C_0805_2012Metric, F.Cu at (49.8, 159.3)
- added C11: C, Capacitor_SMD:C_0805_2012Metric, F.Cu at (48.0, 59.4)
- added C12: C, Capacitor_SMD:C_0603_1608Metric, F.Cu at (55.4, 165.9)
- added C12: C, Capacitor_SMD:C_0603_1608Metric, F.Cu at (53.7, 66.1)
- added C126: 14pF, Capacitor_SMD:C_0603_1608Metric, F.Cu at (52.3, 299.3)
- added C127: 14pF, Capacitor_SMD:C_0603_1608Metric, F.Cu at (50.6, 291.3)
- added C128: 100nF, Capacitor_SMD:C_0603_1608Metric, F.Cu at (43.1, 299.3)
- added C129: 10uF, Capacitor_SMD:C_0603_1608Metric, F.Cu at (48.1, 291.3)
- added C130: 0.1uF, Capacitor_SMD:C_0603_1608Metric, F.Cu at (49.8, 295.3)
- added C131: 0.1uF, Capacitor_SMD:C_0603_1608Metric, F.Cu at (47.3, 295.3)
- added C132: 14pF, Capacitor_SMD:C_0603_1608Metric, F.Cu at (48.1, 299.3)
- added C133: 14pF, Capacitor_SMD:C_0603_1608Metric, F.Cu at (45.6, 291.3)
- added C134: 10uF, Capacitor_SMD:C_0603_1608Metric, F.Cu at (52.3, 295.3)
- added C14: C, Capacitor_SMD:C_0603_1608Metric, F.Cu at (61.2, 164.3)
- added C14: C, Capacitor_SMD:C_0603_1608Metric, F.Cu at (59.5, 64.5)
- added D1: D_TVS, Diode_SMD:D_SMA, F.Cu at (35.0, 289.1)
- added D19: LED, LED_SMD:LED_0603_1608Metric, F.Cu at (68.6, 4.57)
- added D20: LED, LED_SMD:LED_0603_1608Metric, F.Cu at (40.6, 164.1)
- added D20: LED, LED_SMD:LED_0603_1608Metric, F.Cu at (38.8, 64.3)
- added D21: LED, LED_SMD:LED_0603_1608Metric, F.Cu at (71.6, 231.1)
- added D21: LED, LED_SMD:LED_0603_1608Metric, F.Cu at (72.9, 129.3)
- added D21: LED, LED_SMD:LED_0603_1608Metric, F.Cu at (71.1, 29.5)
- added D22: LED, LED_SMD:LED_0603_1608Metric, F.Cu at (32.8, 164.1)
- added D22: LED, LED_SMD:LED_0603_1608Metric, F.Cu at (31.0, 64.3)
- added D23: LED, LED_SMD:LED_0603_1608Metric, F.Cu at (36.8, 161.5)
- added D23: LED, LED_SMD:LED_0603_1608Metric, F.Cu at (35.1, 61.7)
- added D24: LED, LED_SMD:LED_0603_1608Metric, F.Cu at (39.6, 262.4)
- added D24: LED, LED_SMD:LED_0603_1608Metric, F.Cu at (40.9, 160.6)
- added D24: LED, LED_SMD:LED_0603_1608Metric, F.Cu at (39.1, 60.8)
- added IC1: OKR-T_6-W12-C, dg_power:MURATACASEC90, F.Cu at (72.6, 51.1)
- added IC2: OKR-T_6-W12-C, dg_power:MURATACASEC90, F.Cu at (72.6, 25.9)
- added J2: Conn_02x03_Counter_Clockwise, Connector_PinHeader_2.54mm:PinHeader_2x03_P2.54mm_Vertical, F.Cu at (77.5, 43.4)
- added J4: Conn_02x03_Odd_Even, Connector_PinHeader_2.54mm:PinHeader_2x03_P2.54mm_Vertical, F.Cu at (15.8, 287.7)
- added J5: 2x20, Connector_PinHeader_2.54mm:PinHeader_2x20_P2.54mm_Vertical, F.Cu at (15.8, 306.2)
- added J6: Conn_02x03_Odd_Even, Connector:Tag-Connect_TC2030-IDC-FP_2x03_P1.27mm_Vertical, F.Cu at (28.0, 285.2)
- added J7: USB_B, aep:CUI_UJ2-BH-1-TH, F.Cu at (61.7, 270.3)
- added J8: SS-74500-024, aep:BEL_SS-74500-024, F.Cu at (39.4, 338.8)
- added J9: USB_B, aep:CUI_UJ2-BH-1-TH, F.Cu at (61.5, 286.8)
- added JP13: SolderJumper_2_Open, Jumper:SolderJumper-2_P1.3mm_Open_RoundedPad1.0x1.5mm, F.Cu at (44.8, 163.6)
- added JP13: SolderJumper_2_Open, Jumper:SolderJumper-2_P1.3mm_Open_RoundedPad1.0x1.5mm, F.Cu at (43.0, 63.8)
- added JP14: SolderJumper_2_Open, Jumper:SolderJumper-2_P1.3mm_Open_RoundedPad1.0x1.5mm, F.Cu at (47.5, 249.2)
- added JP14: SolderJumper_2_Open, Jumper:SolderJumper-2_P1.3mm_Open_RoundedPad1.0x1.5mm, F.Cu at (48.8, 147.3)
- added JP14: SolderJumper_2_Open, Jumper:SolderJumper-2_P1.3mm_Open_RoundedPad1.0x1.5mm, F.Cu at (47.0, 47.5)
- added JP15: SolderJumper_2_Open, Jumper:SolderJumper-2_P1.3mm_Open_RoundedPad1.0x1.5mm, F.Cu at (36.3, 249.2)
- added JP15: SolderJumper_2_Open, Jumper:SolderJumper-2_P1.3mm_Open_RoundedPad1.0x1.5mm, F.Cu at (37.6, 147.3)
- added JP15: SolderJumper_2_Open, Jumper:SolderJumper-2_P1.3mm_Open_RoundedPad1.0x1.5mm, F.Cu at (35.8, 47.5)
- added JP16: SolderJumper_2_Open, Jumper:SolderJumper-2_P1.3mm_Open_RoundedPad1.0x1.5mm, F.Cu at (35.1, 228.1)
- added JP16: SolderJumper_2_Open, Jumper:SolderJumper-2_P1.3mm_Open_RoundedPad1.0x1.5mm, F.Cu at (36.3, 126.2)
- added JP16: SolderJumper_2_Open, Jumper:SolderJumper-2_P1.3mm_Open_RoundedPad1.0x1.5mm, F.Cu at (34.5, 26.4)
- added M1: Fan_4pin, Connector:FanPinHeader_1x04_P2.54mm_Vertical, F.Cu at (3.23, 4.23)
- added M2: Fan_4pin, Connector:FanPinHeader_1x04_P2.54mm_Vertical, F.Cu at (15.7, 4.06)
- added R100: 10K, Resistor_SMD:R_0603_1608Metric, F.Cu at (59.8, 299.3)
- added R101: 10K, Resistor_SMD:R_0603_1608Metric, F.Cu at (57.3, 299.3)
- added R102: 10K, Resistor_SMD:R_0603_1608Metric, F.Cu at (54.8, 295.3)
- added R18: R, Resistor_SMD:R_0603_1608Metric, F.Cu at (51.4, 166.9)
- added R18: R, Resistor_SMD:R_0603_1608Metric, F.Cu at (49.6, 67.0)
- added R19: R, Resistor_SMD:R_0603_1608Metric, F.Cu at (47.3, 166.9)
- added R19: R, Resistor_SMD:R_0603_1608Metric, F.Cu at (45.5, 67.1)
- added R20: R, Resistor_SMD:R_0603_1608Metric, F.Cu at (71.7, 228.3)
- added R20: R, Resistor_SMD:R_0603_1608Metric, F.Cu at (73.0, 126.5)
- added R20: R, Resistor_SMD:R_0603_1608Metric, F.Cu at (71.2, 26.7)
- added R21: R, Resistor_SMD:R_0603_1608Metric, F.Cu at (28.8, 164.2)
- added R21: R, Resistor_SMD:R_0603_1608Metric, F.Cu at (27.0, 64.3)
- added R22: R, Resistor_SMD:R_0603_1608Metric, F.Cu at (53.2, 164.3)
- added R22: R, Resistor_SMD:R_0603_1608Metric, F.Cu at (51.4, 64.5)
- added R23: R, Resistor_SMD:R_0603_1608Metric, F.Cu at (32.8, 161.6)
- added R23: R, Resistor_SMD:R_0603_1608Metric, F.Cu at (31.1, 61.8)
- added R86: NC, Resistor_SMD:R_0603_1608Metric, F.Cu at (44.8, 295.3)
- added R87: NC, Resistor_SMD:R_0603_1608Metric, F.Cu at (43.1, 291.3)
- added R88: 36K 1%, Resistor_SMD:R_0603_1608Metric, F.Cu at (54.8, 299.3)
- added R89: 36K 1%, Resistor_SMD:R_0603_1608Metric, F.Cu at (45.6, 299.3)
- added R94: 12K 1%, Resistor_SMD:R_0603_1608Metric, F.Cu at (47.4, 287.3)
- added R97: 10K, Resistor_SMD:R_0603_1608Metric, F.Cu at (14.7, 280.8)
- added R98: 10K, Resistor_SMD:R_0603_1608Metric, F.Cu at (34.0, 283.0)
- added R99: 10K, Resistor_SMD:R_0603_1608Metric, F.Cu at (42.2, 295.3)
- added T1: QT24A01, dg_transformers:SOP100P1000X450-24N, F.Cu at (6.86, 36.6)
- added TP12: TestPoint, TestPoint:TestPoint_Pad_D1.0mm, B.Cu at (51.5, 1.95)
- added TP6: TestPoint, TestPoint:TestPoint_Pad_D1.0mm, B.Cu at (57.6, 1.95)
- added U1: rpi_cm4, dg_rpi:rpi_cm4, F.Cu at (14.2, 259.3)
- added U1: rpi_cm4, dg_rpi:rpi_cm4, F.Cu at (11.4, 107.2)
- added U1: rpi_cm4, dg_rpi:rpi_cm4, F.Cu at (13.7, 57.6)
- added U13: EMC2301, Package_SO:MSOP-8_3x3mm_P0.65mm, F.Cu at (39.6, 289.4)
- added U14: STM32L151C8T6, Package_QFP:LQFP-48_7x7mm_P0.5mm, F.Cu at (19.2, 295.7)
- added U15: USB2514B_Bi, Package_DFN_QFN:QFN-36-1EP_6x6mm_P0.5mm_EP3.7x3.7mm, F.Cu at (36.9, 297.2)
- added U2: m.2_pcie_nvme, dg_connectors:m.2_pcie_nvme, B.Cu at (57.7, 113.8)
- added U2: m.2_pcie_nvme, dg_connectors:m.2_pcie_nvme, B.Cu at (55.9, 14.0)
- added Y2: 24Mhz X1E0000210264, Crystal:Crystal_SMD_SeikoEpson_TSX3225-4Pin_3.2x2.5mm, F.Cu at (39.5, 283.1)
- added Y3: 24Mhz X1E0000210264, Crystal:Crystal_SMD_SeikoEpson_TSX3225-4Pin_3.2x2.5mm, F.Cu at (44.0, 283.1)
- C13, TP7: moved to B.Cu
- moved C13 373.9 mm to (47.0, 5.59), turned to 90 degrees
- moved TP7 305.7 mm to (54.6, 1.95), turned to 180 degrees
Other:
- outline, holes or cut-outs redrawn

Commit message: just use two usb hubs
Parts:
- removed the C11 at (48.5, 261.1)
- removed the C11 at (49.8, 159.3)
- removed the C11 at (48.0, 59.4)
- removed the C12 at (55.4, 165.9)
- removed the C12 at (53.7, 66.1)
- removed the C14 at (61.2, 164.3)
- removed the C14 at (59.5, 64.5)
- removed the D20 at (40.6, 164.1)
- removed the D20 at (38.8, 64.3)
- removed the D21 at (71.6, 231.1)
- removed the D21 at (72.9, 129.3)
- removed the D21 at (71.1, 29.5)
- removed the D22 at (32.8, 164.1)
- removed the D22 at (31.0, 64.3)
- removed the D23 at (36.8, 161.5)
- removed the D23 at (35.1, 61.7)
- removed the D24 at (39.6, 262.4)
- removed the D24 at (40.9, 160.6)
- removed the D24 at (39.1, 60.8)
- removed the JP13 at (44.8, 163.6)
- removed the JP13 at (43.0, 63.8)
- removed the JP14 at (47.5, 249.2)
- removed the JP14 at (48.8, 147.3)
- removed the JP14 at (47.0, 47.5)
- removed the JP15 at (36.3, 249.2)
- removed the JP15 at (37.6, 147.3)
- removed the JP15 at (35.8, 47.5)
- removed the JP16 at (35.1, 228.1)
- removed the JP16 at (36.3, 126.2)
- removed the JP16 at (34.5, 26.4)
- removed the R18 at (51.4, 166.9)
- removed the R18 at (49.6, 67.0)
- removed the R19 at (47.3, 166.9)
- removed the R19 at (45.5, 67.1)
- removed the R20 at (71.7, 228.3)
- removed the R20 at (73.0, 126.5)
- removed the R20 at (71.2, 26.7)
- removed the R21 at (28.8, 164.2)
- removed the R21 at (27.0, 64.3)
- removed the R22 at (53.2, 164.3)
- removed the R22 at (51.4, 64.5)
- removed the R23 at (32.8, 161.6)
- removed the R23 at (31.1, 61.8)
- removed the U1 at (14.2, 259.3)
- removed the U1 at (11.4, 107.2)
- removed the U1 at (13.7, 57.6)
- removed the U2 at (57.7, 113.8)
- removed the U2 at (55.9, 14.0)
- added C11: C, Capacitor_SMD:C_0805_2012Metric, F.Cu at (71.0, 57.0)
- added C12: C, Capacitor_SMD:C_0603_1608Metric, F.Cu at (40.4, 42.2)
- added C14: C, Capacitor_SMD:C_0603_1608Metric, F.Cu at (36.4, 43.6)
- added D20: LED, LED_SMD:LED_0603_1608Metric, F.Cu at (41.2, 36.1)
- added D21: LED, LED_SMD:LED_0603_1608Metric, F.Cu at (36.7, 39.6)
- added D22: LED, LED_SMD:LED_0603_1608Metric, F.Cu at (40.8, 39.6)
- added D23: LED, LED_SMD:LED_0603_1608Metric, F.Cu at (44.8, 38.7)
- added D24: LED, LED_SMD:LED_0603_1608Metric, F.Cu at (48.9, 36.1)
- added J1: Conn_02x04_Odd_Even, Connector_Molex:Molex_Mini-Fit_Jr_5569-08A1_2x04_P4.20mm_Horizontal, F.Cu at (58.0, 9.00)
- added JP13: SolderJumper_2_Open, Jumper:SolderJumper-2_P1.3mm_Open_RoundedPad1.0x1.5mm, F.Cu at (32.5, 39.6)
- added JP14: SolderJumper_2_Open, Jumper:SolderJumper-2_P1.3mm_Open_RoundedPad1.0x1.5mm, F.Cu at (37.0, 36.6)
- added JP15: SolderJumper_2_Open, Jumper:SolderJumper-2_P1.3mm_Open_RoundedPad1.0x1.5mm, F.Cu at (75.4, 57.3)
- added JP16: SolderJumper_2_Open, Jumper:SolderJumper-2_P1.3mm_Open_RoundedPad1.0x1.5mm, F.Cu at (33.0, 27.0)
- added R18: R, Resistor_SMD:R_0603_1608Metric, F.Cu at (52.9, 36.0)
- added R19: R, Resistor_SMD:R_0603_1608Metric, F.Cu at (56.9, 36.0)
- added R20: R, Resistor_SMD:R_0603_1608Metric, F.Cu at (48.8, 41.1)
- added R21: R, Resistor_SMD:R_0603_1608Metric, F.Cu at (52.8, 41.1)
- added R22: R, Resistor_SMD:R_0603_1608Metric, F.Cu at (44.4, 42.2)
- added R23: R, Resistor_SMD:R_0603_1608Metric, F.Cu at (52.9, 38.5)
- added U1: rpi_cm4, dg_rpi:rpi_cm4, F.Cu at (12.0, 59.0)
- added U2: m.2_pcie_nvme, dg_connectors:m.2_pcie_nvme, B.Cu at (16.0, 9.00)
- C13, TP12, TP6, TP7: moved to F.Cu
- moved U13 274.5 mm to (46.0, 15.0), turned to 0 degrees
- moved R97 233.9 mm to (203.4, 142.6), turned to 0 degrees
- moved R86 217.4 mm to (199.4, 142.6), turned to 0 degrees
- moved R100 208.0 mm to (199.4, 145.1), turned to 0 degrees
- moved R88 193.9 mm to (188.0, 158.5), turned to 0 degrees
- moved J6 188.9 mm to (172.9, 164.1), turned to 0 degrees
- moved C130 186.8 mm to (179.2, 160.6), turned to 0 degrees
- moved J4 181.7 mm to (158.3, 175.0), turned to 0 degrees
- moved R89 176.1 mm to (169.2, 173.9), turned to 0 degrees
- moved C134 174.4 mm to (166.0, 163.1), turned to 0 degrees
- moved C127 174.4 mm to (166.0, 160.6), turned to 0 degrees
- moved R99 172.8 mm to (165.2, 173.9), turned to 0 degrees
- moved R98 172.2 mm to (169.2, 176.4), turned to 0 degrees
- moved C129 172.0 mm to (170.1, 170.2), turned to 0 degrees
- moved J7 169.0 mm to (173.7, 143.7), turned to 0 degrees
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Routing:
- added copper zone on In3.Cu, net +12V
- added copper zone on In1.Cu, net GND
- added copper zone on In4.Cu, net GND
Other:
- copper layers 2 -> 6
