File: currypi.kicad_pcb (KiCad board)
At the start: 6 copper layers, 80 x 350 mm, 64 parts, among them IC1 OKR-T_6-W12-C, IC2 OKR-T_6-W12-C, J1 Conn_02x04_Odd_Even, J2 Conn_02x03_Counter_Clockwise, J4 Conn_02x03_Odd_Even, J5 2x20, J6 Conn_02x03_Odd_Even, J7 USB_B, J8 SS-74500-024, J9 USB_B, M1 Fan_4pin, M2 Fan_4pin, T1 QT24A01, U1 rpi_cm4, U13 EMC2301, U14 STM32L151C8T6, U15 USB2514B_Bi, U2 m.2_pcie_nvme, Y2 24Mhz X1E0000210264, Y3 24Mhz X1E0000210264

Commit message: use native rpi uarts instead of extra chip
Parts:
- removed C126, C127, C132, C133: 14pF, Capacitor_SMD:C_0603_1608Metric
- removed C128: 100nF, Capacitor_SMD:C_0603_1608Metric
- removed C129, C134: 10uF, Capacitor_SMD:C_0603_1608Metric
- removed C130, C131: 0.1uF, Capacitor_SMD:C_0603_1608Metric
- removed J6: Conn_02x03_Odd_Even, Connector:Tag-Connect_TC2030-IDC-FP_2x03_P1.27mm_Vertical
- removed J7, J9: USB_B, aep:CUI_UJ2-BH-1-TH
- removed R100, R101, R102, R97, R98, R99: 10K, Resistor_SMD:R_0603_1608Metric
- removed R86, R87: NC, Resistor_SMD:R_0603_1608Metric
- removed R88, R89: 36K 1%, Resistor_SMD:R_0603_1608Metric
- removed R94: 12K 1%, Resistor_SMD:R_0603_1608Metric
- removed U13: EMC2301, Package_SO:MSOP-8_3x3mm_P0.65mm
- removed U14: STM32L151C8T6, Package_QFP:LQFP-48_7x7mm_P0.5mm
- removed U15: USB2514B_Bi, Package_DFN_QFN:QFN-36-1EP_6x6mm_P0.5mm_EP3.7x3.7mm
- removed Y2: 24Mhz X1E0000210264, Crystal:Crystal_SMD_SeikoEpson_TSX3225-4Pin_3.2x2.5mm
- added C1: C, Capacitor_SMD:C_0805_2012Metric, F.Cu at (69.0, 287.0)
- added C15: 14pF, Capacitor_SMD:C_0603_1608Metric, F.Cu at (33.6, 261.6)
- added C16: 14pF, Capacitor_SMD:C_0603_1608Metric, F.Cu at (44.4, 250.1)
- added C18: 10uF, Capacitor_SMD:C_0603_1608Metric, F.Cu at (29.6, 261.6)
- added C2: C, Capacitor_SMD:C_0603_1608Metric, F.Cu at (81.6, 284.5)
- added C3: 100nF, Capacitor_SMD:C_0603_1608Metric, F.Cu at (11.2, -7.24)
- added C7: 0.1uF, Capacitor_SMD:C_0603_1608Metric, F.Cu at (44.4, 252.6)
- added C8: 0.1uF, Capacitor_SMD:C_0603_1608Metric, F.Cu at (37.6, 259.0)
- added D2: LED, LED_SMD:LED_0603_1608Metric, F.Cu at (81.6, 281.9)
- added D3: LED, LED_SMD:LED_0603_1608Metric, F.Cu at (73.2, 290.3)
- added D4: LED, LED_SMD:LED_0603_1608Metric, F.Cu at (81.6, 279.3)
- added D5: LED, LED_SMD:LED_0603_1608Metric, F.Cu at (68.8, 293.4)
- added D6: LED, LED_SMD:LED_0603_1608Metric, F.Cu at (81.6, 276.7)
- added D7: D_TVS, Diode_SMD:D_SMA, F.Cu at (103.0, 329.0)
- added H1: MountingHole, MountingHole:MountingHole_3.2mm_M3_Pad, F.Cu at (74.0, 28.0)
- added H2: MountingHole, MountingHole:MountingHole_3.2mm_M3_Pad, F.Cu at (4.73, 173.4)
- added H3: MountingHole, MountingHole:MountingHole_3.2mm_M3_Pad, F.Cu at (5.00, 28.0)
- added H4: MountingHole, MountingHole:MountingHole_3.2mm_M3_Pad, F.Cu at (75.0, 173.4)
- added H5: MountingHole, MountingHole:MountingHole_3.2mm_M3_Pad, F.Cu at (74.0, 313.0)
- added H6: MountingHole, MountingHole:MountingHole_3.2mm_M3_Pad, F.Cu at (6.00, 313.0)
- added IC3: OKR-T_6-W12-C, dg_power:MURATACASEC90, F.Cu at (99.0, 278.6)
- added IC4: OKR-T_6-W12-C, dg_power:MURATACASEC90, F.Cu at (99.0, 269.8)
- added JP1: SolderJumper_2_Open, Jumper:SolderJumper-2_P1.3mm_Open_RoundedPad1.0x1.5mm, F.Cu at (69.0, 290.3)
- added JP2: SolderJumper_2_Open, Jumper:SolderJumper-2_P1.3mm_Open_RoundedPad1.0x1.5mm, F.Cu at (81.8, 273.7)
- added JP3: SolderJumper_2_Open, Jumper:SolderJumper-2_P1.3mm_Open_RoundedPad1.0x1.5mm, F.Cu at (81.8, 270.1)
- added JP4: SolderJumper_2_Open, Jumper:SolderJumper-2_P1.3mm_Open_RoundedPad1.0x1.5mm, F.Cu at (73.4, 287.3)
- added R1: 268, Resistor_SMD:R_0402_1005Metric_Pad0.72x0.64mm_HandSolder, F.Cu at (83.8, 50.0)
- added R10: R, Resistor_SMD:R_0603_1608Metric, F.Cu at (72.8, 293.3)
- added R11: R, Resistor_SMD:R_0603_1608Metric, F.Cu at (77.2, 290.3)
- added R12: R, Resistor_SMD:R_0603_1608Metric, F.Cu at (68.8, 298.4)
- added R13: 1K, Resistor_SMD:R_0402_1005Metric_Pad0.72x0.64mm_HandSolder, F.Cu at (117.5, 279.5)
- added R14: 268, Resistor_SMD:R_0402_1005Metric_Pad0.72x0.64mm_HandSolder, F.Cu at (121.0, 282.5)
- added R15: 436, Resistor_SMD:R_0402_1005Metric_Pad0.72x0.64mm_HandSolder, F.Cu at (120.5, 280.0)
- added R16: 10K, Resistor_SMD:R_0603_1608Metric, F.Cu at (48.5, 255.7)
- added R17: 10K, Resistor_SMD:R_0603_1608Metric, F.Cu at (45.6, 258.2)
- added R2: 436, Resistor_SMD:R_0402_1005Metric_Pad0.72x0.64mm_HandSolder, F.Cu at (83.8, 52.0)
- added R24: 10K, Resistor_SMD:R_0603_1608Metric, F.Cu at (37.6, 261.6)
- added R25: 10K, Resistor_SMD:R_0603_1608Metric, F.Cu at (53.7, 245.7)
- added R26: 10K, Resistor_SMD:R_0603_1608Metric, F.Cu at (33.6, 259.0)
- added R27: 10K, Resistor_SMD:R_0603_1608Metric, F.Cu at (49.7, 243.1)
- added R28: DNC, Resistor_SMD:R_0402_1005Metric_Pad0.72x0.64mm_HandSolder, F.Cu at (119.0, 274.0)
- added R3: DNC, Resistor_SMD:R_0402_1005Metric_Pad0.72x0.64mm_HandSolder, F.Cu at (87.0, 50.0)
- added R4: 1K, Resistor_SMD:R_0402_1005Metric_Pad0.72x0.64mm_HandSolder, F.Cu at (87.0, 52.0)
- added R5: R, Resistor_SMD:R_0603_1608Metric, F.Cu at (77.6, 286.8)
- added R6: 36K 1%, Resistor_SMD:R_0603_1608Metric, F.Cu at (5.99, -2.00)
- added R7: 36K 1%, Resistor_SMD:R_0603_1608Metric, F.Cu at (11.2, -9.75)
- added R8: R, Resistor_SMD:R_0603_1608Metric, F.Cu at (68.8, 295.9)
- added R9: 12K 1%, Resistor_SMD:R_0603_1608Metric, F.Cu at (52.5, 250.7)
- added RLA1: G3VM-61VY2-TR, dg_relay:G3VM-SOP, F.Cu at (73.2, 71.0)
- added RLA2: G3VM-61VY2-TR, dg_relay:G3VM-SOP, F.Cu at (108.4, 271.1)
- added T2: QT24A01, dg_transformers:SOP100P1000X450-24N, F.Cu at (73.2, 276.9)
- added U3: EMC2301, Package_SO:MSOP-8_3x3mm_P0.65mm, F.Cu at (43.3, -7.08)
- added U4: rpi_cm4, dg_rpi:rpi_cm4, F.Cu at (11.2, 308.9)
- added U6: USB2514B_Bi, Package_DFN_QFN:QFN-36-1EP_6x6mm_P0.5mm_EP3.7x3.7mm, F.Cu at (22.4, 246.0)
- J1: footprint Connector_Molex:Molex_Mini-Fit_Jr_5569-08A1_2x04_P4.20mm_Horizontal -> Connector_Molex:Molex_Mini-Fit_Jr_5569-08A2_2x04_P4.20mm_Horizontal
- J4: value Conn_02x03_Odd_Even -> Conn_02x03_Counter_Clockwise
- J5: value 2x20 -> Conn_02x04_Odd_Even; footprint Connector_PinHeader_2.54mm:PinHeader_2x20_P2.54mm_Vertical -> Connector_Molex:Molex_Mini-Fit_Jr_5569-08A2_2x04_P4.20mm_Horizontal
- moved Y3 155.7 mm to (20.9, 260.6)
- moved J4 114.2 mm to (105.3, 276.1)
- moved D1 100.2 mm to (110.0, 294.5)
- moved J5 71.4 mm to (77.2, 336.0), turned to 180 degrees
- moved C11 70.0 mm to (1.75, 67.5)
- moved JP15 70.0 mm to (6.15, 67.8)
- moved M2 32.6 mm to (6.26, -15.3)
- moved M1 31.4 mm to (18.4, -15.3)
- moved C12 13.5 mm to (40.1, 55.7)
- moved C13 13.5 mm to (32.3, 49.8)
- moved C14 13.5 mm to (36.1, 57.1)
- moved D19 13.5 mm to (32.1, 56.1)
- moved D20 13.5 mm to (40.9, 49.6)
- moved D21 13.5 mm to (36.5, 53.1)
- moved D22 13.5 mm to (40.5, 53.1)
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- renumbered J8 to J3
Connections:
- net /sheet613B6EED/3.3V renamed /dcdc/3.3V
- net /sheet613B6EED/5V renamed /dcdc/5V
- net /sheet613B6EED/ETH0+ renamed /pi/ETH0+
- net /sheet613B6EED/ETH0- renamed /pi/ETH0-
- net /sheet613B6EED/ETH1+ renamed /pi/ETH1+
- net /sheet613B6EED/ETH1- renamed /pi/ETH1-
- net /sheet613B6EED/ETH2+ renamed /pi/ETH2+
- net /sheet613B6EED/ETH2- renamed /pi/ETH2-
- net /sheet613B6EED/ETH3+ renamed /pi/ETH3+
- net /sheet613B6EED/ETH3- renamed /pi/ETH3-
- net /sheet613B6EED/RPI_PCIe_CLK_nREQ renamed /pi/RPI_PCIe_CLK_nREQ
- net /sheet613B6EED/RPI_PCIe_RX_N renamed /pi/RPI_PCIe_RX_N
- net /sheet613B6EED/RPI_PCIe_RX_P renamed /pi/RPI_PCIe_RX_P
- net /sheet613B6EED/RPI_PCIe_TX_N renamed /pi/RPI_PCIe_TX_N
- net /sheet613B6EED/RPI_PCIe_TX_P renamed /pi/RPI_PCIe_TX_P
- net /sheet613B6EED/RPI_PCIe_nRST renamed /pi/RPI_PCIe_nRST
- net /sheet613B6EED/pi3.3 renamed /pi/pi3.3
- net /sheet613B6EEE/VIN1 renamed /dcdc/VIN1
- net /sheet613B6EEE/VIN2 renamed /dcdc/VIN2
- IC1 pad 1: /sheet613B6EEE/DISABLE -> /c1_disable
- IC1 pad 5: (no net) -> Net-(IC1-Pad5)
- IC2 pad 1: /sheet613B6EEE/DISABLE -> /c1_disable
- IC2 pad 5: (no net) -> Net-(IC2-Pad5)
- J4 pad 1: (no net) -> /mgm/5V
- J4 pad 2: +3V3 -> /mgm/5V
- J4 pad 3: /mcu_reset -> /sheet61DCBD00/VIN2
- J4 pad 4: Net-(J4-Pad4) -> /sheet61DCBD00/VIN2
- J4 pad 5: GND -> /sheet61DCBD00/VIN1
- J4 pad 6: GND -> /sheet61DCBD00/VIN1
- J5 pad 3: /c1_vref -> GND
- J5 pad 4: /c1_tx -> GND
- J5 pad 5: /c1_wp -> +12V
- J5 pad 6: /c1_rx -> +12V
- J5 pad 7: /c1_boot -> +12V
- J5 pad 8: /c1_act -> +12V
- U1 pad 103: (no net) -> /c1_usb-
- U1 pad 105: (no net) -> /c1_usb+
- U1 pad 46: (no net) -> /c1_boot
- U1 pad 49: (no net) -> /c1_disable
- U1 pad 51: (no net) -> /c1_rx
- U1 pad 55: (no net) -> /c1_tx
- U1 pad 93: (no net) -> /c1_boot
Other:
- outline, holes or cut-outs redrawn

Commit message: use a 2x2 and a magjack
Parts:
- removed D20, D21: LED, LED_SMD:LED_0603_1608Metric
- removed T2: QT24A01, dg_transformers:SOP100P1000X450-24N
- added C10: 100nF, Capacitor_SMD:C_0402_1005Metric, F.Cu at (79.4, -32.0)
- added C17: 10uF, Capacitor_SMD:C_0805_2012Metric, F.Cu at (62.5, -26.8)
- added C19: 10uF, Capacitor_SMD:C_0805_2012Metric, F.Cu at (67.0, -29.8)
- added C20: 10uF, Capacitor_SMD:C_0805_2012Metric, F.Cu at (73.8, -36.5)
- added C21: 10uF, Capacitor_SMD:C_0805_2012Metric, F.Cu at (62.5, -29.8)
- added C22: 100nF, Capacitor_SMD:C_0402_1005Metric, F.Cu at (79.3, -28.1)
- added C23: 100nF, Capacitor_SMD:C_0402_1005Metric, F.Cu at (73.6, -26.7)
- added C24: 100nF, Capacitor_SMD:C_0402_1005Metric, F.Cu at (79.4, -30.0)
- added C25: 1000pF 2kV, Capacitor_SMD:C_1206_3216Metric, F.Cu at (68.8, -36.3)
- added C26: 100nF, Capacitor_SMD:C_0402_1005Metric, F.Cu at (76.5, -30.0)
- added C4: 100uF, Capacitor_SMD:C_1206_3216Metric, F.Cu at (63.1, -33.0)
- added C5: 10uF, Capacitor_SMD:C_0805_2012Metric, F.Cu at (68.2, -33.1)
- added C6: 10uF, Capacitor_SMD:C_0805_2012Metric, F.Cu at (78.3, -36.5)
- added C9: 10uF, Capacitor_SMD:C_0805_2012Metric, F.Cu at (67.0, -26.8)
- added D10: LED, LED_SMD:LED_0603_1608Metric, F.Cu at (75.2, -20.8)
- added D11: LED, LED_SMD:LED_0603_1608Metric, F.Cu at (62.4, -12.0)
- added D8: LED, LED_SMD:LED_0603_1608Metric, F.Cu at (28.4, 18.9)
- added D9: LED, LED_SMD:LED_0603_1608Metric, F.Cu at (41.2, 10.1)
- added J6: 0826-1X1T-GH-F, dg_connectors:BEL_0826-1X1T-GH-F, F.Cu at (70.0, 342.5)
- added R29: 1k, Resistor_SMD:R_0402_1005Metric, F.Cu at (70.7, -30.6)
- added R30: 75, Resistor_SMD:R_0402_1005Metric, F.Cu at (76.3, -34.0)
- added R31: 75, Resistor_SMD:R_0402_1005Metric, F.Cu at (70.7, -28.7)
- added R32: 75, Resistor_SMD:R_0402_1005Metric, F.Cu at (73.6, -30.6)
- added R33: 75, Resistor_SMD:R_0402_1005Metric, F.Cu at (73.6, -28.7)
- added R34: 1k, Resistor_SMD:R_0402_1005Metric, F.Cu at (70.7, -26.7)
- added R35: 1k, Resistor_SMD:R_0402_1005Metric, F.Cu at (79.2, -34.0)
- added R36: 1k, Resistor_SMD:R_0402_1005Metric, F.Cu at (76.5, -32.0)
- C11: value C -> 10uF
- C12: value C -> 100nF; footprint Capacitor_SMD:C_0603_1608Metric -> Capacitor_SMD:C_0402_1005Metric
- C13: value C -> 100uF; footprint Capacitor_SMD:C_0805_2012Metric -> Capacitor_SMD:C_1206_3216Metric
- C14: value C -> 10uF; footprint Capacitor_SMD:C_0603_1608Metric -> Capacitor_SMD:C_0805_2012Metric
- J2, J4: value Conn_02x03_Counter_Clockwise -> Header_2x6_2.54mm
- J3: value SS-74500-024 -> SS-74500-020; footprint aep:BEL_SS-74500-024 -> dg_connectors:BEL_SS-74500-020
- R15: value 436 -> 1k; footprint Resistor_SMD:R_0402_1005Metric_Pad0.72x0.64mm_HandSolder -> Resistor_SMD:R_0402_1005Metric
- R18, R21, R22, R23: value R -> 1k; footprint Resistor_SMD:R_0603_1608Metric -> Resistor_SMD:R_0402_1005Metric
- R19: value R -> DNC; footprint Resistor_SMD:R_0603_1608Metric -> Resistor_SMD:R_0402_1005Metric
- R20: value R -> 436; footprint Resistor_SMD:R_0603_1608Metric -> Resistor_SMD:R_0402_1005Metric_Pad0.72x0.64mm_HandSolder
- R28: footprint Resistor_SMD:R_0402_1005Metric_Pad0.72x0.64mm_HandSolder -> Resistor_SMD:R_0402_1005Metric
- R3: value DNC -> 1k; footprint Resistor_SMD:R_0402_1005Metric_Pad0.72x0.64mm_HandSolder -> Resistor_SMD:R_0402_1005Metric
- moved D7 333.1 mm to (3.58, 11.0)
- moved J5 326.2 mm to (-16.8, 23.7), turned to 0 degrees
- moved J1 321.7 mm to (53.0, 336.0), turned to 180 degrees
- moved IC4 292.0 mm to (69.1, -20.7)
- moved R28 290.6 mm to (69.1, -12.3)
- moved R15 275.0 mm to (35.1, 18.6)
- moved C14 97.3 mm to (72.6, -33.1)
- moved C13 91.5 mm to (63.1, -36.3)
- moved C12 91.3 mm to (76.5, -28.1)
- moved R22 80.2 mm to (74.6, -18.5)
- moved R23 77.7 mm to (78.7, -21.1)
- moved U1 76.7 mm to (-19.8, 2.56)
- moved R21 74.4 mm to (74.6, -16.5)
- moved R20 69.1 mm to (66.0, -12.3)
- moved R2 61.6 mm to (32.0, 18.6)
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Connections:
- net /dcdc/VIN2 renamed /dcdc/VIN_DCDC_3V3
- net /pi/pi3.3 renamed /pi/pi3V3
- net /sheet61DCBD00/VIN2 renamed /sheet61DCBD00/VIN_DCDC_3V3
- C13 pad 1: /dcdc/3.3V -> /dcdc/3V3
- C14 pad 1: /dcdc/3.3V -> /dcdc/3V3
- C18 pad 1: /sheet61DCBD00/3.3V -> /usbhub/3.3V
- IC1 pad 1: /c1_disable -> /dcdc/DISABLE_DCDC
- IC1 pad 2: /dcdc/VIN1 -> /dcdc/VIN_DCDC_5V
- IC2 pad 1: /c1_disable -> /dcdc/DISABLE_DCDC
- IC2 pad 4: /dcdc/3.3V -> /dcdc/3V3
- IC3 pad 1: /sheet61DCBD00/DISABLE -> /sheet61DCBD00/DISABLE_DCDC
- IC3 pad 2: /sheet61DCBD00/VIN1 -> /sheet61DCBD00/VIN_DCDC_5V
- IC4 pad 1: /sheet61DCBD00/DISABLE -> /sheet61DCBD00/DISABLE_DCDC
- IC4 pad 4: /sheet61DCBD00/3.3V -> /sheet61DCBD00/3V3
- J2 pad 5: /dcdc/VIN1 -> /dcdc/VIN_DCDC_5V
- J2 pad 6: /dcdc/VIN1 -> /dcdc/VIN_DCDC_5V
- J3 pad 11_2: /c2_vref -> (no net)
- J3 pad 11_3: /c3_vref -> (no net)
- J3 pad 11_4: /c4_vref -> (no net)
- J3 pad 9_2: /c2_vref -> (no net)
- J3 pad 9_3: /c3_vref -> (no net)
- J3 pad 9_4: /c4_vref -> (no net)
- J4 pad 5: /sheet61DCBD00/VIN1 -> /sheet61DCBD00/VIN_DCDC_5V
- J4 pad 6: /sheet61DCBD00/VIN1 -> /sheet61DCBD00/VIN_DCDC_5V
- R15 pad 1: GND -> Net-(D9-Pad1)
- R15 pad 2: Net-(IC4-Pad5) -> GND
- R16 pad 2: /sheet61DCBD00/3.3V -> /usbhub/3.3V
- R17 pad 2: /sheet61DCBD00/3.3V -> /usbhub/3.3V
- R18 pad 1: Net-(R18-Pad1) -> /dcdc/VIN_DCDC_5V
- R18 pad 2: Net-(D19-Pad1) -> /dcdc/DISABLE_DCDC
- R19 pad 1: GND -> /c1_disable
- R19 pad 2: Net-(D20-Pad1) -> /dcdc/DISABLE_DCDC
- R20 pad 2: Net-(D21-Pad1) -> Net-(IC4-Pad5)
- R21 pad 1: Net-(R21-Pad1) -> Net-(D10-Pad1)
- R21 pad 2: Net-(D22-Pad2) -> GND
- R22 pad 1: Net-(R22-Pad1) -> Net-(D11-Pad1)
- R22 pad 2: Net-(D23-Pad2) -> GND
- R23 pad 1: Net-(R23-Pad1) -> /sheet61DCBD00/VIN_DCDC_5V
- R23 pad 2: Net-(D24-Pad2) -> /sheet61DCBD00/DISABLE_DCDC
- R25 pad 2: /sheet61DCBD00/3.3V -> /usbhub/3.3V
- R26 pad 2: /sheet61DCBD00/3.3V -> /usbhub/3.3V
- R28 pad 2: /sheet61DCBD00/VIN1 -> /sheet61DCBD00/DISABLE_DCDC
- R3 pad 1: /c1_disable -> Net-(D8-Pad1)
- R3 pad 2: /dcdc/VIN1 -> GND
- RLA1 pad 4: /c1_disable -> /dcdc/DISABLE_DCDC
- RLA2 pad 4: /sheet61DCBD00/DISABLE -> /sheet61DCBD00/DISABLE_DCDC
- T1 pad 1: (no net) -> Net-(C26-Pad1)
- T1 pad 10: (no net) -> Net-(C26-Pad1)
- T1 pad 11: (no net) -> /pi/TD4_P
- T1 pad 12: (no net) -> /pi/TD4_N
- T1 pad 13: (no net) -> /pi/ETH3-
- T1 pad 14: (no net) -> /pi/ETH3+
- T1 pad 15: (no net) -> Net-(R33-Pad1)
- T1 pad 16: (no net) -> /pi/ETH2-
- T1 pad 17: (no net) -> /pi/ETH2+
- T1 pad 18: (no net) -> Net-(R32-Pad1)
- T1 pad 19: (no net) -> /pi/ETH1-
- T1 pad 2: (no net) -> /pi/TD1_P
- T1 pad 20: (no net) -> /pi/ETH1+
- T1 pad 21: (no net) -> Net-(R31-Pad1)
- T1 pad 22: (no net) -> /pi/ETH0-
- T1 pad 23: (no net) -> /pi/ETH0+
- T1 pad 24: (no net) -> Net-(R30-Pad1)
- T1 pad 3: (no net) -> /pi/TD1_N
- T1 pad 4: (no net) -> Net-(C26-Pad1)
- T1 pad 5: (no net) -> /pi/TD2_P
- T1 pad 6: (no net) -> /pi/TD2_N
- T1 pad 7: (no net) -> Net-(C26-Pad1)
- T1 pad 8: (no net) -> /pi/TD3_P
- T1 pad 9: (no net) -> /pi/TD3_N
- U1 pad 10: /pi/ETH0- -> /pi/TD1_N
- U1 pad 11: /pi/ETH2+ -> /pi/TD3_P
- U1 pad 110: GND -> /pi/RPI_PCIe_CLK_P
- U1 pad 112: GND -> /pi/RPI_PCIe_CLK_N
- U1 pad 12: /pi/ETH0+ -> /pi/TD1_P
- U1 pad 15: Net-(R23-Pad1) -> Net-(R36-Pad2)
- U1 pad 17: Net-(R22-Pad1) -> Net-(R35-Pad2)
- U1 pad 19: Net-(R21-Pad1) -> Net-(R34-Pad2)
- U1 pad 21: Net-(R18-Pad1) -> Net-(R29-Pad2)
- U1 pad 3: /pi/ETH3+ -> /pi/TD4_P
- U1 pad 4: /pi/ETH1+ -> /pi/TD2_P
- U1 pad 5: /pi/ETH3- -> /pi/TD4_N
- U1 pad 6: /pi/ETH1- -> /pi/TD2_N
- U1 pad 9: /pi/ETH2- -> /pi/TD3_N
- U2 pad 12: /dcdc/3.3V -> /pi/3.3V
- U2 pad 14: /dcdc/3.3V -> /pi/3.3V
- U2 pad 16: /dcdc/3.3V -> /pi/3.3V
- U2 pad 18: /dcdc/3.3V -> /pi/3.3V
- U2 pad 2: /dcdc/3.3V -> /pi/3.3V
- U2 pad 4: /dcdc/3.3V -> /pi/3.3V
- U2 pad 53: GND -> /pi/RPI_PCIe_CLK_N
- U2 pad 55: GND -> /pi/RPI_PCIe_CLK_P
- U2 pad 70: /dcdc/3.3V -> /pi/3.3V
- U2 pad 72: /dcdc/3.3V -> /pi/3.3V
- U2 pad 74: /dcdc/3.3V -> /pi/3.3V
- U6 pad 10: /sheet61DCBD00/3.3V -> /usbhub/3.3V
- U6 pad 15: /sheet61DCBD00/3.3V -> /usbhub/3.3V
- U6 pad 23: /sheet61DCBD00/3.3V -> /usbhub/3.3V
- U6 pad 29: /sheet61DCBD00/3.3V -> /usbhub/3.3V
- U6 pad 36: /sheet61DCBD00/3.3V -> /usbhub/3.3V
- U6 pad 5: /sheet61DCBD00/3.3V -> /usbhub/3.3V
Other:
- outline, holes or cut-outs redrawn

Commit message: Updated PCB Design.
Parts:
- removed D23, D24: LED, LED_SMD:LED_0603_1608Metric
- removed J2, J4: Header_2x6_2.54mm, Connector_PinHeader_2.54mm:PinHeader_2x03_P2.54mm_Vertical
- removed J3: SS-74500-020, dg_connectors:BEL_SS-74500-020
- removed Y3: 24Mhz X1E0000210264, Crystal:Crystal_SMD_SeikoEpson_TSX3225-4Pin_3.2x2.5mm
- added C27: 100uF, Capacitor_SMD:C_1206_3216Metric, F.Cu at (272.2, 187.0)
- added C28: 10uF, Capacitor_SMD:C_0805_2012Metric, F.Cu at (281.7, 186.8)
- added C29: 10uF, Capacitor_SMD:C_0805_2012Metric, F.Cu at (277.2, 186.8)
- added C30: 10uF, Capacitor_SMD:C_0805_2012Metric, F.Cu at (253.7, 233.6)
- added C31: 10uF, Capacitor_SMD:C_0805_2012Metric, F.Cu at (271.6, 190.2)
- added C32: 100nF, Capacitor_SMD:C_0402_1005Metric, F.Cu at (276.6, 201.9)
- added C33: 100nF, Capacitor_SMD:C_0402_1005Metric, F.Cu at (276.6, 199.9)
- added C34: 100uF, Capacitor_SMD:C_1206_3216Metric, F.Cu at (248.6, 233.7)
- added C35: 10uF, Capacitor_SMD:C_0805_2012Metric, F.Cu at (280.5, 189.9)
- added C36: 10uF, Capacitor_SMD:C_0805_2012Metric, F.Cu at (276.0, 193.2)
- added C37: 10uF, Capacitor_SMD:C_0805_2012Metric, F.Cu at (271.6, 196.2)
- added C38: 10uF, Capacitor_SMD:C_0805_2012Metric, F.Cu at (271.6, 193.2)
- added C39: 10uF, Capacitor_SMD:C_0805_2012Metric, F.Cu at (276.0, 190.2)
- added C40: 100nF, Capacitor_SMD:C_0402_1005Metric, F.Cu at (270.8, 203.9)
- added C41: 100nF, Capacitor_SMD:C_0402_1005Metric, F.Cu at (273.7, 201.9)
- added C42: 100nF, Capacitor_SMD:C_0402_1005Metric, F.Cu at (270.8, 201.9)
- added C43: 1000pF 2kV, Capacitor_SMD:C_1206_3216Metric, F.Cu at (328.5, 162.9)
- added C44: 100nF, Capacitor_SMD:C_0402_1005Metric, F.Cu at (273.7, 203.9)
- added C45: 100uF, Capacitor_SMD:C_1206_3216Metric, F.Cu at (418.5, 136.9)
- added C46: 10uF, Capacitor_SMD:C_0805_2012Metric, F.Cu at (450.3, 93.0)
- added C47: 10uF, Capacitor_SMD:C_0805_2012Metric, F.Cu at (423.5, 136.7)
- added C48: 10uF, Capacitor_SMD:C_0805_2012Metric, F.Cu at (441.4, 93.3)
- added C49: 10uF, Capacitor_SMD:C_0805_2012Metric, F.Cu at (447.1, 90.0)
- added C50: 100nF, Capacitor_SMD:C_0402_1005Metric, F.Cu at (440.6, 107.0)
- added C51: 100nF, Capacitor_SMD:C_0402_1005Metric, F.Cu at (446.4, 105.0)
- added C52: 100uF, Capacitor_SMD:C_1206_3216Metric, F.Cu at (442.0, 90.2)
- added C53: 10uF, Capacitor_SMD:C_0805_2012Metric, F.Cu at (445.9, 93.3)
- added C54: 10uF, Capacitor_SMD:C_0805_2012Metric, F.Cu at (445.9, 96.3)
- added C55: 10uF, Capacitor_SMD:C_0805_2012Metric, F.Cu at (441.4, 99.4)
- added C56: 10uF, Capacitor_SMD:C_0805_2012Metric, F.Cu at (451.5, 90.0)
- added C57: 10uF, Capacitor_SMD:C_0805_2012Metric, F.Cu at (441.4, 96.3)
- added C58: 100nF, Capacitor_SMD:C_0402_1005Metric, F.Cu at (446.4, 103.1)
- added C59: 100nF, Capacitor_SMD:C_0402_1005Metric, F.Cu at (440.6, 105.0)
- added C60: 100nF, Capacitor_SMD:C_0402_1005Metric, F.Cu at (443.5, 105.0)
- added C61: 1000pF 2kV, Capacitor_SMD:C_1206_3216Metric, F.Cu at (498.3, 66.0)
- added C62: 100nF, Capacitor_SMD:C_0402_1005Metric, F.Cu at (443.5, 107.0)
- added C63: 100uF, Capacitor_SMD:C_1206_3216Metric, F.Cu at (498.3, 162.9)
- added C64: 10uF, Capacitor_SMD:C_0805_2012Metric, F.Cu at (445.9, 193.2)
- added C65: 10uF, Capacitor_SMD:C_0805_2012Metric, F.Cu at (441.4, 196.2)
- added C66: 10uF, Capacitor_SMD:C_0805_2012Metric, F.Cu at (450.3, 189.9)
- added C67: 10uF, Capacitor_SMD:C_0805_2012Metric, F.Cu at (441.4, 193.2)
- added C68: 100nF, Capacitor_SMD:C_0402_1005Metric, F.Cu at (446.4, 201.9)
- added C69: 100nF, Capacitor_SMD:C_0402_1005Metric, F.Cu at (446.4, 199.9)
- added C70: 100uF, Capacitor_SMD:C_1206_3216Metric, F.Cu at (442.0, 187.0)
- added C71: 10uF, Capacitor_SMD:C_0805_2012Metric, F.Cu at (423.5, 233.6)
- added C72: 10uF, Capacitor_SMD:C_0805_2012Metric, F.Cu at (445.9, 190.2)
- added C73: 10uF, Capacitor_SMD:C_0805_2012Metric, F.Cu at (451.5, 186.8)
- added C74: 10uF, Capacitor_SMD:C_0805_2012Metric, F.Cu at (441.4, 190.2)
- added C75: 10uF, Capacitor_SMD:C_0805_2012Metric, F.Cu at (447.1, 186.8)
- added C76: 100nF, Capacitor_SMD:C_0402_1005Metric, F.Cu at (443.5, 201.9)
- added C77: 100nF, Capacitor_SMD:C_0402_1005Metric, F.Cu at (440.6, 203.9)
- added C78: 100nF, Capacitor_SMD:C_0402_1005Metric, F.Cu at (443.5, 203.9)
- added C79: 1000pF 2kV, Capacitor_SMD:C_1206_3216Metric, F.Cu at (418.5, 233.7)
- added C80: 100nF, Capacitor_SMD:C_0402_1005Metric, F.Cu at (440.6, 201.9)
- added C81: 100uF, Capacitor_SMD:C_1206_3216Metric, F.Cu at (248.6, 283.9)
- added C82: 10uF, Capacitor_SMD:C_0805_2012Metric, F.Cu at (252.5, 287.1)
- added C83: 10uF, Capacitor_SMD:C_0805_2012Metric, F.Cu at (258.1, 284.8)
- added C84: 10uF, Capacitor_SMD:C_0805_2012Metric, F.Cu at (248.0, 287.1)
- added C85: 10uF, Capacitor_SMD:C_0805_2012Metric, F.Cu at (253.7, 283.7)
- added C86: 100nF, Capacitor_SMD:C_0402_1005Metric, F.Cu at (280.6, 285.2)
- added C87: 100nF, Capacitor_SMD:C_0402_1005Metric, F.Cu at (277.8, 285.2)
- added C88: 100nF, Capacitor_SMD:C_0402_1005Metric, F.Cu at (274.9, 285.2)
- added D12: LED, LED_SMD:LED_0603_1608Metric, F.Cu at (398.0, 246.3)
- added D13: LED, LED_SMD:LED_0603_1608Metric, F.Cu at (458.9, 93.3)
- added D14: LED, LED_SMD:LED_0603_1608Metric, F.Cu at (463.0, 93.3)
- added D15: LED, LED_SMD:LED_0603_1608Metric, F.Cu at (360.8, 268.6)
- added D16: LED, LED_SMD:LED_0603_1608Metric, F.Cu at (366.8, 264.5)
- added D17: LED, LED_SMD:LED_0603_1608Metric, F.Cu at (463.0, 190.2)
- added D18: LED, LED_SMD:LED_0603_1608Metric, F.Cu at (458.9, 190.2)
- added D20: LED, LED_SMD:LED_0603_1608Metric, F.Cu at (398.0, 268.6)
- added D21: LED, LED_SMD:LED_0603_1608Metric, F.Cu at (256.8, 287.6)
- added F1: Polyfuse, Fuse:Fuse_1210_3225Metric_Castellated, F.Cu at (361.7, 242.9)
- added F2: Polyfuse, Fuse:Fuse_1210_3225Metric_Castellated, F.Cu at (485.5, 337.0)
- added F3: Polyfuse, Fuse:Fuse_1210_3225Metric_Castellated, F.Cu at (398.9, 242.9)
- added F4: Polyfuse, Fuse:Fuse_1210_3225Metric_Castellated, F.Cu at (361.7, 265.2)
- added F5: Polyfuse, Fuse:Fuse_1210_3225Metric_Castellated, F.Cu at (398.9, 265.2)
- added FID1: Fiducial, Fiducial:Fiducial_1mm_Mask2mm, F.Cu at (477.4, 328.6)
- added FID2: Fiducial, Fiducial:Fiducial_1mm_Mask2mm, F.Cu at (480.9, 328.6)
- added FID3: Fiducial, Fiducial:Fiducial_1mm_Mask2mm, F.Cu at (484.4, 328.6)
- added IC10: OKR-T_6-W12-C, dg_power:MURATACASEC90, F.Cu at (381.7, 264.6)
- added IC5: OKR-T_6-W12-C, dg_power:MURATACASEC90, F.Cu at (381.7, 251.1)
- added IC6: OKR-T_6-W12-C, dg_power:MURATACASEC90, F.Cu at (381.7, 242.3)
- added IC7: OKR-T_6-W12-C, dg_power:MURATACASEC90, F.Cu at (344.5, 273.4)
- added IC8: OKR-T_6-W12-C, dg_power:MURATACASEC90, F.Cu at (344.5, 264.6)
- added IC9: OKR-T_6-W12-C, dg_power:MURATACASEC90, F.Cu at (381.7, 273.4)
- added J10: Header_2x6_2.54mm, Connector_PinHeader_2.54mm:PinHeader_2x03_P2.54mm_Vertical, F.Cu at (388.1, 248.7)
- added J11: Header_2x6_2.54mm, Connector_PinHeader_2.54mm:PinHeader_2x03_P2.54mm_Vertical, F.Cu at (350.9, 270.9)
- added J12: Header_2x6_2.54mm, Connector_PinHeader_2.54mm:PinHeader_2x03_P2.54mm_Vertical, F.Cu at (388.1, 270.9)
- added J13: 0826-1X1T-GH-F, dg_connectors:BEL_0826-1X1T-GH-F, F.Cu at (312.4, 252.6)
- added J7: Header_2x6_2.54mm, Connector_PinHeader_2.54mm:PinHeader_2x03_P2.54mm_Vertical, F.Cu at (350.9, 248.7)
- added J9: Header_2x6_2.54mm, Connector_PinHeader_2.54mm:PinHeader_2x03_P2.54mm_Vertical, F.Cu at (474.7, 342.8)
- added JP10: SolderJumper_2_Open, Jumper:SolderJumper-2_P1.3mm_Open_RoundedPad1.0x1.5mm, F.Cu at (297.9, 187.1)
- added JP11: SolderJumper_2_Open, Jumper:SolderJumper-2_P1.3mm_Open_RoundedPad1.0x1.5mm, F.Cu at (387.9, 257.8)
- added JP12: SolderJumper_2_Open, Jumper:SolderJumper-2_P1.3mm_Open_RoundedPad1.0x1.5mm, F.Cu at (467.8, 90.3)
- added JP17: SolderJumper_2_Open, Jumper:SolderJumper-2_P1.3mm_Open_RoundedPad1.0x1.5mm, F.Cu at (467.8, 187.1)
- added JP18: SolderJumper_2_Open, Jumper:SolderJumper-2_P1.3mm_Open_RoundedPad1.0x1.5mm, F.Cu at (463.4, 187.1)
- added JP19: SolderJumper_2_Open, Jumper:SolderJumper-2_P1.3mm_Open_RoundedPad1.0x1.5mm, F.Cu at (454.7, 190.1)
- added JP20: SolderJumper_2_Open, Jumper:SolderJumper-2_P1.3mm_Open_RoundedPad1.0x1.5mm, F.Cu at (459.1, 187.1)
- added JP21: SolderJumper_2_Open, Jumper:SolderJumper-2_P1.3mm_Open_RoundedPad1.0x1.5mm, F.Cu at (387.9, 280.1)
- added JP22: SolderJumper_2_Open, Jumper:SolderJumper-2_P1.3mm_Open_RoundedPad1.0x1.5mm, F.Cu at (262.5, 287.5)
- added JP23: SolderJumper_2_Open, Jumper:SolderJumper-2_P1.3mm_Open_RoundedPad1.0x1.5mm, F.Cu at (266.9, 284.0)
- added JP24: SolderJumper_2_Open, Jumper:SolderJumper-2_P1.3mm_Open_RoundedPad1.0x1.5mm, F.Cu at (262.5, 284.0)
- added JP25: SolderJumper_2_Open, Jumper:SolderJumper-2_P1.3mm_Open_RoundedPad1.0x1.5mm, F.Cu at (329.4, 242.7)
- added JP26: SolderJumper_2_Open, Jumper:SolderJumper-2_P1.3mm_Open_RoundedPad1.0x1.5mm, F.Cu at (324.9, 247.2)
- added JP5: SolderJumper_2_Open, Jumper:SolderJumper-2_P1.3mm_Open_RoundedPad1.0x1.5mm, F.Cu at (284.9, 93.3)
- added JP6: SolderJumper_2_Open, Jumper:SolderJumper-2_P1.3mm_Open_RoundedPad1.0x1.5mm, F.Cu at (474.5, 351.9)
- added JP7: SolderJumper_2_Open, Jumper:SolderJumper-2_P1.3mm_Open_RoundedPad1.0x1.5mm, F.Cu at (289.2, 187.1)
- added JP8: SolderJumper_2_Open, Jumper:SolderJumper-2_P1.3mm_Open_RoundedPad1.0x1.5mm, F.Cu at (284.9, 190.1)
- added JP9: SolderJumper_2_Open, Jumper:SolderJumper-2_P1.3mm_Open_RoundedPad1.0x1.5mm, F.Cu at (293.6, 187.1)
- added Q1: 2N7002K, Package_TO_SOT_SMD:SOT-23, F.Cu at (325.0, 243.2)
- added R37: 436, Resistor_SMD:R_0402_1005Metric_Pad0.72x0.64mm_HandSolder, F.Cu at (394.6, 248.6)
- added R38: 1K, Resistor_SMD:R_0402_1005Metric_Pad0.72x0.64mm_HandSolder, F.Cu at (397.8, 248.6)
- added R39: 1k, Resistor_SMD:R_0402_1005Metric, F.Cu at (394.4, 250.6)
- added R40: 1k, Resistor_SMD:R_0402_1005Metric, F.Cu at (394.4, 252.6)
- added R41: 1k, Resistor_SMD:R_0402_1005Metric, F.Cu at (391.6, 257.0)
- added R42: 1k, Resistor_SMD:R_0402_1005Metric, F.Cu at (417.1, 139.5)
- added R43: 75, Resistor_SMD:R_0402_1005Metric, F.Cu at (445.1, 99.1)
- added R44: 75, Resistor_SMD:R_0402_1005Metric, F.Cu at (448.0, 99.1)
- added R45: 75, Resistor_SMD:R_0402_1005Metric, F.Cu at (450.9, 99.1)
- added R46: 75, Resistor_SMD:R_0402_1005Metric, F.Cu at (445.1, 101.1)
- added R47: 470, Resistor_SMD:R_0402_1005Metric, F.Cu at (448.0, 101.1)
- added R48: 470, Resistor_SMD:R_0402_1005Metric, F.Cu at (440.6, 103.1)
- added R49: 470, Resistor_SMD:R_0402_1005Metric, F.Cu at (443.6, 103.1)
- added R50: 268, Resistor_SMD:R_0402_1005Metric_Pad0.72x0.64mm_HandSolder, F.Cu at (357.4, 270.8)
- added R51: 436, Resistor_SMD:R_0402_1005Metric_Pad0.72x0.64mm_HandSolder, F.Cu at (360.6, 270.8)
- added R52: 1K, Resistor_SMD:R_0402_1005Metric_Pad0.72x0.64mm_HandSolder, F.Cu at (364.4, 268.2)
- added R53: 1k, Resistor_SMD:R_0402_1005Metric, F.Cu at (354.3, 279.3)
- added R54: 1k, Resistor_SMD:R_0402_1005Metric, F.Cu at (357.2, 274.8)
- added R55: 1k, Resistor_SMD:R_0402_1005Metric, F.Cu at (357.2, 272.8)
- added R56: 1k, Resistor_SMD:R_0402_1005Metric, F.Cu at (445.1, 195.9)
- added R57: 75, Resistor_SMD:R_0402_1005Metric, F.Cu at (448.0, 195.9)
- added R58: 75, Resistor_SMD:R_0402_1005Metric, F.Cu at (450.9, 195.9)
- added R59: 75, Resistor_SMD:R_0402_1005Metric, F.Cu at (445.1, 197.9)
- added R60: 75, Resistor_SMD:R_0402_1005Metric, F.Cu at (448.0, 197.9)
- added R61: 470, Resistor_SMD:R_0402_1005Metric, F.Cu at (440.6, 199.9)
- added R62: 470, Resistor_SMD:R_0402_1005Metric, F.Cu at (443.6, 199.9)
- added R63: 470, Resistor_SMD:R_0402_1005Metric, F.Cu at (417.1, 236.4)
- added R64: 268, Resistor_SMD:R_0402_1005Metric_Pad0.72x0.64mm_HandSolder, F.Cu at (397.8, 270.8)
- added R65: 436, Resistor_SMD:R_0402_1005Metric_Pad0.72x0.64mm_HandSolder, F.Cu at (401.6, 268.2)
- added R66: 1K, Resistor_SMD:R_0402_1005Metric_Pad0.72x0.64mm_HandSolder, F.Cu at (394.6, 270.8)
- added R67: 1k, Resistor_SMD:R_0402_1005Metric, F.Cu at (391.6, 279.3)
- added R68: 1k, Resistor_SMD:R_0402_1005Metric, F.Cu at (394.4, 274.8)
- added R69: 1k, Resistor_SMD:R_0402_1005Metric, F.Cu at (394.4, 272.8)
- added R70: 1k, Resistor_SMD:R_0402_1005Metric, F.Cu at (328.6, 246.4)
- added R71: 470, Resistor_SMD:R_0402_1005Metric, F.Cu at (266.2, 288.7)
- added R72: 470, Resistor_SMD:R_0402_1005Metric, F.Cu at (274.6, 283.2)
- added R73: 470, Resistor_SMD:R_0402_1005Metric, F.Cu at (269.1, 286.9)
- added R74: DNP, Resistor_SMD:R_0402_1005Metric, F.Cu at (324.2, 250.0)
- added R75: 1k, Resistor_SMD:R_0402_1005Metric, F.Cu at (266.2, 286.8)
- added R76: 7.2K, Resistor_SMD:R_0402_1005Metric, F.Cu at (272.0, 286.9)
- added R77: 5K, Resistor_SMD:R_0402_1005Metric, F.Cu at (277.5, 283.2)
- added R78: 1k, Resistor_SMD:R_0402_1005Metric, F.Cu at (280.4, 283.2)
- added R79: 0, Resistor_SMD:R_0402_1005Metric, F.Cu at (283.3, 283.2)
- added R80: 1k, Resistor_SMD:R_0402_1005Metric, F.Cu at (286.2, 283.2)
- added R81: 0, Resistor_SMD:R_0402_1005Metric, F.Cu at (289.1, 283.2)
- added RLA3: G3VM-61VY2-TR, dg_relay:G3VM-SOP, F.Cu at (391.1, 243.6)
- added RLA4: G3VM-61VY2-TR, dg_relay:G3VM-SOP, F.Cu at (353.9, 265.9)
- added RLA5: G3VM-61VY2-TR, dg_relay:G3VM-SOP, F.Cu at (391.1, 265.9)
- added T2: QT24A01, dg_transformers:SOP100P1000X450-24N, F.Cu at (332.1, 152.6)
- added T3: QT24A01, dg_transformers:SOP100P1000X450-24N, F.Cu at (501.9, 55.8)
- added T4: QT24A01, dg_transformers:SOP100P1000X450-24N, F.Cu at (501.9, 152.6)
- added TP1: TestPoint, TestPoint:TestPoint_Pad_D1.0mm, F.Cu at (282.8, 96.6)
- added TP10: TestPoint, TestPoint:TestPoint_Pad_D1.0mm, F.Cu at (458.4, 193.0)
- added TP11: TestPoint, TestPoint:TestPoint_Pad_D1.0mm, F.Cu at (449.6, 193.4)
- added TP2: TestPoint, TestPoint:TestPoint_Pad_D1.0mm, F.Cu at (279.8, 96.6)
- added TP3: TestPoint, TestPoint:TestPoint_Pad_D1.0mm, F.Cu at (288.6, 96.2)
- added TP4: TestPoint, TestPoint:TestPoint_Pad_D1.0mm, F.Cu at (279.8, 193.4)
- added TP5: TestPoint, TestPoint:TestPoint_Pad_D1.0mm, F.Cu at (282.8, 193.4)
- added TP8: TestPoint, TestPoint:TestPoint_Pad_D1.0mm, F.Cu at (458.4, 96.2)
- added TP9: TestPoint, TestPoint:TestPoint_Pad_D1.0mm, F.Cu at (449.6, 96.6)
- added U10: rpi_cm4, dg_rpi:rpi_cm4, F.Cu at (246.6, 281.5)
- added U5: m.2_pcie_nvme, dg_connectors:m.2_pcie_nvme, F.Cu at (257.6, 150.8)
- added U7: m.2_pcie_nvme, dg_connectors:m.2_pcie_nvme, F.Cu at (427.4, 54.0)
- added U8: rpi_cm4, dg_rpi:rpi_cm4, F.Cu at (439.9, 184.6)
- added U9: m.2_pcie_nvme, dg_connectors:m.2_pcie_nvme, F.Cu at (427.4, 150.8)
- added Y1: 24Mhz X1E0000210264, Crystal:Crystal_SMD_SeikoEpson_TSX3225-4Pin_3.2x2.5mm, F.Cu at (256.7, 295.0)
- C1: value C -> 100uF; footprint Capacitor_SMD:C_0805_2012Metric -> Capacitor_SMD:C_1206_3216Metric
- C10, C12: value 100nF -> 10uF; footprint Capacitor_SMD:C_0402_1005Metric -> Capacitor_SMD:C_0805_2012Metric
- C13, C4: value 100uF -> 10uF; footprint Capacitor_SMD:C_1206_3216Metric -> Capacitor_SMD:C_0805_2012Metric
- C14, C20, C21, C6: value 10uF -> 100nF; footprint Capacitor_SMD:C_0805_2012Metric -> Capacitor_SMD:C_0402_1005Metric
- C15, C16: value 14pF -> 100nF; footprint Capacitor_SMD:C_0603_1608Metric -> Capacitor_SMD:C_0402_1005Metric
- C17: value 10uF -> 1000pF 2kV; footprint Capacitor_SMD:C_0805_2012Metric -> Capacitor_SMD:C_1206_3216Metric
- C18: value 10uF -> 100nF; footprint Capacitor_SMD:C_0603_1608Metric -> Capacitor_SMD:C_0402_1005Metric
- C2: value C -> 10uF; footprint Capacitor_SMD:C_0603_1608Metric -> Capacitor_SMD:C_0805_2012Metric
- C22, C23: value 100nF -> 14pF
- C25: value 1000pF 2kV -> 100nF; footprint Capacitor_SMD:C_1206_3216Metric -> Capacitor_SMD:C_0402_1005Metric
- C3: value 100nF -> 10uF; footprint Capacitor_SMD:C_0603_1608Metric -> Capacitor_SMD:C_0805_2012Metric
- C7: value 0.1uF -> 100nF; footprint Capacitor_SMD:C_0603_1608Metric -> Capacitor_SMD:C_0402_1005Metric
- C8: value 0.1uF -> 100uF; footprint Capacitor_SMD:C_0603_1608Metric -> Capacitor_SMD:C_1206_3216Metric
- D2: value LED -> D_TVS; footprint LED_SMD:LED_0603_1608Metric -> Diode_SMD:D_SMA
- D7: value D_TVS -> LED; footprint Diode_SMD:D_SMA -> LED_SMD:LED_0603_1608Metric
- J1: value Conn_02x04_Odd_Even -> SS-74500-020; footprint Connector_Molex:Molex_Mini-Fit_Jr_5569-08A2_2x04_P4.20mm_Horizontal -> dg_connectors:BEL_SS-74500-020
- J6: value 0826-1X1T-GH-F -> Conn_02x04_Odd_Even; footprint dg_connectors:BEL_0826-1X1T-GH-F -> Connector_Molex:Molex_Mini-Fit_Jr_5569-08A2_2x04_P4.20mm_Horizontal
- R10, R11, R8: value R -> 75; footprint Resistor_SMD:R_0603_1608Metric -> Resistor_SMD:R_0402_1005Metric
- R12: value R -> 470; footprint Resistor_SMD:R_0603_1608Metric -> Resistor_SMD:R_0402_1005Metric
- R13: value 1K -> 470; footprint Resistor_SMD:R_0402_1005Metric_Pad0.72x0.64mm_HandSolder -> Resistor_SMD:R_0402_1005Metric
- R14: value 268 -> 470; footprint Resistor_SMD:R_0402_1005Metric_Pad0.72x0.64mm_HandSolder -> Resistor_SMD:R_0402_1005Metric
- R15, R18, R21: value 1k -> 10k
- R16: value 10K -> 10k; footprint Resistor_SMD:R_0603_1608Metric -> Resistor_SMD:R_0402_1005Metric
- R17: value 10K -> 12k %1; footprint Resistor_SMD:R_0603_1608Metric -> Resistor_SMD:R_0402_1005Metric
- R19: value DNC -> 10k
- R20: value 436 -> 10k; footprint Resistor_SMD:R_0402_1005Metric_Pad0.72x0.64mm_HandSolder -> Resistor_SMD:R_0402_1005Metric
- R22, R36: value 1k -> 268; footprint Resistor_SMD:R_0402_1005Metric -> Resistor_SMD:R_0402_1005Metric_Pad0.72x0.64mm_HandSolder
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Connections:
- C1 pad 1: /mgm/5V -> /dcdc/5V
- C10 pad 1: /dcdc/5V -> /dcdc/3V3
- C11 pad 1: /dcdc/5V -> /dcdc/3V3
- C12 pad 1: /dcdc/5V -> /dcdc/3V3
- C15 pad 1: GND -> /dcdc/3V3
- C15 pad 2: Net-(C15-Pad2) -> GND
- C16 pad 1: GND -> /dcdc/3V3
- C16 pad 2: Net-(C16-Pad2) -> GND
- C17 pad 1: /dcdc/3V3 -> GND
- C17 pad 2: GND -> Net-(C17-Pad2)
- C18 pad 1: /usbhub/3.3V -> Net-(C18-Pad1)
- C19 pad 1: /dcdc/3V3 -> /3V3_MGMT
- C2 pad 1: /mgm/5V -> /dcdc/5V
- C20 pad 1: /dcdc/3V3 -> /3V3_MGMT
- C21 pad 1: /dcdc/3V3 -> /3V3_MGMT
- C22 pad 1: /dcdc/3V3 -> /usbhub/XTALIN
- C23 pad 1: /dcdc/3V3 -> /usbhub/XTALOUT
- C24 pad 1: /dcdc/3V3 -> Net-(C24-Pad1)
- C25 pad 1: GND -> Net-(C25-Pad1)
- C25 pad 2: Net-(C25-Pad2) -> GND
- C26 pad 1: Net-(C26-Pad1) -> /usbhub/USB_Hub_RSTn
- C3 pad 1: +3V3 -> /dcdc/5V
- C7 pad 1: GND -> /dcdc/5V
- C7 pad 2: Net-(C7-Pad2) -> GND
- C8 pad 1: GND -> /dcdc/3V3
- C8 pad 2: Net-(C8-Pad2) -> GND
- C9 pad 1: /dcdc/5V -> /dcdc/3V3
- D10 pad 2: /mgm/5V -> /sheet6142DC77/pi3V3
- D11 pad 2: /sheet61DCBD00/3V3 -> /sheet6143BBAB/5V
- D19 pad 2: /pi/pi3V3 -> /mgm/5V
- D2 pad 1: Net-(D2-Pad1) -> +12V
- D2 pad 2: /mgm/pi3.3 -> GND
- D22 pad 1: GND -> Net-(D22-Pad1)
- D22 pad 2: Net-(D22-Pad2) -> /mgm/pi3V3
- D3 pad 2: /mgm/5V -> /dcdc/5V
- D4 pad 1: GND -> Net-(D4-Pad1)
- D4 pad 2: Net-(D4-Pad2) -> /dcdc/3V3
- D5 pad 1: GND -> Net-(D5-Pad1)
- D5 pad 2: Net-(D5-Pad2) -> /pi/pi3V3
- D6 pad 1: GND -> Net-(D6-Pad1)
- D6 pad 2: Net-(D6-Pad2) -> /pi/pi3V3
- D7 pad 1: +12V -> Net-(D7-Pad1)
- D7 pad 2: GND -> /sheet6142DC76/5V
- D8 pad 2: /dcdc/5V -> /sheet6142DC76/3V3
- D9 pad 2: /dcdc/3V3 -> /sheet6142DC77/pi3V3
- IC3 pad 1: /sheet61DCBD00/DISABLE_DCDC -> /sheet6142DC76/DISABLE_DCDC
- IC3 pad 2: /sheet61DCBD00/VIN_DCDC_5V -> /sheet6142DC76/VIN_DCDC_5V
- IC3 pad 4: /mgm/5V -> /sheet6142DC76/5V
- IC4 pad 1: /sheet61DCBD00/DISABLE_DCDC -> /sheet6142DC76/DISABLE_DCDC
- IC4 pad 2: /sheet61DCBD00/VIN_DCDC_3V3 -> /sheet6142DC76/VIN_DCDC_3V3
- IC4 pad 4: /sheet61DCBD00/3V3 -> /sheet6142DC76/3V3
- J6 pad 1: (no net) -> GND
- J6 pad 2: (no net) -> GND
- J6 pad 3: (no net) -> GND
- J6 pad 4: (no net) -> GND
- J6 pad 5: (no net) -> +12V
- J6 pad 6: (no net) -> +12V
- J6 pad 7: (no net) -> +12V
- J6 pad 8: (no net) -> +12V
- JP1 pad 1: GND -> /c1_disable
- JP1 pad 2: Net-(JP1-Pad2) -> /dcdc/DISABLE_DCDC
- JP16 pad 1: GND -> /c4_disable
- JP16 pad 2: Net-(JP16-Pad2) -> /sheet6144BA66/DISABLE_DCDC
- M1 pad 4: Net-(M1-Pad4) -> /mgm/fan_pwm_in
- M2 pad 4: (no net) -> /mgm/fan_pwm_in
- R10 pad 2: Net-(D4-Pad2) -> Net-(C17-Pad2)
- R11 pad 2: Net-(D5-Pad2) -> Net-(C17-Pad2)
- R12 pad 1: Net-(R12-Pad1) -> Net-(D6-Pad1)
- R12 pad 2: Net-(D6-Pad2) -> Net-(R12-Pad2)
- R13 pad 1: /sheet61DCBD00/DISABLE -> /pi/eth_speed_ledy
- R14 pad 1: GND -> /pi/eth_act_ledg
- R14 pad 2: Net-(IC3-Pad5) -> Net-(R14-Pad2)
- R15 pad 1: Net-(D9-Pad1) -> /3V3_MGMT
- R15 pad 2: GND -> /usbhub/USB_Hub_RSTn
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Routing:
- removed copper zone on In3.Cu, net +12V
- removed copper zone on In1.Cu, net GND
- removed copper zone on In4.Cu, net GND
Other:
- outline, holes or cut-outs redrawn

Commit message: Completed PCB Placement.
Parts:
- removed C31, C49, C5, C67, C85: 10uF, Capacitor_SMD:C_0805_2012Metric
- removed C33, C51, C69, C7, C87: 100nF, Capacitor_SMD:C_0402_1005Metric
- removed JP21: SolderJumper_2_Open, Jumper:SolderJumper-2_P1.3mm_Open_RoundedPad1.0x1.5mm
- removed R66: 1K, Resistor_SMD:R_0402_1005Metric_Pad0.72x0.64mm_HandSolder
- removed RLA5: G3VM-61VY2-TR, dg_relay:G3VM-SOP
- moved J6 454.3 mm to (151.9, 30.5)
- moved T3 450.6 mm to (101.5, 262.5), turned to 270 degrees
- moved C61 448.2 mm to (100.1, 271.7)
- moved D2 439.0 mm to (147.0, 33.5), turned to 90 degrees
- moved T4 438.5 mm to (101.5, 331.5), turned to 270 degrees
- moved J5 410.8 mm to (152.0, 359.5), turned to 180 degrees
- moved C63 401.2 mm to (132.6, 327.9), turned to 270 degrees
- moved U6 389.1 mm to (89.4, 256.5)
- moved R43 388.3 mm to (98.9, 275.0)
- moved R45 388.3 mm to (104.7, 275.0)
- moved R46 388.3 mm to (98.9, 277.0)
- moved R44 388.3 mm to (101.8, 275.0)
- moved D8 385.6 mm to (149.0, 157.3), turned to 90 degrees
- moved R23 384.3 mm to (153.0, 152.0)
- moved C62 382.9 mm to (92.4, 259.7), turned to 180 degrees
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Connections:
- U1 pad 24: /c3_boot -> (no net)
- U1 pad 25: /c2_disable -> (no net)
- U1 pad 26: Net-(U1-Pad26) -> (no net)
- U1 pad 27: /c1_disable -> (no net)
- U1 pad 28: /c4_rx -> (no net)
- U1 pad 29: /mgm/tach1 -> (no net)
- U1 pad 30: Net-(U1-Pad30) -> (no net)
- U1 pad 31: /c4_tx -> (no net)
- U1 pad 34: /c2_rx -> (no net)
- U1 pad 37: Net-(U1-Pad37) -> (no net)
- U1 pad 38: Net-(U1-Pad38) -> (no net)
- U1 pad 39: /c3_tx -> (no net)
- U1 pad 40: /c3_rx -> (no net)
- U1 pad 41: /c2_boot -> (no net)
- U1 pad 44: Net-(U1-Pad44) -> (no net)
- U1 pad 45: /c1_boot -> (no net)
- U1 pad 46: /c3_disable -> (no net)
- U1 pad 47: /c4_disable -> (no net)
- U1 pad 48: /c4_boot -> (no net)
- U1 pad 49: /mgm/fanpwm -> (no net)
- U1 pad 50: /mgm/tach2 -> (no net)
- U1 pad 54: /c2_tx -> (no net)
- U1 pad 56: Net-(U1-Pad56) -> (no net)
- U1 pad 58: Net-(U1-Pad58) -> (no net)
- U10 pad 24: (no net) -> /c3_boot
- U10 pad 25: (no net) -> /c2_disable
- U10 pad 26: (no net) -> Net-(U10-Pad26)
- U10 pad 27: (no net) -> /c1_disable
- U10 pad 28: (no net) -> /c4_rx
- U10 pad 29: (no net) -> /mgm/tach1
- U10 pad 30: (no net) -> Net-(U10-Pad30)
- U10 pad 31: (no net) -> /c4_tx
- U10 pad 34: (no net) -> /c2_rx
- U10 pad 37: (no net) -> Net-(U10-Pad37)
- U10 pad 38: (no net) -> Net-(U10-Pad38)
- U10 pad 39: (no net) -> /c3_tx
- U10 pad 40: (no net) -> /c3_rx
- U10 pad 41: (no net) -> /c2_boot
- U10 pad 44: (no net) -> Net-(U10-Pad44)
- U10 pad 45: (no net) -> /c1_boot
- U10 pad 46: (no net) -> /c3_disable
- U10 pad 47: (no net) -> /c4_disable
- U10 pad 48: (no net) -> /c4_boot
- U10 pad 49: (no net) -> /mgm/fanpwm
- U10 pad 50: (no net) -> /mgm/tach2
- U10 pad 54: (no net) -> /c2_tx
- U10 pad 56: (no net) -> Net-(U10-Pad56)
- U10 pad 58: (no net) -> Net-(U10-Pad58)
Routing:
- net /sheet6144BA67/RPI_PCIe_TX_P: track 0.00 -> 22.0 mm
- net /sheet6144BA67/RPI_PCIe_CLK_P: track 0.00 -> 21.4 mm
- net /sheet6144BA67/RPI_PCIe_CLK_N: track 0.00 -> 21.0 mm
- net /sheet6144BA67/RPI_PCIe_TX_N: track 0.00 -> 20.7 mm
- net /sheet6144BA67/TD4_N: track 0.00 -> 18.5 mm
- net /sheet6144BA67/TD4_P: track 0.00 -> 17.6 mm
- net /sheet6144BA67/RPI_PCIe_RX_P: track 0.00 -> 17.5 mm
- net /sheet6144BA67/RPI_PCIe_RX_N: track 0.00 -> 17.0 mm
- net /sheet6144BA67/TD3_N: track 0.00 -> 15.8 mm
- net /sheet6144BA67/TD3_P: track 0.00 -> 15.8 mm
Other:
- board size 80 x 350 mm -> 120 x 350 mm
- net class Default: clearance 0.2 -> 0.11; trace_width 0.25 -> 0.11; via_dia 0.8 -> 0.5; via_drill 0.4 -> 0.2
- rule trace_clearance: 0.2 -> 0.11
- rule trace_min: 0.2 -> 0.11
- rule via_min_drill: 0.3 -> 0.2
- rule via_min_size: 0.4 -> 0.5
