File: currypi.kicad_pcb (KiCad board)
At the start: 6 copper layers, 120 x 350 mm, 272 parts, among them IC1 OKR-T_6-W12-C, IC10 OKR-T_6-W12-C, IC2 OKR-T_6-W12-C, IC3 OKR-T_6-W12-C, IC4 OKR-T_6-W12-C, IC5 OKR-T_6-W12-C, IC6 OKR-T_6-W12-C, IC7 OKR-T_6-W12-C, IC8 OKR-T_6-W12-C, IC9 OKR-T_6-W12-C, J1 SS-74500-020, J10 Header_2x6_2.54mm, J11 Header_2x6_2.54mm, J12 Header_2x6_2.54mm, J13 0826-1X1T-GH-F, J5 Conn_02x04_Odd_Even, J6 Conn_02x04_Odd_Even, J7 Header_2x6_2.54mm, J9 Header_2x6_2.54mm, M1 Fan_4pin, M2 Fan_4pin, Q1 2N7002K, T1 QT24A01, T2 QT24A01, T3 QT24A01, T4 QT24A01, U1 rpi_cm4, U10 rpi_cm4, U2 m.2_pcie_nvme, U3 USB2514B_Bi, U4 rpi_cm4, U5 m.2_pcie_nvme, U6 rpi_cm4, U7 m.2_pcie_nvme, U8 rpi_cm4, U9 m.2_pcie_nvme, Y1 24Mhz X1E0000210264

Commit message: Fixed fan pwm connection.
Parts:
- moved C43 18.1 mm to (85.0, 196.1)
- moved R30 18.1 mm to (88.3, 193.2)
- moved R29 18.1 mm to (85.1, 192.7)
- moved R31 18.1 mm to (88.0, 190.8)
- moved R32 18.1 mm to (85.1, 190.8)
- moved R43 16.4 mm to (84.7, 266.7)
- moved R44 16.4 mm to (87.6, 266.7)
- moved R45 16.4 mm to (90.5, 266.7)
- moved R46 16.4 mm to (84.7, 268.7)
- moved C61 16.4 mm to (85.9, 263.4)
- moved R59 15.6 mm to (86.1, 335.1)
- moved C79 15.6 mm to (82.7, 334.1)
- moved R57 15.6 mm to (89.0, 333.1)
- moved R58 15.6 mm to (91.9, 333.1)
- moved R60 15.6 mm to (89.0, 335.1)
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Connections:
- R76 pad 2: Net-(R76-Pad2) -> /mgm/fan_pwm_in
- R77 pad 1: Net-(R76-Pad2) -> /mgm/fan_pwm_in
Routing:
- net /mgm/ETH0+: track 0.00 -> 57.7 mm
- net /mgm/ETH0-: track 0.00 -> 56.4 mm
- net /mgm/ETH1-: track 0.00 -> 55.9 mm
- net /mgm/ETH1+: track 0.00 -> 54.6 mm
- net /mgm/ETH2+: track 0.00 -> 53.0 mm
- net /mgm/ETH2-: track 0.00 -> 51.7 mm
- net /mgm/ETH3-: track 0.00 -> 45.5 mm
- net /mgm/ETH3+: track 0.00 -> 44.2 mm
- net /pi/TD4_N: track 0.00 -> 20.4 mm
- net /pi/TD3_P: track 0.00 -> 19.8 mm
- net /pi/TD3_N: track 0.00 -> 19.8 mm
- net /pi/TD4_P: track 0.00 -> 19.5 mm
- net /pi/TD1_N: track 0.00 -> 17.2 mm
- net /pi/TD1_P: track 0.00 -> 17.2 mm
- net /pi/TD2_N: track 0.00 -> 15.4 mm
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
Commit message: Started Routing.
Parts:
- moved JP25 291.2 mm to (195.5, 328.5), turned to 180 degrees
- moved R75 19.2 mm to (191.5, 49.2), turned to 180 degrees
- moved D1 18.1 mm to (156.5, 357.0), turned to 270 degrees
- moved M2 17.4 mm to (195.6, 42.0), turned to 90 degrees
- moved R78 16.4 mm to (197.5, 46.5), turned to 90 degrees
- moved R79 14.7 mm to (196.5, 46.5), turned to 90 degrees
- moved R80 13.7 mm to (194.5, 46.5), turned to 90 degrees
- moved R81 13.5 mm to (195.5, 46.5), turned to 90 degrees
- moved R76 13.4 mm to (190.5, 44.5), turned to 0 degrees
- moved R77 13.3 mm to (192.5, 44.5), turned to 0 degrees
- moved Q1 13.3 mm to (192.0, 47.0), turned to 90 degrees
- moved M1 11.5 mm to (195.6, 29.9), turned to 90 degrees
- moved R74 8.35 mm to (189.7, 46.6), turned to 90 degrees
- moved JP26 7.73 mm to (190.0, 42.0), turned to 270 degrees
- moved D2 0.71 mm to (147.5, 33.0)
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Routing:
- net /mgm/fan_pwm_in: track 0.00 -> 46.4 mm
- net Net-(M1-Pad3): track 0.00 -> 24.8 mm
- net Net-(M2-Pad3): track 0.00 -> 12.5 mm
- net /mgm/pi3V3: track 0.00 -> 8.41 mm
- net /mgm/tach2: track 0.00 -> 5.41 mm
- net /mgm/tach1: track 0.00 -> 5.20 mm
- net /mgm/fanpwm: track 0.00 -> 4.19 mm
- net Net-(JP26-Pad2): track 0.00 -> 1.85 mm
- net +12V: track 0.00 -> 1.85 mm, vias 0 -> 1
- net Net-(Q1-Pad1): track 0.00 -> 1.22 mm
- added copper zone on F.Cu, net +12V
- added copper zone on F.Cu, net GND
Other:
- rule via_min_size: 0.5 -> 0.4

Commit message: Created Net Groups.
Routing:
- net /sheet6144BA67/TD4_N: track 18.5 -> 0.00 mm
- net /sheet6144BA67/TD4_P: track 17.6 -> 0.00 mm
- net /sheet6144BA67/TD3_N: track 15.8 -> 0.00 mm
- net /sheet6144BA67/TD3_P: track 15.8 -> 0.00 mm
- net /sheet6143BBAC/TD3_N: track 0.00 -> 1.80 mm
- net /sheet6143BBAC/TD3_P: track 0.00 -> 1.69 mm
Other:
- net class mgm_eth added: clearance 0.11, trace_width 0.11, via_dia 0.5, via_drill 0.2
- net class usb added: clearance 0.11, trace_width 0.11, via_dia 0.5, via_drill 0.2
Changed lines of the file:
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@@
     (thickness 1.6)
     (drawings 8)
-    (tracks 358)
+    (tracks 324)
     (zones 0)
     (modules 272)
@@
     (add_net /c1_rx)
     (add_net /c1_tx)
-    (add_net /c1_usb+)
-    (add_net /c1_usb-)
     (add_net /c2_boot)
     (add_net /c2_disable)
     (add_net /c2_rx)
     (add_net /c2_tx)
-    (add_net /c2_usb+)
-    (add_net /c2_usb-)
     (add_net /c3_boot)
     (add_net /c3_disable)
     (add_net /c3_rx)
     (add_net /c3_tx)
-    (add_net /c3_usb+)
-    (add_net /c3_usb-)
     (add_net /c4_boot)
     (add_net /c4_disable)
     (add_net /c4_rx)
     (add_net /c4_tx)
-    (add_net /c4_usb+)
-    (add_net /c4_usb-)
     (add_net /dcdc/3V3)
     (add_net /dcdc/5V)
@@
     (add_net /dcdc/VIN_DCDC_5V)
     (add_net /mgm/5V)
-    (add_net /mgm/ETH0+)
-    (add_net /mgm/ETH0-)
-    (add_net /mgm/ETH1+)
-    (add_net /mgm/ETH1-)
-    (add_net /mgm/ETH2+)
-    (add_net /mgm/ETH2-)
-    (add_net /mgm/ETH3+)
-    (add_net /mgm/ETH3-)
-    (add_net /mgm/USB+)
-    (add_net /mgm/USB-)
     (add_net /mgm/eth_act_ledg)
     (add_net /mgm/eth_speed_ledy)
@@
     (add_net "Net-(U9-Pad8)")
   )
+  (net_class mgm_eth ""
+    (clearance 0.11)
+    (trace_width 0.11)
+    (via_dia 0.5)
+    (via_drill 0.2)
+    (uvia_dia 0.3)
+    (uvia_drill 0.1)
+    (diff_pair_width 0.11)
+    (diff_pair_gap 0.15)
+    (add_net /mgm/ETH0+)
+    (add_net /mgm/ETH0-)
+    (add_net /mgm/ETH1+)
+    (add_net /mgm/ETH1-)
+    (add_net /mgm/ETH2+)
+    (add_net /mgm/ETH2-)
+    (add_net /mgm/ETH3+)
+    (add_net /mgm/ETH3-)
+  )
+  (net_class usb ""
+    (clearance 0.11)
+    (trace_width 0.11)
+    (via_dia 0.5)
+    (via_drill 0.2)
+    (uvia_dia 0.3)
+    (uvia_drill 0.1)
+    (diff_pair_width 0.11)
+    (diff_pair_gap 0.15)
+    (add_net /c1_usb+)
+    (add_net /c1_usb-)
+    (add_net /c2_usb+)
+    (add_net /c2_usb-)
+    (add_net /c3_usb+)
+    (add_net /c3_usb-)
+    (add_net /c4_usb+)
+    (add_net /c4_usb-)
+    (add_net /mgm/USB+)
+    (add_net /mgm/USB-)
+  )
   (module dg_rpi:rpi_cm4 (layer F.Cu)
     (at 158.5 312.5 270)
@@
   (segment (start 97 119.1245) (end 97 118.412) (width 0.11) (layer F.Cu) (net 216))
   (segment (start 97.37 119.4945) (end 97 119.1245) (width 0.11) (layer F.Cu) (net 216))
-  (segment (start 99.63 324.985749) (end 99.63 324.553848) (width 0.11) (layer F.Cu) (net 237))
-  (segment (start 100 325.355749) (end 99.63 324.985749) (width 0.11) (layer F.Cu) (net 237))
-  (segment (start 100 326.912) (end 100 325.355749) (width 0.11) (layer F.Cu) (net 237))
-  (segment (start 99.63 324.553848) (end 100.153848 324.03) (width 0.11) (layer F.Cu) (net 237))
-  (segment (start 100.153848 324.03) (end 107.346152 324.03) (width 0.11) (layer F.Cu) (net 237))
-  (segment (start 107.346152 324.03) (end 108.246152 324.93) (width 0.11) (layer F.Cu) (net 237))
-  (segment (start 108.246152 324.93) (end 111.19885 324.93) (width 0.11) (layer F.Cu) (net 237))
-  (segment (start 111.61 324.25) (end 111.61 324) (width 0.11) (layer F.Cu) (net 237))
-  (segment (start 111.54 324.32) (end 111.61 324.25) (width 0.11) (layer F.Cu) (net 237))
-  (segment (start 111.54 324.58885) (end 111.54 324.32) (width 0.11) (layer F.Cu) (net 237))
-  (segment (start 111.19885 324.93) (end 111.54 324.58885) (width 0.11) (layer F.Cu) (net 237))
-  (segment (start 99.37 324.985749) (end 99.37 324.446152) (width 0.11) (layer F.Cu) (net 238))
-  (segment (start 99 325.355749) (end 99.37 324.985749) (width 0.11) (layer F.Cu) (net 238))
-  (segment (start 99 326.912) (end 99 325.355749) (width 0.11) (layer F.Cu) (net 238))
-  (segment (start 99.37 324.446152) (end 100.046152 323.77) (width 0.11) (layer F.Cu) (net 238))
-  (segment (start 100.046152 323.77) (end 107.453848 323.77) (width 0.11) (layer F.Cu) (net 238))
-  (segment (start 107.453848 323.77) (end 108.353848 324.67) (width 0.11) (layer F.Cu) (net 238))
-  (segment (start 108.353848 324.67) (end 111.091154 324.67) (width 0.11) (layer F.Cu) (net 238))
-  (segment (start 111.28 324.481154) (end 111.28 324.32) (width 0.11) (layer F.Cu) (net 238))
-  (segment (start 111.21 324.25) (end 111.21 324) (width 0.11) (layer F.Cu) (net 238))
-  (segment (start 111.091154 324.67) (end 111.28 324.481154) (width 0.11) (layer F.Cu) (net 238))
-  (segment (start 111.28 324.32) (end 111.21 324.25) (width 0.11) (layer F.Cu) (net 238))
-  (segment (start 110.01 324) (end 110.01 323.474999) (width 0.11) (layer F.Cu) (net 239))
-  (segment (start 96.63 324.653848) (end 96.63 324.985749) (width 0.11) (layer F.Cu) (net 239))
-  (segment (start 110.08 323.404999) (end 110.08 323.063848) (width 0.11) (layer F.Cu) (net 239))
-  (segment (start 110.08 323.063848) (end 109.946152 322.93) (width 0.11) (layer F.Cu) (net 239))
-  (segment (start 110.01 323.474999) (end 110.08 323.404999) (width 0.11) (layer F.Cu) (net 239))
-  (segment (start 109.946152 322.93) (end 98.353848 322.93) (width 0.11) (layer F.Cu) (net 239))
-  (segment (start 98.353848 322.93) (end 96.63 324.653848) (width 0.11) (layer F.Cu) (net 239))
-  (segment (start 96.63 324.985749) (end 97 325.355749) (width 0.11) (layer F.Cu) (net 239))
-  (segment (start 97 325.355749) (end 97 326.912) (width 0.11) (layer F.Cu) (net 239))
-  (segment (start 96 325.355749) (end 96 326.912) (width 0.11) (layer F.Cu) (net 240))
-  (segment (start 96.37 324.985749) (end 96 325.355749) (width 0.11) (layer F.Cu) (net 240))
-  (segment (start 96.37 324.546152) (end 96.37 324.985749) (width 0.11) (layer F.Cu) (net 240))
-  (segment (start 98.246152 322.67) (end 96.37 324.546152) (width 0.11) (layer F.Cu) (net 240))
-  (segment (start 110.053848 322.67) (end 98.246152 322.67) (width 0.11) (layer F.Cu) (net 240))
-  (segment (start 110.34 323.404999) (end 110.34 322.956152) (width 0.11) (layer F.Cu) (net 240))
-  (segment (start 110.41 324) (end 110.41 323.474999) (width 0.11) (layer F.Cu) (net 240))
-  (segment (start 110.34 322.956152) (end 110.053848 322.67) (width 0.11) (layer F.Cu) (net 240))
-  (segment (start 110.41 323.474999) (end 110.34 323.404999) (width 0.11) (layer F.Cu) (net 240))
+  (segment (start 101 258.6245) (end 100.63 258.9945) (width 0.11) (layer F.Cu) (net 229))
+  (segment (start 101 257.912) (end 101 258.6245) (width 0.11) (layer F.Cu) (net 229))
+  (segment (start 100.63 258.9945) (end 100.63 259.446152) (width 0.11) (layer F.Cu) (net 229))
+  (segment (start 100 257.912) (end 100 258.6245) (width 0.11) (layer F.Cu) (net 230))
+  (segment (start 100 258.6245) (end 100.37 258.9945) (width 0.11) (layer F.Cu) (net 230))
+  (segment (start 100.37 258.9945) (end 100.37 259.553848) (width 0.11) (layer F.Cu) (net 230))
   (segment (start 111.28 286.63) (end 111.28 286.463848) (width 0.11) (layer F.Cu) (net 529))
   (segment (start 111.21 286.7) (end 111.28 286.63) (width 0.11) (layer F.Cu) (net 529))

Commit message: Added 3th Fan Connector.
Parts:
- added M3: Fan_4pin, Connector:FanPinHeader_1x04_P2.54mm_Vertical, F.Cu at (113.0, 25.0)
- added R82: 1k, Resistor_SMD:R_0402_1005Metric, F.Cu at (116.5, 27.0)
- added R83: 0, Resistor_SMD:R_0402_1005Metric, F.Cu at (116.5, 26.0)
- moved M1 105.7 mm to (90.0, 25.0), turned to 180 degrees
- moved M2 95.6 mm to (101.5, 25.0), turned to 180 degrees
- moved R78 84.6 mm to (116.5, 22.0), turned to 180 degrees
- moved R79 83.4 mm to (116.5, 23.0), turned to 180 degrees
- moved R81 82.1 mm to (116.5, 24.0), turned to 180 degrees
- moved R80 80.9 mm to (116.5, 25.0), turned to 180 degrees
- moved R77 75.9 mm to (117.8, 31.2), turned to 90 degrees
- moved R76 74.9 mm to (116.8, 31.2), turned to 270 degrees
- moved JP26 74.9 mm to (116.2, 29.0), turned to 0 degrees
- moved Q1 74.1 mm to (120.0, 29.5), turned to 180 degrees
- moved R75 71.9 mm to (122.2, 30.0), turned to 270 degrees
- moved R74 71.7 mm to (119.5, 31.8), turned to 180 degrees
- moved D11 8.54 mm to (146.0, 236.5)
- moved D12 8.54 mm to (146.0, 219.5)
- moved D15 8.54 mm to (146.0, 305.5)
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Connections:
- U10 pad 26: Net-(U10-Pad26) -> /mgm/tach3
Routing:
- net Net-(M3-Pad3): track 0.00 -> 11.5 mm
- net Net-(M2-Pad3): track 12.5 -> 22.0 mm
- net Net-(M1-Pad3): track 24.8 -> 33.5 mm
- net +12V: track 1.85 -> 8.09 mm, vias 1 -> 0
- net /mgm/fan_pwm_in: track 46.4 -> 49.8 mm
- net /mgm/pi3V3: track 8.41 -> 10.9 mm

Commit message: Completed PCIE and Eth. Routing.
Parts:
- moved TP4 13.9 mm to (130.0, 119.8)
- moved TP5 13.9 mm to (130.0, 122.8)
- moved TP6 13.9 mm to (130.0, 125.8)
- moved TP10 13.2 mm to (130.4, 258.1)
- moved TP11 13.2 mm to (130.4, 261.1)
- moved TP12 13.2 mm to (130.4, 264.1)
- moved C44 8.11 mm to (99.0, 177.2), turned to 90 degrees
- moved C80 8.06 mm to (99.0, 316.2), turned to 90 degrees
- moved C18 8.00 mm to (99.0, 107.8), turned to 90 degrees
- moved C62 7.96 mm to (99.0, 247.2), turned to 90 degrees
- moved TP1 3.71 mm to (117.2, 49.9)
- moved TP2 3.71 mm to (117.2, 52.9)
- moved TP3 3.71 mm to (117.2, 55.9)
- moved C86 0.56 mm to (157.5, 349.7)
- turned JP24 to 90 degrees
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Connections:
- net /dcdc/3V3 renamed /C1/3V3
- net /dcdc/5V renamed /C1/5V
- net /dcdc/DISABLE_DCDC renamed /C1_PWR/DISABLE_DCDC
- net /dcdc/VIN_DCDC_3V3 renamed /C1_PWR/VIN_DCDC_3V3
- net /dcdc/VIN_DCDC_5V renamed /C1_PWR/VIN_DCDC_5V
- net /pi/ETH0+ renamed /C1/ETH0+
- net /pi/ETH0- renamed /C1/ETH0-
- net /pi/ETH1+ renamed /C1/ETH1+
- net /pi/ETH1- renamed /C1/ETH1-
- net /pi/ETH2+ renamed /C1/ETH2+
- net /pi/ETH2- renamed /C1/ETH2-
- net /pi/ETH3+ renamed /C1/ETH3+
- net /pi/ETH3- renamed /C1/ETH3-
- net /pi/RPI_PCIe_CLK_N renamed /C1/RPI_PCIe_CLK_N
- net /pi/RPI_PCIe_CLK_P renamed /C1/RPI_PCIe_CLK_P
- net /pi/RPI_PCIe_CLK_nREQ renamed /C1/RPI_PCIe_CLK_nREQ
- net /pi/RPI_PCIe_RX_N renamed /C1/RPI_PCIe_RX_N
- net /pi/RPI_PCIe_RX_P renamed /C1/RPI_PCIe_RX_P
- net /pi/RPI_PCIe_TX_N renamed /C1/RPI_PCIe_TX_N
- net /pi/RPI_PCIe_TX_P renamed /C1/RPI_PCIe_TX_P
- net /pi/RPI_PCIe_nRST renamed /C1/RPI_PCIe_nRST
- net /pi/TD1_N renamed /C1/TD1_N
- net /pi/TD1_P renamed /C1/TD1_P
- net /pi/TD2_N renamed /C1/TD2_N
- net /pi/TD2_P renamed /C1/TD2_P
- net /pi/TD3_N renamed /C1/TD3_N
- net /pi/TD3_P renamed /C1/TD3_P
- net /pi/TD4_N renamed /C1/TD4_N
- net /pi/TD4_P renamed /C1/TD4_P
- net /pi/eth_act_ledg renamed /C1/eth_act_ledg
- net /pi/eth_speed_ledy renamed /C1/eth_speed_ledy
- net /pi/pi3V3 renamed /C1/pi3V3
- net /sheet6142DC76/3V3 renamed /C2/3V3
- net /sheet6142DC76/5V renamed /C2/5V
- net /sheet6142DC76/DISABLE_DCDC renamed /C2_PWR/DISABLE_DCDC
- net /sheet6142DC76/VIN_DCDC_3V3 renamed /C2_PWR/VIN_DCDC_3V3
- net /sheet6142DC76/VIN_DCDC_5V renamed /C2_PWR/VIN_DCDC_5V
- net /sheet6142DC77/ETH0+ renamed /C2/ETH0+
- net /sheet6142DC77/ETH0- renamed /C2/ETH0-
- net /sheet6142DC77/ETH1+ renamed /C2/ETH1+
- net /sheet6142DC77/ETH1- renamed /C2/ETH1-
- net /sheet6142DC77/ETH2+ renamed /C2/ETH2+
- net /sheet6142DC77/ETH2- renamed /C2/ETH2-
- net /sheet6142DC77/ETH3+ renamed /C2/ETH3+
- net /sheet6142DC77/ETH3- renamed /C2/ETH3-
- net /sheet6142DC77/RPI_PCIe_CLK_N renamed /C2/RPI_PCIe_CLK_N
- net /sheet6142DC77/RPI_PCIe_CLK_P renamed /C2/RPI_PCIe_CLK_P
- net /sheet6142DC77/RPI_PCIe_CLK_nREQ renamed /C2/RPI_PCIe_CLK_nREQ
- net /sheet6142DC77/RPI_PCIe_RX_N renamed /C2/RPI_PCIe_RX_N
- net /sheet6142DC77/RPI_PCIe_RX_P renamed /C2/RPI_PCIe_RX_P
- net /sheet6142DC77/RPI_PCIe_TX_N renamed /C2/RPI_PCIe_TX_N
- net /sheet6142DC77/RPI_PCIe_TX_P renamed /C2/RPI_PCIe_TX_P
- net /sheet6142DC77/RPI_PCIe_nRST renamed /C2/RPI_PCIe_nRST
- net /sheet6142DC77/TD1_N renamed /C2/TD1_N
- net /sheet6142DC77/TD1_P renamed /C2/TD1_P
- net /sheet6142DC77/TD2_N renamed /C2/TD2_N
- net /sheet6142DC77/TD2_P renamed /C2/TD2_P
- net /sheet6142DC77/TD3_N renamed /C2/TD3_N
- net /sheet6142DC77/TD3_P renamed /C2/TD3_P
- net /sheet6142DC77/TD4_N renamed /C2/TD4_N
- net /sheet6142DC77/TD4_P renamed /C2/TD4_P
- net /sheet6142DC77/eth_act_ledg renamed /C2/eth_act_ledg
- net /sheet6142DC77/eth_speed_ledy renamed /C2/eth_speed_ledy
- net /sheet6142DC77/pi3V3 renamed /C2/pi3V3
- net /sheet6143BBAB/3V3 renamed /C3/3V3
- net /sheet6143BBAB/5V renamed /C3/5V
- net /sheet6143BBAB/DISABLE_DCDC renamed /C3_PWR/DISABLE_DCDC
- net /sheet6143BBAB/VIN_DCDC_3V3 renamed /C3_PWR/VIN_DCDC_3V3
- net /sheet6143BBAB/VIN_DCDC_5V renamed /C3_PWR/VIN_DCDC_5V
- net /sheet6143BBAC/ETH0+ renamed /C3/ETH0+
- net /sheet6143BBAC/ETH0- renamed /C3/ETH0-
- net /sheet6143BBAC/ETH1+ renamed /C3/ETH1+
- net /sheet6143BBAC/ETH1- renamed /C3/ETH1-
- net /sheet6143BBAC/ETH2+ renamed /C3/ETH2+
- net /sheet6143BBAC/ETH2- renamed /C3/ETH2-
- net /sheet6143BBAC/ETH3+ renamed /C3/ETH3+
- net /sheet6143BBAC/ETH3- renamed /C3/ETH3-
- net /sheet6143BBAC/RPI_PCIe_CLK_N renamed /C3/RPI_PCIe_CLK_N
- net /sheet6143BBAC/RPI_PCIe_CLK_P renamed /C3/RPI_PCIe_CLK_P
- net /sheet6143BBAC/RPI_PCIe_CLK_nREQ renamed /C3/RPI_PCIe_CLK_nREQ
- net /sheet6143BBAC/RPI_PCIe_RX_N renamed /C3/RPI_PCIe_RX_N
- net /sheet6143BBAC/RPI_PCIe_RX_P renamed /C3/RPI_PCIe_RX_P
- net /sheet6143BBAC/RPI_PCIe_TX_N renamed /C3/RPI_PCIe_TX_N
- net /sheet6143BBAC/RPI_PCIe_TX_P renamed /C3/RPI_PCIe_TX_P
- net /sheet6143BBAC/RPI_PCIe_nRST renamed /C3/RPI_PCIe_nRST
- net /sheet6143BBAC/TD1_N renamed /C3/TD1_N
- net /sheet6143BBAC/TD1_P renamed /C3/TD1_P
- net /sheet6143BBAC/TD2_N renamed /C3/TD2_N
- net /sheet6143BBAC/TD2_P renamed /C3/TD2_P
- net /sheet6143BBAC/TD3_N renamed /C3/TD3_N
- net /sheet6143BBAC/TD3_P renamed /C3/TD3_P
- net /sheet6143BBAC/TD4_N renamed /C3/TD4_N
- net /sheet6143BBAC/TD4_P renamed /C3/TD4_P
- net /sheet6143BBAC/eth_act_ledg renamed /C3/eth_act_ledg
- net /sheet6143BBAC/eth_speed_ledy renamed /C3/eth_speed_ledy
- net /sheet6143BBAC/pi3V3 renamed /C3/pi3V3
- net /sheet6144BA66/3V3 renamed /C4/3V3
- net /sheet6144BA66/5V renamed /C4/5V
- net /sheet6144BA66/DISABLE_DCDC renamed /C4_PWR/DISABLE_DCDC
- net /sheet6144BA66/VIN_DCDC_3V3 renamed /C4_PWR/VIN_DCDC_3V3
- net /sheet6144BA66/VIN_DCDC_5V renamed /C4_PWR/VIN_DCDC_5V
- net /sheet6144BA67/ETH0+ renamed /C4/ETH0+
- net /sheet6144BA67/ETH0- renamed /C4/ETH0-
- net /sheet6144BA67/ETH1+ renamed /C4/ETH1+
- net /sheet6144BA67/ETH1- renamed /C4/ETH1-
- net /sheet6144BA67/ETH2+ renamed /C4/ETH2+
- net /sheet6144BA67/ETH2- renamed /C4/ETH2-
- net /sheet6144BA67/ETH3+ renamed /C4/ETH3+
- net /sheet6144BA67/ETH3- renamed /C4/ETH3-
- net /sheet6144BA67/RPI_PCIe_CLK_N renamed /C4/RPI_PCIe_CLK_N
- net /sheet6144BA67/RPI_PCIe_CLK_P renamed /C4/RPI_PCIe_CLK_P
- net /sheet6144BA67/RPI_PCIe_CLK_nREQ renamed /C4/RPI_PCIe_CLK_nREQ
- net /sheet6144BA67/RPI_PCIe_RX_N renamed /C4/RPI_PCIe_RX_N
- net /sheet6144BA67/RPI_PCIe_RX_P renamed /C4/RPI_PCIe_RX_P
- net /sheet6144BA67/RPI_PCIe_TX_N renamed /C4/RPI_PCIe_TX_N
- net /sheet6144BA67/RPI_PCIe_TX_P renamed /C4/RPI_PCIe_TX_P
- net /sheet6144BA67/RPI_PCIe_nRST renamed /C4/RPI_PCIe_nRST
- net /sheet6144BA67/TD1_N renamed /C4/TD1_N
- net /sheet6144BA67/TD1_P renamed /C4/TD1_P
- net /sheet6144BA67/TD2_N renamed /C4/TD2_N
- net /sheet6144BA67/TD2_P renamed /C4/TD2_P
- net /sheet6144BA67/TD3_N renamed /C4/TD3_N
- net /sheet6144BA67/TD3_P renamed /C4/TD3_P
- net /sheet6144BA67/TD4_N renamed /C4/TD4_N
- net /sheet6144BA67/TD4_P renamed /C4/TD4_P
- net /sheet6144BA67/eth_act_ledg renamed /C4/eth_act_ledg
- net /sheet6144BA67/eth_speed_ledy renamed /C4/eth_speed_ledy
- net /sheet6144BA67/pi3V3 renamed /C4/pi3V3
Routing:
- net /C3/RPI_PCIe_CLK_nREQ: track 0.00 -> 29.1 mm
- net /C2/RPI_PCIe_CLK_nREQ: track 0.00 -> 29.1 mm
- net /C1/RPI_PCIe_CLK_nREQ: track 0.00 -> 29.1 mm
- net /C4/RPI_PCIe_CLK_nREQ: track 0.00 -> 29.1 mm
- net /C3/RPI_PCIe_nRST: track 0.00 -> 26.8 mm
- net /C2/RPI_PCIe_nRST: track 0.00 -> 26.8 mm
- net /C1/RPI_PCIe_nRST: track 0.00 -> 26.8 mm
- net /C4/RPI_PCIe_nRST: track 0.00 -> 26.8 mm
- net /C1/RPI_PCIe_TX_N: track 0.00 -> 22.9 mm
- net /C3/RPI_PCIe_TX_N: track 0.00 -> 22.9 mm
- net /C2/RPI_PCIe_TX_N: track 0.00 -> 22.9 mm
- net /C3/RPI_PCIe_TX_P: track 0.00 -> 22.9 mm
- net /C2/RPI_PCIe_TX_P: track 0.00 -> 22.9 mm
- net /C1/RPI_PCIe_TX_P: track 0.00 -> 22.9 mm
- net /C3/RPI_PCIe_CLK_N: track 0.00 -> 22.2 mm
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- added copper zone on F.Cu, net /mgm/5V
Other:
- net class pcieC1 added: clearance 0.11, trace_width 0.146812, via_dia 0.5, via_drill 0.2
- net class pcieC2 added: clearance 0.11, trace_width 0.146812, via_dia 0.5, via_drill 0.2
- net class pcieC3 added: clearance 0.11, trace_width 0.146812, via_dia 0.5, via_drill 0.2
- net class pcieC4 added: clearance 0.11, trace_width 0.146812, via_dia 0.5, via_drill 0.2
- board text added: "JLC2313 100 ohm DIFF -> Width:4.35mil Spacing:6mil 90 ohm DIFF -> Width: 4.92mil Spacing:4.5mil 50 Ohm SE -> Width:5.78mil"

Commit message: Added Power Planes.
Parts:
- moved C17 14.4 mm to (93.0, 112.0), turned to 270 degrees
- moved R9 13.7 mm to (93.5, 116.0), turned to 180 degrees
- moved R11 13.7 mm to (93.5, 118.0), turned to 180 degrees
- moved TP7 13.1 mm to (128.9, 187.8)
- moved TP8 13.1 mm to (128.9, 190.8)
- moved TP9 13.1 mm to (128.9, 193.8)
- moved R8 12.9 mm to (93.5, 115.0), turned to 180 degrees
- moved R10 12.9 mm to (93.5, 117.0), turned to 180 degrees
- moved C79 11.9 mm to (93.2, 320.8), turned to 270 degrees
- moved TP1 11.4 mm to (128.4, 48.5)
- moved TP2 11.4 mm to (128.4, 51.5)
- moved TP3 11.4 mm to (128.4, 54.5)
- moved R46 10.8 mm to (93.5, 254.5), turned to 180 degrees
- moved C43 10.6 mm to (93.2, 181.5), turned to 270 degrees
- moved R32 9.67 mm to (93.5, 187.5), turned to 180 degrees
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Routing:
- net (no net): track 0.00 -> 46.1 mm
- net /C4/ETH0+: track 0.00 -> 32.9 mm
- net /C4/ETH0-: track 0.00 -> 32.7 mm
- net /C4/ETH2-: track 0.00 -> 29.2 mm
- net /C4/ETH2+: track 0.00 -> 28.9 mm
- net Net-(R8-Pad1): track 0.00 -> 16.7 mm
- net Net-(R29-Pad1): track 0.00 -> 16.7 mm
- net Net-(R9-Pad1): track 0.00 -> 13.3 mm
- net Net-(R30-Pad1): track 0.00 -> 13.3 mm
- net Net-(R31-Pad1): track 0.00 -> 9.76 mm
- net Net-(R10-Pad1): track 0.00 -> 9.76 mm
- net Net-(R32-Pad1): track 0.00 -> 6.43 mm
- net Net-(R11-Pad1): track 0.00 -> 6.43 mm
- net Net-(C17-Pad2): track 0.00 -> 4.53 mm
- net Net-(C61-Pad2): track 0.00 -> 4.53 mm
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- added copper zone on F.Cu, net /C1/3V3
- added copper zone on F.Cu, net /C1/5V
- added copper zone on F.Cu, net /C2/3V3
- added copper zone on F.Cu, net /C2/5V
- added copper zone on F.Cu, net /C3/3V3
- added copper zone on F.Cu, net /C3/5V
- added copper zone on F.Cu, net /C4/3V3
- added copper zone on F.Cu, net /C4/5V
