File: currypi.kicad_pcb (KiCad board)
At the start: 6 copper layers, 120 x 350 mm, 275 parts, among them IC1 OKR-T_6-W12-C, IC10 OKR-T_6-W12-C, IC2 OKR-T_6-W12-C, IC3 OKR-T_6-W12-C, IC4 OKR-T_6-W12-C, IC5 OKR-T_6-W12-C, IC6 OKR-T_6-W12-C, IC7 OKR-T_6-W12-C, IC8 OKR-T_6-W12-C, IC9 OKR-T_6-W12-C, J1 SS-74500-020, J10 Header_2x6_2.54mm, J11 Header_2x6_2.54mm, J12 Header_2x6_2.54mm, J13 0826-1X1T-GH-F, J5 Conn_02x04_Odd_Even, J6 Conn_02x04_Odd_Even, J7 Header_2x6_2.54mm, J9 Header_2x6_2.54mm, M1 Fan_4pin, M2 Fan_4pin, M3 Fan_4pin, Q1 2N7002K, T1 QT24A01, T2 QT24A01, T3 QT24A01, T4 QT24A01, U1 rpi_cm4, U10 rpi_cm4, U2 m.2_pcie_nvme, U3 USB2514B_Bi, U4 rpi_cm4, U5 m.2_pcie_nvme, U6 rpi_cm4, U7 m.2_pcie_nvme, U8 rpi_cm4, U9 m.2_pcie_nvme, Y1 24Mhz X1E0000210264

Commit message: Connected Mgmt. Pi to USB Hub.
Routing:
- net /mgm/USB+: track 0.00 -> 140.2 mm
- net /mgm/USB-: track 0.00 -> 139.0 mm
Changed lines of the file:
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@@
     (thickness 1.6)
     (drawings 9)
-    (tracks 3374)
+    (tracks 3402)
     (zones 0)
     (modules 275)
@@
   (segment (start 117.01 23.99) (end 118 23) (width 0.25) (layer F.Cu) (net 144))
   (segment (start 118 23) (end 122 23) (width 0.25) (layer F.Cu) (net 144))
+  (segment (start 182.630366 224.632134) (end 182.5 224.7625) (width 0.124968) (layer F.Cu) (net 234))
+  (segment (start 183.550444 222.280366) (end 182.630366 223.200444) (width 0.124968) (layer F.Cu) (net 234))
+  (segment (start 194.445001 333.51) (end 194.525367 333.429634) (width 0.124968) (layer F.Cu) (net 234))
+  (segment (start 195.519634 331.850444) (end 172.119634 308.450444) (width 0.124968) (layer F.Cu) (net 234))
+  (segment (start 193.92 333.51) (end 194.445001 333.51) (width 0.124968) (layer F.Cu) (net 234))
+  (segment (start 194.525367 333.429634) (end 195.039556 333.429634) (width 0.124968) (layer F.Cu) (net 234))
+  (segment (start 182.630366 223.200444) (end 182.630366 224.632134) (width 0.124968) (layer F.Cu) (net 234))
+  (segment (start 195.039556 333.429634) (end 195.519634 332.949556) (width 0.124968) (layer F.Cu) (net 234))
+  (segment (start 172.119634 308.450444) (end 172.119634 259.649556) (width 0.124968) (layer F.Cu) (net 234))
+  (segment (start 172.119634 259.649556) (end 191.319634 240.449556) (width 0.124968) (layer F.Cu) (net 234))
+  (segment (start 195.519634 332.949556) (end 195.519634 331.850444) (width 0.124968) (layer F.Cu) (net 234))
+  (segment (start 191.319634 240.449556) (end 191.319634 223.350444) (width 0.124968) (layer F.Cu) (net 234))
+  (segment (start 190.249556 222.280366) (end 183.550444 222.280366) (width 0.124968) (layer F.Cu) (net 234))
+  (segment (start 191.319634 223.350444) (end 190.249556 222.280366) (width 0.124968) (layer F.Cu) (net 234))
+  (segment (start 182.869634 223.299556) (end 182.869634 224.632134) (width 0.124968) (layer F.Cu) (net 235))
+  (segment (start 183.649556 222.519634) (end 182.869634 223.299556) (width 0.124968) (layer F.Cu) (net 235))
+  (segment (start 191.080366 223.449556) (end 190.150444 222.519634) (width 0.124968) (layer F.Cu) (net 235))
+  (segment (start 191.080366 240.350444) (end 191.080366 223.449556) (width 0.124968) (layer F.Cu) (net 235))
+  (segment (start 171.880366 259.550444) (end 191.080366 240.350444) (width 0.124968) (layer F.Cu) (net 235))
+  (segment (start 171.880366 308.549556) (end 171.880366 259.550444) (width 0.124968) (layer F.Cu) (net 235))
+  (segment (start 195.280366 331.949556) (end 171.880366 308.549556) (width 0.124968) (layer F.Cu) (net 235))
+  (segment (start 195.280366 332.850444) (end 195.280366 331.949556) (width 0.124968) (layer F.Cu) (net 235))
+  (segment (start 190.150444 222.519634) (end 183.649556 222.519634) (width 0.124968) (layer F.Cu) (net 235))
+  (segment (start 193.92 333.11) (end 194.445001 333.11) (width 0.124968) (layer F.Cu) (net 235))
+  (segment (start 182.869634 224.632134) (end 183 224.7625) (width 0.124968) (layer F.Cu) (net 235))
+  (segment (start 194.940444 333.190366) (end 195.280366 332.850444) (width 0.124968) (layer F.Cu) (net 235))
+  (segment (start 194.525367 333.190366) (end 194.940444 333.190366) (width 0.124968) (layer F.Cu) (net 235))
+  (segment (start 194.445001 333.11) (end 194.525367 333.190366) (width 0.124968) (layer F.Cu) (net 235))
   (segment (start 110.34 108.095001) (end 110.34 112.043848) (width 0.11) (layer F.Cu) (net 539))
   (segment (start 110.41 108.025001) (end 110.34 108.095001) (width 0.11) (layer F.Cu) (net 539))

Commit message: Fixed Eth. Schematic issue and Completed Eth. Routing.
Parts:
- moved JP25 39.4 mm to (156.4, 323.0), turned to 0 degrees
- moved D20 14.9 mm to (186.5, 289.2), turned to 90 degrees
- moved R68 11.2 mm to (186.5, 291.7), turned to 270 degrees
- moved D19 5.96 mm to (186.5, 303.3), turned to 90 degrees
- moved R67 5.24 mm to (186.5, 305.8), turned to 270 degrees
- moved R69 3.09 mm to (188.5, 310.2), turned to 180 degrees
Connections:
- J1 pad 4_1: /C1/ETH2- -> /C1/ETH2+
- J1 pad 4_2: /C2/ETH2- -> /C2/ETH2+
- J1 pad 4_3: /C3/ETH2- -> /C3/ETH2+
- J1 pad 4_4: /C4/ETH2- -> /C4/ETH2+
- J1 pad 5_1: /C1/ETH2+ -> /C1/ETH2-
- J1 pad 5_2: /C2/ETH2+ -> /C2/ETH2-
- J1 pad 5_3: /C3/ETH2+ -> /C3/ETH2-
- J1 pad 5_4: /C4/ETH2+ -> /C4/ETH2-
Routing:
- net /C1/ETH1+: track 0.00 -> 258.9 mm, vias 0 -> 1
- net /C1/ETH1-: track 0.00 -> 258.8 mm, vias 0 -> 1
- net /C1/ETH3-: track 0.00 -> 255.3 mm, vias 0 -> 1
- net /C1/ETH3+: track 0.00 -> 255.3 mm, vias 0 -> 1
- net /C1/ETH2-: track 0.00 -> 255.3 mm, vias 0 -> 1
- net /C1/ETH0-: track 0.00 -> 255.3 mm, vias 0 -> 1
- net /C1/ETH0+: track 0.00 -> 255.3 mm, vias 0 -> 1
- net /C1/ETH2+: track 0.00 -> 255.3 mm, vias 0 -> 1
- net /C2/ETH3-: track 0.00 -> 176.2 mm, vias 0 -> 1
- net /C2/ETH1+: track 0.00 -> 176.2 mm, vias 0 -> 1
- net /C2/ETH2-: track 0.00 -> 176.2 mm, vias 0 -> 1
- net /C2/ETH2+: track 0.00 -> 176.2 mm, vias 0 -> 1
- net /C2/ETH0-: track 0.00 -> 176.2 mm, vias 0 -> 1
- net /C2/ETH1-: track 0.00 -> 176.2 mm, vias 0 -> 1
- net /C2/ETH3+: track 0.00 -> 176.2 mm, vias 0 -> 1
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Other:
- board text added: "The differential PCIe signals should be routed as 90Ω differential pairs, with suitable clearances. There is no need to match the lengths between pairs, only the signals within a Pair need to be length matched ideally to better than 0.1mm. The differential Ethernet signals should be routed as 100Ω differential pairs, with suitable clearances. Length matching between pairs should be better than 50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"
