File: currypi.kicad_pcb (KiCad board)
At the start: 4 copper layers, 120 x 350 mm, 266 parts, among them IC1 OKR-T_6-W12-C, IC10 OKR-T_6-W12-C, IC2 OKR-T_6-W12-C, IC3 OKR-T_6-W12-C, IC4 OKR-T_6-W12-C, IC5 OKR-T_6-W12-C, IC6 OKR-T_6-W12-C, IC7 OKR-T_6-W12-C, IC8 OKR-T_6-W12-C, IC9 OKR-T_6-W12-C, J1 SS-74500-020, J10 Header_2x6_2.54mm, J11 Header_2x6_2.54mm, J12 Header_2x6_2.54mm, J13 0826-1X1T-GH-F, J5 Conn_02x04_Odd_Even, J6 Conn_02x04_Odd_Even, J7 Header_2x6_2.54mm, J9 Header_2x6_2.54mm, M1 Fan_4pin, M2 Fan_4pin, M3 Fan_4pin, Q1 2N7002K, T1 QT24A01, T2 QT24A01, T3 QT24A01, T4 QT24A01, U1 rpi_cm4, U10 rpi_cm4, U2 m.2_pcie_nvme, U3 USB2514B_Bi, U4 rpi_cm4, U5 m.2_pcie_nvme, U6 rpi_cm4, U7 m.2_pcie_nvme, U8 rpi_cm4, U9 m.2_pcie_nvme, Y1 24Mhz X1E0000210264

Commit message: Completed Design.Will be reviewed.
Parts:
- moved FID1 350.0 mm to (122.0, 22.0)
- moved H1 344.8 mm to (84.0, 37.0)
- moved FID2 327.6 mm to (198.0, 22.0)
- moved H5 309.9 mm to (196.0, 37.0)
- moved H2 154.0 mm to (84.0, 338.0)
- moved H4 113.9 mm to (196.0, 247.0)
- moved FID3 76.4 mm to (198.0, 368.0)
- moved H6 11.1 mm to (245.0, 358.0)
- moved D2 0.50 mm to (147.0, 33.0)
- moved JP26 0.15 mm to (116.4, 29.0)
- moved C22 0.10 mm to (180.8, 221.6)
- moved C23 0.10 mm to (182.7, 221.6)
- moved C63 0.10 mm to (132.7, 319.9)
- moved C74 0.10 mm to (123.2, 259.7)
Routing:
- net GND: track 272.7 -> 906.9 mm, vias 121 -> 850
- net /C3_PWR/DISABLE_DCDC: track 30.7 -> 33.2 mm
- net /c4_boot: track 58.2 -> 60.3 mm
- net /C1_PWR/DISABLE_DCDC: track 31.5 -> 33.3 mm
- net /c1_tx: track 293.6 -> 295.2 mm
- net /c3_boot: track 123.0 -> 123.6 mm
- net /C3/TD3_N: track 22.2 -> 21.6 mm
Other:
- board text added: "C1"
- board text added: "C2"
- board text added: "C3"
- board text added: "C4"
